File: USBTinyISP/schematic/USBISPTiny.sch (EAGLE design)
At the start: 57 parts, among them Q1 12MHz, SW4 SWITCH_DOUBLE(2.54X4MM), T1 BC847, T10 BC847, T2 BC847, T3 BC847, T4 BC847, T5 BC847, T6 BC847, T9 BC847, X1 USB_B, X2 Target_MCU

Commit message: TinyISP. Fix micro usb incorrect pinout. Change transystor levels converter to fast, diode based. Route PCB.
Parts:
- removed C11, C18, C7, C9: 100pF, __MyCommonLib1:CSMD_0805
- removed R13, R14, R15, R19, R20, R26, R35, R36, R9: 4K7, __MyCommonLib1:RSMD_0805
- removed R16: 4K7, __MyCommonLib1:R0207
- removed R28: 1K0, __MyCommonLib1:RSMD_0805
- removed R30: 100R, __MyCommonLib1:RSMD_0805
- removed T1, T10, T2, T3, T4, T5, T9: BC847, __MyCommonLib1:BC847SOT23_SMALL_PADS
- added D10, D2, D3: LL4148, __MyCommonLib1:LL4147SOD-80
- added DD4, DD5, DD6: BAT54C, __MyCommonLib1:BAT54C(SOT23)
- added J10: 0, __MyCommonLib1:RSMD_0805
- added R7: 100R, __MyCommonLib1:RSMD_0805
- added R8: 4K7, __MyCommonLib1:RSMD_0805
- added X3: USB_MICRO, __MyCommonLib1:USB_MICROMICRO
- added ZD3: 5.6V, __MyCommonLib1:ZENNER(SOD_80)
- R12, R18: device __MyCommonLib1:R0204 -> __MyCommonLib1:RSMD_0805
- R27: value 4K7 -> 1K0
- R33: device __MyCommonLib1:R0204 -> __MyCommonLib1:R0207
- R34: device __MyCommonLib1:R0207 -> __MyCommonLib1:RSMD_0805
Connections:
- removed net N$20: R17.PIN1, R18.PIN0, T3.C
- removed net N$22: R15.PIN1, T3.B, T4.C
- removed net N$23: R11.PIN1, R16.PIN0, T6.B
- removed net N$24: R19.PIN1, R20.PIN0, T4.B
- removed net N$33: R28.PIN1, R30.PIN0, T5.C
- removed net N$35: R27.PIN1, T5.B, T6.C
- removed net N$40: R26.PIN1, T10.C, T9.B
- removed net N$41: R35.PIN1, R36.PIN0, T10.B
- new net N$10: J10.PIN1, X3.D-
- new net N$13: D10.ANODE, R17.PIN1, R18.PIN0
- net +5V_USB: now also DD4.CATHODE, DD5.CATHODE, SW4.CENTER1, SW4.CENTER2, SW4.POS_A1, SW4.POS_A2, X3.VBUS, ZD3.CATHODE; no longer R28.PIN0, SW4.POS_B1, SW4.POS_B2
- net GND: now also X3.GND, X3.PACKAGE, ZD3.ANODE; no longer C11.PIN0, C18.PIN0, C7.PIN0, C9.PIN0, R11.PIN0, R13.PIN0, R19.PIN0, R35.PIN0, T1.E, T10.E, T2.E, T3.E, T4.E, T5.E, T6.E, T9.E
- net N$11: now also DD6.ANODE2, R8.PIN0, T6.B; no longer R13.PIN1, R14.PIN0, T2.B
- net N$2: now also D3.ANODE; no longer T1.C
- net N$39: now also D2.ANODE; no longer T9.C
- net N$9: now also DD6.ANODE1, R11.PIN0, R7.PIN0, T6.E; no longer R9.PIN1, T1.B, T2.C
- net SPI_MISO: now also DD4.ANODE2, R27.PIN1, T6.C, U$1.PB5(MOSI/DI/SDA/PCINT5); no longer C11.PIN1, R30.PIN1, U$1.PB6(MISO/DO/PCINT6)
- net SPI_MOSI: now also D10.CATHODE, DD5.ANODE2, U$1.PB6(MISO/DO/PCINT6); no longer R20.PIN1, U$1.PB5(MOSI/DI/SDA/PCINT5)
- net SPI_RST: now also D2.CATHODE, DD4.ANODE1; no longer R36.PIN1
- net SPI_SCK: now also D3.CATHODE, DD5.ANODE1; no longer R14.PIN1
- net T_MISO: now also R7.PIN1; no longer R16.PIN1
- net T_MOSI: no longer C9.PIN1
- net T_RST: no longer C18.PIN1
- net T_SCK: no longer C7.PIN1
- net T_VCC: now also DD6.CATHODE, R11.PIN1, R8.PIN1, SW4.POS_B1, SW4.POS_B2; no longer R15.PIN0, R26.PIN0, R9.PIN0, SW4.CENTER1, SW4.CENTER2
- net USB_D+: now also X3.D+
- net USB_D-: now also J10.PIN0
Other:
- moved on the sheet: C1, C2, LED1, LED2, Q1, R10, R11, R12, R17, R18, R27, R29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
