File: LC_METER/schematic/LCMeter.brd (EAGLE design)
At the start: 60.5 x 30 mm, 50 parts, among them J10 0, Q1 12MHz, T6 BC847, X1 USB_B, X2 Target_MCU, X3 USB_MICRO

Commit message: LMeter new changes
Parts:
- removed C16: 0.1uF, __MyCommonLib1:RSMD_0805
- added C10, C11, C4, C7, C9: 0.1uF, __MyCommonLib1:RSMD_0805
- added C5: 4.7uF, __MyCommonLib1:RSMD_1206
- added D11, D12, D4, D7, D8, D9: LL4148, __MyCommonLib1:SOD-80
- added IC1, IC2, IC3, IC4, IC5: 74HC595, __MyCommonLib1:SOIC16
- added J1: 0, __MyCommonLib1:RSMD_0805
- added J123, J2, J3, J4, J5, J6, J7, J8, J9: 0, __MyCommonLib1:RSMD_1206_BIG_GAP
- added R13: 1K0, __MyCommonLib1:RSMD_0805
- added R14, R15: 4K7, __MyCommonLib1:RSMD_0805
- added R16: 100R, __MyCommonLib1:RSMD_0805
- added R19, R20, R21, R22, R23, R24, R25, R26, R28, R30, R32, R35, R36, R37, R38, R39, R40, R41, R42, R43, R44, R45, R46, R47, R48, R49, R50, R51, R52, R53, R54, R55, R56, R57, R58: 560R, __MyCommonLib1:RSMD_0805
- added R59, R60, R61: 300R, __MyCommonLib1:RSMD_0805
- added R9: 68R, __MyCommonLib1:RSMD_0805
- C8: value 4.7uF -> 0.1uF; device __MyCommonLib1:RSMD_1206 -> __MyCommonLib1:RSMD_0805
- D1: value 1N4001 -> LL4148; device __MyCommonLib1:DO-41_10MM -> __MyCommonLib1:SOD-80
- D2: value LL4148 -> 1N4001; device __MyCommonLib1:SOD-80 -> __MyCommonLib1:DO-41_10MM
- J10: device __MyCommonLib1:RSMD_0805 -> __MyCommonLib1:RSMD_1206_BIG_GAP
- LED1: value green -> Target_Power
- LED3: value Target_Power -> green
- LI1, LI2, LI3, LI4, LI5: device __MyCommonLib1:KEM-5161 -> __MyCommonLib1:KEM-5161(NARROW)
- R1: value 1K5 -> 4K7; device __MyCommonLib1:RSMD_0805 -> __MyCommonLib1:RSMD_1206
- R10: value 1K0 -> 1K5
- R11: value 4K7 -> 1K0
- R17: value 1K0 -> 1K
- R18: value 100R -> 1K
- R2: value 68R -> 1K0
- R27, R29, R31: value 1K0 -> 560R
- R3: value 68R -> 10R; device __MyCommonLib1:RSMD_0805 -> __MyCommonLib1:R0207
- R33: value 10R -> 560R; device __MyCommonLib1:R0207 -> __MyCommonLib1:RSMD_0805
- R34: value 100R -> 560R
- R4: value 4K7 -> 100R; device __MyCommonLib1:RSMD_1206 -> __MyCommonLib1:RSMD_0805
- R5, R6: value 1K -> 1K0
- R8: value 4K7 -> 68R
- X1: value USB_B -> Target_MCU; device __MyCommonLib1:USB_TYPE_B_SMALL_PADS -> __MyCommonLib1:PIN2X5_2.54MM_FEMALE_RIGHT_ANGLE_SMALL_PADS
- X2: value Target_MCU -> USB_MICRO; device __MyCommonLib1:PIN2X5_2.54MM_FEMALE_RIGHT_ANGLE_SMALL_PADS -> __MyCommonLib1:USB_MICRO_TYPE_B
- X3: value USB_MICRO -> USB_B; device __MyCommonLib1:USB_MICRO_TYPE_B -> __MyCommonLib1:USB_TYPE_B_SMALL_PADS
- ZD1: value 3V6 -> 5.6V
- ZD3: value 5.6V -> 3V6
- moved D10 248.1 mm to (-202.4, -28.9), turned to 0 degrees
- moved R29 218.7 mm to (-164.0, 34.1)
- moved R34 213.9 mm to (-156.7, 34.2), turned to 90 degrees
- moved R33 212.9 mm to (-157.1, 50.5), flipped to the bottom, turned to 90 degrees
- moved R31 210.9 mm to (-159.7, 50.6)
- moved R27 204.4 mm to (-168.5, 27.4), turned to 90 degrees
- moved C8 184.6 mm to (-168.5, 23.3), turned to 270 degrees
- moved LI1 169.0 mm to (-174.9, 46.4)
- moved LI2 144.4 mm to (-162.2, 46.4)
- moved J10 133.1 mm to (-124.4, 16.2), turned to 90 degrees
- moved LI3 120.1 mm to (-149.5, 46.4)
- moved LI4 96.3 mm to (-136.8, 46.4)
- moved LI5 73.5 mm to (-124.1, 46.4)
- moved X2 53.8 mm to (0.20, 14.9), flipped to the bottom, turned to 90 degrees
- moved C3 41.4 mm to (15.3, 5.52), turned to 180 degrees
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- renumbered DD4 to DD1, DD5 to DD2, DD6 to DD3, SW4 to SW1, T6 to T1
Connections:
- new net LED_DATA: R59.PAD_0
- new net LED_DATA': D12.ANODE, D9.CATHODE, IC1.14, R59.PAD_1
- new net LED_LATCH: R61.PAD_0
- new net LED_LATCH': D10.ANODE, D7.CATHODE, J10.PAD_0, J2.PAD_0, J4.PAD_0, J6.PAD_0, J8.PAD_0, R61.PAD_1
- new net LED_SCK: R60.PAD_0
- new net LED_SCK': D11.ANODE, D8.CATHODE, J123.PAD_0, J3.PAD_0, J5.PAD_0, J7.PAD_0, J9.PAD_0, R60.PAD_1
- new net N$100: IC1.11, J123.PAD_1
- new net N$101: IC1.12, J2.PAD_1
- new net N$102: IC2.11, J3.PAD_1
- new net N$103: IC2.12, J4.PAD_1
- new net N$104: IC5.11, J9.PAD_1
- new net N$105: IC4.11, J7.PAD_1
- new net N$106: IC3.11, J5.PAD_1
- new net N$107: IC5.12, J10.PAD_1
- new net N$108: IC4.12, J8.PAD_1
- new net N$109: IC3.12, J6.PAD_1
- new net N$15: IC2.1, R28.PAD_0
- new net N$16: IC2.2, R29.PAD_0
- new net N$17: IC2.3, R30.PAD_0
- new net N$18: IC2.4, R31.PAD_0
- new net N$19: LI1.1, R19.PAD_1
- new net N$20: LI1.2, R21.PAD_1
- new net N$21: LI1.4, R24.PAD_1
- new net N$22: IC2.5, R32.PAD_0
- new net N$23: LI1.5, R26.PAD_1
- new net N$24: LI1.10, R20.PAD_1
- new net N$26: IC2.6, R33.PAD_0
- new net N$27: LI1.9, R22.PAD_1
- new net N$28: LI1.7, R23.PAD_1
- new net N$29: LI1.6, R25.PAD_1
- new net N$30: IC1.15, R19.PAD_0
- new net N$31: IC1.1, R20.PAD_0
- new net N$32: IC1.2, R21.PAD_0
- new net N$33: IC1.3, R22.PAD_0
- new net N$34: IC1.4, R23.PAD_0
- new net N$35: IC1.5, R24.PAD_0
- new net N$36: IC1.6, R25.PAD_0
- new net N$37: IC1.7, R26.PAD_0
- new net N$38: IC2.7, R34.PAD_0
- new net N$40: LI2.1, R27.PAD_1
- new net N$41: LI2.2, R29.PAD_1
- new net N$42: LI2.4, R32.PAD_1
- new net N$43: LI2.5, R34.PAD_1
- new net N$44: LI2.10, R28.PAD_1
- new net N$45: LI2.9, R30.PAD_1
- new net N$46: LI2.7, R31.PAD_1
- new net N$47: LI2.6, R33.PAD_1
- new net N$48: IC3.15, R35.PAD_0
- new net N$49: IC3.1, R36.PAD_0
- new net N$50: IC3.2, R37.PAD_0
- new net N$51: IC3.3, R38.PAD_0
- new net N$52: IC3.4, R39.PAD_0
- new net N$53: IC3.5, R40.PAD_0
- new net N$54: IC3.6, R41.PAD_0
- new net N$55: IC3.7, R42.PAD_0
- new net N$56: LI3.1, R35.PAD_1
- new net N$57: LI3.2, R37.PAD_1
- new net N$58: LI3.4, R40.PAD_1
- new net N$59: LI3.5, R42.PAD_1
- new net N$60: LI3.10, R36.PAD_1
- new net N$61: LI3.9, R38.PAD_1
- new net N$62: LI3.7, R39.PAD_1
- new net N$63: LI3.6, R41.PAD_1
- new net N$64: IC4.15, R43.PAD_0
- new net N$65: IC4.1, R44.PAD_0
- new net N$66: IC4.2, R45.PAD_0
- new net N$67: IC4.3, R46.PAD_0
- new net N$68: IC4.4, R47.PAD_0
- new net N$69: IC4.5, R48.PAD_0
- new net N$70: IC4.6, R49.PAD_0
- new net N$71: IC4.7, R50.PAD_0
- new net N$72: LI4.1, R43.PAD_1
- new net N$73: LI4.2, R45.PAD_1
- new net N$74: LI4.4, R48.PAD_1
- new net N$75: LI4.5, R50.PAD_1
- new net N$76: LI4.10, R44.PAD_1
- new net N$77: LI4.9, R46.PAD_1
- new net N$78: LI4.7, R47.PAD_1
- new net N$79: LI4.6, R49.PAD_1
- new net N$80: IC5.15, R51.PAD_0
- new net N$81: IC5.1, R52.PAD_0
- new net N$82: IC5.2, R53.PAD_0
- new net N$83: IC5.3, R54.PAD_0
- new net N$84: IC5.4, R55.PAD_0
- new net N$85: IC5.5, R56.PAD_0
- new net N$86: IC5.6, R57.PAD_0
- new net N$87: IC5.7, R58.PAD_0
- new net N$88: LI5.1, R51.PAD_1
- new net N$89: LI5.2, R53.PAD_1
- new net N$90: LI5.4, R56.PAD_1
- new net N$91: LI5.5, R58.PAD_1
- new net N$92: LI5.10, R52.PAD_1
- new net N$93: LI5.9, R54.PAD_1
- new net N$94: LI5.7, R55.PAD_1
- new net N$95: LI5.6, R57.PAD_1
- new net N$96: IC3.9, IC4.14
- new net N$97: IC2.9, IC3.14
- new net N$98: IC1.9, IC2.14
- new net N$99: IC4.9, IC5.14
- new net VCC_ROUGH: C10.PAD_1, C11.PAD_1, C7.PAD_1, C8.PAD_1, C9.PAD_1, D10.CATHODE, D11.CATHODE, D12.CATHODE, IC1.10, IC1.16, IC2.10, IC2.16, IC3.10, IC3.16, IC4.10, IC4.16, IC5.10, IC5.16
- net +5V_USB: now also C3.PAD_1, C4.PAD_1, R1.PAD_0, R13.PAD_0, X2.1, ZD1.CATHODE; no longer C6.PAD_1, C8.PAD_1, R27.PAD_0, R4.PAD_0, X1.1, ZD3.CATHODE
- net GND: now also C10.PAD_0, C11.PAD_0, C4.PAD_0, C5.PAD_0, C7.PAD_0, C9.PAD_0, D2.ANODE, D7.ANODE, D8.ANODE, D9.ANODE, IC1.13, IC1.8, IC2.13, IC2.8, IC3.13, IC3.8, IC4.13, IC4.8, IC5.13, IC5.8, LI1.3, LI1.8, LI2.3, LI2.8, LI3.3, LI3.8, LI4.3, LI4.8, LI5.3, LI5.8, X1.10, X1.2, X2.5, X2.PACKAGE1, X2.PACKAGE2, X2.PACKAGE3, X2.PACKAGE4, X2.PACKAGE5, X3.4, X3.PACKAGE_PAD1, X3.PACKAGE_PAD2; no longer C16.PAD_0, D1.ANODE, X1.4, X1.PACKAGE_PAD1, X1.PACKAGE_PAD2, X2.10, X2.2, X3.5, X3.PACKAGE1, X3.PACKAGE2, X3.PACKAGE3, X3.PACKAGE4, X3.PACKAGE5
- net LED1: now also R18.PAD_0; no longer R6.PAD_0
- net LED2: now also R17.PAD_0; no longer R5.PAD_0
- net N$10: now also J1.PAD_1, X2.2; no longer J10.PAD_1, X3.2
- net N$11: now also R14.PAD_0; no longer R8.PAD_0
- net N$12: now also LED1.ANODE, R5.PAD_1; no longer LED3.ANODE, R31.PAD_1
- net N$13: now also D1.ANODE, R2.PAD_1, R4.PAD_0; no longer D10.ANODE, R17.PAD_1, R18.PAD_0
- net N$14: now also IC2.15, R27.PAD_0; no longer LI1.3, LI1.8, LI2.3, LI2.8, LI3.3, LI3.8, LI4.3, LI4.8, LI5.3, LI5.8
- net N$2: now also D4.ANODE, R11.PAD_1; no longer D3.ANODE, R10.PAD_1
- net N$25: now also R3.PAD1, X1.4; no longer R33.PAD1, X2.4
- net N$39: now also D3.ANODE, R6.PAD_1, R7.PAD_0; no longer D2.ANODE, R29.PAD_1, R34.PAD_0
- net N$4: now also R8.PAD_0; no longer R3.PAD_0
- net N$5: now also R9.PAD_1; no longer R2.PAD_1
- net N$6: now also R10.PAD_1; no longer R1.PAD_1
- net N$7: now also R17.PAD_1; no longer R5.PAD_1
- net N$8: now also LED3.ANODE, R18.PAD_1; no longer LED1.ANODE, R6.PAD_1
- net N$9: now also R15.PAD_0, R16.PAD_0; no longer R11.PAD_0, R7.PAD_0
- net RST: now also R1.PAD_1; no longer R4.PAD_1
- net SPI_MISO: now also R13.PAD_1; no longer R27.PAD_1
- net SPI_MOSI: now also D1.CATHODE; no longer D10.CATHODE
- net SPI_RST: now also D3.CATHODE; no longer D2.CATHODE
- net SPI_SCK: now also D4.CATHODE; no longer D3.CATHODE
- net T_MISO: now also R16.PAD_1, X1.3; no longer R7.PAD_1, X2.3
- net T_MOSI: now also R4.PAD_1, X1.9; no longer R18.PAD_1, X2.9
- net T_RST: now also R7.PAD_1, X1.6; no longer R34.PAD_1, X2.6
- net T_SCK: now also X1.1; no longer X2.1
- net T_VCC: now also C5.PAD_1, C6.PAD_1, D2.CATHODE, R11.PAD_0, R14.PAD_1, R15.PAD_1, R2.PAD_0, R3.PAD_0, R5.PAD_0, R6.PAD_0; no longer C16.PAD_1, C3.PAD_1, D1.CATHODE, R10.PAD_0, R11.PAD_1, R17.PAD_0, R29.PAD_0, R31.PAD_0, R33.PAD_0, R8.PAD_1
- net USB_D+: now also R8.PAD_1, X2.3, ZD2.CATHODE; no longer R3.PAD_1, X1.3, ZD1.CATHODE
- net USB_D-: now also J1.PAD_0, R10.PAD_0, R9.PAD_0, X3.2, ZD3.CATHODE; no longer J10.PAD_0, R1.PAD_0, R2.PAD_0, X1.2, ZD2.CATHODE
Routing:
- net GND: track 53.8 -> 198.1 mm
- net LED_SCK': track 0.00 -> 49.1 mm
- net LED_LATCH': track 0.00 -> 43.8 mm
- net VCC_ROUGH: track 0.00 -> 27.3 mm
- net N$33: track 0.00 -> 22.4 mm
- net N$17: track 0.00 -> 22.2 mm
- net N$36: track 0.00 -> 22.1 mm
- net N$26: track 0.00 -> 22.1 mm
- net N$18: track 0.00 -> 21.9 mm
- net N$15: track 0.00 -> 21.8 mm
- net N$31: track 0.00 -> 21.6 mm
- net N$34: track 0.00 -> 21.2 mm
- net N$98: track 0.00 -> 11.8 mm
- net N$97: track 0.00 -> 9.25 mm
- net N$96: track 0.00 -> 9.23 mm
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
Commit message: LCMeter next changes
Parts:
- removed DD1, DD2, DD3: BAT54C, __MyCommonLib1:SOT23_SMALL_PADS
- removed J1: 0, __MyCommonLib1:RSMD_0805
- removed LED1: Target_Power, __MyCommonLib1:LED3MM
- removed LED2: red, __MyCommonLib1:LED3MM
- removed LED3: green, __MyCommonLib1:LED3MM
- removed Q1: 12MHz, crystal:HC49U-V
- removed SW1: (no value), __MyCommonLib1:SWITCH_DOUBLE_2.54X4.0MM
- removed U$1: ATTINY2313SOIC20, __MyCommonLib1:SOIC20
- removed X2: USB_MICRO, __MyCommonLib1:USB_MICRO_TYPE_B
- removed X3: USB_B, __MyCommonLib1:USB_TYPE_B_SMALL_PADS
- removed ZD2, ZD3: 3V6, __MyCommonLib1:SOD-80
- added C12, C13: 22pF, __MyCommonLib1:RSMD_0805
- added C14, C15, C16, C17, C19, C23, C24, C25, C26, C27, C29, C30, C32, C33, C34, C35, C36, C37, C38, C39: 0.1uF, __MyCommonLib1:RSMD_0805
- added C18: 4.7uF, __MyCommonLib1:CE_6.3MM
- added C20: 1nF, __MyCommonLib1:RSMD_0805
- added C21: 22nF*, __MyCommonLib1:RSMD_0805
- added C22: 1.0uF, __MyCommonLib1:RSMD_1206_BIG_GAP
- added D13, D14, D15, D16, D5, D6: LL4148, __MyCommonLib1:SOD-80
- added IC6: MEGA8535, atmel:TQFP44
- added J11: 0, __MyCommonLib1:RSMD_0805
- added Q2: 12MHz, crystal:HC49U-V
- added R154, R63, R68, R72, R73: 100R, __MyCommonLib1:RSMD_1206_BIG_GAP
- added R62: 4K7, __MyCommonLib1:RSMD_0805
- added R64: 25K, __MyCommonLib1:RSMD_1206_BIG_GAP
- added R65: 1K5, __MyCommonLib1:RSMD_0805
- added R66: 100K, __MyCommonLib1:RSMD_1206_BIG_GAP
- added R67, R69, R70, R71: 1K0, __MyCommonLib1:RSMD_1206_BIG_GAP
- added T2, T5, T6, T7: BC847, __MyCommonLib1:SOT23_SMALL_PADS
- added T3, T4: BC857, __MyCommonLib1:SOT23_SMALL_PADS
- added U15: LM324, __MyCommonLib1:SOIC14
- added X4: L_X, con-wago-500:W237-102
- added X5: USB_B, __MyCommonLib1:USB_TYPE_B_SMALL_PADS
- added X6: USB_MICRO, __MyCommonLib1:USB_MICRO_TYPE_B
- added ZD4: 3V6, __MyCommonLib1:SOD-80
- C1, C2: value 22pF -> 0.1uF
- C3: value 4.7uF -> 0.1uF; device __MyCommonLib1:RSMD_1206 -> __MyCommonLib1:RSMD_0805
- C4: value 0.1uF -> 1nF
- C5: value 4.7uF -> 0.47uF; device __MyCommonLib1:RSMD_1206 -> __MyCommonLib1:RSMD_1206_BIG_GAP
- D2: value 1N4001 -> LL4148; device __MyCommonLib1:DO-41_10MM -> __MyCommonLib1:SOD-80
- R1: value 4K7 -> 100K; device __MyCommonLib1:RSMD_1206 -> __MyCommonLib1:RSMD_0805
- R10: value 1K5 -> 20K
- R11: value 1K0 -> 100K; device __MyCommonLib1:RSMD_0805 -> __MyCommonLib1:RSMD_1206_BIG_GAP
- R12, R16: value 100R -> 1K0; device __MyCommonLib1:RSMD_0805 -> __MyCommonLib1:RSMD_1206_BIG_GAP
- R13: value 1K0 -> 100R; device __MyCommonLib1:RSMD_0805 -> __MyCommonLib1:RSMD_1206_BIG_GAP
- R14: value 4K7 -> 25K; device __MyCommonLib1:RSMD_0805 -> __MyCommonLib1:RSMD_1206_BIG_GAP
- R15: value 4K7 -> 100K; device __MyCommonLib1:RSMD_0805 -> __MyCommonLib1:RSMD_1206_BIG_GAP
- R17, R18: value 1K -> 68R
- R2: value 1K0 -> 300R
- R3: value 10R -> 4K7; device __MyCommonLib1:R0207 -> __MyCommonLib1:RSMD_0805
- R4: value 100R -> 47R; device __MyCommonLib1:RSMD_0805 -> __MyCommonLib1:RSMD_1206_BIG_GAP
- R5: value 1K0 -> 25K; device __MyCommonLib1:RSMD_0805 -> __MyCommonLib1:RSMD_1206_BIG_GAP
- R6: value 1K0 -> 4K7
- R7: value 100R -> 300R; device __MyCommonLib1:RSMD_0805 -> __MyCommonLib1:RSMD_1206_BIG_GAP
- R8: value 68R -> ***; device __MyCommonLib1:RSMD_0805 -> __MyCommonLib1:RSMD_1206_BIG_GAP
- R9: value 68R -> 4K7
- X1: value Target_MCU -> C_X; device __MyCommonLib1:PIN2X5_2.54MM_FEMALE_RIGHT_ANGLE_SMALL_PADS -> con-wago-500:W237-102
- ZD1: value 5.6V -> 3V6
- moved ZD1 489.0 mm to (-299.2, -372.2), flipped to the top
- moved D3 453.4 mm to (-276.6, -298.5), turned to 0 degrees
- moved D4 447.3 mm to (-276.6, -301.6), turned to 0 degrees
- moved R15 431.9 mm to (-283.4, -264.1), turned to 0 degrees
- moved R16 430.7 mm to (-276.6, -267.6), turned to 0 degrees
- moved R14 430.0 mm to (-276.6, -264.1), turned to 0 degrees
- moved R12 411.8 mm to (-276.6, -242.9), turned to 0 degrees
- moved R5 409.3 mm to (-276.6, -224.2), turned to 0 degrees
- moved R11 405.6 mm to (-276.6, -239.4), turned to 0 degrees
- moved R13 403.1 mm to (-276.6, -246.4)
- moved R4 389.3 mm to (-277.4, -188.7), turned to 0 degrees
- moved C6 388.5 mm to (-295.0, -151.7), turned to 0 degrees
- moved R6 388.3 mm to (-290.7, -154.8), turned to 0 degrees
- moved R3 387.4 mm to (-276.6, -195.3), flipped to the bottom, turned to 0 degrees
- moved D2 383.0 mm to (-277.3, -173.4), flipped to the bottom, turned to 0 degrees
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Connections:
- removed net LED1: R18.PAD_0, U$1.12
- removed net LED2: R17.PAD_0, U$1.9
- removed net N$10: J1.PAD_1, X2.2
- removed net RST: R1.PAD_1, U$1.1
- removed net SPI_MISO: DD1.2, R13.PAD_1, T1.3, U$1.17
- removed net SPI_MOSI: D1.CATHODE, DD2.2, U$1.18
- removed net SPI_RST: D3.CATHODE, DD1.1, U$1.16
- removed net SPI_SCK: D4.CATHODE, DD2.1, U$1.19
- removed net T_MISO: R16.PAD_1, X1.3
- removed net T_MOSI: R4.PAD_1, X1.9
- removed net T_RST: R7.PAD_1, X1.6
- removed net T_SCK: R12.PAD_1, X1.1
- removed net T_VCC: C5.PAD_1, C6.PAD_1, D2.CATHODE, DD3.3, R11.PAD_0, R14.PAD_1, R15.PAD_1, R2.PAD_0, R3.PAD_0, R5.PAD_0, R6.PAD_0, SW1.POS_B1, SW1.POS_B2
- new net +5V_FINE: C14.PAD_1, C15.PAD_1, C16.PAD_1, C17.PAD_1, C18.+, C19.PAD_1, C2.PAD_1, IC6.17, IC6.27, IC6.38, IC6.5, R154.PAD_0, R62.PAD_0, R72.PAD_0, R73.PAD_0, T1.3, T2.3, U15.4
- new net -5V_FINE: C1.PAD_0, U15.11
- new net ESR_ADC: C33.PAD_1, R69.PAD_1
- new net ESR_ADC_100X: C39.PAD_1, R71.PAD_1
- new net ESR_ADC_10X: C36.PAD_1, R70.PAD_1
- new net ESR_PWM: C20.PAD_1, R3.PAD_0
- new net L_ADC: C3.PAD_0, D2.CATHODE, R2.PAD_1
- new net L_PWM: C4.PAD_1, R6.PAD_0
- new net MCU_RST: IC6.4, R62.PAD_1
- new net N$110: C13.PAD_1, IC6.8, Q2.2
- new net N$111: C12.PAD_1, IC6.7, Q2.1
- new net N$112: IC6.11, R65.PAD_1
- new net N$113: C21.PAD_1, C22.PAD_1, R4.PAD_1
- new net N$114: C22.PAD_0, C23.PAD_1, D3.CATHODE, D4.ANODE, X1.1
- new net N$115: C23.PAD_0, R11.PAD_0, R5.PAD_1, T5.1
- new net N$116: C25.PAD_1, C26.PAD_1, R12.PAD_0, T5.3
- new net N$117: R13.PAD_1, T5.2
- new net N$118: C26.PAD_0, R14.PAD_1, R15.PAD_0, T6.1
- new net N$119: C29.PAD_1, C34.PAD_1, R16.PAD_0, T6.3
- new net N$120: R63.PAD_1, T6.2
- new net N$121: C29.PAD_0, R64.PAD_1, R66.PAD_0, T7.1
- new net N$122: C37.PAD_1, R67.PAD_0, T7.3
- new net N$123: R68.PAD_1, T7.2
- new net N$124: C32.PAD_1, D6.CATHODE, R69.PAD_0
- new net N$125: C25.PAD_0, D5.CATHODE, D6.ANODE
- new net N$126: C24.PAD_0, R11.PAD_1, R12.PAD_1, R154.PAD_1
- new net N$127: C35.PAD_1, D14.CATHODE, R70.PAD_0
- new net N$128: C34.PAD_0, D13.CATHODE, D14.ANODE
- new net N$129: C27.PAD_0, R15.PAD_1, R16.PAD_1, R72.PAD_1
- new net N$130: C38.PAD_1, D16.CATHODE, R71.PAD_0
- new net N$131: C37.PAD_0, D15.CATHODE, D16.ANODE
- new net N$132: J11.PAD_1, X6.2
- new net N$134: C30.PAD_0, R66.PAD_1, R67.PAD_1, R73.PAD_1
- net +5V_USB: now also X5.1, X6.1; no longer C3.PAD_1, C4.PAD_1, DD1.3, DD2.3, R1.PAD_0, R13.PAD_0, SW1.CENTER1, SW1.CENTER2, SW1.POS_A1, SW1.POS_A2, U$1.20, X2.1, X3.1, ZD1.CATHODE
- net GND: now also C1.PAD_1, C12.PAD_0, C13.PAD_0, C14.PAD_0, C15.PAD_0, C16.PAD_0, C17.PAD_0, C18.-, C19.PAD_0, C21.PAD_0, C24.PAD_1, C27.PAD_1, C3.PAD_1, C30.PAD_1, C32.PAD_0, C33.PAD_0, C35.PAD_0, C36.PAD_0, C38.PAD_0, C39.PAD_0, D13.ANODE, D15.ANODE, D3.ANODE, D4.CATHODE, D5.ANODE, IC6.18, IC6.28, IC6.39, IC6.6, R13.PAD_0, R14.PAD_0, R5.PAD_0, R63.PAD_0, R64.PAD_0, R68.PAD_0, R9.PAD_1, T3.3, T4.3, U15.10, U15.12, U15.3, U15.5, X4.2, X5.4, X5.PACKAGE_PAD1, X5.PACKAGE_PAD2, X6.5, X6.PACKAGE1, X6.PACKAGE2, X6.PACKAGE3, X6.PACKAGE4, X6.PACKAGE5, ZD4.ANODE; no longer C1.PAD_0, C3.PAD_0, C4.PAD_0, C6.PAD_0, LED1.CATHODE, LED2.CATHODE, LED3.CATHODE, U$1.10, X1.10, X2.5, X2.PACKAGE1, X2.PACKAGE2, X2.PACKAGE3, X2.PACKAGE4, X2.PACKAGE5, X3.4, X3.PACKAGE_PAD1, X3.PACKAGE_PAD2, ZD2.ANODE, ZD3.ANODE
- net N$1: now also U15.13, U15.14; no longer C2.PAD_1, Q1.2, U$1.5
- net N$11: now also R7.PAD_0, T2.2, T3.2; no longer DD3.2, R14.PAD_0, T1.1
- net N$12: now also D1.CATHODE, R7.PAD_1, X4.1; no longer LED1.ANODE, R5.PAD_1
- net N$13: now also R8.PAD_0; no longer R2.PAD_1, R4.PAD_0
- net N$2: now also U15.8, U15.9; no longer D4.ANODE, R11.PAD_1, R12.PAD_0
- net N$25: now also C5.PAD_1, R10.PAD_0, R8.PAD_1, R9.PAD_0; no longer R3.PAD1, X1.4
- net N$3: now also U15.6, U15.7; no longer C1.PAD_1, Q1.1, U$1.4
- net N$39: now also R4.PAD_0, T1.2, T4.2; no longer D3.ANODE, R6.PAD_1, R7.PAD_0
- net N$4: now also C6.PAD_1, R1.PAD_0, R10.PAD_1, U15.2; no longer R8.PAD_0, U$1.6
- net N$5: now also C6.PAD_0, R1.PAD_1, R2.PAD_0, U15.1; no longer R9.PAD_1, U$1.7
- net N$6: now also C20.PAD_0, R3.PAD_1, T1.1, T4.1; no longer R10.PAD_1, U$1.8
- net N$7: now also IC6.13, R17.PAD_0; no longer LED2.ANODE, R17.PAD_1
- net N$8: now also IC6.12; no longer LED3.ANODE
- net N$9: now also C4.PAD_0, R6.PAD_1, T2.1, T3.1; no longer DD3.1, R15.PAD_0, R16.PAD_0, T1.2
- net USB_D+: now also R17.PAD_1, X5.3, X6.3, ZD4.CATHODE; no longer R8.PAD_1, X2.3, X3.3, ZD2.CATHODE
- net USB_D-: now also J11.PAD_0, R18.PAD_0, R65.PAD_0, X5.2, ZD1.CATHODE; no longer J1.PAD_0, R10.PAD_0, R9.PAD_0, X3.2, ZD3.CATHODE
Routing:
- net T_VCC: track 38.5 -> 0.00 mm
- net GND: track 198.1 -> 170.4 mm
- net SPI_RST: track 22.7 -> 0.00 mm
- net SPI_MISO: track 21.9 -> 0.00 mm
- net USB_D+: track 20.0 -> 0.00 mm
- net USB_D-: track 16.9 -> 0.00 mm
- net +5V_USB: track 16.2 -> 0.00 mm
- net N$39: track 15.8 -> 0.00 mm
- net N$9: track 14.6 -> 0.00 mm
- net N$13: track 12.3 -> 0.00 mm
- net N$25: track 11.4 -> 0.00 mm
- net N$3: track 11.1 -> 0.00 mm
- net SPI_MOSI: track 10.2 -> 0.00 mm
- net N$5: track 10.1 -> 0.00 mm
- net N$6: track 9.84 -> 0.00 mm
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
Commit message: LCMeter Another changes
Parts:
- added C105, C43: 470uFx16V, __MyCommonLib1:CE_10MM
- added C28: 1n0*, __MyCommonLib1:RSMD_0805
- added C31, C40, C42: 0.47uFx16V, __MyCommonLib1:RSMD_0805
- added C41: 1000uFx16V, __MyCommonLib1:CE_10MM
- added D104, D17, D18: FR207, __MyCommonLib1:DO-41_10MM
- added IC12: MC34063, __MyCommonLib1:SOIC8
- added R110: 0.62R, __MyCommonLib1:RSMD_1206_BIG_GAP
- added R74: 5K1, __MyCommonLib1:RSMD_1206_BIG_GAP
- added R75: 1K7, __MyCommonLib1:RSMD_1206_BIG_GAP
- added TR1: TRANS, __MyCommonLib1:RING_25X10_3WIND_HOR
Connections:
- new net N$10: D104.CATHODE, IC12.2, TR1.W1_END
- new net N$133: IC12.1, IC12.7, IC12.8, R110.PAD_1
- new net N$135: C28.PAD_1, IC12.3
- new net N$136: D18.ANODE, TR1.W3_START
- new net N$137: C105.-, C31.PAD_1, D104.ANODE
- new net N$138: D17.ANODE, TR1.W2_START
- new net N$139: IC12.5, R74.PAD_0, R75.PAD_1
- net +5V_USB: now also C40.PAD_1, C41.+, IC12.6, R110.PAD_0
- net GND: now also C105.+, C28.PAD_0, C31.PAD_0, C40.PAD_0, C41.-, C42.PAD_0, C43.-, IC12.4, R75.PAD_0, TR1.W1_START, TR1.W2_END, TR1.W3_END
- net VCC_ROUGH: now also C42.PAD_1, C43.+, D18.CATHODE, R74.PAD_1
Changed lines of the file:
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@@
 <element name="X6" library="__MyCommonLib1" package="USB_MICRO_TYPE_B" value="USB_MICRO" x="-295.8" y="-403.4"/>
 <element name="J11" library="__MyCommonLib1" package="RSMD_0805" value="0" x="-293.2" y="-409"/>
+<element name="IC12" library="__MyCommonLib1" package="SOIC8" value="MC34063" x="-306.9" y="-405.2"/>
+<element name="TR1" library="__MyCommonLib1" package="RING_25X10_3WIND_HOR" value="TRANS" x="-296.6" y="-422.7"/>
+<element name="C28" library="__MyCommonLib1" package="RSMD_0805" value="1n0*" x="-308.4" y="-437.1"/>
+<element name="D104" library="__MyCommonLib1" package="DO-41_10MM" value="FR207" x="-304.3" y="-442.7"/>
+<element name="C31" library="__MyCommonLib1" package="RSMD_0805" value="0.47uFx16V" x="-308.4" y="-446"/>
+<element name="C105" library="__MyCommonLib1" package="CE_10MM" value="470uFx16V" x="-315.6" y="-440.3"/>
+<element name="R110" library="__MyCommonLib1" package="RSMD_1206_BIG_GAP" value="0.62R" x="-318.6" y="-449.1"/>
+<element name="C40" library="__MyCommonLib1" package="RSMD_0805" value="0.47uFx16V" x="-319.4" y="-452.6"/>
+<element name="C41" library="__MyCommonLib1" package="CE_10MM" value="1000uFx16V" x="-326.5" y="-446.9"/>
+<element name="D17" library="__MyCommonLib1" package="DO-41_10MM" value="FR207" x="-325.4" y="-458.2"/>
+<element name="D18" library="__MyCommonLib1" package="DO-41_10MM" value="FR207" x="-325.4" y="-464.1"/>
+<element name="C42" library="__MyCommonLib1" package="RSMD_0805" value="0.47uFx16V" x="-329.5" y="-467.4"/>
+<element name="C43" library="__MyCommonLib1" package="CE_10MM" value="470uFx16V" x="-336.6" y="-461.7"/>
+<element name="R74" library="__MyCommonLib1" package="RSMD_1206_BIG_GAP" value="5K1" x="-338.8" y="-470.5"/>
+<element name="R75" library="__MyCommonLib1" package="RSMD_1206_BIG_GAP" value="1K7" x="-338.8" y="-474"/>
 </elements>
 <signals>
@@
 <contactref element="X6" pad="PACKAGE2"/>
 <contactref element="X6" pad="5"/>
+<contactref element="TR1" pad="W1_START"/>
+<contactref element="IC12" pad="4"/>
+<contactref element="C28" pad="PAD_0"/>
+<contactref element="TR1" pad="W2_END"/>
+<contactref element="TR1" pad="W3_END"/>
+<contactref element="C31" pad="PAD_0"/>
+<contactref element="C105" pad="+"/>
+<contactref element="C40" pad="PAD_0"/>
+<contactref element="C41" pad="-"/>
+<contactref element="C42" pad="PAD_0"/>
+<contactref element="C43" pad="-"/>
+<contactref element="R75" pad="PAD_0"/>
 <wire x1="-274.975" y1="-246.4" x2="-274.975" y2="-224.2" width="0" layer="19" extent="16-16"/>
 <wire x1="-276.85" y1="-249.9" x2="-274.975" y2="-246.4" width="0" layer="19" extent="16-16"/>
@@
 <wire x1="-290.8" y1="-398.7" x2="-294.5" y2="-398.2" width="0" layer="19" extent="1-1"/>
 <wire x1="-290.8" y1="-402.1" x2="-290.8" y2="-398.7" width="0" layer="19" extent="1-1"/>
+<wire x1="-309.59875" y1="-407.105" x2="-300.8" y2="-402.1" width="0" layer="19" extent="1-1"/>
+<wire x1="-308.9825" y1="-422.7" x2="-309.59875" y2="-407.105" width="0" layer="19" extent="1-1"/>
+<wire x1="-309.45" y1="-437.1" x2="-308.9825" y2="-422.7" width="0" layer="19" extent="1-1"/>
+<wire x1="-313.06" y1="-440.3" x2="-309.45" y2="-437.1" width="0" layer="19" extent="1-1"/>
+<wire x1="-309.45" y1="-446" x2="-313.06" y2="-440.3" width="0" layer="19" extent="1-1"/>
+<wire x1="-320.45" y1="-452.6" x2="-309.45" y2="-446" width="0" layer="19" extent="1-1"/>
+<wire x1="-329.04" y1="-446.9" x2="-320.45" y2="-452.6" width="0" layer="19" extent="1-1"/>
+<wire x1="-293.1075" y1="-425.24" x2="-308.9825" y2="-422.7" width="0" layer="19" extent="1-1"/>
+<wire x1="-293.1075" y1="-420.16" x2="-293.1075" y2="-425.24" width="0" layer="19" extent="1-1"/>
+<wire x1="-330.55" y1="-467.4" x2="-320.45" y2="-452.6" width="0" layer="19" extent="1-1"/>
+<wire x1="-339.14" y1="-461.7" x2="-330.55" y2="-467.4" width="0" layer="19" extent="1-1"/>
+<wire x1="-340.425" y1="-474" x2="-330.55" y2="-467.4" width="0" layer="19" extent="1-1"/>
 <wire x1="-261.5" y1="-89.17" x2="-285" y2="-145.4" width="0" layer="19" extent="16-16"/>
 <wire x1="-248.2" y1="-88.37" x2="-261.5" y2="-89.17" width="0" layer="19" extent="1-1"/>
@@
 <contactref element="X5" pad="1"/>
 <contactref element="X6" pad="1"/>
+<contactref element="R110" pad="PAD_0"/>
+<contactref element="IC12" pad="6"/>
+<contactref element="C40" pad="PAD_1"/>
+<contactref element="C41" pad="+"/>
+<wire x1="-297.1" y1="-398.2" x2="-304.20125" y2="-405.835" width="0" layer="19" extent="1-1"/>
 <wire x1="-292.63" y1="-379.66" x2="-297.1" y2="-398.2" width="0" layer="19" extent="1-1"/>
+<wire x1="-323.96" y1="-446.9" x2="-304.20125" y2="-405.835" width="0" layer="19" extent="1-1"/>
+<wire x1="-320.225" y1="-449.1" x2="-323.96" y2="-446.9" width="0" layer="19" extent="1-1"/>
+<wire x1="-318.35" y1="-452.6" x2="-320.225" y2="-449.1" width="0" layer="19" extent="1-1"/>
 </signal>
 <signal name="USB_D-">
@@
 <contactref element="D12" pad="CATHODE"/>
 <contactref element="D11" pad="CATHODE"/>
+<contactref element="D18" pad="CATHODE"/>
+<contactref element="C43" pad="+"/>
+<contactref element="C42" pad="PAD_1"/>
+<contactref element="R74" pad="PAD_1"/>
 <wire x1="-200.825" y1="-33" x2="-200.125" y2="-38.4" width="0" layer="19" extent="16-16"/>
 <wire x1="-200.525" y1="-28.9" x2="-200.825" y2="-33" width="0" layer="19" extent="16-16"/>
@@
 <wire x1="-131.325" y1="23.20125" x2="-138.945" y2="23.20125" width="0" layer="19" extent="16-16"/>
 <wire x1="-117.725" y1="23.20125" x2="-125.345" y2="23.20125" width="0" layer="19" extent="16-16"/>
+<wire x1="-320.32" y1="-464.1" x2="-200.125" y2="-38.4" width="0" layer="19" extent="16-16"/>
+<wire x1="-328.45" y1="-467.4" x2="-320.32" y2="-464.1" width="0" layer="19" extent="1-1"/>
+<wire x1="-334.06" y1="-461.7" x2="-328.45" y2="-467.4" width="0" layer="19" extent="1-1"/>
+<wire x1="-337.175" y1="-470.5" x2="-328.45" y2="-467.4" width="0" layer="19" extent="1-1"/>
 </signal>
 <signal name="LED_SCK'">
@@
 <wire x1="-296.45" y1="-398.2" x2="-292.15" y2="-409" width="0" layer="19" extent="1-1"/>
 </signal>
+<signal name="N$10">
+<contactref element="IC12" pad="2"/>
+<contactref element="TR1" pad="W1_END"/>
+<contactref element="D104" pad="CATHODE"/>
+<wire x1="-301.045" y1="-422.7" x2="-299.22" y2="-442.7" width="0" layer="19" extent="1-1"/>
+<wire x1="-309.59875" y1="-404.565" x2="-301.045" y2="-422.7" width="0" layer="19" extent="1-1"/>
+</signal>
+<signal name="N$133">
+<contactref element="IC12" pad="1"/>
+<contactref element="IC12" pad="8"/>
+<contactref element="R110" pad="PAD_1"/>
+<contactref element="IC12" pad="7"/>
+<wire x1="-304.20125" y1="-403.295" x2="-309.59875" y2="-403.295" width="0" layer="19" extent="1-1"/>
+<wire x1="-304.20125" y1="-404.565" x2="-304.20125" y2="-403.295" width="0" layer="19" extent="1-1"/>
+<wire x1="-316.975" y1="-449.1" x2="-304.20125" y2="-404.565" width="0" layer="19" extent="1-1"/>
+</signal>
+<signal name="N$135">
+<contactref element="IC12" pad="3"/>
+<contactref element="C28" pad="PAD_1"/>
+<wire x1="-309.59875" y1="-405.835" x2="-307.35" y2="-437.1" width="0" layer="19" extent="1-1"/>
+</signal>
+<signal name="N$137">
+<contactref element="D104" pad="ANODE"/>
+<contactref element="C31" pad="PAD_1"/>
+<contactref element="C105" pad="-"/>
+<wire x1="-309.38" y1="-442.7" x2="-318.14" y2="-440.3" width="0" layer="19" extent="1-1"/>
+<wire x1="-307.35" y1="-446" x2="-309.38" y2="-442.7" width="0" layer="19" extent="1-1"/>
+</signal>
+<signal name="N$136">
+<contactref element="D18" pad="ANODE"/>
+<contactref element="TR1" pad="W3_START"/>
+<wire x1="-330.48" y1="-464.1" x2="-285.17" y2="-427.78" width="0" layer="19" extent="1-1"/>
+</signal>
+<signal name="N$138">
+<contactref element="TR1" pad="W2_START"/>
+<contactref element="D17" pad="ANODE"/>
+<wire x1="-330.48" y1="-458.2" x2="-285.17" y2="-417.62" width="0" layer="19" extent="1-1"/>
+</signal>
+<signal name="N$139">
+<contactref element="IC12" pad="5"/>
+<contactref element="R75" pad="PAD_1"/>
+<contactref element="R74" pad="PAD_0"/>
+<wire x1="-340.425" y1="-470.5" x2="-304.20125" y2="-407.105" width="0" layer="19" extent="1-1"/>
+<wire x1="-337.175" y1="-474" x2="-340.425" y2="-470.5" width="0" layer="19" extent="1-1"/>
+</signal>
 </signals>
