File: LC_METER/schematic/LCMeter.brd (EAGLE design)
At the start: 60.5 x 30 mm, 179 parts, among them IC1 74HC595, IC12 MC34063, IC2 74HC595, IC3 74HC595, IC4 74HC595, IC5 74HC595, IC6 MEGA8535, J10 0, J11 0, J123 0, J2 0, J3 0, J4 0, J5 0, J6 0, J7 0, J8 0, J9 0, Q2 12MHz, T1 BC847, T2 BC847, T3 BC857, T4 BC857, T5 BC847, T6 BC847, T7 BC847, U15 LM324, X1 C_X, X4 L_X, X5 USB_B, X6 USB_MICRO

Commit message: LCMeter schematic is almost complete
Parts:
- added C215, C51, C52, C53: 22uFx16V, __MyCommonLib1:CE_6.3MM
- added C44, C46, C49: 0.47uFx16V, __MyCommonLib1:RSMD_0805
- added C45, C47, C48: 470uFx16V, __MyCommonLib1:CE_10MM
- added C50: 0.1uF, __MyCommonLib1:RSMD_0805
- added C54, C55: 0.47uF, __MyCommonLib1:RSMD_0805
- added D19, D20, D21, D22, D23, D24, D25, D26, D27, D28: LL4148, __MyCommonLib1:SOD-80
- added IC15: LM317, __MyCommonLib1:D2PAK
- added IC16: 7905, __MyCommonLib1:D2PAK
- added KEY1: MODE, __MyCommonLib1:KEY_7X4.5
- added KEY2: RANGE, __MyCommonLib1:KEY_7X4.5
- added KEY3: RESERVED, __MyCommonLib1:KEY_7X4.5
- added R76: 5K1, __MyCommonLib1:RSMD_1206_BIG_GAP
- added R77: 1K7, __MyCommonLib1:RSMD_1206_BIG_GAP
- added R78, R79, R80, R81, R82, R83: 4K7, __MyCommonLib1:RSMD_0805
- added X2: MCU_PROGRAMMING, __MyCommonLib1:PIN2X3_2.54MM
- moved Q2 63.1 mm to (-182.4, -51.2), turned to 180 degrees
Connections:
- removed net ESR_ADC: C33.PAD_1, R69.PAD_1
- new net ESR_ADC_1X: C33.PAD_1, D23.CATHODE, D24.ANODE, IC6.32, R69.PAD_1
- new net KEY_MODE: IC6.25, R81.PAD_1
- new net KEY_RANGE: IC6.26, R82.PAD_1
- new net KEY_RESERVED: IC6.24, R83.PAD_1
- new net MCU_MISO: IC6.2, X2.6
- new net MCU_MOSI: IC6.1, X2.3
- new net MCU_SCK: IC6.3, X2.4
- new net N$140: C44.PAD_1, C45.+, D17.CATHODE, IC15.3
- new net N$141: C50.PAD_1, IC6.29
- new net N$142: IC15.1, R76.PAD_1, R77.PAD_1
- new net N$144: KEY1.1, KEY1.2, R80.PAD_0, R81.PAD_0
- new net N$145: KEY2.1, KEY2.2, R79.PAD_0, R82.PAD_0
- new net N$146: KEY3.1, KEY3.2, R78.PAD_0, R83.PAD_0
- net +5V_FINE: now also C46.PAD_1, C47.+, C54.PAD_0, C55.PAD_0, D20.CATHODE, D22.CATHODE, D24.CATHODE, D26.CATHODE, D27.CATHODE, IC15.2, R76.PAD_0, R78.PAD_1, R79.PAD_1, R80.PAD_1, X2.5
- net -5V_FINE: now also C48.-, C49.PAD_1, IC16.3
- net ESR_ADC_100X: now also D19.CATHODE, D20.ANODE, IC6.30
- net ESR_ADC_10X: now also D21.CATHODE, D22.ANODE, IC6.31
- net ESR_PWM: now also D27.ANODE, D28.CATHODE, IC6.13
- net GND: now also C215.-, C44.PAD_0, C45.-, C46.PAD_0, C47.-, C48.+, C49.PAD_0, C50.PAD_0, C51.-, C52.-, C53.+, C54.PAD_1, C55.PAD_1, D19.ANODE, D21.ANODE, D23.ANODE, D25.ANODE, D28.ANODE, IC16.1, KEY1.3, KEY1.4, KEY2.3, KEY2.4, KEY3.3, KEY3.4, R77.PAD_0, X2.1
- net LED_DATA: now also IC6.41
- net LED_LATCH: now also IC6.40
- net LED_SCK: now also IC6.42
- net L_ADC: now also IC6.37
- net L_PWM: now also D25.CATHODE, D26.ANODE, IC6.14
- net MCU_RST: now also X2.2
- net N$124: now also C52.+
- net N$127: now also C51.+
- net N$130: now also C215.+
- net N$137: now also IC16.2
- net N$25: now also C53.-
- net N$7: now also IC6.10; no longer IC6.13
Routing:
- net GND: track 170.4 -> 64.9 mm, vias 2 -> 0
- removed copper zone on layer 16, net +5V_USB
- removed copper zone on layer 16, net GND
- removed copper zone on layer 16, net T_VCC
Other:
- board outline removed
- board text removed: "1"
- board text removed: "GND"
- board text removed: "VCC"

Commit message: LCMeter start routing
Parts:
- removed C105: 470uFx16V, __MyCommonLib1:CE_10MM
- removed C215: 22uFx16V, __MyCommonLib1:CE_6.3MM
- removed D104, D17: FR207, __MyCommonLib1:DO-41_10MM
- removed D19, D21: LL4148, __MyCommonLib1:SOD-80
- removed IC12: MC34063, __MyCommonLib1:SOIC8
- removed IC15: LM317, __MyCommonLib1:D2PAK
- removed IC16: 7905, __MyCommonLib1:D2PAK
- removed J123: 0, __MyCommonLib1:RSMD_1206_BIG_GAP
- removed Q2: 12MHz, crystal:HC49U-V
- removed R110: 0.62R, __MyCommonLib1:RSMD_1206_BIG_GAP
- removed R154: 100R, __MyCommonLib1:RSMD_1206_BIG_GAP
- removed U15: LM324, __MyCommonLib1:SOIC14
- removed X6: USB_MICRO, __MyCommonLib1:USB_MICRO_TYPE_B
- removed ZD4: 3V6, __MyCommonLib1:SOD-80
- added C56: 0.47uFx16V, __MyCommonLib1:RSMD_1206_BIG_GAP
- added C57: 470uFx16V, __MyCommonLib1:CE_10MM
- added D29: FR207, __MyCommonLib1:DO-41_10MM
- added IC10: MC34063, __MyCommonLib1:SOIC8
- added IC7: LM324, __MyCommonLib1:SOIC14
- added IC8: 7905, __MyCommonLib1:D2PAK
- added IC9: LM317, __MyCommonLib1:D2PAK
- added J1: 0, __MyCommonLib1:RSMD_1206_BIG_GAP
- added Q1: 12MHz, crystal:HC49U-V
- added R84: 5K1, __MyCommonLib1:RSMD_0805
- added R85: 1K7, __MyCommonLib1:RSMD_0805
- added X3: C_X, con-wago-500:W237-102
- added ZD2: 3V6, __MyCommonLib1:SOD-80
- C1, C2: value 0.1uF -> 22pF
- C12, C13: value 22pF -> 0.1uF
- C15, C38: value 0.1uF -> 0.47uF
- C17, C39: value 0.1uF -> 1nF
- C18: value 4.7uF -> 22uFx16V
- C19: value 0.1uF -> 0.47uF; device __MyCommonLib1:RSMD_0805 -> __MyCommonLib1:RSMD_1206_BIG_GAP
- C20: value 1nF -> 0.1uF
- C21: value 22nF* -> 0.1uF
- C22: value 1.0uF -> 0.1uF; device __MyCommonLib1:RSMD_1206_BIG_GAP -> __MyCommonLib1:RSMD_0805
- C27, C30, C33: value 0.1uF -> 22uFx16V; device __MyCommonLib1:RSMD_0805 -> __MyCommonLib1:CE_6.3MM
- C28: value 1n0* -> 0.1uF
- C31, C42: value 0.47uFx16V -> 0.1uF
- C4: value 1nF -> 4.7uF; device __MyCommonLib1:RSMD_0805 -> __MyCommonLib1:CE_6.3MM
- C40: value 0.47uFx16V -> 1.0uF; device __MyCommonLib1:RSMD_0805 -> __MyCommonLib1:RSMD_1206_BIG_GAP
- C41: value 1000uFx16V -> 0.1uF; device __MyCommonLib1:CE_10MM -> __MyCommonLib1:RSMD_0805
- C43: value 470uFx16V -> 0.1uF; device __MyCommonLib1:CE_10MM -> __MyCommonLib1:RSMD_0805
- C44: value 0.47uFx16V -> 22nF*
- C45, C47: value 470uFx16V -> 0.47uFx16V; device __MyCommonLib1:CE_10MM -> __MyCommonLib1:RSMD_0805
- C46: value 0.47uFx16V -> 470uFx16V; device __MyCommonLib1:RSMD_0805 -> __MyCommonLib1:CE_10MM
- C48: value 470uFx16V -> 47uFx16V; device __MyCommonLib1:CE_10MM -> __MyCommonLib1:CE_6.3MM
- C49: device __MyCommonLib1:RSMD_0805 -> __MyCommonLib1:RSMD_1206
- C5: value 0.47uF -> 0.1uF; device __MyCommonLib1:RSMD_1206_BIG_GAP -> __MyCommonLib1:RSMD_0805
- C50: value 0.1uF -> 470uFx16V; device __MyCommonLib1:RSMD_0805 -> __MyCommonLib1:CE_10MM
- C51: value 22uFx16V -> 0.47uFx16V; device __MyCommonLib1:CE_6.3MM -> __MyCommonLib1:RSMD_0805
- C52: value 22uFx16V -> 47uFx16V; device __MyCommonLib1:CE_6.3MM -> __MyCommonLib1:CE_10MM
- C53: value 22uFx16V -> 1000uFx16V; device __MyCommonLib1:CE_6.3MM -> __MyCommonLib1:CE_10MM
- C54: value 0.47uF -> 0.47uFx16V; device __MyCommonLib1:RSMD_0805 -> __MyCommonLib1:RSMD_1206
- C55: value 0.47uF -> 1n0*
- D18: value FR207 -> LL4148; device __MyCommonLib1:DO-41_10MM -> __MyCommonLib1:SOD-80
- D27, D28: value LL4148 -> FR207; device __MyCommonLib1:SOD-80 -> __MyCommonLib1:DO-41_10MM
- IC1: value 74HC595 -> MEGA8535; device __MyCommonLib1:SOIC16 -> atmel:TQFP44
- IC6: value MEGA8535 -> 74HC595; device atmel:TQFP44 -> __MyCommonLib1:SOIC16
- R1: value 100K -> 4K7
- R10: value 20K -> 68R
- R11, R15: value 100K -> 560R; device __MyCommonLib1:RSMD_1206_BIG_GAP -> __MyCommonLib1:RSMD_0805
- R12, R16: value 1K0 -> 560R; device __MyCommonLib1:RSMD_1206_BIG_GAP -> __MyCommonLib1:RSMD_0805
- R13: value 100R -> 560R; device __MyCommonLib1:RSMD_1206_BIG_GAP -> __MyCommonLib1:RSMD_0805
- R14: value 25K -> 560R; device __MyCommonLib1:RSMD_1206_BIG_GAP -> __MyCommonLib1:RSMD_0805
- R17: value 68R -> 300R
- R18: value 68R -> 560R
- R19, R21: value 560R -> 300R
- R2, R60: value 300R -> 4K7
- R4: value 47R -> 4K7; device __MyCommonLib1:RSMD_1206_BIG_GAP -> __MyCommonLib1:RSMD_0805
- R5: value 25K -> 4K7; device __MyCommonLib1:RSMD_1206_BIG_GAP -> __MyCommonLib1:RSMD_0805
- R54: value 560R -> 100K
- R55: value 560R -> 4K7
- R56: value 560R -> 300R; device __MyCommonLib1:RSMD_0805 -> __MyCommonLib1:RSMD_1206_BIG_GAP
- R57: value 560R -> ***; device __MyCommonLib1:RSMD_0805 -> __MyCommonLib1:RSMD_1206_BIG_GAP
- R58: value 560R -> 20K
- R61: value 300R -> 1K0
- R62: value 4K7 -> 1K0
- R63, R68, R72: value 100R -> 1K0; device __MyCommonLib1:RSMD_1206_BIG_GAP -> __MyCommonLib1:RSMD_0805
- R64: value 25K -> 100R
- R65: value 1K5 -> 100R; device __MyCommonLib1:RSMD_0805 -> __MyCommonLib1:RSMD_1206_BIG_GAP
- R66: value 100K -> 100R
- R67, R69, R71: value 1K0 -> 100K; device __MyCommonLib1:RSMD_1206_BIG_GAP -> __MyCommonLib1:RSMD_0805
- R7: value 300R -> 4K7; device __MyCommonLib1:RSMD_1206_BIG_GAP -> __MyCommonLib1:RSMD_0805
- R70: device __MyCommonLib1:RSMD_1206_BIG_GAP -> __MyCommonLib1:RSMD_0805
- R73: value 100R -> 47R
- R74: value 5K1 -> 4K7; device __MyCommonLib1:RSMD_1206_BIG_GAP -> __MyCommonLib1:RSMD_0805
- R75, R77: value 1K7 -> 25K; device __MyCommonLib1:RSMD_1206_BIG_GAP -> __MyCommonLib1:RSMD_0805
- R76: value 5K1 -> 100R; device __MyCommonLib1:RSMD_1206_BIG_GAP -> __MyCommonLib1:RSMD_0805
- R78, R80: value 4K7 -> 100R
- R79: value 4K7 -> 25K
- R8: value *** -> 68R; device __MyCommonLib1:RSMD_1206_BIG_GAP -> __MyCommonLib1:RSMD_0805
- R81: value 4K7 -> 5K1; device __MyCommonLib1:RSMD_0805 -> __MyCommonLib1:RSMD_1206_BIG_GAP
- R82: value 4K7 -> 1K7; device __MyCommonLib1:RSMD_0805 -> __MyCommonLib1:RSMD_1206_BIG_GAP
- R83: value 4K7 -> 0.62R; device __MyCommonLib1:RSMD_0805 -> __MyCommonLib1:RSMD_1206_BIG_GAP
- R9: value 4K7 -> 1K5
- T2, T7: value BC847 -> BC857
- T3, T4: value BC857 -> BC847
- X1: value C_X -> MCU_PROGRAMMING; device con-wago-500:W237-102 -> __MyCommonLib1:PIN2X3_2.54MM
- X2: value MCU_PROGRAMMING -> L_X; device __MyCommonLib1:PIN2X3_2.54MM -> con-wago-500:W237-102
- X4: value L_X -> USB_MICRO; device con-wago-500:W237-102 -> __MyCommonLib1:USB_MICRO_TYPE_B
- moved R83 792.7 mm to (24.0, 81.0), flipped to the bottom, turned to 180 degrees
- moved R80 775.6 mm to (66.0, 33.0), flipped to the bottom
- moved R79 775.5 mm to (66.0, 36.0), flipped to the bottom
- moved R78 761.8 mm to (66.0, 23.0), flipped to the bottom
- moved D28 760.1 mm to (52.0, 67.0)
- moved C54 749.8 mm to (14.0, 80.0), flipped to the bottom, turned to 90 degrees
- moved C55 748.8 mm to (21.0, 70.0), flipped to the bottom, turned to 180 degrees
- moved C53 735.3 mm to (7.00, 79.0)
- moved D27 728.7 mm to (23.0, 53.0)
- moved X2 719.8 mm to (6.00, 4.90), turned to 180 degrees
- moved C49 710.8 mm to (52.0, 64.0), flipped to the bottom, turned to 180 degrees
- moved D22 708.9 mm to (49.5, 35.0), flipped to the bottom, turned to 90 degrees
- moved C50 708.7 mm to (51.0, 59.0)
- moved D26 704.7 mm to (56.0, 4.00), flipped to the bottom, turned to 90 degrees
- moved D25 704.4 mm to (59.0, 4.00), flipped to the bottom, turned to 270 degrees
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Connections:
- removed net N$98 (its old number): IC1.9, IC2.14
- new net N$99: IC5.9, IC6.14
- net +5V_FINE: now also C15.PAD_0, C21.PAD_1, C38.PAD_0, C4.+, C5.PAD_1, C51.PAD_1, C52.+, C6.PAD_1, C7.PAD_1, C8.PAD_1, C9.PAD_1, D11.CATHODE, D12.CATHODE, D13.CATHODE, D23.CATHODE, D7.CATHODE, IC1.17, IC1.27, IC1.38, IC1.5, IC7.4, IC9.2, R1.PAD_0, R2.PAD_1, R3.PAD_1, R4.PAD_1, R64.PAD_0, R65.PAD_0, R66.PAD_0, R81.PAD_0, T3.3, X1.5; no longer C14.PAD_1, C15.PAD_1, C16.PAD_1, C17.PAD_1, C18.+, C19.PAD_1, C2.PAD_1, C46.PAD_1, C47.+, C54.PAD_0, C55.PAD_0, D20.CATHODE, D22.CATHODE, D24.CATHODE, D26.CATHODE, D27.CATHODE, IC15.2, IC6.17, IC6.27, IC6.38, IC6.5, R154.PAD_0, R62.PAD_0, R72.PAD_0, R73.PAD_0, R76.PAD_0, R78.PAD_1, R79.PAD_1, R80.PAD_1, T2.3, U15.4, X2.5
- net +5V_USB: now also C53.+, C54.PAD_1, IC10.6, R83.PAD_0, X4.1; no longer C40.PAD_1, C41.+, IC12.6, R110.PAD_0, X6.1
- net -5V_FINE: now also C25.PAD_0, C47.PAD_1, IC7.11, IC8.3; no longer C1.PAD_0, C49.PAD_1, IC16.3, U15.11
- net ESR_ADC_100X: now also C32.PAD_1, D13.ANODE, IC1.30, R63.PAD_1; no longer C39.PAD_1, D19.CATHODE, D20.ANODE, IC6.30, R71.PAD_1
- net ESR_ADC_10X: now also C29.PAD_1, D12.ANODE, IC1.31, R62.PAD_1; no longer C36.PAD_1, D21.CATHODE, D22.ANODE, IC6.31, R70.PAD_1
- net ESR_ADC_1X: now also C26.PAD_1, D11.ANODE, IC1.32, R61.PAD_1; no longer C33.PAD_1, D23.CATHODE, D24.ANODE, IC6.32, R69.PAD_1
- net ESR_PWM: now also C39.PAD_1, D23.ANODE, D24.CATHODE, IC1.13, R74.PAD_0; no longer C20.PAD_1, D27.ANODE, D28.CATHODE, IC6.13, R3.PAD_0
- net GND: now also C1.PAD_0, C15.PAD_1, C18.+, C20.PAD_1, C25.PAD_1, C26.PAD_0, C27.-, C29.PAD_0, C3.PAD_0, C30.-, C33.-, C34.PAD_0, C35.PAD_1, C36.PAD_1, C37.PAD_1, C38.PAD_1, C4.-, C45.PAD_0, C46.+, C47.PAD_0, C50.-, C51.PAD_0, C53.-, C54.PAD_0, C55.PAD_0, C56.PAD_0, C57.-, C6.PAD_0, D10.ANODE, D18.ANODE, D20.ANODE, D22.ANODE, D24.ANODE, D26.CATHODE, D4.ANODE, D6.ANODE, IC1.18, IC1.28, IC1.39, IC1.6, IC10.4, IC6.13, IC6.8, IC7.10, IC7.12, IC7.3, IC7.5, IC8.1, R60.PAD_1, R76.PAD_0, R78.PAD_0, R79.PAD_0, R80.PAD_0, R82.PAD_0, R85.PAD_0, T2.3, T7.3, X1.1, X2.2, X3.2, X4.5, X4.PACKAGE1, X4.PACKAGE2, X4.PACKAGE3, X4.PACKAGE4, X4.PACKAGE5, ZD2.ANODE; no longer C1.PAD_1, C105.+, C15.PAD_0, C16.PAD_0, C17.PAD_0, C18.-, C215.-, C24.PAD_1, C27.PAD_1, C3.PAD_1, C30.PAD_1, C33.PAD_0, C35.PAD_0, C36.PAD_0, C38.PAD_0, C39.PAD_0, C40.PAD_0, C41.-, C42.PAD_0, C43.-, C45.-, C46.PAD_0, C47.-, C50.PAD_0, C51.-, C53.+, C54.PAD_1, C55.PAD_1, D13.ANODE, D15.ANODE, D19.ANODE, D2.ANODE, D21.ANODE, D23.ANODE, D28.ANODE, D3.ANODE, D4.CATHODE, D7.ANODE, D8.ANODE, IC1.13, IC1.8, IC12.4, IC16.1, IC6.18, IC6.28, IC6.39, IC6.6, R13.PAD_0, R14.PAD_0, R5.PAD_0, R63.PAD_0, R64.PAD_0, R68.PAD_0, R9.PAD_1, T3.3, T4.3, U15.10, U15.12, U15.3, U15.5, X1.2, X2.1, X4.2, X6.5, X6.PACKAGE1, X6.PACKAGE2, X6.PACKAGE3, X6.PACKAGE4, X6.PACKAGE5, ZD4.ANODE
- net KEY_MODE: now also IC1.25, R5.PAD_1; no longer IC6.25, R81.PAD_1
- net KEY_RANGE: now also IC1.26, R6.PAD_1; no longer IC6.26, R82.PAD_1
- net KEY_RESERVED: now also IC1.24, R7.PAD_1; no longer IC6.24, R83.PAD_1
- net LED_DATA: now also IC1.41, R17.PAD_0; no longer IC6.41, R59.PAD_0
- net LED_DATA': now also D3.ANODE, D6.CATHODE, IC2.14, R17.PAD_1; no longer D12.ANODE, D9.CATHODE, IC1.14, R59.PAD_1
- net LED_LATCH: now also IC1.40, R21.PAD_0; no longer IC6.40, R61.PAD_0
- net LED_LATCH': now also D1.ANODE, D4.CATHODE, R21.PAD_1; no longer D10.ANODE, D7.CATHODE, R61.PAD_1
- net LED_SCK: now also IC1.42, R19.PAD_0; no longer IC6.42, R60.PAD_0
- net LED_SCK': now also D2.ANODE, D5.CATHODE, J1.PAD_0, R19.PAD_1; no longer D11.ANODE, D8.CATHODE, J123.PAD_0, R60.PAD_1
- net L_ADC: now also C20.PAD_0, D10.CATHODE, IC1.37, R59.PAD_1; no longer C3.PAD_0, D2.CATHODE, IC6.37, R2.PAD_1
- net L_PWM: now also C17.PAD_1, D7.ANODE, D9.CATHODE, IC1.14, R55.PAD_0; no longer C4.PAD_1, D25.CATHODE, D26.ANODE, IC6.14, R6.PAD_0
- net MCU_MISO: now also IC1.2, X1.6; no longer IC6.2, X2.6
- net MCU_MOSI: now also IC1.1, X1.3; no longer IC6.1, X2.3
- net MCU_RST: now also IC1.4, R1.PAD_1, X1.2; no longer IC6.4, R62.PAD_1, X2.2
- net MCU_SCK: now also IC1.3, X1.4; no longer IC6.3, X2.4
- net N$1: now also IC7.13, IC7.14; no longer U15.13, U15.14
- net N$10: now also D27.CATHODE, IC10.2; no longer D104.CATHODE, IC12.2
- net N$100: now also IC2.11, J1.PAD_1; no longer IC1.11, J123.PAD_1
- net N$101: now also IC2.12; no longer IC1.12
- net N$102: now also IC3.11; no longer IC2.11
- net N$103: now also IC3.12; no longer IC2.12
- net N$104: now also IC6.11; no longer IC5.11
- net N$105: now also IC5.11; no longer IC4.11
- net N$106: now also IC4.11; no longer IC3.11
- net N$107: now also IC6.12; no longer IC5.12
- net N$108: now also IC5.12; no longer IC4.12
- net N$109: now also IC4.12; no longer IC3.12
- net N$11: now also R56.PAD_0, T1.2; no longer R7.PAD_0, T3.2
- net N$110: now also C2.PAD_1, IC1.8, Q1.2; no longer C13.PAD_1, IC6.8, Q2.2
- net N$111: now also C1.PAD_1, IC1.7, Q1.1; no longer C12.PAD_1, IC6.7, Q2.1
- net N$112: now also IC1.11, R9.PAD_1; no longer IC6.11, R65.PAD_1
- net N$113: now also C40.PAD_1, C44.PAD_1, R73.PAD_1; no longer C21.PAD_1, C22.PAD_1, R4.PAD_1
- net N$114: now also C40.PAD_0, C41.PAD_1, D25.CATHODE, D26.ANODE, X3.1; no longer C22.PAD_0, C23.PAD_1, D3.CATHODE, D4.ANODE, X1.1
- net N$115: now also C41.PAD_0, R67.PAD_0, R75.PAD_1, T4.1; no longer C23.PAD_0, R11.PAD_0, R5.PAD_1, T5.1
- net N$116: now also C22.PAD_1, C42.PAD_1, R68.PAD_0, T4.3; no longer C25.PAD_1, C26.PAD_1, R12.PAD_0, T5.3
- net N$117: now also R76.PAD_1, T4.2; no longer R13.PAD_1, T5.2
- net N$118: now also C42.PAD_0, R69.PAD_0, R77.PAD_1, T5.1; no longer C26.PAD_0, R14.PAD_1, R15.PAD_0, T6.1
- net N$119: now also C23.PAD_1, C43.PAD_1, R70.PAD_0, T5.3; no longer C29.PAD_1, C34.PAD_1, R16.PAD_0, T6.3
- net N$12: now also D8.CATHODE, R56.PAD_1, X2.1; no longer D1.CATHODE, R7.PAD_1, X4.1
- net N$120: now also R78.PAD_1, T5.2; no longer R63.PAD_1, T6.2
- net N$121: now also C43.PAD_0, R71.PAD_0, R79.PAD_1, T6.1; no longer C29.PAD_0, R64.PAD_1, R66.PAD_0, T7.1
- net N$122: now also C24.PAD_1, R72.PAD_0, T6.3; no longer C37.PAD_1, R67.PAD_0, T7.3
- net N$123: now also R80.PAD_1, T6.2; no longer R68.PAD_1, T7.2
- net N$124: now also C27.+, C28.PAD_1, D14.CATHODE, R61.PAD_0; no longer C32.PAD_1, C52.+, D6.CATHODE, R69.PAD_0
- net N$125: now also C22.PAD_0, D14.ANODE, D18.CATHODE; no longer C25.PAD_0, D5.CATHODE, D6.ANODE
- net N$126: now also C35.PAD_0, R64.PAD_1, R67.PAD_1, R68.PAD_1; no longer C24.PAD_0, R11.PAD_1, R12.PAD_1, R154.PAD_1
- net N$127: now also C30.+, C31.PAD_1, D15.CATHODE, R62.PAD_0; no longer C35.PAD_1, C51.+, D14.CATHODE, R70.PAD_0
- net N$128: now also C23.PAD_0, D15.ANODE, D20.CATHODE; no longer C34.PAD_0, D13.CATHODE, D14.ANODE
- net N$129: now also C36.PAD_0, R65.PAD_1, R69.PAD_1, R70.PAD_1; no longer C27.PAD_0, R15.PAD_1, R16.PAD_1, R72.PAD_1
- net N$13: now also D8.ANODE, R57.PAD_0; no longer D1.ANODE, R8.PAD_0
- net N$130: now also C33.+, C34.PAD_1, R63.PAD_0; no longer C215.+, C38.PAD_1, R71.PAD_0
- net N$131: now also C24.PAD_0, D22.CATHODE; no longer C37.PAD_0, D15.CATHODE
- net N$132: now also X4.2; no longer X6.2
- net N$133: now also IC10.1, IC10.7, IC10.8, R83.PAD_1; no longer IC12.1, IC12.7, IC12.8, R110.PAD_1
- net N$134: now also C37.PAD_0, R71.PAD_1, R72.PAD_1; no longer C30.PAD_0, R67.PAD_1, R73.PAD_1
- net N$135: now also C55.PAD_1, IC10.3; no longer C28.PAD_1, IC12.3
- net N$136: now also D29.ANODE, TR1.W2_START; no longer D18.ANODE, TR1.W3_START
- net N$137: now also C45.PAD_1, C46.-, D27.ANODE, IC8.2; no longer C105.-, C31.PAD_1, D104.ANODE, IC16.2
- net N$138: now also D28.ANODE, TR1.W3_START; no longer D17.ANODE, TR1.W2_START
- net N$139: now also IC10.5, R84.PAD_0, R85.PAD_1; no longer IC12.5, R74.PAD_0, R75.PAD_1
- net N$14: now also IC3.15, R22.PAD_0; no longer IC2.15, R27.PAD_0
- net N$140: now also C49.PAD_1, C50.+, D28.CATHODE, IC9.3; no longer C44.PAD_1, C45.+, D17.CATHODE, IC15.3
- net N$141: now also C3.PAD_1, IC1.29; no longer C50.PAD_1, IC6.29
- net N$142: now also IC9.1, R81.PAD_1, R82.PAD_1; no longer IC15.1, R76.PAD_1, R77.PAD_1
- net N$144: now also R2.PAD_0, R5.PAD_0; no longer R80.PAD_0, R81.PAD_0
- net N$145: now also R3.PAD_0, R6.PAD_0; no longer R79.PAD_0, R82.PAD_0
- net N$146: now also R4.PAD_0, R7.PAD_0; no longer R78.PAD_0, R83.PAD_0
- net N$15: now also IC3.1, R23.PAD_0; no longer IC2.1, R28.PAD_0
- net N$16: now also IC3.2, R24.PAD_0; no longer IC2.2, R29.PAD_0
- net N$17: now also IC3.3, R25.PAD_0; no longer IC2.3, R30.PAD_0
- net N$18: now also IC3.4, R26.PAD_0; no longer IC2.4, R31.PAD_0
- net N$19: now also R11.PAD_1; no longer R19.PAD_1
- net N$2: now also IC7.8, IC7.9; no longer U15.8, U15.9
- net N$20: now also R13.PAD_1; no longer R21.PAD_1
- net N$21: now also R16.PAD_1; no longer R24.PAD_1
- net N$22: now also IC3.5, R27.PAD_0; no longer IC2.5, R32.PAD_0
- net N$23: now also R20.PAD_1; no longer R26.PAD_1
- net N$24: now also R12.PAD_1; no longer R20.PAD_1
- net N$25: now also C18.-, C19.PAD_1, R57.PAD_1, R58.PAD_0, R60.PAD_0; no longer C5.PAD_1, C53.-, R10.PAD_0, R8.PAD_1, R9.PAD_0
- net N$26: now also IC3.6, R28.PAD_0; no longer IC2.6, R33.PAD_0
- net N$27: now also R14.PAD_1; no longer R22.PAD_1
- net N$28: now also R15.PAD_1; no longer R23.PAD_1
- net N$29: now also R18.PAD_1; no longer R25.PAD_1
- net N$3: now also IC7.6, IC7.7; no longer U15.6, U15.7
- net N$30: now also IC2.15, R11.PAD_0; no longer IC1.15, R19.PAD_0
- net N$31: now also IC2.1, R12.PAD_0; no longer IC1.1, R20.PAD_0
- net N$32: now also IC2.2, R13.PAD_0; no longer IC1.2, R21.PAD_0
- net N$33: now also IC2.3, R14.PAD_0; no longer IC1.3, R22.PAD_0
- net N$34: now also IC2.4, R15.PAD_0; no longer IC1.4, R23.PAD_0
- net N$35: now also IC2.5, R16.PAD_0; no longer IC1.5, R24.PAD_0
- net N$36: now also IC2.6, R18.PAD_0; no longer IC1.6, R25.PAD_0
- net N$37: now also IC2.7, R20.PAD_0; no longer IC1.7, R26.PAD_0
- net N$38: now also IC3.7, R29.PAD_0; no longer IC2.7, R34.PAD_0
- net N$39: now also R73.PAD_0, T3.2, T7.2; no longer R4.PAD_0, T1.2, T4.2
- net N$4: now also C16.PAD_1, IC7.2, R54.PAD_0, R58.PAD_1; no longer C6.PAD_1, R1.PAD_0, R10.PAD_1, U15.2
- net N$40: now also R22.PAD_1; no longer R27.PAD_1
- net N$41: now also R24.PAD_1; no longer R29.PAD_1
- net N$42: now also R27.PAD_1; no longer R32.PAD_1
- net N$43: now also R29.PAD_1; no longer R34.PAD_1
- net N$44: now also R23.PAD_1; no longer R28.PAD_1
- net N$45: now also R25.PAD_1; no longer R30.PAD_1
- net N$46: now also R26.PAD_1; no longer R31.PAD_1
- net N$47: now also R28.PAD_1; no longer R33.PAD_1
- net N$48: now also IC4.15, R30.PAD_0; no longer IC3.15, R35.PAD_0
- net N$49: now also IC4.1, R31.PAD_0; no longer IC3.1, R36.PAD_0
- net N$5: now also C16.PAD_0, IC7.1, R54.PAD_1, R59.PAD_0; no longer C6.PAD_0, R1.PAD_1, R2.PAD_0, U15.1
- net N$50: now also IC4.2, R32.PAD_0; no longer IC3.2, R37.PAD_0
- net N$51: now also IC4.3, R33.PAD_0; no longer IC3.3, R38.PAD_0
- net N$52: now also IC4.4, R34.PAD_0; no longer IC3.4, R39.PAD_0
- net N$53: now also IC4.5, R35.PAD_0; no longer IC3.5, R40.PAD_0
- net N$54: now also IC4.6, R36.PAD_0; no longer IC3.6, R41.PAD_0
- net N$55: now also IC4.7, R37.PAD_0; no longer IC3.7, R42.PAD_0
- net N$56: now also R30.PAD_1; no longer R35.PAD_1
- net N$57: now also R32.PAD_1; no longer R37.PAD_1
- net N$58: now also R35.PAD_1; no longer R40.PAD_1
- net N$59: now also R37.PAD_1; no longer R42.PAD_1
- net N$6: now also C39.PAD_0, R74.PAD_1, T3.1, T7.1; no longer C20.PAD_0, R3.PAD_1, T1.1, T4.1
- net N$60: now also R31.PAD_1; no longer R36.PAD_1
- net N$61: now also R33.PAD_1; no longer R38.PAD_1
- net N$62: now also R34.PAD_1; no longer R39.PAD_1
- net N$63: now also R36.PAD_1; no longer R41.PAD_1
- net N$64: now also IC5.15, R38.PAD_0; no longer IC4.15, R43.PAD_0
- net N$65: now also IC5.1, R39.PAD_0; no longer IC4.1, R44.PAD_0
- net N$66: now also IC5.2, R40.PAD_0; no longer IC4.2, R45.PAD_0
- net N$67: now also IC5.3, R41.PAD_0; no longer IC4.3, R46.PAD_0
- net N$68: now also IC5.4, R42.PAD_0; no longer IC4.4, R47.PAD_0
- net N$69: now also IC5.5, R43.PAD_0; no longer IC4.5, R48.PAD_0
- net N$7: now also IC1.10, R10.PAD_0; no longer IC6.10, R17.PAD_0
- net N$70: now also IC5.6, R44.PAD_0; no longer IC4.6, R49.PAD_0
- net N$71: now also IC5.7, R45.PAD_0; no longer IC4.7, R50.PAD_0
- net N$72: now also R38.PAD_1; no longer R43.PAD_1
- net N$73: now also R40.PAD_1; no longer R45.PAD_1
- net N$74: now also R43.PAD_1; no longer R48.PAD_1
- net N$75: now also R45.PAD_1; no longer R50.PAD_1
- net N$76: now also R39.PAD_1; no longer R44.PAD_1
- net N$77: now also R41.PAD_1; no longer R46.PAD_1
- net N$78: now also R42.PAD_1; no longer R47.PAD_1
- net N$79: now also R44.PAD_1; no longer R49.PAD_1
- net N$8: now also IC1.12, R8.PAD_1; no longer IC6.12, R18.PAD_1
- net N$80: now also IC6.15, R46.PAD_0; no longer IC5.15, R51.PAD_0
- net N$81: now also IC6.1, R47.PAD_0; no longer IC5.1, R52.PAD_0
- net N$82: now also IC6.2, R48.PAD_0; no longer IC5.2, R53.PAD_0
- net N$83: now also IC6.3, R49.PAD_0; no longer IC5.3, R54.PAD_0
- net N$84: now also IC6.4, R50.PAD_0; no longer IC5.4, R55.PAD_0
- net N$85: now also IC6.5, R51.PAD_0; no longer IC5.5, R56.PAD_0
- net N$86: now also IC6.6, R52.PAD_0; no longer IC5.6, R57.PAD_0
- net N$87: now also IC6.7, R53.PAD_0; no longer IC5.7, R58.PAD_0
- net N$88: now also R46.PAD_1; no longer R51.PAD_1
- net N$89: now also R48.PAD_1; no longer R53.PAD_1
- net N$9: now also C17.PAD_0, R55.PAD_1, T1.1; no longer C4.PAD_0, R6.PAD_1, T3.1
- net N$90: now also R51.PAD_1; no longer R56.PAD_1
- net N$91: now also R53.PAD_1; no longer R58.PAD_1
- net N$92: now also R47.PAD_1; no longer R52.PAD_1
- net N$93: now also R49.PAD_1; no longer R54.PAD_1
- net N$94: now also R50.PAD_1; no longer R55.PAD_1
- net N$95: now also R52.PAD_1; no longer R57.PAD_1
- net USB_D+: now also R10.PAD_1, X4.3, ZD2.CATHODE; no longer R17.PAD_1, X6.3, ZD4.CATHODE
- net USB_D-: now also R8.PAD_0, R9.PAD_0; no longer R18.PAD_0, R65.PAD_0
- net VCC_ROUGH: now also C12.PAD_1, C13.PAD_1, C14.PAD_1, C56.PAD_1, C57.+, D1.CATHODE, D2.CATHODE, D29.CATHODE, D3.CATHODE, IC6.10, IC6.16, R84.PAD_1; no longer C42.PAD_1, C43.+, C7.PAD_1, C8.PAD_1, C9.PAD_1, D10.CATHODE, D11.CATHODE, D12.CATHODE, D18.CATHODE, IC1.10, IC1.16, R74.PAD_1
Routing:
- net VCC_ROUGH: track 27.3 -> 59.6 mm, vias 0 -> 2
- net LED_LATCH': track 43.8 -> 56.3 mm
- net N$98 (its old number): track 11.8 -> 0.00 mm
- net N$99: track 0.00 -> 9.15 mm
- net GND: track 64.9 -> 68.6 mm
- net N$98: track 9.25 -> 11.8 mm
Other:
- board outline added: 70 x 130 mm

Commit message: LCMeter routing
Parts:
- removed D4, D5, D6: LL4148, __MyCommonLib1:SOD-80
- R64, R65, R66: device __MyCommonLib1:RSMD_1206_BIG_GAP -> __MyCommonLib1:RSMD_0805
- moved D1 371.8 mm to (93.9, 106.4)
- moved D2 371.8 mm to (94.2, 110.5)
- moved D3 371.8 mm to (93.5, 115.9)
- moved R17 368.1 mm to (76.7, 83.7)
- moved R19 368.1 mm to (76.2, 88.6)
- moved R21 368.1 mm to (75.0, 95.1)
- moved D13 308.1 mm to (50.5, 37.5), flipped to the bottom, turned to 0 degrees
- moved KEY1 298.2 mm to (66.0, 75.5)
- moved KEY2 287.3 mm to (66.0, 65.5)
- moved KEY3 276.4 mm to (66.0, 55.5), turned to 270 degrees
- moved R2 268.7 mm to (65.0, 75.5), flipped to the bottom
- moved R3 265.9 mm to (65.0, 65.5), flipped to the bottom
- moved R4 265.9 mm to (65.0, 55.5), flipped to the bottom
- moved R5 259.0 mm to (60.5, 64.5), flipped to the bottom, turned to 270 degrees
- moved R6 255.9 mm to (60.5, 59.0), flipped to the bottom, turned to 270 degrees
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Connections:
- net ESR_ADC_100X: now also IC1.32; no longer IC1.30
- net ESR_ADC_10X: now also IC1.33; no longer IC1.31
- net ESR_ADC_1X: now also IC1.34; no longer IC1.32
- net GND: no longer D4.ANODE, D5.ANODE, D6.ANODE
- net KEY_MODE: now also IC1.23; no longer IC1.25
- net KEY_RANGE: now also IC1.24; no longer IC1.26
- net KEY_RESERVED: now also IC1.25; no longer IC1.24
- net LED_DATA: now also IC1.21; no longer IC1.41
- net LED_DATA': no longer D6.CATHODE
- net LED_LATCH: now also IC1.20; no longer IC1.40
- net LED_LATCH': no longer D4.CATHODE
- net LED_SCK: now also IC1.22; no longer IC1.42
- net LED_SCK': no longer D5.CATHODE
Routing:
- net GND: track 68.6 -> 220.5 mm
- net +5V_FINE: track 0.00 -> 64.6 mm
- net ESR_ADC_100X: track 0.00 -> 26.7 mm
- net ESR_ADC_1X: track 0.00 -> 19.6 mm
- net ESR_ADC_10X: track 0.00 -> 18.4 mm
- net N$114: track 0.00 -> 15.2 mm
- net N$126: track 0.00 -> 14.1 mm
- net N$129: track 0.00 -> 14.1 mm
- net N$111: track 0.00 -> 12.9 mm
- net N$121: track 0.00 -> 12.2 mm
- net N$6: track 0.00 -> 12.0 mm
- net MCU_RST: track 0.00 -> 11.8 mm
- net N$118: track 0.00 -> 11.7 mm
- net N$116: track 0.00 -> 10.6 mm
- net N$119: track 0.00 -> 10.5 mm
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
Commit message: LCMeter start routing2
Parts:
- removed J1, J2, J3, J5, J7: 0, __MyCommonLib1:RSMD_1206_BIG_GAP
- added R86, R87, R88: 1K0, __MyCommonLib1:RSMD_0805
- J10, J4, J6, J8, J9: device __MyCommonLib1:RSMD_1206_BIG_GAP -> __MyCommonLib1:RSMD_0805
- moved C14 371.9 mm to (61.5, 92.5), turned to 0 degrees
- moved C13 366.1 mm to (47.9, 92.6), turned to 0 degrees
- moved C12 360.5 mm to (34.3, 92.4), turned to 0 degrees
- moved D3 83.5 mm to (13.8, 91.0), turned to 270 degrees
- moved D1 66.5 mm to (29.4, 90.1), turned to 270 degrees
- moved D2 54.6 mm to (43.2, 91.1), turned to 270 degrees
- moved R17 20.7 mm to (56.2, 81.0), turned to 0 degrees
- moved R5 16.7 mm to (59.6, 47.8)
- moved R6 11.3 mm to (62.3, 47.8)
- moved R11 7.10 mm to (3.60, 105.1)
- moved R7 6.88 mm to (65.0, 47.8)
- moved C11 4.90 mm to (20.7, 92.4), turned to 0 degrees
- moved J8 4.06 mm to (51.3, 89.5)
- moved J10 2.98 mm to (63.1, 87.7)
- moved J4 2.59 mm to (24.5, 89.5)
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Connections:
- removed net N$100: IC2.11, J1.PAD_1
- removed net N$101: IC2.12, J2.PAD_1
- removed net N$102: IC3.11, J3.PAD_1
- removed net N$105: IC5.11, J7.PAD_1
- removed net N$106: IC4.11, J5.PAD_1
- net GND: now also R86.PAD_0, R87.PAD_0, R88.PAD_0
- net LED_DATA: now also IC1.20; no longer IC1.21
- net LED_LATCH: now also IC1.21; no longer IC1.20
- net LED_LATCH': now also IC2.12; no longer J2.PAD_0
- net LED_SCK': now also IC2.11, IC3.11, IC4.11, IC5.11; no longer J1.PAD_0, J3.PAD_0, J5.PAD_0, J7.PAD_0
- net N$124: now also R86.PAD_1
- net N$127: now also R87.PAD_1
- net N$130: now also R88.PAD_1
Routing:
- net GND: track 220.5 -> 518.6 mm
- net VCC_ROUGH: track 59.6 -> 128.4 mm, vias 2 -> 8
- net LED_SCK: track 0.00 -> 62.5 mm
- net LED_DATA: track 0.00 -> 62.2 mm
- net LED_LATCH: track 0.00 -> 62.1 mm
- net +5V_FINE: track 64.6 -> 117.2 mm
- net KEY_RESERVED: track 0.00 -> 39.9 mm
- net KEY_RANGE: track 0.00 -> 36.4 mm
- net KEY_MODE: track 0.00 -> 32.9 mm
- net N$144: track 0.00 -> 32.0 mm
- net N$81: track 0.00 -> 21.7 mm
- net N$83: track 0.00 -> 21.5 mm
- net N$145: track 0.00 -> 21.2 mm
- net N$84: track 0.00 -> 21.1 mm
- net N$68: track 0.00 -> 20.9 mm
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
Commit message: LCMeter start routing2
Parts:
- removed C47: 0.47uFx16V, __MyCommonLib1:RSMD_0805
- removed J11, J9: 0, __MyCommonLib1:RSMD_0805
- D29: device __MyCommonLib1:DO-41_10MM -> __MyCommonLib1:DO-41_5MM
- R81, R82: device __MyCommonLib1:RSMD_1206_BIG_GAP -> __MyCommonLib1:RSMD_0805
- R84: device __MyCommonLib1:RSMD_0805 -> __MyCommonLib1:R0207
- moved ZD1 400.5 mm to (20.2, 45.7), flipped to the bottom, turned to 0 degrees
- moved ZD2 398.1 mm to (18.1, 43.0), flipped to the bottom, turned to 0 degrees
- moved R82 347.3 mm to (47.6, 61.1), flipped to the bottom, turned to 0 degrees
- moved C51 337.6 mm to (31.8, 45.6), flipped to the bottom, turned to 0 degrees
- moved R81 337.1 mm to (39.5, 50.9), flipped to the bottom
- moved C52 334.9 mm to (31.6, 48.8)
- moved C4 245.0 mm to (29.5, 17.2), turned to 0 degrees
- moved C9 220.5 mm to (35.3, 17.1), turned to 90 degrees
- moved R83 21.7 mm to (12.5, 62.6), turned to 90 degrees
- moved C54 20.5 mm to (5.80, 61.2), turned to 180 degrees
- moved R21 19.7 mm to (60.2, 82.1), turned to 90 degrees
- moved R85 16.8 mm to (19.4, 57.3), turned to 0 degrees
- moved R84 15.7 mm to (16.1, 62.4)
- moved C53 14.2 mm to (5.20, 64.9)
- moved IC10 14.2 mm to (18.4, 61.6), turned to 0 degrees
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Connections:
- removed net N$104: IC6.11, J9.PAD_1
- removed net N$132: J11.PAD_1, X4.2
- net -5V_FINE: no longer C47.PAD_1
- net GND: no longer C47.PAD_0
- net LED_SCK': now also IC6.11; no longer J9.PAD_0
- net USB_D-: now also X4.2; no longer J11.PAD_0
- net VCC_ROUGH: now also R84.PAD1; no longer R84.PAD_1
Routing:
- net USB_D+: track 0.00 -> 110.3 mm
- net USB_D-: track 0.00 -> 106.9 mm
- net LED_DATA': track 11.6 -> 61.9 mm
- net LED_SCK': track 64.8 -> 86.1 mm
- net VCC_ROUGH: track 128.4 -> 108.5 mm
- net +5V_FINE: track 117.2 -> 132.2 mm
- net -5V_FINE: track 0.00 -> 13.7 mm
- net GND: track 518.6 -> 532.0 mm
- net LED_LATCH': track 46.7 -> 59.4 mm
- net LED_SCK: track 62.5 -> 68.1 mm
- net N$107: track 0.00 -> 5.49 mm
- net LED_DATA: track 62.2 -> 58.0 mm
- net N$8: track 3.64 -> 0.00 mm
- net LED_LATCH: track 62.1 -> 64.1 mm
- net N$1: track 0.00 -> 1.27 mm
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Other:
- board size 70 x 130 mm -> 70 x 125 mm
