File: LC_METER/schematic/LCMeter.brd (EAGLE design)
At the start: 70 x 125 mm, 205 parts, among them IC1 MEGA8535, IC10 MC34063, IC2 74HC595, IC3 74HC595, IC4 74HC595, IC5 74HC595, IC6 74HC595, IC7 LM324, IC8 7905, IC9 LM317, J10 0, J4 0, J6 0, J8 0, Q1 12MHz, T1 BC847, T2 BC857, T3 BC847, T4 BC847, T5 BC847, T6 BC847, T7 BC857, X1 MCU_PROGRAMMING, X2 L_X, X3 C_X, X4 USB_MICRO, X5 USB_B

Commit message: LCMeter start routing2
Parts:
- removed C4: 4.7uF, __MyCommonLib1:CE_6.3MM
- added C47, C58: 4.7uF, __MyCommonLib1:CE_6.3MM
- added J100: 0, __MyCommonLib1:RSMD_1206_BIG_GAP
- moved C9 28.2 mm to (51.1, 40.4), turned to 180 degrees
- moved R81 14.9 mm to (38.4, 65.8)
- moved C38 11.0 mm to (35.6, 12.0), turned to 90 degrees
- moved R74 7.34 mm to (38.5, 3.10)
- moved D9 6.72 mm to (22.3, 4.50), turned to 270 degrees
- moved D23 5.64 mm to (32.2, 8.10), turned to 270 degrees
- moved R73 5.59 mm to (49.0, 9.00)
- moved C17 5.31 mm to (23.0, 8.80)
- moved R55 5.19 mm to (23.0, 11.4)
- moved C51 5.02 mm to (26.9, 46.7), turned to 180 degrees
- moved C16 4.64 mm to (14.2, 18.7), turned to 270 degrees
- moved T1 4.61 mm to (18.5, 9.00)
- moved ZD1 4.60 mm to (15.6, 45.5)
- moved T2 4.59 mm to (18.5, 4.10), turned to 180 degrees
- moved D7 4.34 mm to (27.9, 8.80), turned to 0 degrees
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Connections:
- new net N$100: IC1.35, J100.PAD_1
- net +5V_FINE: now also C47.+, C58.+; no longer C4.+
- net ESR_PWM: now also IC1.14; no longer IC1.13
- net GND: now also C47.-, C58.-; no longer C4.-
- net L_ADC: now also J100.PAD_0; no longer IC1.37
- net L_PWM: now also IC1.13; no longer IC1.14
Routing:
- net +5V_FINE: track 132.2 -> 239.8 mm, vias 0 -> 8
- net VCC_ROUGH: track 108.5 -> 185.1 mm, vias 8 -> 10
- net ESR_PWM: track 0.00 -> 47.1 mm, vias 0 -> 2
- net L_PWM: track 0.00 -> 44.0 mm, vias 0 -> 2
- net N$140: track 0.00 -> 23.2 mm
- net USB_D-: track 106.9 -> 121.8 mm
- net USB_D+: track 110.3 -> 124.6 mm
- net N$10: track 0.00 -> 14.1 mm
- net L_ADC: track 0.00 -> 11.8 mm
- net N$25: track 0.00 -> 11.8 mm
- net N$4: track 0.00 -> 11.3 mm
- net N$142: track 0.00 -> 10.9 mm
- net N$9: track 0.00 -> 10.3 mm
- net N$100: track 0.00 -> 8.84 mm
- net N$11: track 0.00 -> 8.69 mm
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- added copper zone on layer 16, net +5V_FINE
- added copper zone on layer 16, net GND

Commit message: LCMeter start routing4
Parts:
- added C4: 0.1uF, __MyCommonLib1:RSMD_0805
- added D4: LL4148, __MyCommonLib1:SOD-80
- added J11: 0, __MyCommonLib1:RSMD_0805
- added R100: 10K, __MyCommonLib1:RSMD_0805
- added R89: 1K, __MyCommonLib1:RSMD_0805
- D28: device __MyCommonLib1:DO-41_10MM -> __MyCommonLib1:DO-41_5MM
- R59: device __MyCommonLib1:RSMD_0805 -> __MyCommonLib1:RSMD_1206_BIG_GAP
- moved D3 40.9 mm to (54.8, 84.1)
- moved ZD2 36.6 mm to (19.7, 79.0), turned to 90 degrees
- moved ZD1 36.2 mm to (24.1, 80.7)
- moved R82 11.6 mm to (39.3, 69.1), turned to 270 degrees
- moved R17 4.16 mm to (58.5, 80.9)
- moved C26 3.51 mm to (44.5, 19.2)
- moved C49 3.42 mm to (48.9, 67.6)
- moved C50 3.35 mm to (47.3, 58.0), turned to 270 degrees
- moved R61 3.01 mm to (41.0, 19.2)
- moved D28 2.61 mm to (46.4, 64.6)
- moved C9 2.41 mm to (53.5, 40.2)
- moved D2 2.25 mm to (41.3, 87.3), turned to 0 degrees
- moved C45 1.57 mm to (18.9, 51.5), turned to 270 degrees
- moved R19 1.53 mm to (67.4, 84.1)
- moved R59 1.51 mm to (18.4, 18.9), turned to 180 degrees
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Connections:
- new net BATTERY_ADC: C4.PAD_1, D4.ANODE, IC1.35, R100.PAD_1, R89.PAD_0
- new net N$101: J11.PAD_0, X4.2
- net +5V_FINE: now also D4.CATHODE
- net +5V_USB: now also R100.PAD_0
- net GND: now also C4.PAD_0, R89.PAD_1
- net N$100: now also IC1.37; no longer IC1.35
- net USB_D-: now also J11.PAD_1; no longer X4.2
Routing:
- net +5V_USB: track 0.00 -> 132.5 mm
- net BATTERY_ADC: track 0.00 -> 40.7 mm, vias 0 -> 2
- net +5V_FINE: track 239.8 -> 221.3 mm, vias 8 -> 7
- net GND: track 526.8 -> 510.5 mm
- net VCC_ROUGH: track 185.1 -> 197.0 mm, vias 10 -> 12
- net USB_D-: track 121.8 -> 115.6 mm
- net USB_D+: track 124.6 -> 119.1 mm
- net N$139: track 0.00 -> 5.21 mm
- net N$135: track 0.00 -> 3.24 mm
- net N$140: track 23.2 -> 20.0 mm
- net N$101: track 0.00 -> 2.94 mm
- net LED_DATA: track 58.0 -> 60.7 mm
- net LED_DATA': track 60.1 -> 58.1 mm
- net L_ADC: track 11.8 -> 10.0 mm
- net N$142: track 10.9 -> 9.36 mm
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- added copper zone on layer 16, net N$133
- added copper zone on layer 16, net N$137

Commit message: LCMeter start routing 5
Parts:
- D28: device __MyCommonLib1:DO-41_5MM -> __MyCommonLib1:DO-41_12.5MM
- moved D3 52.5 mm to (2.40, 86.4)
- moved C49 8.00 mm to (48.8, 59.6), turned to 270 degrees
- moved D28 6.89 mm to (43.2, 58.5), turned to 270 degrees
- moved C50 5.02 mm to (52.3, 58.5)
- moved C56 4.12 mm to (46.3, 72.9)
- moved R17 2.91 mm to (55.9, 82.2), turned to 0 degrees
- moved C57 2.04 mm to (50.5, 68.9), turned to 90 degrees
- moved R21 1.70 mm to (59.4, 82.6)
- moved IC9 1.70 mm to (33.0, 58.3)
- moved C26 1.50 mm to (46.0, 19.2)
- moved J10 1.50 mm to (63.2, 84.1)
- moved R19 1.50 mm to (65.9, 84.1)
- moved C22 1.30 mm to (56.2, 15.3)
- moved R82 0.90 mm to (40.2, 69.1)
- moved R81 0.90 mm to (39.3, 65.8)
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Routing:
- net GND: track 510.5 -> 443.2 mm, vias 0 -> 2
- net N$140: track 20.0 -> 0.00 mm
- net VCC_ROUGH: track 197.0 -> 177.6 mm
- net LED_DATA: track 60.7 -> 65.6 mm
- net +5V_FINE: track 221.3 -> 218.0 mm, vias 7 -> 6
- net USB_D-: track 115.6 -> 117.9 mm
- net LED_SCK: track 68.7 -> 70.9 mm
- net LED_DATA': track 58.1 -> 60.1 mm
- net USB_D+: track 119.1 -> 120.8 mm
- net LED_LATCH: track 62.7 -> 64.5 mm
- net +5V_USB: track 132.5 -> 134.2 mm
- net N$126: track 14.1 -> 12.6 mm
- net LED_LATCH': track 59.9 -> 58.4 mm
- net N$129: track 14.1 -> 12.9 mm
- net N$119: track 10.5 -> 9.41 mm
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- added copper zone on layer 16, net +5V_USB
- added copper zone on layer 16, net N$110
- added copper zone on layer 16, net N$111
- added copper zone on layer 16, net N$140
- added copper zone on layer 16, net VCC_ROUGH

Commit message: LCMeter Route finish 1
Parts:
- X1: device __MyCommonLib1:PIN2X3_2.54MM -> __MyCommonLib1:PIN2X3_2.54MM_LOOSE_PADS
- moved C47 2.60 mm to (16.5, 12.5)
- moved C15 2.20 mm to (16.4, 14.7)
Routing:
- net VCC_ROUGH: track 177.6 -> 143.3 mm
- net GND: track 443.2 -> 423.1 mm
- net N$110: track 7.52 -> 6.92 mm
- net N$51: track 20.8 -> 21.4 mm
- net N$99: track 13.5 -> 14.1 mm
- added copper zone on layer 16, net MCU_MISO
- added copper zone on layer 16, net MCU_MOSI
- added copper zone on layer 16, net MCU_RST
- added copper zone on layer 16, net MCU_SCK

Commit message: LCMeter Route finished
Routing:
- net GND: track 423.1 -> 406.6 mm
- net N$114: track 13.9 -> 2.90 mm
- net N$12: track 8.44 -> 0.00 mm
- net +5V_FINE: track 217.7 -> 212.7 mm
- net VCC_ROUGH: track 143.3 -> 141.6 mm
- net L_ADC: track 10.0 -> 9.45 mm
- added copper zone on layer 16, net N$114
- added copper zone on layer 16, net N$12

Commit message: LC meter schematic. Power stabilizer values fix
Parts:
- R81: value 5K1 -> 1K0
- R82: value 1K7 -> 3K0
- R84: value 5K1 -> 4K7
- R85: value 1K7 -> 1K6
Changed lines of the file:
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@@
 <grid distance="0.1" unitdist="mm" unit="mm" style="lines" multiple="1" display="yes" altdistance="0.025" altunitdist="inch" altunit="inch"/>
 <layers>
-<layer number="1" name="Top" color="4" fill="1" visible="no" active="yes"/>
+<layer number="1" name="Top" color="4" fill="1" visible="yes" active="yes"/>
 <layer number="2" name="Route2" color="1" fill="3" visible="no" active="no"/>
 <layer number="3" name="Route3" color="4" fill="3" visible="no" active="no"/>
@@
 <layer number="21" name="tPlace" color="7" fill="1" visible="yes" active="yes"/>
 <layer number="22" name="bPlace" color="7" fill="1" visible="yes" active="yes"/>
-<layer number="23" name="tOrigins" color="15" fill="1" visible="no" active="yes"/>
-<layer number="24" name="bOrigins" color="15" fill="1" visible="no" active="yes"/>
+<layer number="23" name="tOrigins" color="15" fill="1" visible="yes" active="yes"/>
+<layer number="24" name="bOrigins" color="15" fill="1" visible="yes" active="yes"/>
 <layer number="25" name="tNames" color="7" fill="1" visible="no" active="yes"/>
 <layer number="26" name="bNames" color="7" fill="1" visible="no" active="yes"/>
@@
 <element name="C56" library="__MyCommonLib1" package="RSMD_1206_BIG_GAP" value="0.47uFx16V" x="46.3" y="72.9" rot="MR180"/>
 <element name="C57" library="__MyCommonLib1" package="CE_10MM" value="470uFx16V" x="50.5" y="68.9" rot="R90"/>
-<element name="R84" library="__MyCommonLib1" package="R0207" value="5K1" x="15.4" y="63" rot="R90"/>
-<element name="R85" library="__MyCommonLib1" package="RSMD_0805" value="1K7" x="18.7" y="57.9" rot="MR0"/>
+<element name="R84" library="__MyCommonLib1" package="R0207" value="4K7" x="15.4" y="63" rot="R90"/>
+<element name="R85" library="__MyCommonLib1" package="RSMD_0805" value="1K6" x="18.7" y="57.9" rot="MR0"/>
 <element name="C49" library="__MyCommonLib1" package="RSMD_1206" value="0.47uFx16V" x="48.8" y="59.6" rot="MR270"/>
 <element name="C50" library="__MyCommonLib1" package="CE_10MM" value="470uFx16V" x="52.3" y="58.5" rot="R270"/>
@@
 <element name="C51" library="__MyCommonLib1" package="RSMD_0805" value="0.47uFx16V" x="26.9" y="46.7" rot="MR180"/>
 <element name="C52" library="__MyCommonLib1" package="CE_10MM" value="47uFx16V" x="28.3" y="49.9"/>
-<element name="R81" library="__MyCommonLib1" package="RSMD_0805" value="5K1" x="39.3" y="65.8" rot="MR180"/>
-<element name="R82" library="__MyCommonLib1" package="RSMD_0805" value="1K7" x="40.2" y="69.1" rot="MR270"/>
+<element name="R81" library="__MyCommonLib1" package="RSMD_0805" value="1K0" x="39.3" y="65.8" rot="MR180"/>
+<element name="R82" library="__MyCommonLib1" package="RSMD_0805" value="3K0" x="40.2" y="69.1" rot="MR270"/>
 <element name="IC8" library="__MyCommonLib1" package="D2PAK" value="7905" x="6.6" y="49" rot="MR0"/>
 <element name="C3" library="__MyCommonLib1" package="RSMD_0805" value="0.1uF" x="38.8" y="27.5" rot="MR0"/>

Commit message: LC Meter change some values
Parts:
- C47, C58: value 4.7uF -> 100uFx10V
- R54, R67, R69, R71: value 100K -> 120K
- R55, R74: value 4K7 -> 2K2
- R58: value 20K -> 24K
- R59: value 300R -> 1K0
- R75, R77, R79: value 25K -> 24K
- R86, R87, R88: value 1K0 -> 10K
Changed lines of the file:
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@@
 <layer number="49" name="Reference" color="7" fill="1" visible="no" active="yes"/>
 <layer number="51" name="tDocu" color="7" fill="1" visible="no" active="yes"/>
-<layer number="52" name="bDocu" color="7" fill="1" visible="no" active="yes"/>
+<layer number="52" name="bDocu" color="7" fill="1" visible="yes" active="yes"/>
 <layer number="91" name="Nets" color="2" fill="1" visible="no" active="no"/>
 <layer number="92" name="Busses" color="1" fill="1" visible="no" active="no"/>
@@
 <element name="R8" library="__MyCommonLib1" package="RSMD_0805" value="68R" x="25.4" y="40.4" rot="MR270"/>
 <element name="R9" library="__MyCommonLib1" package="RSMD_0805" value="1K5" x="22.5" y="40.4" rot="MR270"/>
-<element name="R55" library="__MyCommonLib1" package="RSMD_0805" value="4K7" x="23" y="11.4" rot="MR0"/>
+<element name="R55" library="__MyCommonLib1" package="RSMD_0805" value="2K2" x="23" y="11.4" rot="MR0"/>
 <element name="C17" library="__MyCommonLib1" package="RSMD_0805" value="1nF" x="23" y="8.8" rot="MR180"/>
 <element name="T1" library="__MyCommonLib1" package="SOT23_SMALL_PADS" value="BC847" x="18.5" y="9" rot="MR180"/>
@@
 <element name="C19" library="__MyCommonLib1" package="RSMD_1206_BIG_GAP" value="0.47uF" x="5.5" y="18.1" rot="MR180"/>
 <element name="R60" library="__MyCommonLib1" package="RSMD_0805" value="4K7" x="5.5" y="12.1" rot="MR0"/>
-<element name="R58" library="__MyCommonLib1" package="RSMD_0805" value="20K" x="11.1" y="15.2" rot="MR180"/>
+<element name="R58" library="__MyCommonLib1" package="RSMD_0805" value="24K" x="11.1" y="15.2" rot="MR180"/>
 <element name="C16" library="__MyCommonLib1" package="RSMD_0805" value="0.1uF" x="14.2" y="18.7" rot="MR270"/>
 <element name="IC7" library="__MyCommonLib1" package="SOIC14" value="LM324" x="6" y="24.4" rot="MR90"/>
 <element name="C25" library="__MyCommonLib1" package="RSMD_0805" value="0.1uF" x="4" y="30.8" rot="MR180"/>
 <element name="C21" library="__MyCommonLib1" package="RSMD_0805" value="0.1uF" x="12.2" y="24.4" rot="MR90"/>
-<element name="R54" library="__MyCommonLib1" package="RSMD_0805" value="100K" x="11.6" y="18.7" rot="MR90"/>
-<element name="R59" library="__MyCommonLib1" package="RSMD_1206_BIG_GAP" value="300R" x="18.4" y="18.9" rot="MR180"/>
+<element name="R54" library="__MyCommonLib1" package="RSMD_0805" value="120K" x="11.6" y="18.7" rot="MR90"/>
+<element name="R59" library="__MyCommonLib1" package="RSMD_1206_BIG_GAP" value="1K0" x="18.4" y="18.9" rot="MR180"/>
 <element name="D10" library="__MyCommonLib1" package="SOD-80" value="LL4148" x="25.2" y="18.7" rot="MR90"/>
 <element name="C20" library="__MyCommonLib1" package="RSMD_0805" value="0.1uF" x="22.6" y="19.5" rot="MR90"/>
-<element name="R74" library="__MyCommonLib1" package="RSMD_0805" value="4K7" x="38.5" y="3.1" rot="MR180"/>
+<element name="R74" library="__MyCommonLib1" package="RSMD_0805" value="2K2" x="38.5" y="3.1" rot="MR180"/>
 <element name="C39" library="__MyCommonLib1" package="RSMD_0805" value="1nF" x="38.5" y="5.7" rot="MR0"/>
 <element name="T3" library="__MyCommonLib1" package="SOT23_SMALL_PADS" value="BC847" x="43.1" y="8.4" rot="MR0"/>
@@
 <element name="T4" library="__MyCommonLib1" package="SOT23_SMALL_PADS" value="BC847" x="61" y="14" rot="MR90"/>
 <element name="C41" library="__MyCommonLib1" package="RSMD_0805" value="0.1uF" x="61" y="9" rot="MR270"/>
-<element name="R75" library="__MyCommonLib1" package="RSMD_0805" value="25K" x="66" y="15" rot="MR0"/>
-<element name="R67" library="__MyCommonLib1" package="RSMD_0805" value="100K" x="64" y="19" rot="MR90"/>
+<element name="R75" library="__MyCommonLib1" package="RSMD_0805" value="24K" x="66" y="15" rot="MR0"/>
+<element name="R67" library="__MyCommonLib1" package="RSMD_0805" value="120K" x="64" y="19" rot="MR90"/>
 <element name="R68" library="__MyCommonLib1" package="RSMD_0805" value="1K0" x="58" y="19" rot="MR90"/>
 <element name="R76" library="__MyCommonLib1" package="RSMD_0805" value="100R" x="66" y="12" rot="MR0"/>
@@
 <element name="T5" library="__MyCommonLib1" package="SOT23_SMALL_PADS" value="BC847" x="61" y="24" rot="MR90"/>
 <element name="C42" library="__MyCommonLib1" package="RSMD_0805" value="0.1uF" x="61" y="19" rot="MR270"/>
-<element name="R77" library="__MyCommonLib1" package="RSMD_0805" value="25K" x="66" y="25.5" rot="MR0"/>
-<element name="R69" library="__MyCommonLib1" package="RSMD_0805" value="100K" x="64" y="29" rot="MR90"/>
+<element name="R77" library="__MyCommonLib1" package="RSMD_0805" value="24K" x="66" y="25.5" rot="MR0"/>
+<element name="R69" library="__MyCommonLib1" package="RSMD_0805" value="120K" x="64" y="29" rot="MR90"/>
 <element name="R70" library="__MyCommonLib1" package="RSMD_0805" value="1K0" x="58" y="29" rot="MR90"/>
 <element name="R78" library="__MyCommonLib1" package="RSMD_0805" value="100R" x="66" y="22.5" rot="MR0"/>
@@
 <element name="T6" library="__MyCommonLib1" package="SOT23_SMALL_PADS" value="BC847" x="61" y="34" rot="MR90"/>
 <element name="C43" library="__MyCommonLib1" package="RSMD_0805" value="0.1uF" x="61" y="29" rot="MR270"/>
-<element name="R79" library="__MyCommonLib1" package="RSMD_0805" value="25K" x="66" y="36" rot="MR0"/>
-<element name="R71" library="__MyCommonLib1" package="RSMD_0805" value="100K" x="62" y="39" rot="MR90"/>
+<element name="R79" library="__MyCommonLib1" package="RSMD_0805" value="24K" x="66" y="36" rot="MR0"/>
+<element name="R71" library="__MyCommonLib1" package="RSMD_0805" value="120K" x="62" y="39" rot="MR90"/>
 <element name="R72" library="__MyCommonLib1" package="RSMD_0805" value="1K0" x="59" y="39" rot="MR90"/>
 <element name="R80" library="__MyCommonLib1" package="RSMD_0805" value="100R" x="66" y="33" rot="MR0"/>
@@
 <element name="X1" library="__MyCommonLib1" package="PIN2X3_2.54MM_LOOSE_PADS" value="MCU_PROGRAMMING" x="17.4" y="23.6"/>
 <element name="C48" library="__MyCommonLib1" package="CE_6.3MM" value="47uFx16V" x="5.9" y="34"/>
-<element name="R86" library="__MyCommonLib1" package="RSMD_0805" value="1K0" x="41" y="14.5" rot="MR90"/>
-<element name="R87" library="__MyCommonLib1" package="RSMD_0805" value="1K0" x="46.5" y="28" rot="MR270"/>
-<element name="R88" library="__MyCommonLib1" package="RSMD_0805" value="1K0" x="46" y="37.5" rot="MR270"/>
+<element name="R86" library="__MyCommonLib1" package="RSMD_0805" value="10K" x="41" y="14.5" rot="MR90"/>
+<element name="R87" library="__MyCommonLib1" package="RSMD_0805" value="10K" x="46.5" y="28" rot="MR270"/>
+<element name="R88" library="__MyCommonLib1" package="RSMD_0805" value="10K" x="46" y="37.5" rot="MR270"/>
 <element name="J100" library="__MyCommonLib1" package="RSMD_1206_BIG_GAP" value="0" x="29.4" y="15.9" rot="MR180"/>
-<element name="C47" library="__MyCommonLib1" package="CE_6.3MM" value="4.7uF" x="16.5" y="12.5"/>
-<element name="C58" library="__MyCommonLib1" package="CE_6.3MM" value="4.7uF" x="38.4" y="12" rot="R270"/>
+<element name="C47" library="__MyCommonLib1" package="CE_6.3MM" value="100uFx10V" x="16.5" y="12.5"/>
+<element name="C58" library="__MyCommonLib1" package="CE_6.3MM" value="100uFx10V" x="38.4" y="12" rot="R270"/>
 <element name="J11" library="__MyCommonLib1" package="RSMD_0805" value="0" x="8.5" y="77.2" rot="MR90"/>
 <element name="R100" library="__MyCommonLib1" package="RSMD_0805" value="10K" x="34" y="47.3" rot="MR270"/>

Commit message: LC Meter. Battery voltage metter resistors values changed
Parts:
- R89: value 1K -> 3K0
Changed lines of the file:
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@@
 <element name="J11" library="__MyCommonLib1" package="RSMD_0805" value="0" x="8.5" y="77.2" rot="MR90"/>
 <element name="R100" library="__MyCommonLib1" package="RSMD_0805" value="10K" x="34" y="47.3" rot="MR270"/>
-<element name="R89" library="__MyCommonLib1" package="RSMD_0805" value="1K" x="35.3" y="19.8" rot="MR90"/>
+<element name="R89" library="__MyCommonLib1" package="RSMD_0805" value="3K0" x="35.3" y="19.8" rot="MR90"/>
 <element name="C4" library="__MyCommonLib1" package="RSMD_0805" value="0.1uF" x="38" y="19.8" rot="MR270"/>
 <element name="D4" library="__MyCommonLib1" package="SOD-80" value="LL4148" x="30.5" y="45.6" rot="MR270"/>
