File: LC_METER/schematic/LCMeter.brd (EAGLE design)
At the start: 70 x 125 mm, 212 parts, among them IC1 MEGA8535, IC10 MC34063, IC2 74HC595, IC3 74HC595, IC4 74HC595, IC5 74HC595, IC6 74HC595, IC7 LM324, IC8 7905, IC9 LM317, J10 0, J100 0, J11 0, J4 0, J6 0, J8 0, Q1 12MHz, T1 BC847, T2 BC857, T3 BC847, T4 BC847, T5 BC847, T6 BC847, T7 BC857, X1 MCU_PROGRAMMING, X2 L_X, X3 C_X, X4 USB_MICRO, X5 USB_B

Commit message: LC Metter. Adjust +5v stabilizer values
Parts:
- added R90: 100K*, __MyCommonLib1:RSMD_0805
- R81: value 1K0 -> 1K1 1%
- R82: value 3K0 -> 3K3 1%
Connections:
- net GND: now also R90.PAD_0
- net N$142: now also R90.PAD_1
Changed lines of the file:
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@@
 <element name="C51" library="__MyCommonLib1" package="RSMD_0805" value="0.47uFx16V" x="26.9" y="46.7" rot="MR180"/>
 <element name="C52" library="__MyCommonLib1" package="CE_10MM" value="47uFx16V" x="28.3" y="49.9"/>
-<element name="R81" library="__MyCommonLib1" package="RSMD_0805" value="1K0" x="39.3" y="65.8" rot="MR180"/>
-<element name="R82" library="__MyCommonLib1" package="RSMD_0805" value="3K0" x="40.2" y="69.1" rot="MR270"/>
+<element name="R81" library="__MyCommonLib1" package="RSMD_0805" value="1K1 1%" x="39.3" y="65.8" rot="MR180"/>
+<element name="R82" library="__MyCommonLib1" package="RSMD_0805" value="3K3 1%" x="40.2" y="69.1" rot="MR270"/>
 <element name="IC8" library="__MyCommonLib1" package="D2PAK" value="7905" x="6.6" y="49" rot="MR0"/>
 <element name="C3" library="__MyCommonLib1" package="RSMD_0805" value="0.1uF" x="38.8" y="27.5" rot="MR0"/>
@@
 <element name="C4" library="__MyCommonLib1" package="RSMD_0805" value="0.1uF" x="38" y="19.8" rot="MR270"/>
 <element name="D4" library="__MyCommonLib1" package="SOD-80" value="LL4148" x="30.5" y="45.6" rot="MR270"/>
+<element name="R90" library="__MyCommonLib1" package="RSMD_0805" value="100K*" x="-1.2" y="-5"/>
 </elements>
 <signals>
@@
 <vertex x="54.3" y="93.6"/>
 </polygon>
+<contactref element="R90" pad="PAD_0"/>
+<wire x1="3.5" y1="6.17" x2="-2.25" y2="-5" width="0" layer="19" extent="1-1"/>
 </signal>
 <signal name="+5V_USB">
@@
 <wire x1="44.17" y1="60.84" x2="43.71" y2="61.3" width="0.8" layer="16"/>
 <wire x1="43.71" y1="61.3" x2="42.8" y2="61.3" width="0.8" layer="16"/>
+<contactref element="R90" pad="PAD_1"/>
+<wire x1="-0.15" y1="-5" x2="42.8" y2="61.3" width="0" layer="19" extent="1-16"/>
 </signal>
 <signal name="N$141">
