File: LC_METER/schematic/LCMeter.sch (EAGLE design)
At the start: 212 parts, among them IC1 MEGA8535, IC10 MC34063, IC2 74HC595, IC3 74HC595, IC4 74HC595, IC5 74HC595, IC6 74HC595, IC7 LM324, IC8 7905, IC9 LM317, J10 0, J100 0, J11 0, J4 0, J6 0, J8 0, Q1 12MHz, T1 BC847, T2 BC857, T3 BC847, T4 BC847, T5 BC847, T6 BC847, T7 BC857, X1 MCU_PROGRAMMING, X2 L_X, X3 C_X, X4 USB_MICRO, X5 USB_B

Commit message: LC meter schematic. Power stabilizer values fix
Parts:
- R81: value 5K1 -> 1K0
- R82: value 1K7 -> 3K0
- R84: value 5K1 -> 4K7
- R85: value 1K7 -> 1K6
Changed lines of the file:
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@@
 <setting verticaltext="up"/>
 </settings>
-<grid distance="0.05" unitdist="inch" unit="inch" style="lines" multiple="2" display="yes" altdistance="0.01" altunitdist="inch" altunit="inch"/>
+<grid distance="0.1" unitdist="inch" unit="inch" style="lines" multiple="1" display="no" altdistance="0.01" altunitdist="inch" altunit="inch"/>
 <layers>
-<layer number="1" name="Top" color="4" fill="1" visible="yes" active="no"/>
-<layer number="2" name="Route2" color="1" fill="3" visible="yes" active="no"/>
-<layer number="3" name="Route3" color="4" fill="3" visible="yes" active="no"/>
-<layer number="4" name="Route4" color="1" fill="4" visible="yes" active="no"/>
-<layer number="5" name="Route5" color="4" fill="4" visible="yes" active="no"/>
-<layer number="6" name="Route6" color="1" fill="8" visible="yes" active="no"/>
-<layer number="7" name="Route7" color="4" fill="8" visible="yes" active="no"/>
-<layer number="8" name="Route8" color="1" fill="2" visible="yes" active="no"/>
-<layer number="9" name="Route9" color="4" fill="2" visible="yes" active="no"/>
-<layer number="10" name="Route10" color="1" fill="7" visible="yes" active="no"/>
-<layer number="11" name="Route11" color="4" fill="7" visible="yes" active="no"/>
-<layer number="12" name="Route12" color="1" fill="5" visible="yes" active="no"/>
-<layer number="13" name="Route13" color="4" fill="5" visible="yes" active="no"/>
-<layer number="14" name="Route14" color="1" fill="6" visible="yes" active="no"/>
-<layer number="15" name="Route15" color="4" fill="6" visible="yes" active="no"/>
-<layer number="16" name="Bottom" color="1" fill="1" visible="yes" active="no"/>
-<layer number="17" name="Pads" color="2" fill="1" visible="yes" active="no"/>
-<layer number="18" name="Vias" color="2" fill="1" visible="yes" active="no"/>
-<layer number="19" name="Unrouted" color="6" fill="1" visible="yes" active="no"/>
-<layer number="20" name="Dimension" color="15" fill="1" visible="yes" active="no"/>
-<layer number="21" name="tPlace" color="7" fill="1" visible="yes" active="no"/>
-<layer number="22" name="bPlace" color="7" fill="1" visible="yes" active="no"/>
-<layer number="23" name="tOrigins" color="15" fill="1" visible="yes" active="no"/>
-<layer number="24" name="bOrigins" color="15" fill="1" visible="yes" active="no"/>
-<layer number="25" name="tNames" color="7" fill="1" visible="yes" active="no"/>
-<layer number="26" name="bNames" color="7" fill="1" visible="yes" active="no"/>
-<layer number="27" name="tValues" color="7" fill="1" visible="yes" active="no"/>
-<layer number="28" name="bValues" color="7" fill="1" visible="yes" active="no"/>
+<layer number="1" name="Top" color="4" fill="1" visible="no" active="no"/>
+<layer number="2" name="Route2" color="1" fill="3" visible="no" active="no"/>
+<layer number="3" name="Route3" color="4" fill="3" visible="no" active="no"/>
+<layer number="4" name="Route4" color="1" fill="4" visible="no" active="no"/>
+<layer number="5" name="Route5" color="4" fill="4" visible="no" active="no"/>
+<layer number="6" name="Route6" color="1" fill="8" visible="no" active="no"/>
+<layer number="7" name="Route7" color="4" fill="8" visible="no" active="no"/>
+<layer number="8" name="Route8" color="1" fill="2" visible="no" active="no"/>
+<layer number="9" name="Route9" color="4" fill="2" visible="no" active="no"/>
+<layer number="10" name="Route10" color="1" fill="7" visible="no" active="no"/>
+<layer number="11" name="Route11" color="4" fill="7" visible="no" active="no"/>
+<layer number="12" name="Route12" color="1" fill="5" visible="no" active="no"/>
+<layer number="13" name="Route13" color="4" fill="5" visible="no" active="no"/>
+<layer number="14" name="Route14" color="1" fill="6" visible="no" active="no"/>
+<layer number="15" name="Route15" color="4" fill="6" visible="no" active="no"/>
+<layer number="16" name="Bottom" color="1" fill="1" visible="no" active="no"/>
+<layer number="17" name="Pads" color="2" fill="1" visible="no" active="no"/>
+<layer number="18" name="Vias" color="2" fill="1" visible="no" active="no"/>
+<layer number="19" name="Unrouted" color="6" fill="1" visible="no" active="no"/>
+<layer number="20" name="Dimension" color="15" fill="1" visible="no" active="no"/>
+<layer number="21" name="tPlace" color="7" fill="1" visible="no" active="no"/>
+<layer number="22" name="bPlace" color="7" fill="1" visible="no" active="no"/>
+<layer number="23" name="tOrigins" color="15" fill="1" visible="no" active="no"/>
+<layer number="24" name="bOrigins" color="15" fill="1" visible="no" active="no"/>
+<layer number="25" name="tNames" color="7" fill="1" visible="no" active="no"/>
+<layer number="26" name="bNames" color="7" fill="1" visible="no" active="no"/>
+<layer number="27" name="tValues" color="7" fill="1" visible="no" active="no"/>
+<layer number="28" name="bValues" color="7" fill="1" visible="no" active="no"/>
 <layer number="29" name="tStop" color="7" fill="3" visible="no" active="no"/>
 <layer number="30" name="bStop" color="7" fill="6" visible="no" active="no"/>
@@
 <layer number="35" name="tGlue" color="7" fill="4" visible="no" active="no"/>
 <layer number="36" name="bGlue" color="7" fill="5" visible="no" active="no"/>
-<layer number="37" name="tTest" color="7" fill="1" visible="yes" active="no"/>
-<layer number="38" name="bTest" color="7" fill="1" visible="yes" active="no"/>
+<layer number="37" name="tTest" color="7" fill="1" visible="no" active="no"/>
+<layer number="38" name="bTest" color="7" fill="1" visible="no" active="no"/>
 <layer number="39" name="tKeepout" color="4" fill="11" visible="no" active="no"/>
 <layer number="40" name="bKeepout" color="1" fill="11" visible="no" active="no"/>
@@
 <layer number="44" name="Drills" color="7" fill="1" visible="no" active="no"/>
 <layer number="45" name="Holes" color="7" fill="1" visible="no" active="no"/>
-<layer number="46" name="Milling" color="3" fill="1" visible="yes" active="no"/>
-<layer number="47" name="Measures" color="7" fill="1" visible="yes" active="no"/>
-<layer number="48" name="Document" color="7" fill="1" visible="yes" active="no"/>
-<layer number="49" name="Reference" color="7" fill="1" visible="yes" active="no"/>
-<layer number="51" name="tDocu" color="7" fill="1" visible="yes" active="no"/>
-<layer number="52" name="bDocu" color="7" fill="1" visible="yes" active="no"/>
+<layer number="46" name="Milling" color="3" fill="1" visible="no" active="no"/>
+<layer number="47" name="Measures" color="7" fill="1" visible="no" active="no"/>
+<layer number="48" name="Document" color="7" fill="1" visible="no" active="no"/>
+<layer number="49" name="Reference" color="7" fill="1" visible="no" active="no"/>
+<layer number="51" name="tDocu" color="7" fill="1" visible="no" active="no"/>
+<layer number="52" name="bDocu" color="7" fill="1" visible="no" active="no"/>
 <layer number="91" name="Nets" color="2" fill="1" visible="yes" active="yes"/>
 <layer number="92" name="Busses" color="1" fill="1" visible="yes" active="yes"/>
@@
 <part name="GND73" library="supply1" deviceset="GND" device=""/>
 <part name="GND74" library="supply1" deviceset="GND" device=""/>
-<part name="R84" library="__MyCommonLib1" deviceset="R" device="0207" value="5K1"/>
-<part name="R85" library="__MyCommonLib1" deviceset="R" device="SMD_0805" value="1K7"/>
+<part name="R84" library="__MyCommonLib1" deviceset="R" device="0207" value="4K7"/>
+<part name="R85" library="__MyCommonLib1" deviceset="R" device="SMD_0805" value="1K6"/>
 <part name="GND75" library="supply1" deviceset="GND" device=""/>
 <part name="C49" library="__MyCommonLib1" deviceset="C" device="SMD_1206" value="0.47uFx16V"/>
@@
 <part name="GND79" library="supply1" deviceset="GND" device=""/>
 <part name="GND80" library="supply1" deviceset="GND" device=""/>
-<part name="R81" library="__MyCommonLib1" deviceset="R" device="SMD_0805" value="5K1"/>
-<part name="R82" library="__MyCommonLib1" deviceset="R" device="SMD_0805" value="1K7"/>
+<part name="R81" library="__MyCommonLib1" deviceset="R" device="SMD_0805" value="1K0"/>
+<part name="R82" library="__MyCommonLib1" deviceset="R" device="SMD_0805" value="3K0"/>
 <part name="IC8" library="__MyCommonLib1" deviceset="7905" device="(D2PAK)" value="7905"/>
 <part name="GND82" library="supply1" deviceset="GND" device=""/>
@@
 </sheet>
 </sheets>
+<errors>
+</errors>
 </schematic>
 </drawing>

Commit message: LC Meter change some values
Parts:
- C47, C58: value 4.7uF -> 100uFx10V
- R54, R67, R69, R71: value 100K -> 120K
- R55, R74: value 4K7 -> 2K2
- R58: value 20K -> 24K
- R59: value 300R -> 1K0
- R75, R77, R79: value 25K -> 24K
- R86, R87, R88: value 1K0 -> 10K
Changed lines of the file:
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@@
 <part name="R9" library="__MyCommonLib1" deviceset="R" device="SMD_0805" value="1K5"/>
 <part name="FRAME3" library="frames" deviceset="A4L-LOC" device="" value="L_METER"/>
-<part name="R55" library="__MyCommonLib1" deviceset="R" device="SMD_0805" value="4K7"/>
+<part name="R55" library="__MyCommonLib1" deviceset="R" device="SMD_0805" value="2K2"/>
 <part name="C17" library="__MyCommonLib1" deviceset="C" device="SMD_0805" value="1nF"/>
 <part name="T1" library="__MyCommonLib1" deviceset="BC847" device="SOT23_SMALL_PADS" value="BC847"/>
@@
 <part name="GND8" library="supply1" deviceset="GND" device=""/>
 <part name="R60" library="__MyCommonLib1" deviceset="R" device="SMD_0805" value="4K7"/>
-<part name="R58" library="__MyCommonLib1" deviceset="R" device="SMD_0805" value="20K"/>
+<part name="R58" library="__MyCommonLib1" deviceset="R" device="SMD_0805" value="24K"/>
 <part name="C16" library="__MyCommonLib1" deviceset="C" device="SMD_0805" value="0.1uF"/>
 <part name="IC7" library="__MyCommonLib1" deviceset="LM324" device=""/>
@@
 <part name="GND3" library="supply1" deviceset="GND" device=""/>
 <part name="GND4" library="supply1" deviceset="GND" device=""/>
-<part name="R54" library="__MyCommonLib1" deviceset="R" device="SMD_0805" value="100K"/>
+<part name="R54" library="__MyCommonLib1" deviceset="R" device="SMD_0805" value="120K"/>
 <part name="GND12" library="supply1" deviceset="GND" device=""/>
-<part name="R59" library="__MyCommonLib1" deviceset="R" device="SMD_1206_BIG_GAP" value="300R"/>
+<part name="R59" library="__MyCommonLib1" deviceset="R" device="SMD_1206_BIG_GAP" value="1K0"/>
 <part name="D10" library="__MyCommonLib1" deviceset="LL4147" device="SOD-80" value="LL4148"/>
 <part name="C20" library="__MyCommonLib1" deviceset="C" device="SMD_0805" value="0.1uF"/>
 <part name="GND13" library="supply1" deviceset="GND" device=""/>
 <part name="GND15" library="supply1" deviceset="GND" device=""/>
-<part name="R74" library="__MyCommonLib1" deviceset="R" device="SMD_0805" value="4K7"/>
+<part name="R74" library="__MyCommonLib1" deviceset="R" device="SMD_0805" value="2K2"/>
 <part name="C39" library="__MyCommonLib1" deviceset="C" device="SMD_0805" value="1nF"/>
 <part name="T3" library="__MyCommonLib1" deviceset="BC847" device="SOT23_SMALL_PADS" value="BC847"/>
@@
 <part name="T4" library="__MyCommonLib1" deviceset="BC847" device="SOT23_SMALL_PADS" value="BC847"/>
 <part name="C41" library="__MyCommonLib1" deviceset="C" device="SMD_0805" value="0.1uF"/>
-<part name="R75" library="__MyCommonLib1" deviceset="R" device="SMD_0805" value="25K"/>
+<part name="R75" library="__MyCommonLib1" deviceset="R" device="SMD_0805" value="24K"/>
 <part name="GND44" library="supply1" deviceset="GND" device=""/>
 <part name="GND46" library="supply1" deviceset="GND" device=""/>
-<part name="R67" library="__MyCommonLib1" deviceset="R" device="SMD_0805" value="100K"/>
+<part name="R67" library="__MyCommonLib1" deviceset="R" device="SMD_0805" value="120K"/>
 <part name="R68" library="__MyCommonLib1" deviceset="R" device="SMD_0805" value="1K0"/>
 <part name="R76" library="__MyCommonLib1" deviceset="R" device="SMD_0805" value="100R"/>
@@
 <part name="T5" library="__MyCommonLib1" deviceset="BC847" device="SOT23_SMALL_PADS" value="BC847"/>
 <part name="C42" library="__MyCommonLib1" deviceset="C" device="SMD_0805" value="0.1uF"/>
-<part name="R77" library="__MyCommonLib1" deviceset="R" device="SMD_0805" value="25K"/>
-<part name="R69" library="__MyCommonLib1" deviceset="R" device="SMD_0805" value="100K"/>
+<part name="R77" library="__MyCommonLib1" deviceset="R" device="SMD_0805" value="24K"/>
+<part name="R69" library="__MyCommonLib1" deviceset="R" device="SMD_0805" value="120K"/>
 <part name="R70" library="__MyCommonLib1" deviceset="R" device="SMD_0805" value="1K0"/>
 <part name="R78" library="__MyCommonLib1" deviceset="R" device="SMD_0805" value="100R"/>
@@
 <part name="T6" library="__MyCommonLib1" deviceset="BC847" device="SOT23_SMALL_PADS" value="BC847"/>
 <part name="C43" library="__MyCommonLib1" deviceset="C" device="SMD_0805" value="0.1uF"/>
-<part name="R79" library="__MyCommonLib1" deviceset="R" device="SMD_0805" value="25K"/>
-<part name="R71" library="__MyCommonLib1" deviceset="R" device="SMD_0805" value="100K"/>
+<part name="R79" library="__MyCommonLib1" deviceset="R" device="SMD_0805" value="24K"/>
+<part name="R71" library="__MyCommonLib1" deviceset="R" device="SMD_0805" value="120K"/>
 <part name="R72" library="__MyCommonLib1" deviceset="R" device="SMD_0805" value="1K0"/>
 <part name="R80" library="__MyCommonLib1" deviceset="R" device="SMD_0805" value="100R"/>
@@
 <part name="GND98" library="supply1" deviceset="GND" device=""/>
 <part name="C48" library="__MyCommonLib1" deviceset="CE" device="6.3MM" value="47uFx16V"/>
-<part name="R86" library="__MyCommonLib1" deviceset="R" device="SMD_0805" value="1K0"/>
+<part name="R86" library="__MyCommonLib1" deviceset="R" device="SMD_0805" value="10K"/>
 <part name="GND33" library="supply1" deviceset="GND" device=""/>
-<part name="R87" library="__MyCommonLib1" deviceset="R" device="SMD_0805" value="1K0"/>
+<part name="R87" library="__MyCommonLib1" deviceset="R" device="SMD_0805" value="10K"/>
 <part name="GND34" library="supply1" deviceset="GND" device=""/>
-<part name="R88" library="__MyCommonLib1" deviceset="R" device="SMD_0805" value="1K0"/>
+<part name="R88" library="__MyCommonLib1" deviceset="R" device="SMD_0805" value="10K"/>
 <part name="GND35" library="supply1" deviceset="GND" device=""/>
 <part name="J100" library="__MyCommonLib1" deviceset="R" device="SMD_1206_BIG_GAP" value="0"/>
-<part name="C47" library="__MyCommonLib1" deviceset="CE" device="6.3MM" value="4.7uF"/>
-<part name="C58" library="__MyCommonLib1" deviceset="CE" device="6.3MM" value="4.7uF"/>
+<part name="C47" library="__MyCommonLib1" deviceset="CE" device="6.3MM" value="100uFx10V"/>
+<part name="C58" library="__MyCommonLib1" deviceset="CE" device="6.3MM" value="100uFx10V"/>
 <part name="GND81" library="supply1" deviceset="GND" device=""/>
 <part name="GND86" library="supply1" deviceset="GND" device=""/>

Commit message: LC Meter. Battery voltage metter resistors values changed
Parts:
- R89: value 1K -> 3K0
Changed lines of the file:
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@@
 <part name="J11" library="__MyCommonLib1" deviceset="R" device="SMD_0805" value="0"/>
 <part name="R100" library="__MyCommonLib1" deviceset="R" device="SMD_0805" value="10K"/>
-<part name="R89" library="__MyCommonLib1" deviceset="R" device="SMD_0805" value="1K"/>
+<part name="R89" library="__MyCommonLib1" deviceset="R" device="SMD_0805" value="3K0"/>
 <part name="C4" library="__MyCommonLib1" deviceset="C" device="SMD_0805" value="0.1uF"/>
 <part name="D4" library="__MyCommonLib1" deviceset="LL4147" device="SOD-80" value="LL4148"/>

Commit message: LC Metter. Adjust +5v stabilizer values
Parts:
- added R90: 100K*, __MyCommonLib1:RSMD_0805
- R81: value 1K0 -> 1K1 1%
- R82: value 3K0 -> 3K3 1%
Connections:
- net GND: now also R90.PIN0
- net N$142: now also R90.PIN1
Other:
- moved on the sheet: R82
Changed lines of the file:
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@@
 <setting verticaltext="up"/>
 </settings>
-<grid distance="0.1" unitdist="inch" unit="inch" style="lines" multiple="1" display="no" altdistance="0.01" altunitdist="inch" altunit="inch"/>
+<grid distance="0.05" unitdist="inch" unit="inch" style="lines" multiple="2" display="yes" altdistance="0.01" altunitdist="inch" altunit="inch"/>
 <layers>
 <layer number="1" name="Top" color="4" fill="1" visible="no" active="no"/>
@@
 <part name="GND79" library="supply1" deviceset="GND" device=""/>
 <part name="GND80" library="supply1" deviceset="GND" device=""/>
-<part name="R81" library="__MyCommonLib1" deviceset="R" device="SMD_0805" value="1K0"/>
-<part name="R82" library="__MyCommonLib1" deviceset="R" device="SMD_0805" value="3K0"/>
+<part name="R81" library="__MyCommonLib1" deviceset="R" device="SMD_0805" value="1K1 1%"/>
+<part name="R82" library="__MyCommonLib1" deviceset="R" device="SMD_0805" value="3K3 1%"/>
 <part name="IC8" library="__MyCommonLib1" deviceset="7905" device="(D2PAK)" value="7905"/>
 <part name="GND82" library="supply1" deviceset="GND" device=""/>
@@
 <part name="GND43" library="supply1" deviceset="GND" device=""/>
 <part name="GND88" library="supply1" deviceset="GND" device=""/>
+<part name="R90" library="__MyCommonLib1" deviceset="R" device="SMD_0805" value="100K*"/>
 </parts>
 <sheets>
@@
 </instance>
 <instance part="C49" gate="C$1" x="177.8" y="66.04" smashed="yes">
-<attribute name="NAME" x="176.53" y="68.58" size="1.27" layer="95" font="vector" ratio="20" rot="R180"/>
+<attribute name="NAME" x="175.26" y="66.04" size="1.27" layer="95" font="vector" ratio="20" rot="R180"/>
 <attribute name="VALUE" x="175.26" y="64.77" size="1.27" layer="96" font="vector" ratio="20" rot="R180"/>
 </instance>
 <instance part="C50" gate="C$1" x="182.88" y="66.04" smashed="yes">
-<attribute name="NAME" x="184.15" y="67.31" size="1.27" layer="95" font="vector" ratio="20"/>
-<attribute name="VALUE" x="184.15" y="63.5" size="1.27" layer="96" font="vector" ratio="20"/>
+<attribute name="NAME" x="175.26" y="63.5" size="1.27" layer="95" font="vector" ratio="20" rot="R180"/>
+<attribute name="VALUE" x="175.26" y="62.23" size="1.27" layer="96" font="vector" ratio="20" rot="R180"/>
 </instance>
 <instance part="GND76" gate="1" x="177.8" y="58.42" smashed="yes">
@@
 </instance>
 <instance part="GND77" gate="1" x="182.88" y="58.42" smashed="yes">
-<attribute name="VALUE" x="180.34" y="53.34" size="1.27" layer="96" font="vector" ratio="20"/>
+<attribute name="VALUE" x="181.61" y="55.88" size="1.27" layer="96" font="vector" ratio="20"/>
 </instance>
 <instance part="IC9" gate="G$1" x="193.04" y="71.12" smashed="yes">
@@
 <attribute name="VALUE" x="190.5" y="74.295" size="1.27" layer="96" font="vector" ratio="20"/>
 </instance>
-<instance part="GND78" gate="1" x="208.28" y="55.88" smashed="yes">
-<attribute name="VALUE" x="205.74" y="50.8" size="1.27" layer="96" font="vector" ratio="20"/>
+<instance part="GND78" gate="1" x="193.04" y="43.18" smashed="yes">
+<attribute name="VALUE" x="190.5" y="38.1" size="1.27" layer="96" font="vector" ratio="20"/>
 </instance>
 <instance part="C51" gate="C$1" x="213.36" y="66.04" smashed="yes">
@@
 </instance>
 <instance part="GND79" gate="1" x="213.36" y="58.42" smashed="yes">
-<attribute name="VALUE" x="210.82" y="53.34" size="1.27" layer="96" font="vector" ratio="20"/>
+<attribute name="VALUE" x="210.82" y="55.88" size="1.27" layer="96" font="vector" ratio="20"/>
 </instance>
 <instance part="GND80" gate="1" x="218.44" y="58.42" smashed="yes">
-<attribute name="VALUE" x="215.9" y="53.34" size="1.27" layer="96" font="vector" ratio="20"/>
+<attribute name="VALUE" x="218.44" y="55.88" size="1.27" layer="96" font="vector" ratio="20"/>
 </instance>
 <instance part="R81" gate="R$1" x="200.66" y="63.5" smashed="yes" rot="R90">
-<attribute name="NAME" x="201.93" y="67.31" size="1.27" layer="95" font="vector" ratio="20" rot="R180"/>
-<attribute name="VALUE" x="201.93" y="66.04" size="1.27" layer="96" font="vector" ratio="20" rot="R180"/>
+<attribute name="NAME" x="199.39" y="67.31" size="1.27" layer="95" font="vector" ratio="20"/>
+<attribute name="VALUE" x="204.47" y="66.04" size="1.27" layer="96" font="vector" ratio="20" rot="R180"/>
 </instance>
-<instance part="R82" gate="R$1" x="200.66" y="60.96" smashed="yes" rot="R90">
-<attribute name="NAME" x="198.12" y="58.42" size="1.27" layer="95" font="vector" ratio="20"/>
-<attribute name="VALUE" x="198.12" y="57.15" size="1.27" layer="96" font="vector" ratio="20"/>
+<instance part="R82" gate="R$1" x="193.04" y="55.88" smashed="yes">
+<attribute name="NAME" x="195.58" y="58.42" size="1.27" layer="95" font="vector" ratio="20"/>
+<attribute name="VALUE" x="195.58" y="57.15" size="1.27" layer="96" font="vector" ratio="20"/>
 </instance>
 <instance part="IC8" gate="G$1" x="182.88" y="149.86" smashed="yes">
@@
 <attribute name="VALUE" x="41.91" y="157.48" size="1.27" layer="96" font="vector" ratio="20" rot="R180"/>
 </instance>
+<instance part="R90" gate="R$1" x="190.5" y="55.88" smashed="yes">
+<attribute name="NAME" x="195.58" y="54.61" size="1.27" layer="95" font="vector" ratio="20"/>
+<attribute name="VALUE" x="195.58" y="53.34" size="1.27" layer="96" font="vector" ratio="20"/>
+</instance>
 </instances>
 <busses>
@@
 <pinref part="R82" gate="R$1" pin="PIN0"/>
 <pinref part="GND78" gate="1" pin="GND"/>
-<wire x1="205.74" y1="60.96" x2="208.28" y2="60.96" width="0.1524" layer="91"/>
-<wire x1="208.28" y1="60.96" x2="208.28" y2="58.42" width="0.1524" layer="91"/>
+<wire x1="193.04" y1="50.8" x2="193.04" y2="48.26" width="0.1524" layer="91"/>
+<pinref part="R90" gate="R$1" pin="PIN0"/>
+<wire x1="193.04" y1="48.26" x2="193.04" y2="45.72" width="0.1524" layer="91"/>
+<wire x1="193.04" y1="48.26" x2="190.5" y2="48.26" width="0.1524" layer="91"/>
+<wire x1="190.5" y1="48.26" x2="190.5" y2="50.8" width="0.1524" layer="91"/>
+<junction x="193.04" y="48.26"/>
 </segment>
 <segment>
@@
 <pinref part="R82" gate="R$1" pin="PIN1"/>
 <pinref part="IC9" gate="G$1" pin="ADJ"/>
-<wire x1="195.58" y1="60.96" x2="193.04" y2="60.96" width="0.1524" layer="91"/>
 <wire x1="193.04" y1="60.96" x2="193.04" y2="63.5" width="0.1524" layer="91"/>
 <pinref part="R81" gate="R$1" pin="PIN1"/>
@@
 <wire x1="195.58" y1="63.5" x2="193.04" y2="63.5" width="0.1524" layer="91"/>
 <junction x="193.04" y="63.5"/>
+<pinref part="R90" gate="R$1" pin="PIN1"/>
+<wire x1="193.04" y1="63.5" x2="190.5" y2="63.5" width="0.1524" layer="91"/>
+<wire x1="190.5" y1="63.5" x2="190.5" y2="60.96" width="0.1524" layer="91"/>
 </segment>
 </net>
