File: L_Saturation_Meter/schematic/L_SaturationMeter.brd (EAGLE design)
At the start: 40 parts, among them IC1 LM317, IC4 LM358, T1 IRF830, T2 BC847, T3 BC857, X2 POWER_12V, X3 L_TEST, X4 I_SENSE

Commit message: Fix inconsistancy error
Parts:
- removed C11: 1000uFx25V, __MyCommonLib1:CE_10MM
- removed C12: 470uFx16V, __MyCommonLib1:CE_10MM
- added C104: 470uFx16V, __MyCommonLib1:CE_8.2MM
- added C8: 1000uFx25V, __MyCommonLib1:CE_10MM
- moved X2 137.1 mm to (100.3, 5.08)
- moved X3 132.0 mm to (71.1, 29.2)
- moved C2 131.2 mm to (29.2, 31.8)
- moved D100 131.2 mm to (68.6, 19.1)
- moved C1 130.3 mm to (21.6, 27.9)
- moved C10 130.3 mm to (49.5, 17.8)
- moved C13 130.3 mm to (81.3, 19.1)
- moved C3 130.3 mm to (30.5, 22.9)
- moved C4 130.3 mm to (27.9, 22.9)
- moved C5 130.3 mm to (47.0, 7.62)
- moved C6 130.3 mm to (39.4, 2.54)
- moved C7 130.3 mm to (35.6, 15.2)
- moved D1 130.3 mm to (53.3, 3.81)
- moved D2 130.3 mm to (48.3, 15.2)
- moved D3 130.3 mm to (21.6, 26.7)
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Connections:
- net GND: now also C100.-, C8.-
- net N$6: now also C104.-; no longer C12.+
- net N$9: now also C100.+, C104.+, C8.+; no longer C12.-

Commit message: Fix CE packages pads naming, to avoid inconsistance after package change
Parts:
- C2: device __MyCommonLib1:CE_10MM -> __MyCommonLib1:CE_8.2MM
- C4: device __MyCommonLib1:CE_6.3MM -> __MyCommonLib1:CE_5.2MM
- moved C3 8.98 mm to (21.6, 21.6), turned to 270 degrees
- moved C4 4.02 mm to (24.1, 21.6), turned to 90 degrees
- moved D3 3.81 mm to (21.6, 30.5)
- moved C1 2.54 mm to (21.6, 30.5)
- moved C2 1.80 mm to (27.9, 30.5)
Connections:
- net +VCC: now also C4.PLUS; no longer C4.+
- net GND: now also C100.MINUS, C2.MINUS, C4.MINUS, C8.MINUS; no longer C100.-, C2.-, C4.-, C8.-
- net N$11: now also C2.PLUS; no longer C2.+
- net N$6: now also C104.MINUS; no longer C104.-
- net N$9: now also C100.PLUS, C104.PLUS, C8.PLUS; no longer C100.+, C104.+, C8.+
Changed lines of the file:
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@@
 <element name="C14" library="__MyCommonLib1" package="RSMD_1206_BIG_GAP" value="1uFx25V" x="91.44" y="19.05" rot="MR180"/>
 <element name="IC1" library="__MyCommonLib1" package="D2PAK" value="LM317" x="13.97" y="24.13" rot="MR180"/>
-<element name="C1" library="__MyCommonLib1" package="RSMD_1206_BIG_GAP" value="0.1uFx25V" x="21.59" y="27.94" rot="MR270"/>
-<element name="C2" library="__MyCommonLib1" package="CE_10MM" value="470uFx16V" x="29.21" y="31.75" rot="R90"/>
-<element name="D3" library="__MyCommonLib1" package="DO-41_10MM" value="1N4001" x="21.59" y="26.67" rot="R90"/>
+<element name="C1" library="__MyCommonLib1" package="RSMD_1206_BIG_GAP" value="0.1uFx25V" x="21.59" y="30.48" rot="MR270"/>
+<element name="C2" library="__MyCommonLib1" package="CE_8.2MM" value="470uFx16V" x="27.94" y="30.48" rot="R90"/>
+<element name="D3" library="__MyCommonLib1" package="DO-41_10MM" value="1N4001" x="21.59" y="30.48" rot="R90"/>
 <element name="R1" library="__MyCommonLib1" package="RSMD_0805" value="1K0" x="2.54" y="22.86" rot="MR90"/>
 <element name="R2" library="__MyCommonLib1" package="RSMD_0805" value="3K0" x="6.35" y="22.86" rot="MR270"/>
-<element name="C3" library="__MyCommonLib1" package="RSMD_0805" value="0.1uFx25V" x="30.48" y="22.86" rot="MR90"/>
-<element name="C4" library="__MyCommonLib1" package="CE_6.3MM" value="47uFx16V" x="27.94" y="22.86" rot="R270"/>
+<element name="C3" library="__MyCommonLib1" package="RSMD_0805" value="0.1uFx25V" x="21.59" y="21.59" rot="MR270"/>
+<element name="C4" library="__MyCommonLib1" package="CE_5.2MM" value="47uFx16V" x="24.13" y="21.59" rot="R90"/>
 <element name="C5" library="__MyCommonLib1" package="RSMD_0805" value="0.1uFx25V" x="46.99" y="7.62" rot="MR270"/>
 <element name="D4" library="__MyCommonLib1" package="SOD-80" value="LL4148" x="35.56" y="7.62" rot="MR270"/>
@@
 <contactref element="C14" pad="PAD_1"/>
 <contactref element="C1" pad="PAD_1"/>
-<contactref element="C2" pad="-"/>
+<contactref element="C2" pad="MINUS"/>
 <contactref element="R1" pad="PAD_0"/>
 <contactref element="C3" pad="PAD_1"/>
-<contactref element="C4" pad="-"/>
+<contactref element="C4" pad="MINUS"/>
 <contactref element="C5" pad="PAD_1"/>
 <contactref element="C6" pad="PAD_1"/>
@@
 <contactref element="R102" pad="PACKAGE1"/>
 <contactref element="R102" pad="PACKAGE2"/>
-<contactref element="C100" pad="-"/>
-<contactref element="C8" pad="-"/>
+<contactref element="C100" pad="MINUS"/>
+<contactref element="C8" pad="MINUS"/>
 <wire x1="93.065" y1="19.05" x2="91.44" y2="24.13" width="0" layer="19" extent="16-16"/>
 <wire x1="91.44" y1="13.97" x2="93.065" y2="19.05" width="0" layer="19" extent="16-16"/>
@@
 <wire x1="46.99" y1="6.57" x2="44.45" y2="1.49" width="0" layer="19" extent="16-16"/>
 <wire x1="39.4" y1="20.32" x2="46.99" y2="6.57" width="0" layer="19" extent="16-16"/>
-<wire x1="30.48" y1="23.91" x2="39.4" y2="20.32" width="0" layer="19" extent="16-16"/>
-<wire x1="27.94" y1="24.13" x2="30.48" y2="23.91" width="0" layer="19" extent="16-16"/>
-<wire x1="29.21" y1="29.21" x2="27.94" y2="24.13" width="0" layer="19" extent="1-1"/>
-<wire x1="21.59" y1="26.315" x2="27.94" y2="24.13" width="0" layer="19" extent="16-16"/>
-<wire x1="2.54" y1="21.81" x2="21.59" y2="26.315" width="0" layer="19" extent="16-16"/>
-<wire x1="1.16" y1="8.89" x2="2.54" y2="21.81" width="0" layer="19" extent="16-16"/>
-<wire x1="10.16" y1="8.89" x2="1.16" y2="8.89" width="0" layer="19" extent="1-1"/>
+<wire x1="27.94" y1="28.78" x2="39.4" y2="20.32" width="0" layer="19" extent="16-16"/>
+<wire x1="21.59" y1="28.855" x2="27.94" y2="28.78" width="0" layer="19" extent="16-16"/>
+<wire x1="21.59" y1="20.54" x2="21.59" y2="28.855" width="0" layer="19" extent="16-16"/>
+<wire x1="24.13" y1="20.59" x2="21.59" y2="20.54" width="0" layer="19" extent="16-16"/>
+<wire x1="10.16" y1="8.89" x2="21.59" y2="20.54" width="0" layer="19" extent="16-16"/>
+<wire x1="1.16" y1="8.89" x2="10.16" y2="8.89" width="0" layer="19" extent="1-1"/>
+<wire x1="2.54" y1="21.81" x2="1.16" y2="8.89" width="0" layer="19" extent="16-16"/>
 </signal>
 <signal name="N$1">
@@
 <contactref element="R14" pad="PAD_0"/>
 <contactref element="C13" pad="PAD_1"/>
-<contactref element="C104" pad="-"/>
+<contactref element="C104" pad="MINUS"/>
 <wire x1="81.28" y1="13.97" x2="81.28" y2="17.425" width="0" layer="19" extent="16-16"/>
 <wire x1="74.93" y1="17.35" x2="81.28" y2="17.425" width="0" layer="19" extent="16-16"/>
@@
 <contactref element="X3" pad="1"/>
 <contactref element="C14" pad="PAD_0"/>
-<contactref element="C100" pad="+"/>
-<contactref element="C8" pad="+"/>
-<contactref element="C104" pad="+"/>
+<contactref element="C100" pad="PLUS"/>
+<contactref element="C8" pad="PLUS"/>
+<contactref element="C104" pad="PLUS"/>
 <wire x1="81.28" y1="31.75" x2="83.82" y2="31.75" width="0" layer="19" extent="1-1"/>
 <wire x1="73.62" y1="30.48" x2="81.28" y2="31.75" width="0" layer="19" extent="1-1"/>
@@
 <contactref element="IC1" pad="3"/>
 <contactref element="C1" pad="PAD_0"/>
-<contactref element="C2" pad="+"/>
+<contactref element="C2" pad="PLUS"/>
 <contactref element="X2" pad="1"/>
 <contactref element="R13" pad="PAD_0"/>
@@
 <wire x1="96.52" y1="22.86" x2="104.14" y2="31.75" width="0" layer="19" extent="1-1"/>
 <wire x1="99.06" y1="7.58" x2="96.52" y2="22.86" width="0" layer="19" extent="1-1"/>
-<wire x1="29.21" y1="34.29" x2="96.52" y2="22.86" width="0" layer="19" extent="1-1"/>
-<wire x1="21.59" y1="31.75" x2="29.21" y2="34.29" width="0" layer="19" extent="1-1"/>
-<wire x1="21.59" y1="29.565" x2="21.59" y2="31.75" width="0" layer="19" extent="16-16"/>
-<wire x1="16.51" y1="35.3" x2="21.59" y2="31.75" width="0" layer="19" extent="16-16"/>
+<wire x1="27.94" y1="32.18" x2="96.52" y2="22.86" width="0" layer="19" extent="1-1"/>
+<wire x1="21.59" y1="32.105" x2="27.94" y2="32.18" width="0" layer="19" extent="16-16"/>
+<wire x1="21.59" y1="35.56" x2="21.59" y2="32.105" width="0" layer="19" extent="16-16"/>
+<wire x1="16.51" y1="35.3" x2="21.59" y2="35.56" width="0" layer="19" extent="16-16"/>
 </signal>
 <signal name="N$7">
@@
 <contactref element="IC1" pad="2"/>
 <contactref element="R2" pad="PAD_1"/>
-<contactref element="C4" pad="+"/>
+<contactref element="C4" pad="PLUS"/>
 <contactref element="C3" pad="PAD_0"/>
 <contactref element="D3" pad="ANODE"/>
@@
 <wire x1="46.99" y1="8.67" x2="46.77" y2="11.43" width="0" layer="19" extent="16-16"/>
 <wire x1="49.53" y1="8.89" x2="46.99" y2="8.67" width="0" layer="19" extent="16-16"/>
-<wire x1="30.48" y1="21.81" x2="33.02" y2="15.24" width="0" layer="19" extent="1-16"/>
-<wire x1="27.94" y1="21.59" x2="30.48" y2="21.81" width="0" layer="19" extent="16-16"/>
-<wire x1="21.59" y1="21.59" x2="27.94" y2="21.59" width="0" layer="19" extent="1-1"/>
-<wire x1="13.97" y1="24.13" x2="21.59" y2="21.59" width="0" layer="19" extent="16-16"/>
+<wire x1="24.13" y1="22.59" x2="33.02" y2="15.24" width="0" layer="19" extent="1-1"/>
+<wire x1="21.59" y1="22.64" x2="24.13" y2="22.59" width="0" layer="19" extent="16-16"/>
+<wire x1="21.59" y1="25.4" x2="21.59" y2="22.64" width="0" layer="19" extent="16-16"/>
+<wire x1="13.97" y1="24.13" x2="21.59" y2="25.4" width="0" layer="19" extent="16-16"/>
 <wire x1="6.35" y1="21.81" x2="13.97" y2="24.13" width="0" layer="19" extent="16-16"/>
 </signal>

Commit message: Start routing
Parts:
- added X1: (no value), con-wago-500:W237-102
- D5: device __MyCommonLib1:DO-41_10MM -> __MyCommonLib1:DO-41_5MM
- R12: device __MyCommonLib1:R_2.0W -> __MyCommonLib1:R_1.0W_VERTICAL
- R14: device __MyCommonLib1:R_1.0W -> __MyCommonLib1:R_1.0W_VERTICAL
- X3: value L_TEST -> (none)
- moved D5 19.0 mm to (82.8, 4.62)
- moved C100 12.5 mm to (83.4, 25.2)
- moved R14 10.8 mm to (73.0, 16.0), turned to 0 degrees
- moved C8 10.5 mm to (83.6, 15.1)
- moved C13 10.1 mm to (74.0, 26.1), turned to 0 degrees
- moved X2 9.81 mm to (90.5, 5.08)
- moved R13 9.48 mm to (91.5, 22.6), turned to 90 degrees
- moved C14 8.15 mm to (83.4, 20.1)
- moved R12 6.59 mm to (68.8, 12.7)
- moved C1 5.55 mm to (25.1, 34.8)
- moved T2 5.22 mm to (41.5, 24.6)
- moved C7 4.97 mm to (38.1, 19.5)
- moved R8 4.97 mm to (41.9, 19.5)
- moved R3 4.97 mm to (48.3, 15.7)
- moved R5 4.97 mm to (43.2, 15.7)
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Connections:
- net N$10: now also X3.1
- net N$9: now also X1.1, X1.2; no longer X3.1
Routing:
- net +VCC: track 10.2 -> 13.2 mm
Other:
- board outline added: 96 x 40 mm

Commit message: L saturation metter routed
Parts:
- X1: value (none) -> L_TEST_START
- X3: value (none) -> L_TEST_END
- moved R1 11.5 mm to (2.98, 35.6)
- moved R2 11.5 mm to (5.99, 35.6)
- moved C4 4.26 mm to (27.0, 26.1)
- moved C3 3.98 mm to (23.9, 25.8)
- moved T3 2.30 mm to (38.7, 24.5)
- moved T2 2.30 mm to (43.8, 24.5)
- moved D4 1.00 mm to (38.1, 9.89)
- moved D5 0.58 mm to (82.5, 5.12)
- moved C6 0.41 mm to (41.5, 5.91)
- moved R6 0.41 mm to (41.5, 11.0)
- moved D1 0.40 mm to (55.5, 6.08)
- moved D2 0.30 mm to (51.1, 18.5)
- moved C104 0.30 mm to (74.0, 22.6)
- moved R14 0.22 mm to (73.0, 15.8)
Routing:
- net GND: track 0.00 -> 33.3 mm
- net N$15: track 0.00 -> 28.8 mm
- net N$2: track 0.00 -> 20.1 mm
- net N$1: track 0.00 -> 14.6 mm
- net N$14: track 0.00 -> 14.5 mm
- net N$7: track 0.00 -> 10.6 mm
- net N$16: track 0.00 -> 9.80 mm
- net +VCC: track 13.2 -> 21.4 mm, vias 1 -> 2
- net N$8: track 0.00 -> 8.04 mm
- net N$17: track 0.00 -> 7.68 mm
- net N$10: track 0.00 -> 5.47 mm
- net N$13: track 0.00 -> 2.54 mm
- net N$18: track 0.00 -> 2.43 mm
- net N$6: track 0.00 -> 2.26 mm
- added copper zone on layer 16, net +VCC
- added copper zone on layer 16, net GND
- added copper zone on layer 16, net N$10
- added copper zone on layer 16, net N$11
- added copper zone on layer 16, net N$3
- added copper zone on layer 16, net N$6
- added copper zone on layer 16, net N$9

Commit message: L saturation meter. Ver2 schematic complete
Parts:
- added C11: 1n0, __MyCommonLib1:RSMD_0805
- added C12: 10nF, __MyCommonLib1:RSMD_0805
- added C15, C9: 0.1uF, __MyCommonLib1:RSMD_0805
- added D10, D11, D12, D6, D7, D8, D9: LL4148, __MyCommonLib1:SOD-80
- added D101: BAT54C, __MyCommonLib1:SOT23_SMALL_PADS
- added D13: FR207, __MyCommonLib1:DO-41_10MM
- added R10: 1K0, __MyCommonLib1:RSMD_0805
- added R15, R16, R17, R18: 10K, __MyCommonLib1:RSMD_0805
- added R19: 510R, __MyCommonLib1:RSMD_0805
- added R20: 100K, __MyCommonLib1:SP3-4AM
- added R21, R22: 330R, __MyCommonLib1:RSMD_0805
- added R23: 1K, __MyCommonLib1:RSMD_0805
- added R24: 330R, __MyCommonLib1:RSMD_1206_BIG_GAP
- added R25, R26: 510R, __MyCommonLib1:RSMD_1206_BIG_GAP
- added R27: 20R, __MyCommonLib1:RSMD_1206_BIG_GAP
- added R28, R29: 20R, __MyCommonLib1:RSMD_0805
- added R30: 10R, __MyCommonLib1:R_0.5W
- added R31: 0.01R, __MyCommonLib1:RSMD_2512
- added R9: 10K, __MyCommonLib1:SP3-4AM
- added SW1: DUR_10X, __MyCommonLib1:SWITCH_DOUBLE_2.54X4.0MM
- added T4, T5: BC847, __MyCommonLib1:SOT23_SMALL_PADS
- added T6, T7: IRF830, __MyCommonLib1:TO-220(HORIZONTAL)
- added X5: Synchro, con-wago-500:W237-102
- added X6: L_TEST_END, con-wago-500:W237-102
- C10: value 1n0 -> 0.1uFx25V
- C7: value 1n0 -> 47uFx16V; device __MyCommonLib1:RSMD_0805 -> __MyCommonLib1:CE_5.2MM
- R13: value 10R -> 1R0
- R6: value 100K -> 1K0
- R8: value 10K -> 2K
- T3: value BC857 -> BC847
- X1: value L_TEST_START -> I_SENSE_100x
- X4: value I_SENSE -> I_SENSE_10x
- moved X1 238.7 mm to (-109.4, -111.1), turned to 0 degrees
- moved C10 173.2 mm to (-63.5, -109.6), flipped to the top
- moved C7 160.1 mm to (-62.5, -105.1), flipped to the top, turned to 0 degrees
- moved T3 130.2 mm to (-54.5, -66.4), turned to 0 degrees
- moved R6 83.0 mm to (-26.7, -36.3), turned to 0 degrees
- moved D4 77.2 mm to (-25.9, -33.2), turned to 0 degrees
- moved D3 55.1 mm to (22.1, 86.8)
- moved C2 51.7 mm to (43.9, 84.2)
- moved C3 49.2 mm to (17.6, 74.6)
- moved C1 47.3 mm to (18.2, 81.5)
- moved C4 41.3 mm to (24.9, 67.3)
- moved R1 29.2 mm to (25.5, 54.2)
- moved IC1 29.2 mm to (36.2, 43.7)
- moved R2 28.9 mm to (28.1, 54.2)
- moved C104 0.13 mm to (74.2, 22.6), turned to 180 degrees
Connections:
- removed net N$9: C100.PLUS, C104.PLUS, C13.PAD_0, C14.PAD_0, C8.PLUS, R13.PAD1, R14.PAD1, X1.1, X1.2
- new net +12V_FILTERED: C100.PLUS, C104.MINUS, C13.PAD_0, C14.PAD_0, C8.PLUS, R13.PAD1, R14.PAD1, R30.PAD1, X3.2, X6.2
- new net N$12: IC4.5, R15.PAD_1, R16.PAD_0, R17.PAD_1
- new net N$19: R18.PAD_0, T4.1
- new net N$20: R19.PAD_0, T4.2, X5.1
- new net N$21: D6.CATHODE, R21.PAD_0, R22.PAD_1
- new net N$22: C12.PAD_0, SW1.POS_A1, SW1.POS_A2
- new net N$23: IC4.1, R20.END_A, R20.MIDDLE, R23.PAD_1, R5.PAD_0
- new net N$24: R23.PAD_0, T5.1
- new net N$25: R24.PAD_0, R8.PAD_0, T5.2
- new net N$26: D101.2, R8.PAD_1, T3.1
- new net N$27: D101.3, D7.CATHODE, D8.CATHODE, T3.3
- new net N$28: D11.CATHODE, D9.ANODE, R28.PAD_1, T7.1
- new net N$29: R27.PAD_1, T2.3
- new net N$30: D8.ANODE, R11.PAD_0, R28.PAD_0, R29.PAD_0, T2.2
- new net N$31: D10.ANODE, D12.CATHODE, R29.PAD_1, T1.1
- new net N$32: R31.PAD1, T6.3, T7.3, X1.1
- new net N$33: C10.PAD_0, C7.PLUS, D10.CATHODE, D2.CATHODE, D9.CATHODE, R26.PAD_0, R27.PAD_0, R30.PAD_0
- new net N$34: D13.ANODE, T6.2, T7.2, X6.1
- new net N$4: C9.PAD_0, IC4.6, R10.PAD_0
- new net N$5: R10.PAD_1, R9.END_A
- net +VCC: now also C15.PAD_0, R16.PAD_1, R21.PAD_1, R6.PAD_0, T4.3, T5.3; no longer D2.CATHODE, T2.3
- net GND: now also C10.PAD_1, C12.PAD_1, C15.PAD_1, C7.MINUS, C9.PAD_1, D11.ANODE, D12.ANODE, R15.PAD_0, R19.PAD_1, R20.PACKAGE1, R20.PACKAGE2, R22.PAD_0, R24.PAD_1, R31.PAD0, R9.PACKAGE1, R9.PACKAGE2, T3.2, X1.2, X5.2; no longer IC4.5, T3.3
- net N$1: now also D7.ANODE, R25.PAD_1, T2.1; no longer C10.PAD_1, R11.PAD_0, T2.2, T3.2
- net N$10: no longer X3.2
- net N$13: now also C11.PAD_1, R17.PAD_0, R18.PAD_1, R9.END_B, R9.MIDDLE; no longer IC4.6
- net N$14: now also D4.ANODE
- net N$15: now also R20.END_B; no longer C7.PAD_1, IC4.1, R5.PAD_0, R6.PAD_0, R8.PAD_0
- net N$16: now also R25.PAD_0, R26.PAD_1; no longer C7.PAD_0, R8.PAD_1, T2.1, T3.1
- net N$18: now also C11.PAD_0, D4.CATHODE, R6.PAD_1; no longer D4.ANODE, R7.PAD_1
- net N$2: now also T6.1; no longer C10.PAD_0, T1.1
- net N$6: now also C104.PLUS, D13.CATHODE; no longer C104.MINUS
- net N$7: now also D6.ANODE, R7.PAD_1, SW1.CENTER1, SW1.CENTER2; no longer D4.CATHODE, R6.PAD_1
Routing:
- net GND: track 33.3 -> 0.00 mm
- net N$15: track 28.8 -> 0.00 mm
- net N$2: track 20.1 -> 0.00 mm
- net N$1: track 14.6 -> 0.00 mm
- net N$14: track 14.5 -> 0.00 mm
- net N$7: track 10.6 -> 0.00 mm
- net N$16: track 9.80 -> 0.00 mm
- net N$8: track 8.04 -> 0.00 mm
- net N$17: track 7.68 -> 0.00 mm
- net N$10: track 5.47 -> 0.00 mm
- net +VCC: track 21.4 -> 18.8 mm
- net N$13: track 2.54 -> 0.00 mm
- net N$18: track 2.43 -> 0.00 mm
- net N$6: track 2.26 -> 0.00 mm
- removed copper zone on layer 16, net +VCC
- removed copper zone on layer 16, net GND
- removed copper zone on layer 16, net N$10
- removed copper zone on layer 16, net N$11
- removed copper zone on layer 16, net N$3
- removed copper zone on layer 16, net N$6
- removed copper zone on layer 16, net N$9
Other:
- board size 96 x 40 mm -> 96 x 58.9 mm

Commit message: L saturation meter. Parts locating
Parts:
- added C16, C17: 1000uFx25V, __MyCommonLib1:CE_10MM
- T1, T6, T7: device __MyCommonLib1:TO-220(HORIZONTAL) -> __MyCommonLib1:TO-220(HORIZONTAL_WITH_SCREW_PAD)
- moved D13 262.6 mm to (91.2, 46.5)
- moved X6 231.1 mm to (92.1, 52.0), turned to 180 degrees
- moved R31 230.5 mm to (91.1, 11.1)
- moved X1 221.0 mm to (78.0, 6.10)
- moved T6 211.3 mm to (84.0, 15.9)
- moved T7 211.0 mm to (72.4, 16.0)
- moved R30 191.3 mm to (62.0, 32.4), turned to 90 degrees
- moved T1 60.4 mm to (119.0, 15.6)
- moved D5 57.7 mm to (117.5, 51.0)
- moved X2 56.6 mm to (123.5, 51.1), turned to 90 degrees
- moved R12 55.7 mm to (124.4, 9.20), turned to 270 degrees
- moved X4 46.7 mm to (115.5, 7.38)
- moved D100 44.0 mm to (103.7, 46.6), turned to 180 degrees
- moved X3 36.7 mm to (102.0, 52.0)
- moved R14 35.8 mm to (102.5, 36.0)
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Connections:
- net +12V_FILTERED: now also C16.PLUS, C17.PLUS, X6.1; no longer R30.PAD1, X6.2
- net GND: now also C16.MINUS, C17.MINUS, R12.PAD1, X1.1, X2.1, X4.1; no longer R12.PAD_0, X1.2, X2.2, X4.2
- net N$10: now also T1.SCREW_PAD
- net N$11: now also R30.PAD1, X2.2; no longer X2.1
- net N$3: now also R12.PAD_0, X4.2; no longer R12.PAD1, X4.1
- net N$32: now also X1.2; no longer X1.1
- net N$34: now also T6.SCREW_PAD, T7.SCREW_PAD, X6.2; no longer X6.1
Routing:
- net N$32: track 0.00 -> 21.0 mm
- net +VCC: track 18.8 -> 0.00 mm, vias 2 -> 0
- net N$2: track 0.00 -> 12.8 mm
Other:
- board size 96 x 58.9 mm -> 130 x 60 mm

Commit message: L saturation meter. Routing step 1
Parts:
- removed C17: 1000uFx25V, __MyCommonLib1:CE_10MM
- removed D1, D10, D11, D12, D9: LL4148, __MyCommonLib1:SOD-80
- added D14: LL4148, __MyCommonLib1:SOD-80
- D100: device __MyCommonLib1:DO-41_10MM -> __MyCommonLib1:DO-41_20MM
- D13: device __MyCommonLib1:DO-41_10MM -> __MyCommonLib1:DO-41_5MM
- D3: device __MyCommonLib1:DO-41_10MM -> __MyCommonLib1:DO-41_15MM
- D5: device __MyCommonLib1:DO-41_5MM -> __MyCommonLib1:DO-41_15MM
- R19, R23: device __MyCommonLib1:RSMD_0805 -> __MyCommonLib1:RSMD_1206_BIG_GAP
- T1, T6, T7: device __MyCommonLib1:TO-220(HORIZONTAL_WITH_SCREW_PAD) -> __MyCommonLib1:D2PAK
- moved R29 212.9 mm to (121.7, 23.8), turned to 270 degrees
- moved C10 198.7 mm to (67.2, 40.0), turned to 180 degrees
- moved C7 196.6 mm to (67.3, 42.6), turned to 180 degrees
- moved R28 181.3 mm to (84.5, 24.0), turned to 270 degrees
- moved R26 168.3 mm to (60.3, 38.4), turned to 270 degrees
- moved R27 168.0 mm to (56.4, 38.4), turned to 270 degrees
- moved R25 166.5 mm to (63.9, 35.5), turned to 270 degrees
- moved D7 156.3 mm to (63.7, 27.8), turned to 90 degrees
- moved D8 154.5 mm to (60.2, 25.9), turned to 90 degrees
- moved D101 150.2 mm to (65.4, 19.4), turned to 180 degrees
- moved T3 143.2 mm to (60.2, 19.4), turned to 180 degrees
- moved R24 135.6 mm to (64.0, 7.50), turned to 270 degrees
- moved D6 134.1 mm to (46.9, 40.6), turned to 180 degrees
- moved R23 133.3 mm to (54.2, 26.0)
- moved T5 130.3 mm to (57.1, 13.3), turned to 90 degrees
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Connections:
- removed net N$17: R102.END_B, R7.PAD_0
- new net N$35: R20.END_A, R7.PAD_0
- net +12V_FILTERED: no longer C17.PLUS
- net GND: now also D14.ANODE, X1.2, X4.2; no longer C17.MINUS, D1.ANODE, D11.ANODE, D12.ANODE, X1.1, X4.1
- net N$10: no longer T1.SCREW_PAD
- net N$15: now also R20.MIDDLE; no longer R102.MIDDLE
- net N$2: no longer D1.CATHODE, D2.ANODE
- net N$23: now also R102.END_B, R102.MIDDLE; no longer R20.END_A, R20.MIDDLE
- net N$28: no longer D11.CATHODE, D9.ANODE
- net N$3: now also X4.1; no longer X4.2
- net N$30: now also D14.CATHODE, D2.ANODE
- net N$31: no longer D10.ANODE, D12.CATHODE
- net N$32: now also X1.1; no longer X1.2
- net N$33: no longer D10.CATHODE, D9.CATHODE
- net N$34: no longer T6.SCREW_PAD, T7.SCREW_PAD
Routing:
- net GND: track 0.00 -> 96.7 mm, vias 0 -> 2
- net +VCC: track 0.00 -> 86.8 mm
- net N$30: track 0.00 -> 77.8 mm, vias 0 -> 4
- net N$23: track 0.00 -> 36.1 mm, vias 0 -> 2
- net N$13: track 0.00 -> 35.0 mm
- net N$35: track 0.00 -> 32.1 mm, vias 0 -> 2
- net N$8: track 0.00 -> 27.6 mm
- net N$7: track 0.00 -> 23.3 mm
- net N$33: track 0.00 -> 22.5 mm
- net N$14: track 0.00 -> 17.2 mm
- net N$20: track 0.00 -> 15.0 mm
- net N$15: track 0.00 -> 14.0 mm
- net N$27: track 0.00 -> 13.5 mm
- net N$24: track 0.00 -> 13.3 mm
- net N$4: track 0.00 -> 12.5 mm
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- added copper zone on layer 16, net +12V_FILTERED
- added copper zone on layer 16, net GND
- added copper zone on layer 16, net N$10
- added copper zone on layer 16, net N$11
- added copper zone on layer 16, net N$3
- added copper zone on layer 16, net N$32
- added copper zone on layer 16, net N$34
- added copper zone on layer 16, net N$6

Commit message: L saturation meter. Routing step 2
Routing:
- net GND: track 96.7 -> 49.1 mm
- net +VCC: track 86.8 -> 67.1 mm
- net N$13: track 35.0 -> 35.6 mm
- added copper zone on layer 16, net +VCC
