File: L_Saturation_Meter/schematic/L_SaturationMeter.sch (EAGLE design)
At the start: 77 parts, among them IC1 LM317, IC4 LM358, SW1 DUR_10X, T1 IRF830, T2 BC847, T3 BC847, T4 BC847, T5 BC847, T6 IRF830, T7 IRF830, X1 I_SENSE_100x, X2 POWER_12V, X3 L_TEST_END, X4 I_SENSE_10x, X5 Synchro, X6 L_TEST_END

Commit message: L saturation meter. Final changes
Parts:
- R1: value 5K6 -> 4K7
- R13: value 1R0 -> 1R5
- R25, R26: value 510R -> 240R
- R27: value 20R -> 10R
- R6: value 1K0 -> 4K7
Changed lines of the file:
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@@
 <part name="GND1" library="supply1" deviceset="GND" device=""/>
 <part name="D2" library="__MyCommonLib1" deviceset="LL4147" device="SOD-80" value="LL4148"/>
-<part name="R13" library="__MyCommonLib1" deviceset="R" device="2.0W" value="1R0"/>
+<part name="R13" library="__MyCommonLib1" deviceset="R" device="2.0W" value="1R5"/>
 <part name="X2" library="con-wago-500" deviceset="W237-102" device="" value="POWER_12V"/>
 <part name="X3" library="con-wago-500" deviceset="W237-102" device="" value="L_TEST_END"/>
@@
 <part name="C2" library="__MyCommonLib1" deviceset="CE" device="8.2MM" value="470uFx16V"/>
 <part name="D3" library="__MyCommonLib1" deviceset="1N4001" device="DO-41_15MM" value="1N4001"/>
-<part name="R1" library="__MyCommonLib1" deviceset="R" device="SMD_0805" value="5K6"/>
+<part name="R1" library="__MyCommonLib1" deviceset="R" device="SMD_0805" value="4K7"/>
 <part name="R2" library="__MyCommonLib1" deviceset="R" device="SMD_0805" value="1K0"/>
 <part name="GND9" library="supply1" deviceset="GND" device=""/>
@@
 <part name="C11" library="__MyCommonLib1" deviceset="C" device="SMD_0805" value="1n0"/>
 <part name="D4" library="__MyCommonLib1" deviceset="LL4147" device="SOD-80" value="LL4148"/>
-<part name="R6" library="__MyCommonLib1" deviceset="R" device="SMD_0805" value="1K0"/>
+<part name="R6" library="__MyCommonLib1" deviceset="R" device="SMD_0805" value="4K7"/>
 <part name="SW1" library="__MyCommonLib1" deviceset="SWITCH_DOUBLE" device="(2.54X4MM)" value="DUR_10X"/>
 <part name="C12" library="__MyCommonLib1" deviceset="C" device="SMD_0805" value="10nF"/>
@@
 <part name="D7" library="__MyCommonLib1" deviceset="LL4147" device="SOD-80" value="LL4148"/>
 <part name="D8" library="__MyCommonLib1" deviceset="LL4147" device="SOD-80" value="LL4148"/>
-<part name="R25" library="__MyCommonLib1" deviceset="R" device="SMD_1206_BIG_GAP" value="510R"/>
-<part name="R26" library="__MyCommonLib1" deviceset="R" device="SMD_1206_BIG_GAP" value="510R"/>
-<part name="R27" library="__MyCommonLib1" deviceset="R" device="SMD_1206_BIG_GAP" value="20R"/>
+<part name="R25" library="__MyCommonLib1" deviceset="R" device="SMD_1206_BIG_GAP" value="240R"/>
+<part name="R26" library="__MyCommonLib1" deviceset="R" device="SMD_1206_BIG_GAP" value="240R"/>
+<part name="R27" library="__MyCommonLib1" deviceset="R" device="SMD_1206_BIG_GAP" value="10R"/>
 <part name="R28" library="__MyCommonLib1" deviceset="R" device="SMD_0805" value="20R"/>
 <part name="R29" library="__MyCommonLib1" deviceset="R" device="SMD_0805" value="20R"/>
