File: LC_METER/TestPowerInverter/LCMeter_test_power_inverter.sch (EAGLE design)
At the start: 34 parts, among them IC10 MC34063, T1 H772, X1 VCC_IN, X2 GND, X3 +5V_STAB, X4 +7V, X5 -7V, X6 GND

Commit message: LC meter test power supply inverter. parts Located
Parts:
- D1, D3: device __MyCommonLib1:1N4001DO-41_5MM -> __MyCommonLib1:1N4001DO-41_12.5MM
- R2: device __MyCommonLib1:RSMD_1206_BIG_GAP -> __MyCommonLib1:RSMD_0805
- R84: device __MyCommonLib1:RSMD_0805 -> __MyCommonLib1:R0204
Connections:
- removed net N$9: C3.PIN1, R6.PIN0
- new net N$1: C3.PIN0, R6.PIN1
- net +7V: now also R6.PIN0; no longer C3.PIN0
- net N$8: now also C3.PIN1; no longer R6.PIN1
Other:
- moved on the sheet: C3, R6
Changed lines of the file:
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@@
 <part name="GND71" library="supply1" deviceset="GND" device=""/>
 <part name="GND72" library="supply1" deviceset="GND" device=""/>
-<part name="R84" library="__MyCommonLib1" deviceset="R" device="SMD_0805" value="4K7"/>
+<part name="R84" library="__MyCommonLib1" deviceset="R" device="0204" value="4K7"/>
 <part name="R85" library="__MyCommonLib1" deviceset="R" device="SMD_0805" value="1K6"/>
 <part name="GND75" library="supply1" deviceset="GND" device=""/>
@@
 <part name="T1" library="__MyCommonLib1" deviceset="H772_PNP" device="DPAK" value="H772"/>
 <part name="R1" library="__MyCommonLib1" deviceset="R" device="SMD_1206_BIG_GAP" value="51R"/>
-<part name="R2" library="__MyCommonLib1" deviceset="R" device="SMD_1206_BIG_GAP" value="100R"/>
+<part name="R2" library="__MyCommonLib1" deviceset="R" device="SMD_0805" value="100R"/>
 <part name="L1" library="__MyCommonLib1" deviceset="TRANS_2.5_WIND" device="16X8" value="2.5wind"/>
 <part name="GND2" library="supply1" deviceset="GND" device=""/>
 <part name="R3" library="__MyCommonLib1" deviceset="R" device="SMD_1206_BIG_GAP" value="*"/>
 <part name="GND3" library="supply1" deviceset="GND" device=""/>
-<part name="D1" library="__MyCommonLib1" deviceset="1N4001" device="DO-41_5MM" value="SB2100"/>
+<part name="D1" library="__MyCommonLib1" deviceset="1N4001" device="DO-41_12.5MM" value="SB2100"/>
 <part name="D2" library="__MyCommonLib1" deviceset="1N4001" device="DO-41_5MM" value="SB2100"/>
-<part name="D3" library="__MyCommonLib1" deviceset="1N4001" device="DO-41_5MM" value="SB2100"/>
+<part name="D3" library="__MyCommonLib1" deviceset="1N4001" device="DO-41_12.5MM" value="SB2100"/>
 <part name="R4" library="__MyCommonLib1" deviceset="R" device="SMD_1206_BIG_GAP" value="10R"/>
 <part name="C1" library="__MyCommonLib1" deviceset="C" device="SMD_0805" value="1n0"/>
@@
 <attribute name="VALUE" x="176.53" y="123.19" size="1.27" layer="96" font="vector" ratio="20"/>
 </instance>
-<instance part="C3" gate="C$1" x="175.26" y="137.16" smashed="yes" rot="R90">
-<attribute name="NAME" x="173.99" y="139.7" size="1.27" layer="95" font="vector" ratio="20"/>
-<attribute name="VALUE" x="177.8" y="139.7" size="1.27" layer="96" font="vector" ratio="20"/>
-</instance>
-<instance part="R6" gate="R$1" x="165.1" y="137.16" smashed="yes" rot="R90">
-<attribute name="NAME" x="163.83" y="138.43" size="1.27" layer="95" font="vector" ratio="20"/>
-<attribute name="VALUE" x="167.64" y="138.43" size="1.27" layer="96" font="vector" ratio="20"/>
+<instance part="C3" gate="C$1" x="162.56" y="137.16" smashed="yes" rot="R90">
+<attribute name="NAME" x="161.29" y="139.7" size="1.27" layer="95" font="vector" ratio="20"/>
+<attribute name="VALUE" x="165.1" y="139.7" size="1.27" layer="96" font="vector" ratio="20"/>
+</instance>
+<instance part="R6" gate="R$1" x="172.72" y="137.16" smashed="yes" rot="R90">
+<attribute name="NAME" x="171.45" y="138.43" size="1.27" layer="95" font="vector" ratio="20"/>
+<attribute name="VALUE" x="175.26" y="138.43" size="1.27" layer="96" font="vector" ratio="20"/>
 </instance>
 <instance part="C4" gate="C$1" x="182.88" y="124.46" smashed="yes">
@@
 <pinref part="D2" gate="D$1" pin="ANODE"/>
 <wire x1="152.4" y1="134.62" x2="157.48" y2="134.62" width="0.1524" layer="91"/>
-<pinref part="R6" gate="R$1" pin="PIN1"/>
 <wire x1="157.48" y1="134.62" x2="167.64" y2="134.62" width="0.1524" layer="91"/>
-<wire x1="160.02" y1="137.16" x2="157.48" y2="137.16" width="0.1524" layer="91"/>
 <wire x1="157.48" y1="137.16" x2="157.48" y2="134.62" width="0.1524" layer="91"/>
 <junction x="157.48" y="134.62"/>
-</segment>
-</net>
-<net name="N$9" class="0">
-<segment>
-<pinref part="R6" gate="R$1" pin="PIN0"/>
 <pinref part="C3" gate="C$1" pin="PIN1"/>
-<wire x1="172.72" y1="137.16" x2="170.18" y2="137.16" width="0.1524" layer="91"/>
+<wire x1="157.48" y1="137.16" x2="160.02" y2="137.16" width="0.1524" layer="91"/>
 </segment>
 </net>
@@
 <pinref part="D2" gate="D$1" pin="CATHODE"/>
 <wire x1="172.72" y1="134.62" x2="180.34" y2="134.62" width="0.1524" layer="91"/>
-<pinref part="C3" gate="C$1" pin="PIN0"/>
-<wire x1="177.8" y1="137.16" x2="180.34" y2="137.16" width="0.1524" layer="91"/>
 <wire x1="180.34" y1="137.16" x2="180.34" y2="134.62" width="0.1524" layer="91"/>
 <junction x="180.34" y="134.62"/>
@@
 <label x="215.9" y="135.89" size="1.27" layer="95" font="vector" ratio="20" rot="R180"/>
 <pinref part="X4" gate="X$1" pin="1"/>
+<pinref part="R6" gate="R$1" pin="PIN0"/>
+<wire x1="180.34" y1="137.16" x2="177.8" y2="137.16" width="0.1524" layer="91"/>
 </segment>
 </net>
@@
 </segment>
 </net>
+<net name="N$1" class="0">
+<segment>
+<pinref part="R6" gate="R$1" pin="PIN1"/>
+<pinref part="C3" gate="C$1" pin="PIN0"/>
+<wire x1="165.1" y1="137.16" x2="167.64" y2="137.16" width="0.1524" layer="91"/>
+</segment>
+</net>

Commit message: LC meter test power supply inverter. almost routed
Parts:
- added C10: 0.1uF, __MyCommonLib1:CSMD_0805
- R84: device __MyCommonLib1:R0204 -> __MyCommonLib1:R0207
Connections:
- net +5V_STAB: now also C10.PIN1
- net GND: now also C10.PIN0
Changed lines of the file:
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@@
 <part name="GND71" library="supply1" deviceset="GND" device=""/>
 <part name="GND72" library="supply1" deviceset="GND" device=""/>
-<part name="R84" library="__MyCommonLib1" deviceset="R" device="0204" value="4K7"/>
+<part name="R84" library="__MyCommonLib1" deviceset="R" device="0207" value="4K7"/>
 <part name="R85" library="__MyCommonLib1" deviceset="R" device="SMD_0805" value="1K6"/>
 <part name="GND75" library="supply1" deviceset="GND" device=""/>
@@
 <part name="R7" library="__MyCommonLib1" deviceset="R" device="SMD_0805" value="***"/>
 <part name="GND13" library="supply1" deviceset="GND" device=""/>
+<part name="C10" library="__MyCommonLib1" deviceset="C" device="SMD_0805" value="0.1uF"/>
+<part name="GND14" library="supply1" deviceset="GND" device=""/>
 </parts>
 <sheets>
@@
 <attribute name="VALUE" x="93.98" y="67.31" size="1.27" layer="96" font="vector" ratio="20"/>
 </instance>
+<instance part="C10" gate="C$1" x="116.84" y="81.28" smashed="yes" rot="MR0">
+<attribute name="NAME" x="118.11" y="83.82" size="1.27" layer="95" font="vector" ratio="20" rot="MR180"/>
+<attribute name="VALUE" x="119.38" y="80.01" size="1.27" layer="96" font="vector" ratio="20" rot="MR180"/>
+</instance>
+<instance part="GND14" gate="1" x="116.84" y="71.12" smashed="yes">
+<attribute name="VALUE" x="114.3" y="67.31" size="1.27" layer="96" font="vector" ratio="20"/>
+</instance>
 </instances>
 <busses>
@@
 <pinref part="GND13" gate="1" pin="GND"/>
 <wire x1="96.52" y1="76.2" x2="96.52" y2="73.66" width="0.1524" layer="91"/>
+</segment>
+<segment>
+<pinref part="C10" gate="C$1" pin="PIN0"/>
+<pinref part="GND14" gate="1" pin="GND"/>
+<wire x1="116.84" y1="78.74" x2="116.84" y2="73.66" width="0.1524" layer="91"/>
 </segment>
 </net>
@@
 <segment>
 <pinref part="R84" gate="R$1" pin="PIN1"/>
-<wire x1="114.3" y1="88.9" x2="124.46" y2="88.9" width="0.1524" layer="91"/>
+<wire x1="114.3" y1="88.9" x2="116.84" y2="88.9" width="0.1524" layer="91"/>
+<wire x1="116.84" y1="88.9" x2="124.46" y2="88.9" width="0.1524" layer="91"/>
 <wire x1="124.46" y1="88.9" x2="124.46" y2="81.28" width="0.1524" layer="91"/>
 <pinref part="D1" gate="D$1" pin="CATHODE"/>
@@
 <label x="215.9" y="130.81" size="1.27" layer="95" font="vector" ratio="20" rot="R180"/>
 <pinref part="X3" gate="X$1" pin="1"/>
-</segment>
-</net>
+<pinref part="C10" gate="C$1" pin="PIN1"/>
+<wire x1="116.84" y1="83.82" x2="116.84" y2="88.9" width="0.1524" layer="91"/>
+<junction x="116.84" y="88.9"/>
+</segment>
+</net>
