File: LC_METER/TestPowerInverter/LCMeter_test_power_inverter.brd (EAGLE design)
At the start: 70 x 125 mm, 34 parts, among them IC10 MC34063, T1 H772, X1 VCC_IN, X2 GND, X3 +5V_STAB, X4 +7V, X5 -7V, X6 GND

Commit message: LC meter test power supply inverter. parts Located
Parts:
- D1, D3: device __MyCommonLib1:DO-41_5MM -> __MyCommonLib1:DO-41_12.5MM
- R2: device __MyCommonLib1:RSMD_1206_BIG_GAP -> __MyCommonLib1:RSMD_0805
- R84: device __MyCommonLib1:RSMD_0805 -> __MyCommonLib1:R0204
- moved X6 151.8 mm to (55.0, 19.0)
- moved X5 147.5 mm to (49.0, 24.0)
- moved X4 131.9 mm to (49.1, 7.10)
- moved X3 130.7 mm to (54.1, 4.40)
- moved C9 127.3 mm to (38.0, 22.6), turned to 90 degrees
- moved R7 123.0 mm to (12.5, 5.60), turned to 90 degrees
- moved C8 121.2 mm to (41.3, 21.7), turned to 270 degrees
- moved C6 109.9 mm to (47.6, 12.2), turned to 270 degrees
- moved C7 109.3 mm to (44.2, 12.0), turned to 270 degrees
- moved C5 107.1 mm to (54.5, 11.9), turned to 270 degrees
- moved C4 102.8 mm to (51.1, 12.2), turned to 270 degrees
- moved C3 93.3 mm to (40.0, 15.2)
- moved R6 91.7 mm to (39.9, 10.8), turned to 90 degrees
- moved C1 87.0 mm to (31.8, 24.3)
- moved C2 85.6 mm to (43.8, 4.10)
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Connections:
- removed net N$9: C3.PAD_1, R6.PAD_0
- new net N$1: C3.PAD_0, R6.PAD_1
- net +5V_STAB: now also R84.PAD1; no longer R84.PAD_1
- net +7V: now also R6.PAD_0; no longer C3.PAD_0
- net N$8: now also C3.PAD_1; no longer R6.PAD_1
Other:
- board size 70 x 125 mm -> 60 x 28 mm

Commit message: LC meter test power supply inverter. almost routed
Parts:
- added C10: 0.1uF, __MyCommonLib1:RSMD_0805
- R84: device __MyCommonLib1:R0204 -> __MyCommonLib1:R0207
- moved C54 5.74 mm to (2.90, 10.2)
- moved R84 2.24 mm to (16.0, 5.00), turned to 180 degrees
- moved C53 1.63 mm to (6.50, 10.0)
- moved R7 1.17 mm to (13.5, 5.00)
- moved R85 1.08 mm to (16.1, 5.00)
- moved R2 1.00 mm to (21.8, 19.4), turned to 90 degrees
- moved X3 0.76 mm to (53.4, 4.70)
- moved C55 0.63 mm to (21.8, 8.90)
- moved X5 0.30 mm to (49.0, 24.3)
Connections:
- net +5V_STAB: now also C10.PAD_1
- net GND: now also C10.PAD_0
Routing:
- net +5V_STAB: track 0.00 -> 50.9 mm
- net N$3: track 0.00 -> 21.9 mm
- net VCC_IN: track 0.00 -> 19.1 mm
- net N$139: track 0.00 -> 8.36 mm
- net N$133: track 0.00 -> 8.31 mm
- net N$8: track 0.00 -> 6.59 mm
- net N$2: track 0.00 -> 6.54 mm
- net N$7: track 0.00 -> 6.26 mm
- net N$1: track 0.00 -> 3.64 mm
- net N$135: track 0.00 -> 2.82 mm
- net N$5: track 0.00 -> 2.62 mm
- net N$10: track 0.00 -> 2.62 mm
- net N$4: track 0.00 -> 2.52 mm
- net -7V: track 0.00 -> 2.20 mm
- added copper zone on layer 16, net +5V_STAB
- added copper zone on layer 16, net +7V
- added copper zone on layer 16, net -7V
- added copper zone on layer 16, net N$3
- added copper zone on layer 16, net N$4
- added copper zone on layer 16, net VCC_IN

Commit message: LC meter test power supply iverter. Finished
Parts:
- moved X6 1.00 mm to (55.0, 20.0)
Routing:
- net GND: track 0.00 -> 1.76 mm
- added copper zone on layer 16, net GND
Changed lines of the file:
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@@
 <param name="mtCopper" value="0.035mm 0.035mm 0.035mm 0.035mm 0.035mm 0.035mm 0.035mm 0.035mm 0.035mm 0.035mm 0.035mm 0.035mm 0.035mm 0.035mm 0.035mm 0.035mm"/>
 <param name="mtIsolate" value="1.5mm 0.15mm 0.2mm 0.15mm 0.2mm 0.15mm 0.2mm 0.15mm 0.2mm 0.15mm 0.2mm 0.15mm 0.2mm 0.15mm 0.2mm"/>
-<param name="mdWireWire" value="0.25mm"/>
-<param name="mdWirePad" value="0.25mm"/>
+<param name="mdWireWire" value="0.35mm"/>
+<param name="mdWirePad" value="0.35mm"/>
 <param name="mdWireVia" value="0.35mm"/>
-<param name="mdPadPad" value="0.25mm"/>
+<param name="mdPadPad" value="0.35mm"/>
 <param name="mdPadVia" value="0.35mm"/>
 <param name="mdViaVia" value="0.35mm"/>
-<param name="mdSmdPad" value="8mil"/>
-<param name="mdSmdVia" value="8mil"/>
-<param name="mdSmdSmd" value="8mil"/>
+<param name="mdSmdPad" value="0.1mm"/>
+<param name="mdSmdVia" value="0.1mm"/>
+<param name="mdSmdSmd" value="0.1mm"/>
 <param name="mdViaViaSameLayer" value="8mil"/>
 <param name="mnLayersViaInSmd" value="2"/>
@@
 <element name="X4" library="__MyCommonLib1" package="PIN1X1_3.5MM_PWR" value="+7V" x="49.1" y="7.1"/>
 <element name="X5" library="__MyCommonLib1" package="PIN1X1_3.5MM_PWR" value="-7V" x="49" y="24.3"/>
-<element name="X6" library="__MyCommonLib1" package="PIN1X1_3.5MM_PWR" value="GND" x="55" y="19"/>
+<element name="X6" library="__MyCommonLib1" package="PIN1X1_3.5MM_PWR" value="GND" x="55" y="20"/>
 <element name="R7" library="__MyCommonLib1" package="RSMD_0805" value="***" x="13.5" y="5" rot="MR90"/>
 <element name="C10" library="__MyCommonLib1" package="RSMD_0805" value="0.1uF" x="23.7" y="3.3" rot="MR270"/>
@@
 <contactref element="R7" pad="PAD_0"/>
 <contactref element="C10" pad="PAD_0"/>
-<wire x1="54.5" y1="14.44" x2="55" y2="19" width="0" layer="19" extent="1-1"/>
-<wire x1="51.1" y1="13.825" x2="54.5" y2="14.44" width="0" layer="19" extent="16-16"/>
-<wire x1="47.6" y1="13.825" x2="51.1" y2="13.825" width="0" layer="19" extent="16-16"/>
-<wire x1="44.2" y1="14.54" x2="47.6" y2="13.825" width="0" layer="19" extent="16-16"/>
-<wire x1="41.3" y1="19.16" x2="44.2" y2="14.54" width="0" layer="19" extent="1-1"/>
-<wire x1="38" y1="20.975" x2="41.3" y2="19.16" width="0" layer="19" extent="16-16"/>
-<wire x1="33.4" y1="17.78" x2="38" y2="20.975" width="0" layer="19" extent="16-16"/>
-<wire x1="25.4" y1="12.7" x2="33.4" y2="17.78" width="0" layer="19" extent="1-1"/>
-<wire x1="21.8" y1="7.85" x2="25.4" y2="12.7" width="0" layer="19" extent="16-16"/>
-<wire x1="18.99875" y1="8.695" x2="21.8" y2="7.85" width="0" layer="19" extent="16-16"/>
-<wire x1="18.99875" y1="11.235" x2="18.99875" y2="8.695" width="0" layer="19" extent="16-16"/>
-<wire x1="23.7" y1="4.35" x2="21.8" y2="7.85" width="0" layer="19" extent="16-16"/>
-<wire x1="16.1" y1="3.95" x2="18.99875" y2="8.695" width="0" layer="19" extent="16-16"/>
-<wire x1="13.5" y1="3.95" x2="16.1" y2="3.95" width="0" layer="19" extent="16-16"/>
-<wire x1="6.5" y1="7.46" x2="13.5" y2="3.95" width="0" layer="19" extent="16-16"/>
-<wire x1="2.9" y1="8.65" x2="6.5" y2="7.46" width="0" layer="19" extent="16-16"/>
-<wire x1="3.5" y1="3.2" x2="6.5" y2="7.46" width="0" layer="19" extent="1-1"/>
+<polygon width="0.5" layer="16" thermals="no">
+<vertex x="51.1" y="13.6"/>
+<vertex x="52.6" y="13.6"/>
+<vertex x="53" y="13.2"/>
+<vertex x="57.7" y="13.2"/>
+<vertex x="58.7" y="14.2"/>
+<vertex x="58.7" y="26"/>
+<vertex x="58" y="26.7"/>
+<vertex x="53.9" y="26.7"/>
+<vertex x="53.2" y="26"/>
+<vertex x="53.2" y="22.9"/>
+<vertex x="51.1" y="20.8"/>
+<vertex x="40.1" y="20.8"/>
+<vertex x="39.6" y="21.3"/>
+<vertex x="31.5" y="21.3"/>
+<vertex x="31" y="20.8"/>
+<vertex x="30.3" y="20.1"/>
+<vertex x="30.3" y="19.1"/>
+<vertex x="30.3" y="17"/>
+<vertex x="28.2" y="14.9"/>
+<vertex x="27.6" y="14.3"/>
+<vertex x="25.1" y="14.3"/>
+<vertex x="24.3" y="13.5"/>
+<vertex x="24.3" y="11.6"/>
+<vertex x="24.3" y="9.1"/>
+<vertex x="23.3" y="8.1"/>
+<vertex x="23.3" y="4.4"/>
+<vertex x="23.4" y="4.3"/>
+<vertex x="29.5" y="4.3"/>
+<vertex x="30.7" y="5.5"/>
+<vertex x="30.7" y="13.8"/>
+<vertex x="32.1" y="15.2"/>
+<vertex x="32.3" y="15.4"/>
+<vertex x="34.5" y="15.4"/>
+<vertex x="36.4" y="17.3"/>
+<vertex x="40.6" y="17.3"/>
+<vertex x="42" y="17.3"/>
+<vertex x="42.8" y="16.5"/>
+<vertex x="42.8" y="14.1"/>
+<vertex x="43.3" y="13.6"/>
+</polygon>
+<polygon width="0.5" layer="16" thermals="no">
+<vertex x="4.7" y="8.9"/>
+<vertex x="1.5" y="8.9"/>
+<vertex x="1.2" y="8.6"/>
+<vertex x="1.2" y="2"/>
+<vertex x="1.9" y="1.3"/>
+<vertex x="19" y="1.3"/>
+<vertex x="19.6" y="1.9"/>
+<vertex x="19.6" y="3.7"/>
+<vertex x="19.3" y="4"/>
+<vertex x="19.3" y="5.7"/>
+<vertex x="20.3" y="6.7"/>
+<vertex x="21.8" y="6.7"/>
+<vertex x="23.2" y="5.3"/>
+<vertex x="23.9" y="5.3"/>
+<vertex x="23.9" y="8"/>
+<vertex x="20.8" y="8"/>
+<vertex x="20.1" y="8.7"/>
+<vertex x="17.8" y="8.7"/>
+<vertex x="17.4" y="9.1"/>
+<vertex x="17.4" y="10.9"/>
+<vertex x="17.7" y="11.2"/>
+<vertex x="17.6" y="11.3"/>
+<vertex x="15.4" y="11.3"/>
+<vertex x="15.2" y="11.1"/>
+<vertex x="15.2" y="7.8"/>
+<vertex x="15.6" y="7.4"/>
+<vertex x="17.6" y="7.4"/>
+<vertex x="17.9" y="7.1"/>
+<vertex x="17.9" y="4.6"/>
+<vertex x="17.4" y="4.1"/>
+<vertex x="12.9" y="4.1"/>
+<vertex x="11.9" y="3.1"/>
+<vertex x="10" y="3.1"/>
+<vertex x="9.1" y="4"/>
+<vertex x="9.1" y="5.9"/>
+<vertex x="9.9" y="6.7"/>
+<vertex x="9.9" y="8.1"/>
+<vertex x="9.5" y="8.5"/>
+<vertex x="7.8" y="8.5"/>
+<vertex x="7" y="9.3"/>
+<vertex x="5.1" y="9.3"/>
+</polygon>
+<wire x1="18.99875" y1="11.235" x2="17.235" y2="11.235" width="0.6" layer="16"/>
 </signal>
 <signal name="N$133">
@@
 <vertex x="11.1" y="10"/>
 <vertex x="5.6" y="15.6"/>
-<vertex x="5.6" y="17.5"/>
-<vertex x="4.4" y="17.5"/>
+<vertex x="5.6" y="21"/>
+<vertex x="4.4" y="21"/>
 <vertex x="4.4" y="14.1"/>
 <vertex x="4" y="13.7"/>
