File: LC_METER/TestPowerInverter/LCMeter_test_power_inverter_VER2.sch (EAGLE design)
At the start: 51 parts, among them IC1 MC34063, IC10 MC34063, T1 H772, T2 H772, X1 VCC_IN, X2 GND, X3 +5V_STAB, X4 +8.5V_STAB, X5 -8.5V, X6 GND

Commit message: PoverInverter_V2
Parts:
- added C16: 0.47uFx16V, __MyCommonLib1:CSMD_1206
- added C18, C21, C23: 470uFx16V, __MyCommonLib1:CE10MM
- added C19, C20, C22: 0.47uFx16V, __MyCommonLib1:CSMD_1206_BIG_GAP
- added C4: 1n0, __MyCommonLib1:CSMD_0805
- added C5: 1000uFx16V, __MyCommonLib1:CE10MM
- added L1, L2, L3: 3.3uHx0.9A, __MyCommonLib1:L(SENIA)
- added R14: 10R, __MyCommonLib1:RSMD_0805
- D1: device __MyCommonLib1:1N4001DO-41_5MM -> __MyCommonLib1:1N4001DO-41_10MM
- D2, D3: device __MyCommonLib1:1N4001DO-41_12.5MM -> __MyCommonLib1:1N4001DO-41_10MM
- D4: device __MyCommonLib1:1N4001DO-41_20MM -> __MyCommonLib1:1N4001DO-41_10MM
- R15, R4, R6: device __MyCommonLib1:RSMD_1206_BIG_GAP -> __MyCommonLib1:RSMD_0805
Connections:
- removed net -8.5V: C1.PIN0, C8.MINUS, C9.PIN1, D3.ANODE, D4.ANODE, R8.PIN0, X5.1
- new net -8.5V_STABILIZED: C22.PIN1, C23.MINUS, L1.END, X5.1
- new net N$13: C4.PIN1, R14.PIN0
- new net N$17: C1.PIN0, C4.PIN0, C8.MINUS, C9.PIN1, D3.ANODE, D4.ANODE, L1.START, R8.PIN0
- new net N$18: C13.PIN1, C14.PLUS, D1.CATHODE, L3.START, R15.PIN0
- new net N$19: C6.PIN1, C7.PLUS, D2.CATHODE, L2.START, R6.PIN0
- net +5V_STABILIZED: now also C18.PLUS, C19.PIN1, L3.END; no longer C13.PIN1, C14.PLUS, D1.CATHODE, R15.PIN0
- net +8.5V_STABILIZED: now also C20.PIN1, C21.PLUS, L2.END; no longer C6.PIN1, C7.PLUS, D2.CATHODE, R6.PIN0
- net GND: now also C16.PIN0, C18.MINUS, C19.PIN0, C20.PIN0, C21.MINUS, C22.PIN0, C23.PLUS, C5.MINUS
- net N$12: now also R14.PIN1
- net VCC_IN: now also C16.PIN1, C5.PLUS
Other:
- moved on the sheet: C13, C14, C6, C7, C8, C9, X6
