File: LC_METER/TestPowerInverter/LCMeter_test_power_inverter_VER2.sch (EAGLE design)
At the start: 64 parts, among them IC1 MC34063, IC10 MC34063, T1 H772, T2 H772, X1 VCC_IN, X2 GND, X3 +5V_STAB, X4 +8.5V_STAB, X5 -8.5V, X6 GND

Commit message: PowerInverter_V2
Parts:
- removed C4: 1n0, __MyCommonLib1:CSMD_0805
- removed C53: 1000uFx16V, __MyCommonLib1:CE10MM
- removed C54: 0.47uFx16V, __MyCommonLib1:CSMD_1206
- removed R14: 10R, __MyCommonLib1:RSMD_0805
- added X7: GND, __MyCommonLib1:PIN1X13.5MM_PWR
- D1, D3: device __MyCommonLib1:1N4001DO-41_10MM -> __MyCommonLib1:1N4001DO-41_5MM
- D4: device __MyCommonLib1:1N4001DO-41_10MM -> __MyCommonLib1:1N4001DO-41_20MM
Connections:
- removed net N$13: C4.PIN1, R14.PIN0
- net GND: now also TR2.PRI_START, TR2.SEC_END, X7.1; no longer C53.MINUS, C54.PIN0, TR2.PRI_END, TR2.SEC_START
- net N$12: now also TR2.PRI_END; no longer R14.PIN1, TR2.SEC_END
- net N$14: now also TR2.SEC_START; no longer TR2.PRI_START
- net N$17: no longer C4.PIN0
- net N$4: now also TR1.PRI_START; no longer TR1.SEC_END
- net N$8: now also TR1.SEC_END; no longer TR1.PRI_START
- net VCC_IN: no longer C53.PLUS, C54.PIN1
Other:
- moved on the sheet: D4, TR2

Commit message: PowerInverter_V2 PCB routed
Parts:
- D2: device __MyCommonLib1:1N4001DO-41_10MM -> __MyCommonLib1:1N4001DO-41_5MM
Changed lines of the file:
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@@
 <part name="R3" library="__MyCommonLib1" deviceset="R" device="SMD_1206_BIG_GAP" value="*"/>
 <part name="GND3" library="supply1" deviceset="GND" device=""/>
-<part name="D2" library="__MyCommonLib1" deviceset="1N4001" device="DO-41_10MM" value="SB2100"/>
+<part name="D2" library="__MyCommonLib1" deviceset="1N4001" device="DO-41_5MM" value="SB2100"/>
 <part name="D3" library="__MyCommonLib1" deviceset="1N4001" device="DO-41_5MM" value="SB2100"/>
 <part name="R4" library="__MyCommonLib1" deviceset="R" device="SMD_0805" value="10R"/>

Commit message: Test LC meter power supply changes
Parts:
- C2, C55: value 330pf* -> 220pF
- R1, R11: value 51R -> 68R
- R10: value 1K6 -> 1K3
- R7: value *** -> 1K3
- R84: value 4K7 -> 7K5
- R85: value 1K6 -> ***
- R9: value 4K7 -> 3K9
