File: LC_METER/TestPowerInverter/LCMeter_test_power_inverter_VER2.brd (EAGLE design)
At the start: 60 x 28 mm, 51 parts, among them IC1 MC34063, IC10 MC34063, T1 H772, T2 H772, X1 VCC_IN, X2 GND, X3 +5V_STAB, X4 +8.5V_STAB, X5 -8.5V, X6 GND

Commit message: PoverInverter_V2
Parts:
- added C16: 0.47uFx16V, __MyCommonLib1:RSMD_1206
- added C18, C21, C23: 470uFx16V, __MyCommonLib1:CE_10MM
- added C19, C20, C22: 0.47uFx16V, __MyCommonLib1:RSMD_1206_BIG_GAP
- added C4: 1n0, __MyCommonLib1:RSMD_0805
- added C5: 1000uFx16V, __MyCommonLib1:CE_10MM
- added L1, L2, L3: 3.3uHx0.9A, __MyCommonLib1:L_SENIA
- added R14: 10R, __MyCommonLib1:RSMD_0805
- D1: device __MyCommonLib1:DO-41_5MM -> __MyCommonLib1:DO-41_10MM
- D2, D3: device __MyCommonLib1:DO-41_12.5MM -> __MyCommonLib1:DO-41_10MM
- D4: device __MyCommonLib1:DO-41_20MM -> __MyCommonLib1:DO-41_10MM
- R15, R4, R6: device __MyCommonLib1:RSMD_1206_BIG_GAP -> __MyCommonLib1:RSMD_0805
- moved X2 52.0 mm to (2.50, -15.8)
- moved C54 20.8 mm to (20.3, -18.2), turned to 0 degrees
- moved C53 20.7 mm to (20.4, -14.3), turned to 180 degrees
- moved R8 15.9 mm to (55.1, -29.1), turned to 90 degrees
- moved D4 12.3 mm to (47.5, -35.9), turned to 180 degrees
- moved C13 9.68 mm to (53.7, -55.1)
- moved C1 8.64 mm to (49.6, -32.8)
- moved C8 7.92 mm to (58.7, -30.1)
- moved D3 7.87 mm to (47.5, -32.8)
- moved R4 7.49 mm to (45.5, -32.8)
- moved C9 5.85 mm to (62.1, -30.0)
- moved R1 5.30 mm to (25.3, -23.9)
- moved C14 5.00 mm to (57.4, -54.8)
- moved C12 4.85 mm to (54.3, -44.5)
- moved R15 4.57 mm to (58.4, -44.5)
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Connections:
- removed net -8.5V: C1.PAD_0, C8.MINUS, C9.PAD_1, D3.ANODE, D4.ANODE, R8.PAD_0, X5.1
- new net -8.5V_STABILIZED: C22.PAD_1, C23.MINUS, L1.1, X5.1
- new net N$13: C4.PAD_1, R14.PAD_0
- new net N$17: C1.PAD_0, C4.PAD_0, C8.MINUS, C9.PAD_1, D3.ANODE, D4.ANODE, L1.2, R8.PAD_0
- new net N$18: C13.PAD_1, C14.PLUS, D1.CATHODE, L3.2, R15.PAD_0
- new net N$19: C6.PAD_1, C7.PLUS, D2.CATHODE, L2.2, R6.PAD_0
- net +5V_STABILIZED: now also C18.PLUS, C19.PAD_1, L3.1; no longer C13.PAD_1, C14.PLUS, D1.CATHODE, R15.PAD_0
- net +8.5V_STABILIZED: now also C20.PAD_1, C21.PLUS, L2.1; no longer C6.PAD_1, C7.PLUS, D2.CATHODE, R6.PAD_0
- net GND: now also C16.PAD_0, C18.MINUS, C19.PAD_0, C20.PAD_0, C21.MINUS, C22.PAD_0, C23.PLUS, C5.MINUS
- net N$12: now also R14.PAD_1
- net VCC_IN: now also C16.PAD_1, C5.PLUS
Routing:
- net VCC_IN: track 0.00 -> 29.4 mm, vias 0 -> 2
- net GND: track 0.00 -> 24.6 mm, vias 0 -> 2

Commit message: PowerInverter_V2
Parts:
- removed C4: 1n0, __MyCommonLib1:RSMD_0805
- removed C53: 1000uFx16V, __MyCommonLib1:CE_10MM
- removed C54: 0.47uFx16V, __MyCommonLib1:RSMD_1206
- removed R14: 10R, __MyCommonLib1:RSMD_0805
- added X7: GND, __MyCommonLib1:PIN1X1_3.5MM_PWR
- D1, D3: device __MyCommonLib1:DO-41_10MM -> __MyCommonLib1:DO-41_5MM
- D4: device __MyCommonLib1:DO-41_10MM -> __MyCommonLib1:DO-41_20MM
- moved C5 70.0 mm to (8.20, 27.6)
- moved TR2 67.6 mm to (28.9, 14.2), turned to 90 degrees
- moved C18 66.0 mm to (56.6, 10.4)
- moved C14 66.0 mm to (46.3, 10.3)
- moved C19 66.0 mm to (52.9, 10.6)
- moved R2 65.9 mm to (9.40, 34.3)
- moved C13 65.8 mm to (49.5, 10.6)
- moved R4 65.7 mm to (33.8, 31.9)
- moved C1 65.7 mm to (38.0, 31.9)
- moved L3 65.4 mm to (50.9, 16.4)
- moved R83 65.2 mm to (7.70, 38.4)
- moved R3 65.0 mm to (7.80, 42.0)
- moved D1 65.0 mm to (44.4, 19.4)
- moved T1 64.8 mm to (19.1, 34.3)
- moved R9 64.8 mm to (12.8, 23.7), turned to 180 degrees
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Connections:
- removed net N$13: C4.PAD_1, R14.PAD_0
- net GND: now also TR2.W1_START, TR2.W2_END, X7.1; no longer C53.MINUS, C54.PAD_0, TR2.W1_END, TR2.W2_START
- net N$12: now also TR2.W1_END; no longer R14.PAD_1, TR2.W2_END
- net N$14: now also TR2.W2_START; no longer TR2.W1_START
- net N$17: no longer C4.PAD_0
- net N$4: now also TR1.W1_START; no longer TR1.W2_END
- net N$8: now also TR1.W2_END; no longer TR1.W1_START
- net VCC_IN: no longer C53.PLUS, C54.PAD_1
Routing:
- net GND: track 24.6 -> 176.1 mm, vias 2 -> 0
- net +5V_STABILIZED: track 0.00 -> 47.7 mm, vias 0 -> 2
- net +8.5V_STABILIZED: track 0.00 -> 44.5 mm
- net VCC_IN: track 29.4 -> 0.00 mm, vias 2 -> 0
- net N$4: track 0.28 -> 26.5 mm, vias 0 -> 2
- net N$8: track 0.00 -> 16.5 mm, vias 0 -> 2
- net N$14: track 0.00 -> 13.3 mm
- net N$12: track 0.00 -> 12.9 mm
- net N$18: track 0.00 -> 10.6 mm
- net N$7: track 0.00 -> 2.72 mm
- net N$15: track 0.00 -> 2.35 mm
Other:
- board size 60 x 28 mm -> 63 x 54 mm

Commit message: PowerInverter_V2 PCB routed
Parts:
- D2: device __MyCommonLib1:DO-41_10MM -> __MyCommonLib1:DO-41_5MM
- moved C12 4.59 mm to (37.4, 16.9)
- moved R6 4.55 mm to (33.9, 49.9)
- moved R15 3.05 mm to (41.1, 15.3)
- moved C55 2.81 mm to (22.6, 45.8), turned to 270 degrees
- moved C3 1.91 mm to (33.9, 46.5), turned to 180 degrees
- moved X2 1.90 mm to (5.60, 33.9)
- moved D2 1.34 mm to (37.4, 47.8), turned to 90 degrees
- moved L2 1.20 mm to (50.2, 50.0)
- moved R11 0.90 mm to (12.3, 10.6)
- moved R1 0.73 mm to (15.7, 39.6)
- moved C1 0.60 mm to (38.6, 31.9)
- moved R4 0.30 mm to (34.1, 31.9)
- moved C10 0.20 mm to (19.8, 50.2)
- moved R7 0.10 mm to (15.4, 49.4)
- moved R83 0.10 mm to (7.80, 38.4)
Routing:
- net GND: track 176.1 -> 98.5 mm
- net N$4: track 26.5 -> 7.20 mm
- net N$14: track 13.3 -> 0.00 mm
- net N$12: track 12.9 -> 0.00 mm
- net N$2: track 0.00 -> 11.9 mm
- net N$10: track 0.00 -> 11.3 mm
- net N$18: track 10.6 -> 0.00 mm
- net +5V_STABILIZED: track 47.7 -> 38.3 mm
- net N$133: track 0.00 -> 8.83 mm
- net N$6: track 0.00 -> 8.33 mm
- net N$9: track 0.00 -> 7.61 mm
- net N$139: track 0.00 -> 7.36 mm
- net N$11: track 0.00 -> 5.78 mm
- net +8.5V_STABILIZED: track 44.5 -> 40.0 mm
- net VCC_IN: track 0.00 -> 4.42 mm
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- added copper zone on layer 16, net +5V_STABILIZED
- added copper zone on layer 16, net +8.5V_STABILIZED
- added copper zone on layer 16, net -8.5V_STABILIZED
- added copper zone on layer 16, net GND
- added copper zone on layer 16, net N$11
- added copper zone on layer 16, net N$12
- added copper zone on layer 16, net N$14
- added copper zone on layer 16, net N$17
- added copper zone on layer 16, net N$18
- added copper zone on layer 16, net N$19
- added copper zone on layer 16, net N$3
- added copper zone on layer 16, net N$4
- added copper zone on layer 16, net VCC_IN
