File: LC_METER/TestPowerInverter/LCMeter_test_power_inverter_VER2.brd (EAGLE design)
At the start: 63 x 54 mm, 61 parts, among them IC1 MC34063, IC10 MC34063, T1 H772, T2 H772, X1 VCC_IN, X2 GND, X3 +5V_STAB, X4 +8.5V_STAB, X5 -8.5V, X6 GND, X7 GND

Commit message: Test LC meter power supply changes
Parts:
- C2, C55: value 330pf* -> 220pF
- R1, R11: value 51R -> 68R
- R10: value 1K6 -> 1K3
- R7: value *** -> 1K3
- R84: value 4K7 -> 7K5
- R85: value 1K6 -> ***
- R9: value 4K7 -> 3K9
