File: CurrentSensor/hw/CurrentSensor.brd (EAGLE design)
At the start: 52 x 50 mm, 45 parts, among them IC1 LM317, IC2 74HC595, IC3 ATTINY45, X1 VCC_IN, X2 CHARGE_IN, X3 GND_TO_ACC, X4 GND_FROM_CHARGE

Commit message: Current sensor
Parts:
- D1, D2: value 1N4148 -> 1N4001
- LED2, LED7: value YELLOW -> GREEN
- LED4: value GREEN -> YELLOW
- LED5: value RED -> YELLOW
- LED8: value GREEN -> RED

Commit message: Current sensor
Parts:
- R13: value 10K -> 3K3
Changed lines of the file:
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@@
 <attribute name="VALUE" x="35.84" y="37.84" size="1.27" layer="28" font="vector" ratio="20" rot="MR180"/>
 </element>
-<element name="R13" library="__MyCommonLib1" package="RSMD_0805" value="10K" x="32.84" y="40.45" smashed="yes" rot="MR0">
+<element name="R13" library="__MyCommonLib1" package="RSMD_0805" value="3K3" x="32.84" y="40.45" smashed="yes" rot="MR0">
 <attribute name="NAME" x="39.04" y="39.85" size="1.27" layer="26" font="vector" ratio="20" rot="MR0"/>
 <attribute name="VALUE" x="38.84" y="39.85" size="1.27" layer="28" font="vector" ratio="20" rot="MR0"/>

Commit message: Current Sensor board update.
Parts:
- C5: value 0.1uF -> 10nF
Changed lines of the file:
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@@
 <attribute name="VALUE" x="23.62" y="43.92" size="1.27" layer="28" font="vector" ratio="20" rot="MR90"/>
 </element>
-<element name="C5" library="__MyCommonLib1" package="RSMD_0805" value="0.1uF" x="24.8" y="26.4" smashed="yes" rot="MR180">
+<element name="C5" library="__MyCommonLib1" package="RSMD_0805" value="10nF" x="24.8" y="26.4" smashed="yes" rot="MR180">
 <attribute name="NAME" x="23.4" y="27" size="1.27" layer="26" font="vector" ratio="20" rot="MR180"/>
 <attribute name="VALUE" x="22.6" y="24.8" size="1.27" layer="28" font="vector" ratio="20" rot="MR180"/>
