File: CurrentSensor/hw/CurrentSensor.sch (EAGLE design)
At the start: 45 parts, among them IC1 LM317, IC2 74HC595, IC3 ATTINY45, X1 VCC_IN, X2 CHARGE_IN, X3 GND_TO_ACC, X4 GND_FROM_CHARGE

Commit message: Curent sensor. Routed.
Parts:
- R1: device __MyCommonLib1:RSMD_0805 -> __MyCommonLib1:RSMD_1206
Changed lines of the file:
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@@
 <part name="GND14" library="supply1" deviceset="GND" device=""/>
 <part name="IC2" library="__MyCommonLib1" deviceset="74HC595" device="(SOIC16)" value="74HC595"/>
-<part name="R1" library="__MyCommonLib1" deviceset="R" device="SMD_0805" value="1K0"/>
+<part name="R1" library="__MyCommonLib1" deviceset="R" device="SMD_1206" value="1K0"/>
 <part name="R2" library="__MyCommonLib1" deviceset="R" device="SMD_0805" value="1K0"/>
 <part name="R4" library="__MyCommonLib1" deviceset="R" device="SMD_0805" value="1K0"/>
