File: CurrentSensor/hw/CurrentSensor.sch (EAGLE design)
At the start: 45 parts, among them IC1 LM317, IC2 74HC595, IC3 ATTINY45, X1 VCC_IN, X2 CHARGE_IN, X3 GND_TO_ACC, X4 GND_FROM_CHARGE

Commit message: Current sensor
Parts:
- D1, D2: value 1N4148 -> 1N4001
- LED2, LED7: value YELLOW -> GREEN
- LED4: value GREEN -> YELLOW
- LED5: value RED -> YELLOW
- LED8: value GREEN -> RED
Changed lines of the file:
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@@
 <part name="R16" library="__MyCommonLib1" deviceset="R" device="1.0W" value="0.1Ohm"/>
 <part name="X2" library="__MyCommonLib1" deviceset="PIN1X1" device="3.5MM_SIDE_BOARD" value="CHARGE_IN"/>
-<part name="D1" library="__MyCommonLib1" deviceset="1N4001" device="DO-41_10MM" value="1N4148"/>
-<part name="D2" library="__MyCommonLib1" deviceset="1N4001" device="DO-41_10MM" value="1N4148"/>
+<part name="D1" library="__MyCommonLib1" deviceset="1N4001" device="DO-41_10MM" value="1N4001"/>
+<part name="D2" library="__MyCommonLib1" deviceset="1N4001" device="DO-41_10MM" value="1N4001"/>
 <part name="C1" library="__MyCommonLib1" deviceset="CE" device="6.3MM" value="470uFx25V"/>
 <part name="C2" library="__MyCommonLib1" deviceset="C" device="SMD_0805" value="0.1uF"/>
@@
 <part name="GND27" library="supply1" deviceset="GND" device=""/>
 <part name="LED1" library="__MyCommonLib1" deviceset="LED3MM" device="" value="RED"/>
-<part name="LED2" library="__MyCommonLib1" deviceset="LED3MM" device="" value="YELLOW"/>
+<part name="LED2" library="__MyCommonLib1" deviceset="LED3MM" device="" value="GREEN"/>
 <part name="LED3" library="__MyCommonLib1" deviceset="LED3MM" device="" value="YELLOW"/>
-<part name="LED4" library="__MyCommonLib1" deviceset="LED3MM" device="" value="GREEN"/>
-<part name="LED5" library="__MyCommonLib1" deviceset="LED3MM" device="" value="RED"/>
+<part name="LED4" library="__MyCommonLib1" deviceset="LED3MM" device="" value="YELLOW"/>
+<part name="LED5" library="__MyCommonLib1" deviceset="LED3MM" device="" value="YELLOW"/>
 <part name="LED6" library="__MyCommonLib1" deviceset="LED3MM" device="" value="YELLOW"/>
-<part name="LED7" library="__MyCommonLib1" deviceset="LED3MM" device="" value="YELLOW"/>
-<part name="LED8" library="__MyCommonLib1" deviceset="LED3MM" device="" value="GREEN"/>
+<part name="LED7" library="__MyCommonLib1" deviceset="LED3MM" device="" value="GREEN"/>
+<part name="LED8" library="__MyCommonLib1" deviceset="LED3MM" device="" value="RED"/>
 <part name="C6" library="__MyCommonLib1" deviceset="C" device="SMD_0805" value="0.1uF"/>
 <part name="C9" library="__MyCommonLib1" deviceset="C" device="SMD_0805" value="0.1uF"/>

Commit message: Current sensor
Parts:
- R13: value 10K -> 3K3
Changed lines of the file:
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@@
 <part name="R12" library="__MyCommonLib1" deviceset="R" device="SMD_1206_BIG_GAP" value="10K"/>
 <part name="C7" library="__MyCommonLib1" deviceset="C" device="SMD_0805" value="0.1uF"/>
-<part name="R13" library="__MyCommonLib1" deviceset="R" device="SMD_0805" value="10K"/>
+<part name="R13" library="__MyCommonLib1" deviceset="R" device="SMD_0805" value="3K3"/>
 <part name="GND8" library="supply1" deviceset="GND" device=""/>
 <part name="GND9" library="supply1" deviceset="GND" device=""/>
@@
 <instance part="R12" gate="R$1" x="30.48" y="116.84" smashed="yes" rot="R270">
 <attribute name="NAME" x="29.21" y="118.745" size="1.27" layer="95" font="vector" ratio="20"/>
-<attribute name="VALUE" x="33.02" y="118.745" size="1.27" layer="96" font="vector" ratio="20"/>
+<attribute name="VALUE" x="27.94" y="113.665" size="1.27" layer="96" font="vector" ratio="20"/>
 </instance>
 <instance part="C7" gate="C$1" x="43.18" y="109.22" smashed="yes" rot="MR180">

Commit message: Current Sensor board update.
Parts:
- C5: value 0.1uF -> 10nF
Changed lines of the file:
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@@
 <part name="GND5" library="supply1" deviceset="GND" device=""/>
 <part name="D4" library="__MyCommonLib1" deviceset="LL4147" device="SOD-80" value="LL4148"/>
-<part name="C5" library="__MyCommonLib1" deviceset="C" device="SMD_0805" value="0.1uF"/>
+<part name="C5" library="__MyCommonLib1" deviceset="C" device="SMD_0805" value="10nF"/>
 <part name="R6" library="__MyCommonLib1" deviceset="R" device="SMD_0805" value="1K0"/>
 <part name="GND6" library="supply1" deviceset="GND" device=""/>
