File: KLineAdapter/schematic/KLineAdapter.brd (EAGLE design)
At the start: 44 x 21 mm, 25 parts, among them T1 BC847, T2 BC847, X2 OBD2_+12V, X3 USB_MICRO, X4 OBD2_KLINE, X5 OBD2_GND

Commit message: KLine adapter. Almost routed.
Parts:
- LED4: device __MyCommonLib1:LED3MM -> __MyCommonLib1:LED_0805
- X2, X4, X5: device __MyCommonLib1:PIN1X1_3.5MM_PWR -> __MyCommonLib1:PIN1X1_2.54MM
- moved X5 118.6 mm to (41.4, 9.80)
- moved X2 108.2 mm to (9.00, 19.0)
- moved D4 99.2 mm to (33.0, 8.80), turned to 270 degrees
- moved R16 98.2 mm to (35.8, 8.20), turned to 270 degrees
- moved X4 92.4 mm to (4.00, 10.0)
- moved C6 84.4 mm to (13.0, 15.0), turned to 180 degrees
- moved D22 79.0 mm to (9.00, 14.0), turned to 90 degrees
- moved R15 76.6 mm to (10.0, 1.60), turned to 180 degrees
- moved LED4 72.3 mm to (15.6, 9.60), turned to 180 degrees
- moved R13 69.0 mm to (15.6, 12.4), turned to 180 degrees
- moved R14 66.2 mm to (8.00, 9.00), turned to 90 degrees
- moved C2 62.1 mm to (31.0, 19.0), turned to 270 degrees
- moved R4 58.7 mm to (13.8, 5.00), turned to 90 degrees
- moved L1 54.8 mm to (33.0, 15.0), turned to 180 degrees
- moved R3 54.6 mm to (11.4, 9.20), turned to 90 degrees
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Connections:
- net N$1: no longer U$2.4
- net VCC: now also U$2.4
Routing:
- net GND: track 0.00 -> 78.0 mm
- net RXD: track 0.00 -> 31.9 mm
- net VCC: track 0.00 -> 29.1 mm
- net KLINE: track 0.00 -> 19.0 mm
- net N$5: track 0.00 -> 16.0 mm
- net VCC_USB: track 0.00 -> 12.7 mm
- net TXD: track 0.00 -> 9.47 mm
- net N$3: track 0.00 -> 6.64 mm
- net N$4: track 0.00 -> 6.07 mm
- net USB_D-: track 0.00 -> 5.62 mm
- net USB_D+: track 0.00 -> 3.14 mm
- net +12V: track 0.00 -> 3.12 mm
- net N$10: track 0.00 -> 2.80 mm
- net N$1: track 0.00 -> 2.28 mm

Commit message: KLine adapter. Almost routed.
Parts:
- L1: device __MyCommonLib1:RSMD_0805 -> __MyCommonLib1:RSMD_1206
- R13: value 1K0 -> 4K7
- moved R13 9.62 mm to (6.40, 9.60), turned to 90 degrees
- moved LED4 7.60 mm to (8.80, 13.0)
- moved R4 4.62 mm to (14.2, 9.60)
- moved R1 4.39 mm to (17.8, 9.20), turned to 180 degrees
- moved R15 3.74 mm to (9.00, 5.20), turned to 90 degrees
- moved T2 3.03 mm to (13.0, 5.40)
- moved C4 2.88 mm to (34.4, 10.8)
- moved D4 2.63 mm to (32.6, 6.20)
- moved D22 2.55 mm to (10.8, 15.8), turned to 180 degrees
- moved C1 2.42 mm to (17.8, 12.4)
- moved C6 2.01 mm to (13.2, 13.0)
- moved X4 1.71 mm to (2.40, 10.6)
- moved U$2 1.61 mm to (26.6, 6.80)
- moved R2 1.61 mm to (20.8, 3.80), turned to 90 degrees
- moved R16 1.46 mm to (35.4, 6.80)
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Connections:
- removed net N$10: LED4.ANODE, R13.PAD_0
- new net N$9: LED4.CATHODE, R13.PAD_1
- net KLINE: now also R13.PAD_0; no longer LED4.CATHODE
- net N$5: now also LED4.ANODE; no longer R13.PAD_1
Routing:
- net VCC: track 29.1 -> 3.14 mm
- net RXD: track 31.9 -> 23.4 mm
- net GND: track 78.0 -> 71.8 mm
- net KLINE: track 19.0 -> 12.9 mm
- net N$4: track 6.07 -> 11.3 mm
- net N$1: track 2.28 -> 5.83 mm
- net N$9: track 0.00 -> 3.35 mm
- net N$10: track 2.80 -> 0.00 mm
- net N$5: track 16.0 -> 13.6 mm
- net USB_D-: track 5.62 -> 7.05 mm
- net N$3: track 6.64 -> 5.36 mm
- net TXD: track 9.47 -> 10.5 mm
- net USB_D+: track 3.14 -> 4.19 mm
- net VCC_USB: track 12.7 -> 12.0 mm

Commit message: KLine adapter. Routed.
Parts:
- added J1: 0 Ohm, __MyCommonLib1:RSMD_0805
- added LED1: red, __MyCommonLib1:LED_0805
- added R5: 1K0, __MyCommonLib1:RSMD_0805
- X2, X4, X5: device __MyCommonLib1:PIN1X1_2.54MM -> __MyCommonLib1:PIN1X1_3.5MM_PWR
- moved R15 21.7 mm to (30.4, 1.90), turned to 180 degrees
- moved C5 11.4 mm to (33.6, 6.80)
- moved X2 9.80 mm to (9.20, 9.20)
- moved R3 8.99 mm to (18.3, 3.60), turned to 0 degrees
- moved X5 8.30 mm to (41.5, 2.50)
- moved X4 7.91 mm to (2.70, 2.70)
- moved LED4 6.65 mm to (2.60, 10.6), turned to 270 degrees
- moved T2 6.34 mm to (6.70, 4.70)
- moved R4 6.26 mm to (10.3, 4.70)
- moved D4 5.28 mm to (35.8, 2.00), turned to 180 degrees
- moved R2 5.26 mm to (17.5, 7.90)
- moved R13 4.84 mm to (2.60, 6.60)
- moved R1 3.91 mm to (14.0, 8.30)
- moved T1 3.81 mm to (13.9, 4.50)
- moved R14 3.54 mm to (5.50, 9.10)
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Connections:
- new net N$2: J1.PAD_0, U$2.5
- new net N$6: LED1.CATHODE, R5.PAD_1
- net GND: now also R5.PAD_0
- net N$5: no longer R3.PAD_1
- net RXD: now also J1.PAD_1; no longer U$2.5
- net VCC: now also LED1.ANODE, R3.PAD_1
Routing:
- net VCC: track 3.14 -> 33.8 mm
- net GND: track 71.8 -> 47.5 mm, vias 0 -> 2
- net RXD: track 23.4 -> 9.06 mm
- net N$5: track 13.6 -> 19.6 mm
- net TXD: track 10.5 -> 15.8 mm
- net N$6: track 0.00 -> 2.77 mm, vias 1 -> 0
- net N$2: track 0.00 -> 2.73 mm, vias 1 -> 0
- net N$1: track 5.83 -> 3.47 mm
- net USB_D-: track 7.05 -> 5.06 mm
- net N$4: track 11.3 -> 9.69 mm
- net N$9: track 3.35 -> 1.90 mm
- net VCC_USB: track 12.0 -> 13.2 mm
- net KLINE: track 12.9 -> 12.0 mm
- net +12V: track 3.20 -> 4.05 mm
- net USB_D+: track 4.19 -> 3.56 mm
- added copper zone on layer 1, net GND
- added copper zone on layer 1, net KLINE
- added copper zone on layer 1, net VCC

Commit message: KLine adapter. Routed.
Routing:
- net GND: track 47.5 -> 43.7 mm
- net VCC: track 33.8 -> 35.3 mm
Changed lines of the file:
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@@
 <wire x1="20.7" y1="15.6" x2="20.7" y2="18" width="0.4" layer="1"/>
 <wire x1="21.3" y1="10.375" x2="23.525" y2="10.375" width="0.4" layer="1"/>
-<wire x1="23.525" y1="10.375" x2="26.2" y2="7.7" width="0.4" layer="1"/>
 <wire x1="28.3" y1="7.775" x2="26.275" y2="7.775" width="0.4" layer="1"/>
 <wire x1="26.275" y1="7.775" x2="26.2" y2="7.7" width="0.4" layer="1"/>
@@
 <vertex x="0.7" y="14"/>
 <vertex x="1.1" y="13.6"/>
-<vertex x="6.5" y="13.6"/>
-<vertex x="8.9" y="16"/>
-<vertex x="10.1" y="16"/>
-<vertex x="10.7" y="16.6"/>
-<vertex x="10.7" y="18.6"/>
-<vertex x="11.9" y="19.8"/>
-<vertex x="13.3" y="19.8"/>
-<vertex x="14.2" y="18.9"/>
+<vertex x="6.4" y="13.6"/>
+<vertex x="8.9" y="16.1"/>
+<vertex x="10.3" y="16.1"/>
+<vertex x="10.8" y="16.6"/>
+<vertex x="10.8" y="19"/>
+<vertex x="11.7" y="19.9"/>
+<vertex x="13.3" y="19.9"/>
+<vertex x="14.2" y="19"/>
 <vertex x="14.2" y="17.5"/>
 <vertex x="14.3" y="17.4"/>
@@
 <vertex x="15.9" y="14.4"/>
 <vertex x="19" y="14.4"/>
-<vertex x="19" y="16.3"/>
-<vertex x="20.2" y="17.5"/>
-<vertex x="24" y="17.5"/>
-<vertex x="24.8" y="16.7"/>
+<vertex x="19" y="16.9"/>
+<vertex x="19.6" y="17.5"/>
+<vertex x="24.2" y="17.5"/>
+<vertex x="24.8" y="16.9"/>
 <vertex x="24.8" y="15.7"/>
-<vertex x="25.3" y="15.2"/>
-<vertex x="29.5" y="15.2"/>
-<vertex x="29.9" y="15.6"/>
+<vertex x="25.2" y="15.3"/>
+<vertex x="29.5" y="15.3"/>
+<vertex x="29.9" y="15.7"/>
 <vertex x="29.9" y="18.4"/>
 <vertex x="30.4" y="18.9"/>
@@
 <wire x1="21.3" y1="10.375" x2="20.275" y2="10.375" width="0.4" layer="1"/>
 <wire x1="20.275" y1="10.375" x2="19.8" y2="9.9" width="0.4" layer="1"/>
+<polygon width="0.4" layer="1">
+<vertex x="22.7" y="10.4"/>
+<vertex x="23.7" y="11.4"/>
+<vertex x="23.7" y="12"/>
+<vertex x="23.9" y="12.2"/>
+<vertex x="26.3" y="12.2"/>
+<vertex x="26.4" y="12.1"/>
+<vertex x="26.4" y="9.2"/>
+<vertex x="26.4" y="8.2"/>
+<vertex x="26.8" y="7.8"/>
+<vertex x="26.4" y="7.4"/>
+<vertex x="23.8" y="10"/>
+<vertex x="23.2" y="10"/>
+<vertex x="23.1" y="10"/>
+</polygon>
 </signal>
 <signal name="USB_D-">
@@
 <contactref element="C2" pad="PAD_1"/>
 <wire x1="23.3" y1="15.6" x2="23.3" y2="14.4" width="0.4" layer="1"/>
-<wire x1="23.3" y1="14.4" x2="23.8" y2="13.9" width="0.4" layer="1"/>
-<wire x1="23.8" y1="13.9" x2="24.8" y2="13.9" width="0.4" layer="1"/>
-<wire x1="24.8" y1="13.9" x2="31.6" y2="13.9" width="1" layer="1"/>
+<wire x1="23.3" y1="14.4" x2="23.9" y2="13.8" width="0.4" layer="1"/>
+<wire x1="23.9" y1="13.8" x2="24.9" y2="13.8" width="0.4" layer="1"/>
+<wire x1="24.9" y1="13.8" x2="31.6" y2="13.8" width="1" layer="1"/>
 <wire x1="31.65" y1="14.1" x2="31.6" y2="14.05" width="1" layer="1"/>
-<wire x1="31.6" y1="14.05" x2="31.6" y2="13.9" width="1" layer="1"/>
+<wire x1="31.6" y1="14.05" x2="31.6" y2="13.8" width="1" layer="1"/>
 <wire x1="31.45" y1="17.2" x2="31.45" y2="14.1" width="1" layer="1"/>
 <wire x1="31.45" y1="14.1" x2="31.65" y2="14.1" width="1" layer="1"/>
@@
 <wire x1="21.3" y1="9.075" x2="23.325" y2="9.075" width="0.4" layer="1"/>
 <wire x1="28.3" y1="5.825" x2="26.625" y2="5.825" width="0.4" layer="1"/>
-<wire x1="20.2" y1="2.9" x2="22.9" y2="2.9" width="0.4" layer="1"/>
 <wire x1="28.3" y1="5.825" x2="29.275" y2="5.825" width="0.4" layer="1"/>
 <wire x1="29.275" y1="5.825" x2="29.6" y2="5.5" width="0.4" layer="1"/>
@@
 <vertex x="26.9" y="5.8"/>
 <vertex x="26.4" y="6.3"/>
-<vertex x="25.8" y="6.3"/>
-<vertex x="23.8" y="8.3"/>
-<vertex x="23.8" y="8.6"/>
+<vertex x="26.1" y="6.3"/>
 <vertex x="23.3" y="9.1"/>
 </polygon>
@@
 <wire x1="33.85" y1="5.5" x2="37.9" y2="5.5" width="0.4" layer="1"/>
 <wire x1="38.2" y1="5.8" x2="38.2" y2="5.2" width="0.8" layer="1"/>
-<wire x1="20.2" y1="2.9" x2="20.1" y2="3" width="0.4" layer="1"/>
-<wire x1="20.1" y1="3" x2="19.6" y2="3" width="0.4" layer="1"/>
-<wire x1="19.35" y1="3.6" x2="19.6" y2="3.35" width="0.4" layer="1"/>
-<wire x1="19.6" y1="3.35" x2="19.6" y2="3" width="0.4" layer="1"/>
+<wire x1="19.35" y1="3.6" x2="19.6" y2="3.35" width="0.5" layer="1"/>
+<wire x1="19.6" y1="3.35" x2="19.6" y2="3.1" width="0.5" layer="1"/>
+<wire x1="19.6" y1="3.1" x2="19.9" y2="2.8" width="0.5" layer="1"/>
+<wire x1="19.9" y1="2.8" x2="22.4" y2="2.8" width="0.5" layer="1"/>
+<wire x1="22.4" y1="2.8" x2="23.8" y2="4.2" width="0.5" layer="1"/>
 </signal>
 <signal name="N$3">
@@
 <contactref element="R13" pad="PAD_0"/>
 <wire x1="27" y1="1" x2="17.7" y2="1" width="0.4" layer="1"/>
-<polygon width="0.4" layer="1">
+<polygon width="0.4" layer="1" thermals="no">
 <vertex x="0.8" y="5.7"/>
 <vertex x="3.9" y="5.7"/>

Commit message: KLine adapter complete.
Parts:
- R16: value 2K7 -> 3K3
- R3: value 10K -> 3K3
Changed lines of the file:
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@@
 <element name="R1" library="__MyCommonLib1" package="RSMD_0805" value="3K3" x="14" y="8.3" rot="R180"/>
 <element name="R2" library="__MyCommonLib1" package="RSMD_0805" value="3K3" x="17.5" y="7.9" rot="R90"/>
-<element name="R3" library="__MyCommonLib1" package="RSMD_0805" value="10K" x="18.3" y="3.6"/>
+<element name="R3" library="__MyCommonLib1" package="RSMD_0805" value="3K3" x="18.3" y="3.6"/>
 <element name="T2" library="__MyCommonLib1" package="SOT23_SMALL_PADS" value="BC847" x="6.7" y="4.7" rot="R270"/>
 <element name="R4" library="__MyCommonLib1" package="RSMD_0805" value="3K3" x="10.3" y="4.7" rot="R90"/>
@@
 <element name="C100" library="__MyCommonLib1" package="CE_5.2MM" value="47uF x 25V" x="13.5" y="18.4" rot="MR0"/>
 <element name="R15" library="__MyCommonLib1" package="RSMD_0805" value="10K" x="30.4" y="1.9" rot="R180"/>
-<element name="R16" library="__MyCommonLib1" package="RSMD_0805" value="2K7" x="36.1" y="5.5" rot="R270"/>
+<element name="R16" library="__MyCommonLib1" package="RSMD_0805" value="3K3" x="36.1" y="5.5" rot="R270"/>
 <element name="D4" library="__MyCommonLib1" package="SOD-80" value="LL4148" x="35.8" y="2" rot="R180"/>
 <element name="X4" library="__MyCommonLib1" package="PIN1X1_3.5MM_PWR" value="OBD2_KLINE" x="2.7" y="2.7"/>
