File: KLineAdapter/schematic/KLineAdapter_TO_PRINT.brd (EAGLE design)
At the start: 44 x 46 mm, 56 parts, among them J1 0 Ohm, J2 0 Ohm, T1 BC847, T2 BC847, T3 BC847, T4 BC847, X1 USB_MICRO, X2 OBD2_+12V, X3 USB_MICRO, X4 OBD2_KLINE, X5 OBD2_GND, X6 OBD2_KLINE, X7 OBD2_+12V, X8 OBD2_GND

Commit message: KLine adapter complete.
Parts:
- added LED5, LED6: yellow, __MyCommonLib1:LED_0805
- added R19, R20: 4K7, __MyCommonLib1:RSMD_0805
- added U$3, U$4: ODB2, __MyCommonLib1:ODB2
- added X10, X13: K_Line, __MyCommonLib1:PIN1X1_3.5MM_SIDE_BOARD
- added X11, X14: GND, __MyCommonLib1:PIN1X1_3.5MM_SIDE_BOARD
- added X12, X9: +12V, __MyCommonLib1:PIN1X1_3.5MM_SIDE_BOARD
Connections:
- new net BAT_+12V: LED5.ANODE, U$3.16, X9.1
- new net BAT_+12V1: LED6.ANODE, U$4.16, X12.1
- new net GND2: R19.PAD_1, U$3.4, U$3.5, X11.1
- new net GND3: R20.PAD_1, U$4.4, U$4.5, X14.1
- new net N$15: U$3.7, X10.1
- new net N$16: LED5.CATHODE, R19.PAD_0
- new net N$17: U$4.7, X13.1
- new net N$18: LED6.CATHODE, R20.PAD_0
Routing:
- net N$18: track 0.00 -> 3.30 mm
- net N$16: track 0.00 -> 3.30 mm
- added copper zone on layer 1, net BAT_+12V
- added copper zone on layer 1, net BAT_+12V1
- added copper zone on layer 1, net GND2
- added copper zone on layer 1, net GND3
- added copper zone on layer 1, net N$15
- added copper zone on layer 1, net N$17
Other:
- board size 44 x 46 mm -> 44 x 96 mm
- board text added: "+12V"
- board text added: "1"
- board text added: "GND"
- board text added: "K"
