File: 12_to_200V_inverter/schematic/12to220inverter.sch (EAGLE design)
At the start: 29 parts, among them IC10 MC34063, T11 BC857, X2 200VDC_OUTPUT

Commit message: 12 to 200V inverter start.
Parts:
- removed TR1: TRANS, __MyCommonLib1:TRANS_3WINDRING25X10_HOR
- removed U$1: IRF830TO-220_VER2, __MyCommonLib1:IRF830TO-220_VER2
- added R10, R9: 10K, __MyCommonLib1:RSMD_0805
- added R7, R8: 4K7, __MyCommonLib1:RSMD_0805
- added T15: IRL5602S, __MyCommonLib1:IRL5602(D2PAK)
- added T16: BC847, __MyCommonLib1:BC847SOT23_SMALL_PADS
- added T17: IRF830TO-220_VER2, __MyCommonLib1:IRF830TO-220_VER2
- added X3: TURN_ON, con-wago-500:W237-102
- C53, C57: device __MyCommonLib1:CE10MM -> __MyCommonLib1:CE16MM
- IC10: device __MyCommonLib1:MC34063(SO-8) -> __MyCommonLib1:MC34063(DIP8)
- TR2: device __MyCommonLib1:TRANS_2WIND(RING_16X8) -> __MyCommonLib1:TRANS_2WIND(RING_25X10)
- X1: value (none) -> +12V_INPUT
Connections:
- removed net N$138: TR1.SEC2_START
- new net N$13: R7.PIN1, T15.SOURCE, X1-1.KL
- new net N$14: R7.PIN0, R8.PIN1, T15.GATE
- new net N$15: R10.PIN1, X3-1.KL
- new net N$16: R10.PIN0, R9.PIN1, T16.B
- new net N$17: R8.PIN0, T16.C
- net +12V: now also T15.DRAIN
- net GND: now also R9.PIN0, T16.E, T17.SOURCE, X1-2.KL, X3-2.KL; no longer TR1.PRI_START, TR1.SEC1_END, TR1.SEC2_END, U$1.SOURCE
- net N$1: now also T17.DRAIN; no longer U$1.DRAIN
- net N$8: now also T17.GATE; no longer U$1.GATE
Other:
- moved on the sheet: C1, C53, C54, C55, C57, D1, D10, D29, D3, D4, D5, IC10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

Commit message: 12 to 200V inverter. Routed.
Parts:
- added C2: *, __MyCommonLib1:CSMD_1206
- added R11: *, __MyCommonLib1:RSMD_1206
- D10: device __MyCommonLib1:1N4001DO-41_12.5MM -> __MyCommonLib1:1N4001DO-41_15MM
- D29: device __MyCommonLib1:1N4001DO-41_5MM -> __MyCommonLib1:1N4001DO-41_10MM
- R5: device __MyCommonLib1:RSMD_0805 -> __MyCommonLib1:RSMD_1206
- R83: device __MyCommonLib1:RSMD_1206_BIG_GAP -> __MyCommonLib1:RSMD_2512
- T17: value IRF830TO-220_VER2 -> IRF830TO-220; device __MyCommonLib1:IRF830TO-220_VER2 -> __MyCommonLib1:IRF830TO-220
Connections:
- new net N$18: C2.PIN0, R11.PIN1
- net +200V: now also R11.PIN0
- net N$11: now also C2.PIN1
Changed lines of the file:
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@@
 <setting verticaltext="up"/>
 </settings>
-<grid distance="0.1" unitdist="inch" unit="inch" style="lines" multiple="1" display="yes" altdistance="0.01" altunitdist="inch" altunit="inch"/>
+<grid distance="0.05" unitdist="inch" unit="inch" style="lines" multiple="2" display="yes" altdistance="0.01" altunitdist="inch" altunit="inch"/>
 <layers>
 <layer number="1" name="Top" color="4" fill="1" visible="yes" active="no"/>
@@
 <part name="C55" library="__MyCommonLib1" deviceset="C" device="SMD_0805" value="1n0*"/>
 <part name="GND10" library="supply1" deviceset="GND" device=""/>
-<part name="R83" library="__MyCommonLib1" deviceset="R" device="SMD_1206_BIG_GAP" value="0.62R"/>
+<part name="R83" library="__MyCommonLib1" deviceset="R" device="SMD_2512" value="0.62R"/>
 <part name="C54" library="__MyCommonLib1" deviceset="C" device="SMD_1206" value="0.47uFx16V"/>
 <part name="C53" library="__MyCommonLib1" deviceset="CE" device="16MM" value="1000uFx16V"/>
 <part name="GND71" library="supply1" deviceset="GND" device=""/>
 <part name="GND72" library="supply1" deviceset="GND" device=""/>
-<part name="D29" library="__MyCommonLib1" deviceset="1N4001" device="DO-41_5MM" value="UF4007"/>
+<part name="D29" library="__MyCommonLib1" deviceset="1N4001" device="DO-41_10MM" value="UF4007"/>
 <part name="C57" library="__MyCommonLib1" deviceset="CE" device="16MM" value="20uF x 450V"/>
 <part name="GND74" library="supply1" deviceset="GND" device=""/>
@@
 <part name="GND3" library="supply1" deviceset="GND" device=""/>
 <part name="R4" library="__MyCommonLib1" deviceset="R" device="SMD_0805" value="20R"/>
-<part name="T17" library="__MyCommonLib1" deviceset="IRF830" device="TO-220_VER2"/>
+<part name="T17" library="__MyCommonLib1" deviceset="IRF830" device="TO-220"/>
 <part name="GND4" library="supply1" deviceset="GND" device=""/>
 <part name="TR2" library="__MyCommonLib1" deviceset="TRANS_2WIND" device="(RING_25X10)" value="test_ring"/>
-<part name="D10" library="__MyCommonLib1" deviceset="1N4001" device="DO-41_12.5MM" value="UF4001"/>
-<part name="R5" library="__MyCommonLib1" deviceset="R" device="SMD_0805" value="*"/>
+<part name="D10" library="__MyCommonLib1" deviceset="1N4001" device="DO-41_15MM" value="UF4001"/>
+<part name="R5" library="__MyCommonLib1" deviceset="R" device="SMD_1206" value="*"/>
 <part name="C1" library="__MyCommonLib1" deviceset="C" device="SMD_1206" value="0.1uF x 50V"/>
 <part name="GND5" library="supply1" deviceset="GND" device=""/>
@@
 <part name="GND13" library="supply1" deviceset="GND" device=""/>
 <part name="GND14" library="supply1" deviceset="GND" device=""/>
+<part name="C2" library="__MyCommonLib1" deviceset="C" device="SMD_1206" value="*"/>
+<part name="R11" library="__MyCommonLib1" deviceset="R" device="SMD_1206" value="*"/>
 </parts>
 <sheets>
@@
 <instance part="GND14" gate="1" x="43.18" y="68.58" smashed="yes">
 <attribute name="VALUE" x="40.64" y="66.04" size="1.27" layer="96" font="vector" ratio="20"/>
+</instance>
+<instance part="C2" gate="C$1" x="205.74" y="152.4" smashed="yes" rot="R90">
+<attribute name="NAME" x="203.2" y="154.94" size="1.27" layer="95" font="vector" ratio="20"/>
+<attribute name="VALUE" x="208.28" y="154.94" size="1.27" layer="96" font="vector" ratio="20" rot="R90"/>
+</instance>
+<instance part="R11" gate="R$1" x="215.9" y="152.4" smashed="yes" rot="R90">
+<attribute name="NAME" x="213.36" y="154.94" size="1.27" layer="95" font="vector" ratio="20"/>
+<attribute name="VALUE" x="218.44" y="154.94" size="1.27" layer="96" font="vector" ratio="20"/>
 </instance>
 </instances>
@@
 <pinref part="R6" gate="R$1" pin="PIN0"/>
 <pinref part="X2" gate="-1" pin="KL"/>
+<pinref part="R11" gate="R$1" pin="PIN0"/>
+<wire x1="220.98" y1="152.4" x2="223.52" y2="152.4" width="0.1524" layer="91"/>
+<wire x1="223.52" y1="152.4" x2="223.52" y2="147.32" width="0.1524" layer="91"/>
+<wire x1="223.52" y1="147.32" x2="210.82" y2="147.32" width="0.1524" layer="91"/>
+<wire x1="210.82" y1="147.32" x2="210.82" y2="142.24" width="0.1524" layer="91"/>
 </segment>
 </net>
@@
 <pinref part="TR2" gate="G$1" pin="SEC_START"/>
 <pinref part="D29" gate="D$1" pin="ANODE"/>
-<wire x1="198.12" y1="142.24" x2="203.2" y2="142.24" width="0.1524" layer="91"/>
+<wire x1="198.12" y1="142.24" x2="200.66" y2="142.24" width="0.1524" layer="91"/>
+<pinref part="C2" gate="C$1" pin="PIN1"/>
+<wire x1="200.66" y1="142.24" x2="203.2" y2="142.24" width="0.1524" layer="91"/>
+<wire x1="203.2" y1="152.4" x2="200.66" y2="152.4" width="0.1524" layer="91"/>
+<wire x1="200.66" y1="152.4" x2="200.66" y2="142.24" width="0.1524" layer="91"/>
+<junction x="200.66" y="142.24"/>
 </segment>
 </net>
@@
 </segment>
 </net>
+<net name="N$18" class="0">
+<segment>
+<pinref part="C2" gate="C$1" pin="PIN0"/>
+<pinref part="R11" gate="R$1" pin="PIN1"/>
+<wire x1="208.28" y1="152.4" x2="210.82" y2="152.4" width="0.1524" layer="91"/>
+</segment>
+</net>
