File: 12_to_200V_inverter/schematic/12to220inverter.brd (EAGLE design)
At the start: 160 x 100 mm, 29 parts, among them IC10 MC34063, T11 BC857, X2 200VDC_OUTPUT

Commit message: 12 to 200V inverter start.
Parts:
- removed TR1: TRANS, __MyCommonLib1:RING_25X10_3WIND_HOR
- removed U$1: IRF830TO-220_VER2, __MyCommonLib1:TO-220(VER2)
- added R10, R9: 10K, __MyCommonLib1:RSMD_0805
- added R7, R8: 4K7, __MyCommonLib1:RSMD_0805
- added T15: IRL5602S, __MyCommonLib1:D2PAK
- added T16: BC847, __MyCommonLib1:SOT23_SMALL_PADS
- added T17: IRF830TO-220_VER2, __MyCommonLib1:TO-220(VER2)
- added X3: TURN_ON, con-wago-500:W237-102
- C53, C57: device __MyCommonLib1:CE_10MM -> __MyCommonLib1:CE_16MM
- IC10: device __MyCommonLib1:SOIC8 -> __MyCommonLib1:DIP8
- TR2: device __MyCommonLib1:RING_16X8_2WIND -> __MyCommonLib1:RING_25X10_2WIND_VERT
- X1: value (none) -> +12V_INPUT
- moved X2 208.7 mm to (95.0, 19.0), turned to 270 degrees
- moved R85 185.2 mm to (28.0, -87.0)
- moved R84 183.4 mm to (32.0, -75.0)
- moved C55 167.8 mm to (-10.0, -87.0)
- moved C54 155.5 mm to (7.00, -75.0)
- moved TR2 155.5 mm to (61.0, 30.0), turned to 90 degrees
- moved R83 149.7 mm to (-9.00, -79.0)
- moved C57 140.7 mm to (80.0, 16.0), turned to 90 degrees
- moved ZD2 134.9 mm to (31.0, -83.0)
- moved X1 131.5 mm to (7.00, 34.0), turned to 270 degrees
- moved ZD1 127.5 mm to (24.0, -83.0)
- moved D29 124.3 mm to (-9.00, -71.0)
- moved R5 119.7 mm to (34.0, -87.0)
- moved D1 113.8 mm to (23.0, -79.0)
- moved R1 110.7 mm to (16.0, -79.0)
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Connections:
- removed net N$138: TR1.W3_START
- new net N$13: R7.PAD_1, T15.3, X1.1
- new net N$14: R7.PAD_0, R8.PAD_1, T15.1
- new net N$15: R10.PAD_1, X3.1
- new net N$16: R10.PAD_0, R9.PAD_1, T16.1
- new net N$17: R8.PAD_0, T16.3
- net +12V: now also T15.2
- net GND: now also R9.PAD_0, T16.2, T17.3, X1.2, X3.2; no longer TR1.W1_START, TR1.W2_END, TR1.W3_END, U$1.3
- net N$1: now also T17.2; no longer U$1.2
- net N$8: now also T17.1; no longer U$1.1
Other:
- board size 160 x 100 mm -> 100 x 40 mm

Commit message: 12 to 200V inverter. Routed.
Parts:
- added C2, R11: *, __MyCommonLib1:RSMD_1206
- D10: device __MyCommonLib1:DO-41_12.5MM -> __MyCommonLib1:DO-41_15MM
- D29: device __MyCommonLib1:DO-41_5MM -> __MyCommonLib1:DO-41_10MM
- R5: device __MyCommonLib1:RSMD_0805 -> __MyCommonLib1:RSMD_1206
- R83: device __MyCommonLib1:RSMD_1206_BIG_GAP -> __MyCommonLib1:RSMD_2512
- T17: value IRF830TO-220_VER2 -> IRF830TO-220; device __MyCommonLib1:TO-220(VER2) -> __MyCommonLib1:TO-220
- moved C55 125.8 mm to (39.6, 28.6), flipped to the bottom, turned to 270 degrees
- moved D29 124.2 mm to (77.6, 18.0)
- moved R85 119.8 mm to (30.2, 32.8), flipped to the bottom
- moved C1 115.8 mm to (63.8, 15.0), flipped to the bottom
- moved R4 113.6 mm to (50.0, 14.0), flipped to the bottom, turned to 270 degrees
- moved R6 113.1 mm to (38.0, 37.0), flipped to the bottom
- moved R84 112.0 mm to (30.6, 37.0), flipped to the bottom, turned to 180 degrees
- moved ZD1 109.8 mm to (66.2, 18.4), flipped to the bottom
- moved D3 106.9 mm to (40.0, 12.0), flipped to the bottom, turned to 90 degrees
- moved R83 105.9 mm to (20.2, 22.8), flipped to the bottom, turned to 180 degrees
- moved ZD2 105.5 mm to (60.0, 18.4), flipped to the bottom
- moved R5 103.0 mm to (63.8, 11.6), flipped to the bottom
- moved D10 102.2 mm to (60.8, 15.0)
- moved D4 100.2 mm to (34.0, 12.0), flipped to the bottom
- moved D5 99.8 mm to (32.0, 15.0), flipped to the bottom, turned to 180 degrees
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Connections:
- new net N$18: C2.PAD_0, R11.PAD_1
- net +12V: now also R83.PAD0; no longer R83.PAD_0
- net +200V: now also R11.PAD_0
- net N$10: now also R83.PAD1; no longer R83.PAD_1
- net N$11: now also C2.PAD_1
Routing:
- net GND: track 0.00 -> 87.1 mm
- net +200V: track 0.00 -> 49.7 mm
- net N$10: track 0.00 -> 26.9 mm, vias 0 -> 2
- net N$7: track 0.00 -> 20.2 mm
- net N$6: track 0.00 -> 19.2 mm
- net N$14: track 0.00 -> 15.6 mm
- net +12V: track 0.00 -> 11.2 mm
- net N$9: track 0.00 -> 10.0 mm
- net N$15: track 0.00 -> 9.38 mm
- net N$4: track 0.00 -> 8.30 mm
- net N$139: track 0.00 -> 7.25 mm
- net N$8: track 0.00 -> 6.09 mm
- net N$16: track 0.00 -> 5.76 mm
- net N$17: track 0.00 -> 5.13 mm
- net N$2: track 0.00 -> 4.49 mm
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- added copper zone on layer 16, net +12V
- added copper zone on layer 16, net +200V
- added copper zone on layer 16, net GND
- added copper zone on layer 16, net N$1
- added copper zone on layer 16, net N$10
- added copper zone on layer 16, net N$11
- added copper zone on layer 16, net N$13
- added copper zone on layer 16, net N$15
Other:
- board size 100 x 40 mm -> 91 x 40 mm

Commit message: 12 to 200V converter v2. Forward 2 conversion.
Parts:
- R83: value 0.62R -> 0.1R
- T17: value IRF830TO-220 -> IRF830
Routing:
- net GND: track 87.1 -> 58.3 mm, vias 0 -> 1
- net +200V: vias 0 -> 1
