File: 12_to_200V_inverter/schematic/12to220inverterVer2.brd (EAGLE design)
At the start: 91 x 40 mm, 37 parts, among them IC10 MC34063, T11 BC857, T15 IRL5602S, T16 BC847, T17 IRF830TO-220, X1 +12V_INPUT, X2 200VDC_OUTPUT, X3 TURN_ON

Commit message: 12 to 200V converter v2. Forward 2 conversion.
Parts:
- removed C53: 1000uFx16V, __MyCommonLib1:CE_16MM
- removed C54: 0.47uFx16V, __MyCommonLib1:RSMD_1206
- removed C55: 1n0*, __MyCommonLib1:RSMD_0805
- removed C57: 20uF x 450V, __MyCommonLib1:CE_16MM
- removed D10: UF4001, __MyCommonLib1:DO-41_15MM
- removed D29: UF4007, __MyCommonLib1:DO-41_10MM
- removed D4, D5: LL4148, __MyCommonLib1:SOD-80
- removed IC10: MC34063, __MyCommonLib1:DIP8
- removed R83: 0.62R, __MyCommonLib1:RSMD_2512
- removed R84: 130K*, __MyCommonLib1:RSMD_1206
- removed R85: 1K6, __MyCommonLib1:RSMD_0805
- removed T11: BC857, __MyCommonLib1:SOT23_SMALL_PADS
- removed T17: IRF830TO-220, __MyCommonLib1:TO-220
- removed TR2: test_ring, __MyCommonLib1:RING_25X10_2WIND_VERT
- removed ZD2: 10V, __MyCommonLib1:SOD-80
- added C10: 12uF x 10V, __MyCommonLib1:RSMD_0805
- added C11: 100uF x 25V, __MyCommonLib1:CE_5.2MM
- added C3: 10nF x 50V, __MyCommonLib1:RSMD_1206
- added C4: 20uF x 450V, __MyCommonLib1:CE_16MM
- added C5, C7: 0.47uFx16V, __MyCommonLib1:RSMD_1206
- added C6: 100uF x 16V, __MyCommonLib1:CE_8.2MM
- added C8: 2.2uF x 10V, __MyCommonLib1:RSMD_0805
- added C9: 5.5uF, __MyCommonLib1:RSMD_0805
- added D11, D7, D8, D9: UF4007, __MyCommonLib1:DO-41_10MM
- added D2, D6: LL4148, __MyCommonLib1:SOD-80
- added R12, R13: 4K7, __MyCommonLib1:RSMD_0805
- added R14, R15: 5R1, __MyCommonLib1:RSMD_1206
- added R16: 22K, __MyCommonLib1:RSMD_0805
- added R17: 33K, __MyCommonLib1:RSMD_0805
- added R18: 47K, __MyCommonLib1:RSMD_0805
- added T1, T2: IRF830, __MyCommonLib1:TO-220
- added T3, T4: BC857, __MyCommonLib1:SOT23_SMALL_PADS
- added TR3: 12_to_200_trans, __MyCommonLib1:TRANS_38X35MM
- added U1: TL494, __MyCommonLib1:SOIC16
- C1: value 0.1uF x 50V -> 4n7 x 16V; device __MyCommonLib1:RSMD_1206 -> __MyCommonLib1:RSMD_0805
- C2: value * -> 1000uF x 16V; device __MyCommonLib1:RSMD_1206 -> __MyCommonLib1:CE_16MM
- R1: value 10R -> 3K3; device __MyCommonLib1:RSMD_1206_BIG_GAP -> __MyCommonLib1:RSMD_0805
- R11: value * -> 7K5; device __MyCommonLib1:RSMD_1206 -> __MyCommonLib1:RSMD_0805
- R2: value 240R -> 33R; device __MyCommonLib1:RSMD_1206_BIG_GAP -> __MyCommonLib1:RSMD_0805
- R3: value 240R -> 39K; device __MyCommonLib1:RSMD_1206_BIG_GAP -> __MyCommonLib1:RSMD_0805
- R4: value 20R -> 1K2
- R5: value * -> 47K; device __MyCommonLib1:RSMD_1206 -> __MyCommonLib1:RSMD_0805
- R6: value 130K* -> 15K; device __MyCommonLib1:RSMD_1206 -> __MyCommonLib1:RSMD_0805
- ZD1: value 10V -> *
- moved R11 145.6 mm to (-53.5, -43.1)
- moved ZD1 133.9 mm to (-54.3, -40.0)
- moved C2 133.6 mm to (22.9, -108.8), flipped to the top
- moved R5 125.8 mm to (-53.5, -33.8)
- moved D1 123.6 mm to (-54.3, -58.6)
- moved C1 121.9 mm to (-54.3, -15.2)
- moved D3 119.7 mm to (-54.3, -61.7), turned to 0 degrees
- moved R6 117.6 mm to (-53.5, -36.9)
- moved R4 110.4 mm to (-53.5, -24.5), turned to 0 degrees
- moved R1 104.3 mm to (-53.5, -12.1), turned to 0 degrees
- moved R2 96.9 mm to (-53.5, -18.3)
- moved R3 92.0 mm to (-53.5, -21.4)
- moved X2 18.4 mm to (81.8, -12.6)
Connections:
- removed net +12V: C53.PLUS, C54.PAD_1, D5.CATHODE, IC10.6, R83.PAD0, T15.2
- removed net +200V: C57.PLUS, D29.CATHODE, R11.PAD_0, R6.PAD_0, X2.1
- removed net N$1: D10.ANODE, T17.2, TR2.W1_START
- removed net N$10: C1.PAD_1, IC10.1, IC10.7, IC10.8, R5.PAD_1, R83.PAD1, TR2.W1_END, ZD2.ANODE
- removed net N$11: C2.PAD_1, D29.ANODE, TR2.W2_START
- removed net N$135: C55.PAD_1, IC10.3
- removed net N$139: IC10.5, R84.PAD_0, R85.PAD_1
- new net +12V_CONTROL: C11.PLUS, C5.PAD_1, C6.PLUS, R18.PAD_1, R2.PAD_1, T15.2, U1.12
- new net +12V_POWER: C2.PLUS, C7.PAD_1, R7.PAD_1, T15.3, TR3.4, TR3.5, X1.1
- new net I_OUT_SENSE: R15.PAD_0, R5.PAD_1, X2.2
- new net N$19: D2.CATHODE, T2.1, T3.2
- new net N$20: D11.CATHODE, D7.ANODE, TR3.9
- new net N$21: D6.CATHODE, T1.1, T4.2
- new net N$23: D8.ANODE, D9.CATHODE, TR3.10
- new net N$24: C3.PAD_1, T2.2, TR3.6
- new net N$25: R14.PAD_0, T1.2, TR3.3
- new net N$26: C3.PAD_0, R14.PAD_1
- new net N$28: C4.PLUS, D7.CATHODE, D8.CATHODE, X2.1
- new net PWM1: D2.ANODE, R12.PAD_1, T3.1, U1.9
- new net PWM2: D6.ANODE, R13.PAD_1, T4.1, U1.10
- new net V_REF: R11.PAD_1, R3.PAD_1, U1.13, U1.14
- net GND: now also C1.PAD_1, C10.PAD_0, C2.MINUS, C4.MINUS, C5.PAD_0, C6.MINUS, C7.PAD_0, C9.PAD_0, D11.ANODE, D3.ANODE, D9.ANODE, R1.PAD_0, R12.PAD_0, R13.PAD_0, R15.PAD_1, R17.PAD_1, R4.PAD_1, T1.3, T2.3, T3.3, T4.3, U1.4, U1.7; no longer C53.MINUS, C54.PAD_0, C55.PAD_0, C57.MINUS, D4.ANODE, IC10.4, R1.PAD_1, R3.PAD_1, R85.PAD_0, T17.3, TR2.W2_END, X2.2
- net N$12: now also R11.PAD_0, R16.PAD_0, U1.16; no longer ZD1.ANODE, ZD2.CATHODE
- net N$13: now also C11.MINUS, D1.ANODE, D3.CATHODE; no longer R7.PAD_1, T15.3, X1.1
- net N$18: now also C10.PAD_1, D1.CATHODE, R17.PAD_0, R18.PAD_0, U1.15; no longer C2.PAD_0, R11.PAD_1
- net N$2: now also C1.PAD_0, U1.5; no longer R1.PAD_0, T11.3
- net N$3: now also R1.PAD_1, U1.6; no longer R6.PAD_1, R84.PAD_1
- net N$4: now also U1.11, U1.8; no longer D3.CATHODE, T11.1
- net N$5: now also R4.PAD_0, U1.2; no longer R2.PAD_1
- net N$6: now also C8.PAD_0, R16.PAD_1, U1.3; no longer D1.ANODE, D3.ANODE, IC10.2
- net N$7: now also C8.PAD_1, C9.PAD_1, R5.PAD_0, R6.PAD_0, U1.1; no longer D1.CATHODE, D4.CATHODE, D5.ANODE, R4.PAD_0, T11.2
- net N$8: now also R6.PAD_1, ZD1.ANODE; no longer R4.PAD_1, T17.1
- net N$9: no longer C1.PAD_0, D10.CATHODE, R5.PAD_0
Routing:
- net GND: track 87.1 -> 7.83 mm
- net +200V: track 49.7 -> 0.00 mm
- net N$10: track 26.9 -> 0.00 mm, vias 2 -> 0
- net N$7: track 20.2 -> 0.00 mm
- net N$6: track 19.2 -> 0.00 mm
- net +12V: track 11.2 -> 0.00 mm
- net N$9: track 10.0 -> 0.00 mm
- net N$4: track 8.30 -> 0.00 mm
- net N$139: track 7.25 -> 0.00 mm
- net N$8: track 6.09 -> 0.00 mm
- net N$2: track 4.49 -> 0.00 mm
- net N$3: track 4.30 -> 0.00 mm
- net N$11: track 3.62 -> 0.00 mm
- net N$135: track 2.91 -> 0.00 mm
- net N$18: track 2.90 -> 0.00 mm
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- added copper zone on layer 16, net +12V_POWER
- removed copper zone on layer 16, net +12V
- removed copper zone on layer 16, net +200V
- removed copper zone on layer 16, net N$1
- removed copper zone on layer 16, net N$10
- removed copper zone on layer 16, net N$11
- removed copper zone on layer 16, net N$13
Other:
- board size 91 x 40 mm -> 91 x 50 mm

Commit message: 12 to 200V converter v2. Schematic done.
Parts:
- removed ZD1: *, __MyCommonLib1:SOD-80
- added R19: 680K, __MyCommonLib1:RSMD_0805
- added ZD2: 4.7V, __MyCommonLib1:SOD-80
- R5: value 47K -> 1K0
- R6: value 15K -> 680K
Connections:
- removed net N$28: C4.PLUS, D7.CATHODE, D8.CATHODE, X2.1
- removed net N$8: R6.PAD_1, ZD1.ANODE
- removed net N$9: ZD1.CATHODE
- new net +200VDC_OUT: C4.PLUS, D7.CATHODE, D8.CATHODE, R19.PAD_1, X2.1
- new net N$1: R19.PAD_0, R6.PAD_1
- net GND: now also ZD2.ANODE
- net N$7: now also ZD2.CATHODE
Changed lines of the file:
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@@
 <element name="C8" library="__MyCommonLib1" package="RSMD_0805" value="2.2uF x 10V" x="-53.5" y="-27.6" rot="MR0"/>
 <element name="C9" library="__MyCommonLib1" package="RSMD_0805" value="5.5uF" x="-53.5" y="-30.7" rot="MR0"/>
-<element name="R5" library="__MyCommonLib1" package="RSMD_0805" value="47K" x="-53.5" y="-33.8" rot="MR0"/>
-<element name="R6" library="__MyCommonLib1" package="RSMD_0805" value="15K" x="-53.5" y="-36.9" rot="MR0"/>
-<element name="ZD1" library="__MyCommonLib1" package="SOD-80" value="*" x="-54.3" y="-40" rot="MR0"/>
+<element name="R5" library="__MyCommonLib1" package="RSMD_0805" value="1K0" x="-53.5" y="-33.8" rot="MR0"/>
+<element name="R6" library="__MyCommonLib1" package="RSMD_0805" value="680K" x="-53.5" y="-36.9" rot="MR0"/>
 <element name="R11" library="__MyCommonLib1" package="RSMD_0805" value="7K5" x="-53.5" y="-43.1" rot="MR0"/>
 <element name="R16" library="__MyCommonLib1" package="RSMD_0805" value="22K" x="-53.5" y="-46.2" rot="MR0"/>
@@
 <element name="D3" library="__MyCommonLib1" package="SOD-80" value="LL4148" x="-54.3" y="-61.7" rot="MR0"/>
 <element name="C11" library="__MyCommonLib1" package="CE_5.2MM" value="100uF x 25V" x="70.9" y="-99"/>
+<element name="ZD2" library="__MyCommonLib1" package="SOD-80" value="4.7V" x="-109.6" y="-121.4" rot="MR0"/>
+<element name="R19" library="__MyCommonLib1" package="RSMD_0805" value="680K" x="-110.4" y="-124.5" rot="MR0"/>
 </elements>
 <signals>
@@
 <contactref element="C10" pad="PAD_0"/>
 <contactref element="D3" pad="ANODE"/>
+<contactref element="ZD2" pad="ANODE"/>
+<wire x1="-104.6" y1="-57.2" x2="-111.475" y2="-121.4" width="0" layer="19" extent="1-16"/>
 <wire x1="-103.25" y1="-42.4" x2="-104.6" y2="-57.2" width="0" layer="19" extent="16-16"/>
 <wire x1="-104.6" y1="-36.5" x2="-103.25" y2="-42.4" width="0" layer="19" extent="16-16"/>
@@
 <wire x1="79.3" y1="-11.33" x2="-54.55" y2="-33.8" width="0" layer="19" extent="16-16"/>
 </signal>
-<signal name="N$28">
+<signal name="+200VDC_OUT">
 <contactref element="X2" pad="1"/>
 <contactref element="D7" pad="CATHODE"/>
 <contactref element="C4" pad="PLUS"/>
 <contactref element="D8" pad="CATHODE"/>
-<wire x1="38.21" y1="-55.5" x2="84.3" y2="-11.33" width="0" layer="19" extent="1-1"/>
-<wire x1="32.18" y1="-77.2" x2="38.21" y2="-55.5" width="0" layer="19" extent="1-1"/>
-<wire x1="31.98" y1="-84" x2="32.18" y2="-77.2" width="0" layer="19" extent="1-1"/>
+<contactref element="R19" pad="PAD_1"/>
+<wire x1="31.98" y1="-84" x2="-111.45" y2="-124.5" width="0" layer="19" extent="1-1"/>
+<wire x1="32.18" y1="-77.2" x2="31.98" y2="-84" width="0" layer="19" extent="1-1"/>
+<wire x1="38.21" y1="-55.5" x2="32.18" y2="-77.2" width="0" layer="19" extent="1-1"/>
+<wire x1="84.3" y1="-11.33" x2="38.21" y2="-55.5" width="0" layer="19" extent="1-1"/>
 </signal>
 <signal name="+12V_CONTROL">
@@
 <contactref element="C9" pad="PAD_1"/>
 <contactref element="R5" pad="PAD_0"/>
+<contactref element="C8" pad="PAD_1"/>
+<contactref element="ZD2" pad="CATHODE"/>
 <contactref element="R6" pad="PAD_0"/>
-<contactref element="C8" pad="PAD_1"/>
+<wire x1="-52.45" y1="-36.9" x2="-107.725" y2="-121.4" width="0" layer="19" extent="1-16"/>
 <wire x1="-52.45" y1="-33.8" x2="-52.45" y2="-36.9" width="0" layer="19" extent="16-16"/>
 <wire x1="-54.55" y1="-30.7" x2="-52.45" y2="-33.8" width="0" layer="19" extent="16-16"/>
 <wire x1="-54.55" y1="-27.6" x2="-54.55" y2="-30.7" width="0" layer="19" extent="16-16"/>
 <wire x1="-71.80125" y1="-13.755" x2="-54.55" y2="-27.6" width="0" layer="19" extent="16-16"/>
-</signal>
-<signal name="N$8">
-<contactref element="R6" pad="PAD_1"/>
-<contactref element="ZD1" pad="ANODE"/>
-<wire x1="-54.55" y1="-36.9" x2="-56.175" y2="-40" width="0" layer="19" extent="16-16"/>
-</signal>
-<signal name="N$9">
-<contactref element="ZD1" pad="CATHODE"/>
 </signal>
 <signal name="N$12">
@@
 <wire x1="69.9" y1="-99" x2="-52.425" y2="-61.7" width="0" layer="19" extent="16-16"/>
 </signal>
+<signal name="N$1">
+<contactref element="R6" pad="PAD_1"/>
+<contactref element="R19" pad="PAD_0"/>
+<wire x1="-54.55" y1="-36.9" x2="-109.35" y2="-124.5" width="0" layer="19" extent="1-16"/>
+</signal>
 </signals>

Commit message: 12 to 200V converter v2. Routed.
Parts:
- C2: device __MyCommonLib1:CE_16MM -> __MyCommonLib1:CE_12.5MM
- C5: device __MyCommonLib1:RSMD_1206 -> __MyCommonLib1:RSMD_0805
- C6: device __MyCommonLib1:CE_8.2MM -> __MyCommonLib1:CE_6.3MM
- R15: device __MyCommonLib1:RSMD_1206 -> __MyCommonLib1:RSMD_2512
- moved ZD2 232.1 mm to (59.9, 37.1), turned to 270 degrees
- moved R19 224.8 mm to (45.7, 37.2)
- moved R12 165.9 mm to (54.7, 4.80)
- moved T3 165.0 mm to (54.6, 8.30), turned to 270 degrees
- moved D2 162.7 mm to (50.8, 7.60), turned to 270 degrees
- moved T4 156.7 mm to (37.3, 10.6), turned to 180 degrees
- moved D6 155.4 mm to (33.4, 10.7), turned to 90 degrees
- moved U1 150.3 mm to (68.3, 28.6)
- moved R16 144.8 mm to (63.9, 38.6), turned to 180 degrees
- moved D11 143.1 mm to (11.6, 47.7), turned to 90 degrees
- moved R18 141.6 mm to (62.0, 29.6), turned to 270 degrees
- moved C5 141.6 mm to (56.3, 27.5), turned to 90 degrees
- moved R11 141.4 mm to (63.9, 35.8), turned to 180 degrees
- moved D3 141.0 mm to (51.9, 31.0), turned to 90 degrees
- moved R4 140.4 mm to (74.9, 32.3), turned to 180 degrees
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Connections:
- net GND: now also R15.PAD1; no longer R15.PAD_1
- net I_OUT_SENSE: now also R15.PAD0; no longer R15.PAD_0
Routing:
- net GND: track 7.83 -> 84.2 mm, vias 0 -> 6
- net PWM2: track 0.00 -> 46.9 mm, vias 0 -> 2
- net I_OUT_SENSE: track 0.00 -> 43.4 mm
- net +12V_CONTROL: track 0.00 -> 34.5 mm, vias 0 -> 2
- net +200VDC_OUT: track 0.00 -> 33.7 mm
- net PWM1: track 0.00 -> 30.3 mm
- net N$7: track 0.00 -> 28.0 mm
- net N$18: track 0.00 -> 18.6 mm
- net +12V_POWER: track 0.00 -> 16.4 mm, vias 0 -> 2
- net N$4: track 0.00 -> 13.3 mm
- net N$6: track 0.00 -> 13.0 mm
- net V_REF: track 0.00 -> 10.2 mm
- net N$5: track 0.00 -> 8.61 mm
- net N$13: track 0.00 -> 8.49 mm
- net N$12: track 0.00 -> 7.52 mm
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- added copper zone on layer 16, net +12V_CONTROL
- added copper zone on layer 16, net +200VDC_OUT
- added copper zone on layer 16, net I_OUT_SENSE
- added copper zone on layer 16, net N$20
- added copper zone on layer 16, net N$23
- added copper zone on layer 16, net N$24
- added copper zone on layer 16, net N$25
Other:
- board size 91 x 50 mm -> 80 x 55 mm
