File: 12_to_200V_inverter/schematic/12to220inverterVer2.sch (EAGLE design)
At the start: 37 parts, among them IC10 MC34063, T11 BC857, T15 IRL5602S, T16 BC847, T17 IRF830, X1 +12V_INPUT, X2 200VDC_OUTPUT, X3 TURN_ON

Commit message: 12 to 200V converter v2. Forward 2 conversion.
Parts:
- removed C53: 1000uFx16V, __MyCommonLib1:CE16MM
- removed C54: 0.47uFx16V, __MyCommonLib1:CSMD_1206
- removed C55: 1n0*, __MyCommonLib1:CSMD_0805
- removed C57: 20uF x 450V, __MyCommonLib1:CE16MM
- removed D10: UF4001, __MyCommonLib1:1N4001DO-41_15MM
- removed D29: UF4007, __MyCommonLib1:1N4001DO-41_10MM
- removed D4, D5: LL4148, __MyCommonLib1:LL4147SOD-80
- removed IC10: MC34063, __MyCommonLib1:MC34063(DIP8)
- removed R83: 0.1R, __MyCommonLib1:RSMD_2512
- removed R84: 130K*, __MyCommonLib1:RSMD_1206
- removed R85: 1K6, __MyCommonLib1:RSMD_0805
- removed T11: BC857, __MyCommonLib1:BC857SOT23_SMALL_PADS
- removed T17: IRF830, __MyCommonLib1:IRF830TO-220
- removed TR2: test_ring, __MyCommonLib1:TRANS_2WIND(RING_25X10)
- removed ZD2: 10V, __MyCommonLib1:ZENNER(SOD_80)
- added C10: 12uF x 10V, __MyCommonLib1:CSMD_0805
- added C11: 100uF x 25V, __MyCommonLib1:CE5.2MM
- added C3: 10nF x 50V, __MyCommonLib1:CSMD_1206
- added C4: 20uF x 450V, __MyCommonLib1:CE16MM
- added C5, C7: 0.47uFx16V, __MyCommonLib1:CSMD_1206
- added C6: 100uF x 16V, __MyCommonLib1:CE8.2MM
- added C8: 2.2uF x 10V, __MyCommonLib1:CSMD_0805
- added C9: 5.5uF, __MyCommonLib1:CSMD_0805
- added D11, D7, D8, D9: UF4007, __MyCommonLib1:1N4001DO-41_10MM
- added D2, D6: LL4148, __MyCommonLib1:LL4147SOD-80
- added R12, R13: 4K7, __MyCommonLib1:RSMD_0805
- added R14, R15: 5R1, __MyCommonLib1:RSMD_1206
- added R16: 22K, __MyCommonLib1:RSMD_0805
- added R17: 33K, __MyCommonLib1:RSMD_0805
- added R18: 47K, __MyCommonLib1:RSMD_0805
- added T1, T2: IRF830, __MyCommonLib1:IRF830TO-220
- added T3, T4: BC857, __MyCommonLib1:BC857SOT23_SMALL_PADS
- added TR3: 12_to_200_trans, __MyCommonLib1:TRANS_38X30MM
- added U1: TL494, __MyCommonLib1:TL494(SOIC-16)
- C1: value 0.1uF x 50V -> 4n7 x 16V; device __MyCommonLib1:CSMD_1206 -> __MyCommonLib1:CSMD_0805
- C2: value * -> 1000uF x 16V; device __MyCommonLib1:CSMD_1206 -> __MyCommonLib1:CE16MM
- R1: value 10R -> 3K3; device __MyCommonLib1:RSMD_1206_BIG_GAP -> __MyCommonLib1:RSMD_0805
- R11: value * -> 7K5; device __MyCommonLib1:RSMD_1206 -> __MyCommonLib1:RSMD_0805
- R2: value 240R -> 33R; device __MyCommonLib1:RSMD_1206_BIG_GAP -> __MyCommonLib1:RSMD_0805
- R3: value 240R -> 39K; device __MyCommonLib1:RSMD_1206_BIG_GAP -> __MyCommonLib1:RSMD_0805
- R4: value 20R -> 1K2
- R5: value * -> 47K; device __MyCommonLib1:RSMD_1206 -> __MyCommonLib1:RSMD_0805
- R6: value 130K* -> 15K; device __MyCommonLib1:RSMD_1206 -> __MyCommonLib1:RSMD_0805
- ZD1: value 10V -> *
Connections:
- removed net +12V: C53.PLUS, C54.PIN1, D5.CATHODE, IC10.VCC, R83.PIN0, T15.DRAIN
- removed net +200V: C57.PLUS, D29.CATHODE, R11.PIN0, R6.PIN0, X2-1.KL
- removed net N$1: D10.ANODE, T17.DRAIN, TR2.PRI_START
- removed net N$10: C1.PIN1, IC10.DR_C, IC10.I_PEAK, IC10.SW_C, R5.PIN1, R83.PIN1, TR2.PRI_END, ZD2.ANODE
- removed net N$11: C2.PIN1, D29.ANODE, TR2.SEC_START
- removed net N$135: C55.PIN1, IC10.CT
- removed net N$139: IC10.INV_IN, R84.PIN0, R85.PIN1
- new net +12V_CONTROL: C11.PLUS, C5.PIN1, C6.PLUS, R18.PIN1, R2.PIN1, T15.DRAIN, U1.VCC
- new net +12V_POWER: C2.PLUS, C7.PIN1, R7.PIN1, T15.SOURCE, TR3.SEC1_END, TR3.SEC2_START, X1-1.KL
- new net I_OUT_SENSE: R15.PIN0, R5.PIN1, X2-2.KL
- new net N$19: D2.CATHODE, T2.GATE, T3.E
- new net N$20: D11.CATHODE, D7.ANODE, TR3.PRI_START
- new net N$21: D6.CATHODE, T1.GATE, T4.E
- new net N$23: D8.ANODE, D9.CATHODE, TR3.PRI_END
- new net N$24: C3.PIN1, T2.DRAIN, TR3.SEC1_START
- new net N$25: R14.PIN0, T1.DRAIN, TR3.SEC2_END
- new net N$26: C3.PIN0, R14.PIN1
- new net N$28: C4.PLUS, D7.CATHODE, D8.CATHODE, X2-1.KL
- new net PWM1: D2.ANODE, R12.PIN1, T3.B, U1.E1
- new net PWM2: D6.ANODE, R13.PIN1, T4.B, U1.E2
- new net V_REF: R11.PIN1, R3.PIN1, U1.OUT_CTRL, U1.REF
- net GND: now also C1.PIN1, C10.PIN0, C2.MINUS, C4.MINUS, C5.PIN0, C6.MINUS, C7.PIN0, C9.PIN0, D11.ANODE, D3.ANODE, D9.ANODE, R1.PIN0, R12.PIN0, R13.PIN0, R15.PIN1, R17.PIN1, R4.PIN1, T1.SOURCE, T2.SOURCE, T3.C, T4.C, U1.DTC, U1.GND; no longer C53.MINUS, C54.PIN0, C55.PIN0, C57.MINUS, D4.ANODE, IC10.GND, R1.PIN1, R3.PIN1, R85.PIN0, T17.SOURCE, TR2.SEC_END, X2-2.KL
- net N$12: now also R11.PIN0, R16.PIN0, U1.2IN+; no longer ZD1.ANODE, ZD2.CATHODE
- net N$13: now also C11.MINUS, D1.ANODE, D3.CATHODE; no longer R7.PIN1, T15.SOURCE, X1-1.KL
- net N$18: now also C10.PIN1, D1.CATHODE, R17.PIN0, R18.PIN0, U1.2IN-; no longer C2.PIN0, R11.PIN1
- net N$2: now also C1.PIN0, U1.CT; no longer R1.PIN0, T11.C
- net N$3: now also R1.PIN1, U1.RT; no longer R6.PIN1, R84.PIN1
- net N$4: now also U1.C1, U1.C2; no longer D3.CATHODE, T11.B
- net N$5: now also R4.PIN0, U1.1IN-; no longer R2.PIN1
- net N$6: now also C8.PIN0, R16.PIN1, U1.FEEDBACK; no longer D1.ANODE, D3.ANODE, IC10.SW_E
- net N$7: now also C8.PIN1, C9.PIN1, R5.PIN0, R6.PIN0, U1.1IN+; no longer D1.CATHODE, D4.CATHODE, D5.ANODE, R4.PIN0, T11.E
- net N$8: now also R6.PIN1, ZD1.ANODE; no longer R4.PIN1, T17.GATE
- net N$9: no longer C1.PIN0, D10.CATHODE, R5.PIN0
Other:
- moved on the sheet: C1, D1, D3, R1, R10, R11, R2, R3, R4, R5, R6, R7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

Commit message: 12 to 200V converter v2. Schematic done.
Parts:
- removed ZD1: *, __MyCommonLib1:ZENNER(SOD_80)
- added R19: 680K, __MyCommonLib1:RSMD_0805
- added ZD2: 4.7V, __MyCommonLib1:ZENNER(SOD_80)
- R5: value 47K -> 1K0
- R6: value 15K -> 680K
Connections:
- removed net N$28: C4.PLUS, D7.CATHODE, D8.CATHODE, X2-1.KL
- removed net N$8: R6.PIN1, ZD1.ANODE
- removed net N$9: ZD1.CATHODE
- new net +200VDC_OUT: C4.PLUS, D7.CATHODE, D8.CATHODE, R19.PIN1, X2-1.KL
- new net N$1: R19.PIN0, R6.PIN1
- net GND: now also ZD2.ANODE
- net N$7: now also ZD2.CATHODE
Other:
- moved on the sheet: R6
Changed lines of the file:
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@@
 <part name="C9" library="__MyCommonLib1" deviceset="C" device="SMD_0805" value="5.5uF"/>
 <part name="GND10" library="supply1" deviceset="GND" device=""/>
-<part name="R5" library="__MyCommonLib1" deviceset="R" device="SMD_0805" value="47K"/>
-<part name="R6" library="__MyCommonLib1" deviceset="R" device="SMD_0805" value="15K"/>
-<part name="ZD1" library="__MyCommonLib1" deviceset="ZENNER" device="(SOD_80)" value="*"/>
+<part name="R5" library="__MyCommonLib1" deviceset="R" device="SMD_0805" value="1K0"/>
+<part name="R6" library="__MyCommonLib1" deviceset="R" device="SMD_0805" value="680K"/>
 <part name="R11" library="__MyCommonLib1" deviceset="R" device="SMD_0805" value="7K5"/>
 <part name="R16" library="__MyCommonLib1" deviceset="R" device="SMD_0805" value="22K"/>
@@
 <part name="C11" library="__MyCommonLib1" deviceset="CE" device="5.2MM" value="100uF x 25V"/>
 <part name="GND24" library="supply1" deviceset="GND" device=""/>
+<part name="ZD2" library="__MyCommonLib1" deviceset="ZENNER" device="(SOD_80)" value="4.7V"/>
+<part name="R19" library="__MyCommonLib1" deviceset="R" device="SMD_0805" value="680K"/>
+<part name="GND25" library="supply1" deviceset="GND" device=""/>
 </parts>
 <sheets>
@@
 <attribute name="VALUE" x="35.56" y="119.38" size="1.27" layer="96" font="vector" ratio="20" rot="R90"/>
 </instance>
-<instance part="R6" gate="R$1" x="35.56" y="124.46" smashed="yes" rot="R90">
-<attribute name="NAME" x="38.1" y="129.54" size="1.27" layer="95" font="vector" ratio="20" rot="R180"/>
-<attribute name="VALUE" x="38.1" y="127" size="1.27" layer="96" font="vector" ratio="20" rot="R180"/>
-</instance>
-<instance part="ZD1" gate="G$1" x="27.94" y="129.54"/>
+<instance part="R6" gate="R$1" x="45.72" y="137.16" smashed="yes">
+<attribute name="NAME" x="50.8" y="134.62" size="1.27" layer="95" font="vector" ratio="20" rot="R90"/>
+<attribute name="VALUE" x="48.26" y="134.62" size="1.27" layer="96" font="vector" ratio="20" rot="R90"/>
+</instance>
 <instance part="R11" gate="R$1" x="71.12" y="106.68" smashed="yes" rot="R90">
 <attribute name="NAME" x="71.12" y="109.22" size="1.27" layer="95" font="vector" ratio="20" rot="R180"/>
@@
 <instance part="GND24" gate="1" x="109.22" y="93.98" smashed="yes" rot="R90">
 <attribute name="VALUE" x="114.3" y="91.44" size="1.27" layer="96" font="vector" ratio="20" rot="R90"/>
+</instance>
+<instance part="ZD2" gate="G$1" x="40.64" y="129.54" smashed="yes" rot="R270">
+<attribute name="NAME" x="38.1" y="133.35" size="1.27" layer="95" font="vector" ratio="20"/>
+<attribute name="VALUE" x="38.1" y="132.08" size="1.27" layer="96" font="vector" ratio="20"/>
+</instance>
+<instance part="R19" gate="R$1" x="45.72" y="149.86" smashed="yes">
+<attribute name="NAME" x="50.8" y="147.32" size="1.27" layer="95" font="vector" ratio="20" rot="R90"/>
+<attribute name="VALUE" x="48.26" y="147.32" size="1.27" layer="96" font="vector" ratio="20" rot="R90"/>
+</instance>
+<instance part="GND25" gate="1" x="33.02" y="129.54" smashed="yes" rot="R270">
+<attribute name="VALUE" x="27.94" y="132.08" size="1.27" layer="96" font="vector" ratio="20" rot="R270"/>
 </instance>
 </instances>
@@
 <pinref part="GND24" gate="1" pin="GND"/>
 <wire x1="106.68" y1="93.98" x2="104.14" y2="93.98" width="0.1524" layer="91"/>
+</segment>
+<segment>
+<pinref part="ZD2" gate="G$1" pin="ANODE"/>
+<pinref part="GND25" gate="1" pin="GND"/>
+<wire x1="35.56" y1="129.54" x2="38.1" y2="129.54" width="0.1524" layer="91"/>
 </segment>
 </net>
@@
 </segment>
 </net>
-<net name="N$28" class="0">
+<net name="+200VDC_OUT" class="0">
 <segment>
 <pinref part="X2" gate="-1" pin="KL"/>
@@
 <wire x1="213.36" y1="129.54" x2="213.36" y2="111.76" width="0.1524" layer="91"/>
 <junction x="213.36" y="111.76"/>
+<label x="223.52" y="132.08" size="1.27" layer="95" font="vector" ratio="20" rot="R180"/>
+</segment>
+<segment>
+<pinref part="R19" gate="R$1" pin="PIN1"/>
+<wire x1="45.72" y1="154.94" x2="45.72" y2="157.48" width="0.1524" layer="91"/>
+<wire x1="45.72" y1="157.48" x2="55.88" y2="157.48" width="0.1524" layer="91"/>
+<label x="55.88" y="160.02" size="1.27" layer="95" font="vector" ratio="20" rot="R180"/>
 </segment>
 </net>
@@
 <wire x1="45.72" y1="114.3" x2="45.72" y2="109.22" width="0.1524" layer="91"/>
 <wire x1="45.72" y1="114.3" x2="45.72" y2="116.84" width="0.1524" layer="91"/>
-<wire x1="45.72" y1="116.84" x2="45.72" y2="124.46" width="0.1524" layer="91"/>
-<wire x1="45.72" y1="124.46" x2="40.64" y2="124.46" width="0.1524" layer="91"/>
+<wire x1="45.72" y1="116.84" x2="45.72" y2="129.54" width="0.1524" layer="91"/>
 <wire x1="45.72" y1="116.84" x2="40.64" y2="116.84" width="0.1524" layer="91"/>
 <pinref part="R5" gate="R$1" pin="PIN0"/>
-<pinref part="R6" gate="R$1" pin="PIN0"/>
 <junction x="45.72" y="116.84"/>
 <junction x="45.72" y="114.3"/>
@@
 <wire x1="50.8" y1="109.22" x2="50.8" y2="114.3" width="0.1524" layer="91"/>
 <junction x="50.8" y="114.3"/>
-</segment>
-</net>
-<net name="N$8" class="0">
-<segment>
-<pinref part="R6" gate="R$1" pin="PIN1"/>
-<pinref part="ZD1" gate="G$1" pin="ANODE"/>
-<wire x1="30.48" y1="124.46" x2="27.94" y2="124.46" width="0.1524" layer="91"/>
-<wire x1="27.94" y1="124.46" x2="27.94" y2="127" width="0.1524" layer="91"/>
-</segment>
-</net>
-<net name="N$9" class="0">
-<segment>
-<pinref part="ZD1" gate="G$1" pin="CATHODE"/>
-<wire x1="27.94" y1="132.08" x2="27.94" y2="139.7" width="0.1524" layer="91"/>
+<pinref part="ZD2" gate="G$1" pin="CATHODE"/>
+<wire x1="43.18" y1="129.54" x2="45.72" y2="129.54" width="0.1524" layer="91"/>
+<pinref part="R6" gate="R$1" pin="PIN0"/>
+<wire x1="45.72" y1="132.08" x2="45.72" y2="129.54" width="0.1524" layer="91"/>
+<junction x="45.72" y="129.54"/>
 </segment>
 </net>
@@
 </segment>
 </net>
+<net name="N$1" class="0">
+<segment>
+<pinref part="R6" gate="R$1" pin="PIN1"/>
+<pinref part="R19" gate="R$1" pin="PIN0"/>
+<wire x1="45.72" y1="144.78" x2="45.72" y2="142.24" width="0.1524" layer="91"/>
+</segment>
+</net>

Commit message: 12 to 200V converter v2. Routed.
Parts:
- C2: device __MyCommonLib1:CE16MM -> __MyCommonLib1:CE12.5MM
- C5: device __MyCommonLib1:CSMD_1206 -> __MyCommonLib1:CSMD_0805
- C6: device __MyCommonLib1:CE8.2MM -> __MyCommonLib1:CE6.3MM
- R15: device __MyCommonLib1:RSMD_1206 -> __MyCommonLib1:RSMD_2512
Changed lines of the file:
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@@
 <part name="D11" library="__MyCommonLib1" deviceset="1N4001" device="DO-41_10MM" value="UF4007"/>
 <part name="GND19" library="supply1" deviceset="GND" device=""/>
-<part name="R15" library="__MyCommonLib1" deviceset="R" device="SMD_1206" value="5R1"/>
-<part name="C5" library="__MyCommonLib1" deviceset="C" device="SMD_1206" value="0.47uFx16V"/>
-<part name="C6" library="__MyCommonLib1" deviceset="CE" device="8.2MM" value="100uF x 16V"/>
+<part name="R15" library="__MyCommonLib1" deviceset="R" device="SMD_2512" value="5R1"/>
+<part name="C5" library="__MyCommonLib1" deviceset="C" device="SMD_0805" value="0.47uFx16V"/>
+<part name="C6" library="__MyCommonLib1" deviceset="CE" device="6.3MM" value="100uF x 16V"/>
 <part name="GND20" library="supply1" deviceset="GND" device=""/>
 <part name="GND21" library="supply1" deviceset="GND" device=""/>
-<part name="C2" library="__MyCommonLib1" deviceset="CE" device="16MM" value="1000uF x 16V"/>
+<part name="C2" library="__MyCommonLib1" deviceset="CE" device="12.5MM" value="1000uF x 16V"/>
 <part name="C7" library="__MyCommonLib1" deviceset="C" device="SMD_1206" value="0.47uFx16V"/>
 <part name="GND1" library="supply1" deviceset="GND" device=""/>
@@
 <wire x1="114.3" y1="144.78" x2="114.3" y2="147.32" width="0.1524" layer="91"/>
 <wire x1="114.3" y1="147.32" x2="127" y2="147.32" width="0.1524" layer="91"/>
-<label x="106.68" y="149.86" size="1.27" layer="95" font="vector" ratio="20" rot="R180"/>
-</segment>
-<segment>
+<label x="127" y="149.86" size="1.27" layer="95" font="vector" ratio="20" rot="R180"/>
+</segment>
+<segment>
