File: 12_to_200V_inverter/schematic/12to220inverterVer2_to_print.brd (EAGLE design)
At the start: 80 x 55 mm, 50 parts, among them T1 IRF830, T15 IRL5602S, T16 BC847, T2 IRF830, T3 BC857, T4 BC857, U1 TL494, X1 +12V_INPUT, X2 200VDC_OUTPUT, X3 TURN_ON

Commit message: 12 to 200VDC converter. Ver3. Converter schematic done. Add overcurrent/overvoltage protection.
Parts:
- R15: device __MyCommonLib1:RSMD_1206 -> __MyCommonLib1:RSMD_2512
- moved R15 1.91 mm to (17.2, 10.9)
- moved R7 1.80 mm to (63.2, 51.8)
- moved C11 1.60 mm to (51.5, 24.3)
- moved C1 1.50 mm to (74.9, 29.5)
- moved R4 1.42 mm to (74.9, 32.3), turned to 180 degrees
- moved R1 1.40 mm to (74.9, 26.8)
- moved R8 1.30 mm to (66.4, 51.8)
- moved D6 0.50 mm to (33.4, 10.7)
- moved T15 0.50 mm to (47.3, 48.3)
- moved R9 0.20 mm to (70.4, 47.4)
- moved C5 0.10 mm to (56.3, 27.5)
- moved C10 0.10 mm to (54.8, 31.7)
Connections:
- net GND: now also R15.PAD1; no longer R15.PAD_1
- net I_OUT_SENSE: now also R15.PAD0; no longer R15.PAD_0
Routing:
- net GND: track 203.6 -> 80.9 mm, vias 4 -> 6
- net +12V_POWER: track 63.5 -> 16.4 mm
- net N$23: track 27.6 -> 0.00 mm
- net N$20: track 24.7 -> 0.00 mm
- net +200VDC_OUT: track 51.5 -> 28.9 mm
- net N$25: track 16.6 -> 0.00 mm
- net N$24: track 14.6 -> 0.00 mm
- net I_OUT_SENSE: track 57.4 -> 43.4 mm
- net N$14: track 0.00 -> 9.68 mm
- net +12V_CONTROL: track 27.0 -> 34.5 mm
- net N$16: track 0.00 -> 5.22 mm
- net N$17: track 0.00 -> 4.17 mm
- net N$26: track 0.00 -> 4.00 mm
- net N$5: track 11.3 -> 8.61 mm
- net N$15: track 0.00 -> 2.12 mm
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- added copper zone on layer 16, net +12V_CONTROL
- added copper zone on layer 16, net +12V_POWER
- added copper zone on layer 16, net +200VDC_OUT
- added copper zone on layer 16, net GND
- added copper zone on layer 16, net I_OUT_SENSE
- added copper zone on layer 16, net N$15
- added copper zone on layer 16, net N$20
- added copper zone on layer 16, net N$23
- added copper zone on layer 16, net N$24
- added copper zone on layer 16, net N$25
