File: 12_to_200V_inverter/schematic/12to220inverterVer3.brd (EAGLE design)
At the start: 80 x 55 mm, 50 parts, among them T1 IRF830, T15 IRL5602S, T16 BC847, T2 IRF830, T3 BC857, T4 BC857, U1 TL494, X1 +12V_INPUT, X2 200VDC_OUTPUT, X3 TURN_ON

Commit message: 12 to 200VDC converter. Ver3. Converter schematic done. Add overcurrent/overvoltage protection.
Parts:
- removed C10: 12uF x 10V, __MyCommonLib1:RSMD_0805
- removed C11: 100uF x 25V, __MyCommonLib1:CE_5.2MM
- removed D11, D7, D8: UF4007, __MyCommonLib1:DO-41_10MM
- added C12: 20uF x 450V, __MyCommonLib1:CE_13MM
- added D4: UF4007, __MyCommonLib1:DO-41_10MM
- added R20: 10K, __MyCommonLib1:RSMD_0805
- added R21: 150R, __MyCommonLib1:RSMD_0805
- added R22: 1M0, __MyCommonLib1:RSMD_0805
- added R23: 51K, __MyCommonLib1:RSMD_0805
- C1: value 4n7 x 16V -> 4n3 x 16V
- C2: value 1000uF x 16V -> 1000uFx25V; device __MyCommonLib1:CE_12.5MM -> __MyCommonLib1:CE_10MM
- C3: value 10nF x 50V -> 2.2nF x 50V
- C4: device __MyCommonLib1:CE_16MM -> __MyCommonLib1:CE_13MM
- C5, C7: value 0.47uFx16V -> 0.47uFx25V
- C6: value 100uF x 16V -> 100uFx25V
- C8: value 2.2uF x 10V -> 47uF x 10V; device __MyCommonLib1:RSMD_0805 -> __MyCommonLib1:CE_5.2MM
- C9: value 5.5uF -> 0.1uF x 10V
- D1: value LL4148 -> 1N4001; device __MyCommonLib1:SOD-80 -> __MyCommonLib1:DO-41_10MM
- D3: value LL4148 -> MBR0540
- R11: value 7K5 -> 56K
- R14: value 5R1 -> 20R
- R15: value 5R1 -> 1R0; device __MyCommonLib1:RSMD_1206 -> __MyCommonLib1:R_1.0W_VERTICAL
- R16: value 22K -> 160K
- R17: value 33K -> 51K
- R18: value 47K -> 51K
- R19, R6: value 680K -> 510K; device __MyCommonLib1:RSMD_0805 -> __MyCommonLib1:RSMD_1206
- R3: value 39K -> 160K
- R4: value 1K2 -> 10K
- R5: value 1K0 -> 4K7
- R7: value 4K7 -> 10K
- R8: value 4K7 -> 1K0
- T1, T2: value IRF830 -> IRFZ24N
- moved C9 107.0 mm to (-19.0, -39.2), flipped to the top, turned to 0 degrees
- moved C8 103.3 mm to (-18.0, -18.4), flipped to the top, turned to 0 degrees
- moved D3 94.9 mm to (-18.2, -33.0), flipped to the top, turned to 0 degrees
- moved R6 77.3 mm to (-10.3, -10.9), flipped to the top
- moved R19 76.1 mm to (-10.3, -14.4), flipped to the top
- moved D1 75.9 mm to (-6.90, -20.4), flipped to the top, turned to 0 degrees
- moved R15 1.91 mm to (17.2, 10.9)
- moved R7 1.80 mm to (63.2, 51.8)
- moved C1 1.50 mm to (74.9, 29.5)
- moved R4 1.42 mm to (74.9, 32.3), turned to 180 degrees
- moved R1 1.40 mm to (74.9, 26.8)
- moved R8 1.30 mm to (66.4, 51.8)
- moved D6 0.50 mm to (33.4, 10.7)
- moved T15 0.50 mm to (47.3, 48.3)
- moved R9 0.20 mm to (70.4, 47.4)
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Connections:
- removed net +12V_POWER: C2.PLUS, C7.PAD_1, R7.PAD_1, T15.3, TR3.4, TR3.5, X1.1
- removed net I_OUT_SENSE: R15.PAD_0, R5.PAD_1, X2.2
- removed net N$13: C11.MINUS, D1.ANODE, D3.CATHODE
- removed net N$20: D11.CATHODE, D7.ANODE, TR3.9
- removed net N$23: D8.ANODE, D9.CATHODE, TR3.10
- new net +12V_BAT: C2.PLUS, C7.PAD_1, D1.ANODE, TR3.4, TR3.5, X1.1
- new net +200VDC_I_SENSE: D3.ANODE, R15.PAD_0, R5.PAD_1, X2.2
- new net FEEDBACK: R16.PAD_1, R22.PAD_1, U1.3
- new net N$10: C4.PLUS, D4.ANODE, D9.CATHODE
- new net N$11: D3.CATHODE, R21.PAD_1
- new net N$8: C4.MINUS, TR3.10
- new net N$9: D1.CATHODE, R7.PAD_1, T15.3
- net +12V_CONTROL: now also R11.PAD_1; no longer C11.PLUS, R18.PAD_1
- net +200VDC_OUT: now also C12.PLUS, D4.CATHODE, R6.PAD_1; no longer C4.PLUS, D7.CATHODE, D8.CATHODE, R19.PAD_1
- net GND: now also C12.MINUS, C8.MINUS, C9.PAD_1, R15.PAD1, R19.PAD_0, R20.PAD_1, TR3.9; no longer C10.PAD_0, C4.MINUS, C9.PAD_0, D11.ANODE, D3.ANODE, R15.PAD_1
- net N$1: now also R19.PAD_1, R6.PAD_0; no longer R19.PAD_0, R6.PAD_1
- net N$12: now also R20.PAD_0
- net N$18: no longer C10.PAD_1, D1.CATHODE
- net N$6: now also R22.PAD_0, R23.PAD_1, U1.1; no longer C8.PAD_0, R16.PAD_1, U1.3
- net N$7: now also C8.PLUS, C9.PAD_0, R21.PAD_0, R23.PAD_0; no longer C8.PAD_1, C9.PAD_1, R6.PAD_0, U1.1
- net V_REF: now also R18.PAD_1; no longer R11.PAD_1
Routing:
- net GND: track 203.6 -> 73.7 mm, vias 4 -> 6
- net +12V_POWER: track 63.5 -> 0.00 mm, vias 2 -> 0
- net I_OUT_SENSE: track 57.4 -> 0.00 mm
- net +200VDC_OUT: track 51.5 -> 0.00 mm
- net +200VDC_I_SENSE: track 0.00 -> 43.4 mm
- net N$23: track 27.6 -> 0.00 mm
- net N$20: track 24.7 -> 0.00 mm
- net N$25: track 16.6 -> 0.00 mm
- net N$24: track 14.6 -> 0.00 mm
- net N$7: track 28.6 -> 16.5 mm
- net N$18: track 19.1 -> 7.17 mm
- net +12V_BAT: track 0.00 -> 11.9 mm, vias 0 -> 2
- net FEEDBACK: track 0.00 -> 10.1 mm
- net N$14: track 0.00 -> 9.68 mm
- net N$6: track 13.8 -> 6.48 mm
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- added copper zone on layer 16, net +12V_BAT
- added copper zone on layer 16, net +12V_CONTROL
- added copper zone on layer 16, net +200VDC_I_SENSE
- added copper zone on layer 16, net +200VDC_OUT
- added copper zone on layer 16, net GND
- added copper zone on layer 16, net N$15
- added copper zone on layer 16, net N$20
- added copper zone on layer 16, net N$23
- added copper zone on layer 16, net N$24
- added copper zone on layer 16, net N$25

Commit message: 12 to 200VDC converter. Ver3. Start with battery charger.
Parts:
- added U$1: TRANS_FLYBACK_AUX_SINGLE_OUT(TRANS29.5X23), __MyCommonLib1:TRANS_29.5X23_1234567_910
- added U$2: TRANS_FLYBACK_AUX_SINGLE_OUT(TRANS_37X26), __MyCommonLib1:TRANS_37X26_3578_11_13_15_17
- added U$3: TRANS_FLYBACK_AUX_SINGLE_OUT_WITH_SHIELD(TIO20-V2), __MyCommonLib1:TIO20_V2
Connections:
- new net N$13: U$1.1, U$2.3, U$3.1
- new net N$20: U$1.2, U$2.5, U$3.2
- new net N$22: U$1.10, U$2.17, U$3.10
- new net N$23: U$1.9, U$2.15, U$3.9
- new net N$27: U$1.5, U$2.8, U$3.5
- new net N$28: U$1.4, U$2.7, U$3.4
- new net N$29: U$1.7, U$2.13, U$3.7
- new net N$31: U$1.6, U$2.11, U$3.6
Changed lines of the file:
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@@
 <element name="R21" library="__MyCommonLib1" package="RSMD_0805" value="150R" x="-19" y="-36.1"/>
 <element name="C9" library="__MyCommonLib1" package="RSMD_0805" value="0.1uF x 10V" x="-19" y="-39.2"/>
+<element name="U$1" library="__MyCommonLib1" package="TRANS_29.5X23_1234567_910" value="TRANS_FLYBACK_AUX_SINGLE_OUT(TRANS29.5X23)" x="47.2" y="-76"/>
+<element name="U$2" library="__MyCommonLib1" package="TRANS_37X26_3578_11_13_15_17" value="TRANS_FLYBACK_AUX_SINGLE_OUT(TRANS_37X26)" x="46.2" y="-82.2"/>
+<element name="U$3" library="__MyCommonLib1" package="TIO20_V2" value="TRANS_FLYBACK_AUX_SINGLE_OUT_WITH_SHIELD(TIO20-V2)" x="47.2" y="-78.5"/>
 </elements>
 <signals>
@@
 <vertex x="11.2" y="53.9"/>
 </polygon>
+<contactref element="U$1" pad="2"/>
+<contactref element="U$2" pad="5"/>
+<contactref element="U$3" pad="2"/>
+<wire x1="46.2" y1="-92.2" x2="42.12" y2="-84.9" width="0" layer="19" extent="1-1"/>
 </signal>
 <signal name="N$23">
@@
 <vertex x="8.6" y="53.6"/>
 </polygon>
+<contactref element="U$1" pad="9"/>
+<contactref element="U$2" pad="15"/>
+<contactref element="U$3" pad="9"/>
+<wire x1="42.12" y1="-67.1" x2="42.12" y2="-72.1" width="0" layer="19" extent="1-1"/>
+<wire x1="42.2" y1="-72.2" x2="42.12" y2="-67.1" width="0" layer="19" extent="1-1"/>
 </signal>
 <signal name="+200VDC_OUT">
@@
 <wire x1="-20.075" y1="-33" x2="-17.95" y2="-36.1" width="0" layer="19" extent="1-1"/>
 </signal>
+<signal name="N$13">
+<contactref element="U$1" pad="1"/>
+<contactref element="U$2" pad="3"/>
+<contactref element="U$3" pad="1"/>
+<wire x1="38.2" y1="-92.2" x2="37.04" y2="-84.9" width="0" layer="19" extent="1-1"/>
+</signal>
+<signal name="N$22">
+<contactref element="U$1" pad="10"/>
+<contactref element="U$2" pad="17"/>
+<contactref element="U$3" pad="10"/>
+<wire x1="37.04" y1="-67.1" x2="37.04" y2="-72.1" width="0" layer="19" extent="1-1"/>
+<wire x1="34.2" y1="-72.2" x2="37.04" y2="-67.1" width="0" layer="19" extent="1-1"/>
+</signal>
+<signal name="N$27">
+<contactref element="U$1" pad="5"/>
+<contactref element="U$2" pad="8"/>
+<contactref element="U$3" pad="5"/>
+<wire x1="58.2" y1="-92.2" x2="57.36" y2="-84.9" width="0" layer="19" extent="1-1"/>
+</signal>
+<signal name="N$28">
+<contactref element="U$1" pad="4"/>
+<contactref element="U$2" pad="7"/>
+<contactref element="U$3" pad="4"/>
+<wire x1="54.2" y1="-92.2" x2="52.28" y2="-84.9" width="0" layer="19" extent="1-1"/>
+</signal>
+<signal name="N$29">
+<contactref element="U$3" pad="7"/>
+<contactref element="U$1" pad="7"/>
+<contactref element="U$2" pad="13"/>
+<wire x1="52.28" y1="-67.1" x2="52.28" y2="-72.1" width="0" layer="19" extent="1-1"/>
+<wire x1="50.2" y1="-72.2" x2="52.28" y2="-67.1" width="0" layer="19" extent="1-1"/>
+</signal>
+<signal name="N$31">
+<contactref element="U$2" pad="11"/>
+<contactref element="U$1" pad="6"/>
+<contactref element="U$3" pad="6"/>
+<wire x1="57.36" y1="-67.1" x2="57.36" y2="-72.1" width="0" layer="19" extent="1-1"/>
+<wire x1="58.2" y1="-72.2" x2="57.36" y2="-67.1" width="0" layer="19" extent="1-1"/>
+</signal>
 </signals>

Commit message: 12_to_200V inverter. Ver3 Start schematic.
Parts:
- removed U$1: TRANS_FLYBACK_AUX_SINGLE_OUT(TRANS29.5X23), __MyCommonLib1:TRANS_29.5X23_1234567_910
- removed U$2: TRANS_FLYBACK_AUX_SINGLE_OUT(TRANS_37X26), __MyCommonLib1:TRANS_37X26_3578_11_13_15_17
- removed U$3: TRANS_FLYBACK_AUX_SINGLE_OUT_WITH_SHIELD(TIO20-V2), __MyCommonLib1:TIO20_V2
- added C10, C101: 0.1uF x 275VAC X2, __MyCommonLib1:MKP_18X6
- added CE101: 22uF x 400V, __MyCommonLib1:CE_13MM
- added D101, D102, D103, D104: 1N4007, __MyCommonLib1:DO-41_10MM
- added D105: UF4007, __MyCommonLib1:DO-41_10MM
- added F1: 0.3A, __MyCommonLib1:FUSE_20X5.6MM
- added R101, R24: 240K, __MyCommonLib1:RSMD_0805
- added RT1: 5 Ohm, __MyCommonLib1:NTC_9.0X4.2
- added TR101: EMI, __MyCommonLib1:EMI_CM_21X17
- added TR102: Self made transformer. From TR8 sat reciever., __MyCommonLib1:TRANS_37X26_3578_11_13_15_17
- added X101: 220VAC, __MyCommonLib1:BRD_CONNECTOR_12X10.2
- added ZD101: P6KE200, __MyCommonLib1:DO-41_10MM
Connections:
- removed net N$20: U$1.2, U$2.5, U$3.2
- removed net N$23: U$1.9, U$2.15, U$3.9
- new net N$30: D101.ANODE, D103.CATHODE, RT1.PAD1
- new net N$32: CE101.PLUS, D101.CATHODE, D102.CATHODE, TR102.5, ZD101.ANODE
- new net N$33: CE101.MINUS, D103.ANODE, D104.ANODE
- new net N$34: TR102.15, TR102.3
- new net N$35: D105.ANODE, TR102.17
- new net N$36: D105.CATHODE, ZD101.CATHODE
- net N$13: now also F1.PAD1, X101.1; no longer U$1.1, U$2.3, U$3.1
- net N$22: now also C101.1, R24.PAD_0, TR101.W2_START, X101.2; no longer U$1.10, U$2.17, U$3.10
- net N$27: now also C101.2, F1.PAD_0, R101.PAD_1, TR101.W1_START; no longer U$1.5, U$2.8, U$3.5
- net N$28: now also C10.1, D102.ANODE, D104.CATHODE, TR101.W2_END; no longer U$1.4, U$2.7, U$3.4
- net N$29: now also C10.2, RT1.PAD_0, TR101.W1_END; no longer U$1.7, U$2.13, U$3.7
- net N$31: now also R101.PAD_0, R24.PAD_1; no longer U$1.6, U$2.11, U$3.6
Changed lines of the file:
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@@
 <element name="R21" library="__MyCommonLib1" package="RSMD_0805" value="150R" x="-19" y="-36.1"/>
 <element name="C9" library="__MyCommonLib1" package="RSMD_0805" value="0.1uF x 10V" x="-19" y="-39.2"/>
-<element name="U$1" library="__MyCommonLib1" package="TRANS_29.5X23_1234567_910" value="TRANS_FLYBACK_AUX_SINGLE_OUT(TRANS29.5X23)" x="47.2" y="-76"/>
-<element name="U$2" library="__MyCommonLib1" package="TRANS_37X26_3578_11_13_15_17" value="TRANS_FLYBACK_AUX_SINGLE_OUT(TRANS_37X26)" x="46.2" y="-82.2"/>
-<element name="U$3" library="__MyCommonLib1" package="TIO20_V2" value="TRANS_FLYBACK_AUX_SINGLE_OUT_WITH_SHIELD(TIO20-V2)" x="47.2" y="-78.5"/>
+<element name="X101" library="__MyCommonLib1" package="BRD_CONNECTOR_12X10.2" value="220VAC" x="-16.1" y="-44.2" rot="R180"/>
+<element name="F1" library="__MyCommonLib1" package="FUSE_20X5.6MM" value="0.3A" x="-12.2" y="-54.3"/>
+<element name="C101" library="__MyCommonLib1" package="MKP_18X6" value="0.1uF x 275VAC X2" x="-28.5" y="-47.1"/>
+<element name="TR101" library="__MyCommonLib1" package="EMI_CM_21X17" value="EMI" x="-41" y="-46.4" rot="R180"/>
+<element name="C10" library="__MyCommonLib1" package="MKP_18X6" value="0.1uF x 275VAC X2" x="-52.8" y="-48"/>
+<element name="RT1" library="__MyCommonLib1" package="NTC_9.0X4.2" value="5 Ohm" x="-61.1" y="-55.3" rot="R180"/>
+<element name="D101" library="__MyCommonLib1" package="DO-41_10MM" value="1N4007" x="-61.6" y="-46.9" rot="R90"/>
+<element name="D102" library="__MyCommonLib1" package="DO-41_10MM" value="1N4007" x="-58.1" y="-46.9" rot="R90"/>
+<element name="D103" library="__MyCommonLib1" package="DO-41_10MM" value="1N4007" x="-65" y="-46.9" rot="R270"/>
+<element name="D104" library="__MyCommonLib1" package="DO-41_10MM" value="1N4007" x="-68.4" y="-46.9" rot="R270"/>
+<element name="CE101" library="__MyCommonLib1" package="CE_13MM" value="22uF x 400V" x="-63.8" y="-33.7"/>
+<element name="R101" library="__MyCommonLib1" package="RSMD_0805" value="240K" x="-28.5" y="-50" rot="MR270"/>
+<element name="R24" library="__MyCommonLib1" package="RSMD_0805" value="240K" x="-28.5" y="-43.2" rot="MR270"/>
+<element name="TR102" library="__MyCommonLib1" package="TRANS_37X26_3578_11_13_15_17" value="Self made transformer. From TR8 sat reciever." x="-51.8" y="-70.6"/>
+<element name="D105" library="__MyCommonLib1" package="DO-41_10MM" value="UF4007" x="-64.1" y="-88"/>
+<element name="ZD101" library="__MyCommonLib1" package="DO-41_10MM" value="P6KE200" x="-64.1" y="-93.9"/>
 </elements>
 <signals>
@@
 <vertex x="11.2" y="53.9"/>
 </polygon>
-<contactref element="U$1" pad="2"/>
-<contactref element="U$2" pad="5"/>
-<contactref element="U$3" pad="2"/>
-<wire x1="46.2" y1="-92.2" x2="42.12" y2="-84.9" width="0" layer="19" extent="1-1"/>
 </signal>
 <signal name="N$23">
@@
 <vertex x="8.6" y="53.6"/>
 </polygon>
-<contactref element="U$1" pad="9"/>
-<contactref element="U$2" pad="15"/>
-<contactref element="U$3" pad="9"/>
-<wire x1="42.12" y1="-67.1" x2="42.12" y2="-72.1" width="0" layer="19" extent="1-1"/>
-<wire x1="42.2" y1="-72.2" x2="42.12" y2="-67.1" width="0" layer="19" extent="1-1"/>
 </signal>
 <signal name="+200VDC_OUT">
@@
 </signal>
 <signal name="N$13">
-<contactref element="U$1" pad="1"/>
-<contactref element="U$2" pad="3"/>
-<contactref element="U$3" pad="1"/>
-<wire x1="38.2" y1="-92.2" x2="37.04" y2="-84.9" width="0" layer="19" extent="1-1"/>
+<contactref element="X101" pad="1"/>
+<contactref element="F1" pad="PAD1"/>
+<wire x1="-0.45" y1="-54.3" x2="-12.1" y2="-44.2" width="0" layer="19" extent="1-1"/>
 </signal>
 <signal name="N$22">
-<contactref element="U$1" pad="10"/>
-<contactref element="U$2" pad="17"/>
-<contactref element="U$3" pad="10"/>
-<wire x1="37.04" y1="-67.1" x2="37.04" y2="-72.1" width="0" layer="19" extent="1-1"/>
-<wire x1="34.2" y1="-72.2" x2="37.04" y2="-67.1" width="0" layer="19" extent="1-1"/>
+<contactref element="X101" pad="2"/>
+<contactref element="C101" pad="1"/>
+<contactref element="TR101" pad="W2_START"/>
+<contactref element="R24" pad="PAD_0"/>
+<wire x1="-28.5" y1="-39.48" x2="-35.92" y2="-40" width="0" layer="19" extent="1-1"/>
+<wire x1="-28.5" y1="-42.15" x2="-28.5" y2="-39.48" width="0" layer="19" extent="16-16"/>
+<wire x1="-20.1" y1="-44.2" x2="-28.5" y2="-42.15" width="0" layer="19" extent="16-16"/>
 </signal>
 <signal name="N$27">
-<contactref element="U$1" pad="5"/>
-<contactref element="U$2" pad="8"/>
-<contactref element="U$3" pad="5"/>
-<wire x1="58.2" y1="-92.2" x2="57.36" y2="-84.9" width="0" layer="19" extent="1-1"/>
+<contactref element="F1" pad="PAD_0"/>
+<contactref element="C101" pad="2"/>
+<contactref element="TR101" pad="W1_START"/>
+<contactref element="R101" pad="PAD_1"/>
+<wire x1="-28.5" y1="-51.05" x2="-35.92" y2="-52.8" width="0" layer="19" extent="16-16"/>
+<wire x1="-28.5" y1="-54.72" x2="-28.5" y2="-51.05" width="0" layer="19" extent="16-16"/>
+<wire x1="-23.95" y1="-54.3" x2="-28.5" y2="-54.72" width="0" layer="19" extent="1-1"/>
 </signal>
 <signal name="N$28">
-<contactref element="U$1" pad="4"/>
-<contactref element="U$2" pad="7"/>
-<contactref element="U$3" pad="4"/>
-<wire x1="54.2" y1="-92.2" x2="52.28" y2="-84.9" width="0" layer="19" extent="1-1"/>
+<contactref element="TR101" pad="W2_END"/>
+<contactref element="C10" pad="1"/>
+<contactref element="D102" pad="ANODE"/>
+<contactref element="D104" pad="CATHODE"/>
+<wire x1="-58.1" y1="-51.98" x2="-68.4" y2="-51.98" width="0" layer="19" extent="1-1"/>
+<wire x1="-52.8" y1="-40.38" x2="-58.1" y2="-51.98" width="0" layer="19" extent="1-1"/>
+<wire x1="-46.08" y1="-40" x2="-52.8" y2="-40.38" width="0" layer="19" extent="1-1"/>
 </signal>
 <signal name="N$29">
-<contactref element="U$3" pad="7"/>
-<contactref element="U$1" pad="7"/>
-<contactref element="U$2" pad="13"/>
-<wire x1="52.28" y1="-67.1" x2="52.28" y2="-72.1" width="0" layer="19" extent="1-1"/>
-<wire x1="50.2" y1="-72.2" x2="52.28" y2="-67.1" width="0" layer="19" extent="1-1"/>
+<contactref element="TR101" pad="W1_END"/>
+<contactref element="C10" pad="2"/>
+<contactref element="RT1" pad="PAD_0"/>
+<wire x1="-52.8" y1="-55.62" x2="-57.85" y2="-56.4" width="0" layer="19" extent="1-1"/>
+<wire x1="-46.08" y1="-52.8" x2="-52.8" y2="-55.62" width="0" layer="19" extent="1-1"/>
+</signal>
+<signal name="N$30">
+<contactref element="RT1" pad="PAD1"/>
+<contactref element="D103" pad="CATHODE"/>
+<contactref element="D101" pad="ANODE"/>
+<wire x1="-65" y1="-51.98" x2="-64.35" y2="-54.2" width="0" layer="19" extent="1-1"/>
+<wire x1="-61.6" y1="-51.98" x2="-65" y2="-51.98" width="0" layer="19" extent="1-1"/>
+</signal>
+<signal name="N$32">
+<contactref element="D102" pad="CATHODE"/>
+<contactref element="D101" pad="CATHODE"/>
+<contactref element="CE101" pad="PLUS"/>
+<contactref element="TR102" pad="5"/>
+<contactref element="ZD101" pad="ANODE"/>
+<wire x1="-51.8" y1="-80.6" x2="-69.18" y2="-93.9" width="0" layer="19" extent="1-1"/>
+<wire x1="-58.1" y1="-41.82" x2="-51.8" y2="-80.6" width="0" layer="19" extent="1-1"/>
+<wire x1="-61.6" y1="-41.82" x2="-58.1" y2="-41.82" width="0" layer="19" extent="1-1"/>
+<wire x1="-61.26" y1="-33.7" x2="-61.6" y2="-41.82" width="0" layer="19" extent="1-1"/>
+</signal>
+<signal name="N$33">
+<contactref element="D103" pad="ANODE"/>
+<contactref element="D104" pad="ANODE"/>
+<contactref element="CE101" pad="MINUS"/>
+<wire x1="-65" y1="-41.82" x2="-68.4" y2="-41.82" width="0" layer="19" extent="1-1"/>
+<wire x1="-66.34" y1="-33.7" x2="-65" y2="-41.82" width="0" layer="19" extent="1-1"/>
 </signal>
 <signal name="N$31">
-<contactref element="U$2" pad="11"/>
-<contactref element="U$1" pad="6"/>
-<contactref element="U$3" pad="6"/>
-<wire x1="57.36" y1="-67.1" x2="57.36" y2="-72.1" width="0" layer="19" extent="1-1"/>
-<wire x1="58.2" y1="-72.2" x2="57.36" y2="-67.1" width="0" layer="19" extent="1-1"/>
+<contactref element="R101" pad="PAD_0"/>
+<contactref element="R24" pad="PAD_1"/>
+<wire x1="-28.5" y1="-44.25" x2="-28.5" y2="-48.95" width="0" layer="19" extent="16-16"/>
+</signal>
+<signal name="N$34">
+<contactref element="TR102" pad="3"/>
+<contactref element="TR102" pad="15"/>
+<wire x1="-55.8" y1="-60.6" x2="-59.8" y2="-80.6" width="0" layer="19" extent="1-1"/>
+</signal>
+<signal name="N$35">
+<contactref element="TR102" pad="17"/>
+<contactref element="D105" pad="ANODE"/>
+<wire x1="-63.8" y1="-60.6" x2="-69.18" y2="-88" width="0" layer="19" extent="1-1"/>
+</signal>
+<signal name="N$36">
+<contactref element="D105" pad="CATHODE"/>
+<contactref element="ZD101" pad="CATHODE"/>
+<wire x1="-59.02" y1="-88" x2="-59.02" y2="-93.9" width="0" layer="19" extent="1-1"/>
 </signal>
 </signals>

Commit message: 12_to_200V inverter. Ver3 Start schematic.
Parts:
- added C11: 0.1uF x 50V, __MyCommonLib1:RSMD_0805
- added C13: 0.1uF 16V, __MyCommonLib1:RSMD_0805
- added C14: 5n1 x 16V, __MyCommonLib1:RSMD_0805
- added C15: 1n0 x 16V, __MyCommonLib1:RSMD_0805
- added CE1: 22uFx50V, __MyCommonLib1:CE_6.3MM
- added IC101: UC3842, __MyCommonLib1:SOIC8
- added R25: 3R9, __MyCommonLib1:RSMD_1206
- added R26, R27, R28, R29: 120K, __MyCommonLib1:RSMD_1206
- added R30: 16R, __MyCommonLib1:RSMD_0805
- added R31, R34: 10K, __MyCommonLib1:RSMD_0805
- added R32, R36: 3K9*, __MyCommonLib1:RSMD_0805
- added R33, R35: 22K, __MyCommonLib1:RSMD_0805
- added R37: 82K, __MyCommonLib1:RSMD_0805
- added RT2: 22K_20deg, __MyCommonLib1:NTC_5.5X3
- added T101: 16N60, __MyCommonLib1:TO-220(VER2)
- added T102, T103: BC847, __MyCommonLib1:SOT23_SMALL_PADS
Connections:
- new net N$20: R30.PAD_0, T101.1
- new net N$23: IC101.6, R30.PAD_1
- new net N$37: R25.PAD_1, R32.PAD_0, T101.3
- new net N$38: C11.PAD_0, C13.PAD_1, C14.PAD_0, C15.PAD_0, CE1.MINUS, CE101.MINUS, D103.ANODE, D104.ANODE, IC101.2, IC101.5, R25.PAD_0, R33.PAD_0, R34.PAD_0, RT2.PAD_0
- new net N$39: C14.PAD_1, IC101.4, R31.PAD_1
- new net N$40: R27.PAD_0, R29.PAD_1
- new net N$41: R26.PAD_0, R28.PAD_1
- new net N$42: C11.PAD_1, CE1.PLUS, IC101.7, R28.PAD_0, R29.PAD_0
- new net N$43: C15.PAD_1, IC101.3, R32.PAD_1
- new net N$44: R34.PAD_1, T102.2, T103.2
- new net N$45: R36.PAD_0, RT2.PAD1, T103.1
- new net N$46: R37.PAD_1, T103.3
- new net N$47: R33.PAD_1, R35.PAD_0, R37.PAD_0, T102.1
- net N$32: now also R26.PAD_1, R27.PAD_1
- net N$33: now also C13.PAD_0, IC101.8, R31.PAD_0, R35.PAD_1, R36.PAD_1, T102.3; no longer CE101.MINUS, D103.ANODE, D104.ANODE
- net N$35: now also T101.2

Commit message: 12_to_200V inverter. Ver3 Start schematic.
Parts:
- added C16: 2n2 x 50V, __MyCommonLib1:RSMD_0805
- added C17: 10nF x 2kV, __MyCommonLib1:CAP_CER_11X4
- added CE2: 2.2uF x 50V, __MyCommonLib1:CE_5.2MM
- added D106, D5: LL4148, __MyCommonLib1:SOD-80
- added R38: 22K, __MyCommonLib1:RSMD_0805
- added R39, R40: 120R, __MyCommonLib1:RSMD_0805
- added R41, R46: 5K6, __MyCommonLib1:RSMD_0805
- added R42, R43, R44, R45: 33K, __MyCommonLib1:RSMD_1206
- added R47: 560R, __MyCommonLib1:RSMD_0805
- added T104, T5: BC857, __MyCommonLib1:SOT23_SMALL_PADS
- C15: value 1n0 x 16V -> 1n0 x 16V*
Connections:
- new net N$48: C16.PAD_1, D106.ANODE, TR102.7
- new net N$49: C16.PAD_0, R39.PAD_0, R40.PAD_0
- new net N$50: C11.PAD_0, C13.PAD_1, C14.PAD_0, C15.PAD_0, CE1.MINUS, CE101.MINUS, CE2.MINUS, D103.ANODE, D104.ANODE, IC101.2, IC101.5, R25.PAD_0, R33.PAD_0, R34.PAD_0, R39.PAD_1, R40.PAD_1, R47.PAD_0, RT2.PAD_0, T5.3, TR102.8
- new net N$51: CE2.PLUS, D106.CATHODE, D5.CATHODE, R41.PAD_1, T104.2
- new net N$52: R42.PAD_0, R43.PAD_1
- new net N$53: R44.PAD_1, R45.PAD_0
- new net N$54: R46.PAD_0, R47.PAD_1, T5.1
- net N$23: now also R46.PAD_1
- net N$32: now also C17.PAD_0, R42.PAD_1, R45.PAD_1
- net N$36: now also C17.PAD1, R43.PAD_0, R44.PAD_0
- net N$38: now also C11.PAD_1, CE1.PLUS, D5.ANODE, IC101.7, R28.PAD_0, R29.PAD_0, T104.3; no longer C11.PAD_0, C13.PAD_1, C14.PAD_0, C15.PAD_0, CE1.MINUS, CE101.MINUS, D103.ANODE, D104.ANODE, IC101.2, IC101.5, R25.PAD_0, R33.PAD_0, R34.PAD_0, RT2.PAD_0
- net N$42: now also R38.PAD_0, R41.PAD_0, T104.1; no longer C11.PAD_1, CE1.PLUS, IC101.7, R28.PAD_0, R29.PAD_0
- net N$43: now also T5.2
- net N$46: now also R38.PAD_1
