File: 12_to_200V_inverter/schematic/12to220inverterVer3.brd (EAGLE design)
At the start: 80 x 55 mm, 107 parts, among them IC101 UC3842, T1 IRFZ24N, T101 16N60, T102 BC847, T103 BC847, T104 BC857, T15 IRL5602S, T16 BC847, T2 IRFZ24N, T3 BC857, T4 BC857, T5 BC857, U1 TL494, X1 +12V_INPUT, X101 220VAC, X2 200VDC_OUTPUT, X3 TURN_ON

Commit message: 12_to_200V inverter. Ver3 Start schematic.
Parts:
- removed X3: TURN_ON, con-wago-500:W237-102
- added C18: 2n2 x 50V, __MyCommonLib1:RSMD_0805
- added C19: 1n0 275VAC Y2, __MyCommonLib1:MKP_13.4X4
- added C20: 100pF, __MyCommonLib1:RSMD_0805
- added CE3, CE4: 1000uF x 25V, __MyCommonLib1:CE_5.2MM
- added D107: SR3A0, __MyCommonLib1:DO-27_15MM
- added IC102: PC817, __MyCommonLib1:DIP4
- added IC103: TL431, __MyCommonLib1:SOT23
- added L1: 20uH, __MyCommonLib1:COIL_10MM
- added R48, R49: 120R, __MyCommonLib1:RSMD_0805
- added R50: 5K6, __MyCommonLib1:RSMD_0805
- added R51, R53, R55: 10K, __MyCommonLib1:RSMD_0805
- added R52, R54: 1K0, __MyCommonLib1:RSMD_0805
- added T23, T6: IRF830, __MyCommonLib1:TO-220
- X1: value +12V_INPUT -> LAMP1; device con-wago-500:W237-102 -> __MyCommonLib1:BRD_CONNECTOR_12X10.2
- X2: value 200VDC_OUTPUT -> LAMP1; device con-wago-500:W237-102 -> __MyCommonLib1:BRD_CONNECTOR_12X10.2
- moved X1 363.8 mm to (-120.2, -299.1), turned to 0 degrees
- moved X2 344.8 mm to (-120.2, -309.3)
Connections:
- net PWM1 renamed CONV_PWM1
- net PWM2 renamed CONV_PWM2
- removed net GND: C1.PAD_1, C12.MINUS, C2.MINUS, C5.PAD_0, C6.MINUS, C7.PAD_0, C8.MINUS, C9.PAD_1, D9.ANODE, R1.PAD_0, R12.PAD_0, R13.PAD_0, R15.PAD1, R17.PAD_1, R19.PAD_0, R20.PAD_1, R4.PAD_1, R9.PAD_0, T1.3, T16.2, T2.3, T3.3, T4.3, TR3.9, U1.4, U1.7, X1.2, X3.2, ZD2.ANODE
- new net CONV_GND: C1.PAD_1, C2.MINUS, C5.PAD_0, C6.MINUS, C7.PAD_0, C8.MINUS, C9.PAD_1, R1.PAD_0, R12.PAD_0, R13.PAD_0, R15.PAD1, R17.PAD_1, R20.PAD_1, R4.PAD_1, R53.PAD_1, R55.PAD_1, R9.PAD_0, T1.3, T16.2, T2.3, T3.3, T4.3, U1.4, U1.7, ZD2.ANODE
- new net CONV_TURN_ON: R10.PAD_1
- new net LAMP1_ON: R52.PAD_1
- new net LAMP2_ON: R54.PAD_0
- new net N$55: IC101.1, IC102.4
- new net N$56: C18.PAD_0, R48.PAD_0, R49.PAD_0
- new net N$57: C19.1, CE3.MINUS, CE4.MINUS, R48.PAD_1, R49.PAD_1, TR102.11
- new net N$58: C18.PAD_1, D107.ANODE, TR102.13
- new net N$59: CE3.PLUS, D107.CATHODE, L1.1
- new net N$60: CE4.PLUS, L1.2
- new net N$61: IC102.2, R50.PAD_1
- new net N$62: IC102.1, IC103.1, R51.PAD_1
- new net N$63: IC103.3
- new net N$64: R52.PAD_0, R53.PAD_0, T23.1
- new net N$65: T23.2, X1.2
- new net N$66: T6.2, X2.2
- new net N$67: R54.PAD_1, R55.PAD_0, T6.1
- net +12V_BAT: no longer X1.1
- net +200VDC_I_SENSE: now also T23.3, T6.3; no longer X2.2
- net +200VDC_OUT: now also X1.1
- net N$15: now also C12.MINUS, D9.ANODE, R19.PAD_0, TR3.9; no longer R10.PAD_1, X3.1
- net N$50: now also C19.2, IC102.3
Routing:
- net GND: track 73.7 -> 28.9 mm, vias 6 -> 4
- net CONV_GND: track 0.00 -> 31.6 mm, vias 0 -> 2
- net N$15: track 2.12 -> 0.00 mm
- net CONV_TURN_ON: track 0.00 -> 2.12 mm
- added copper zone on layer 16, net CONV_TURN_ON
- removed copper zone on layer 16, net N$15

Commit message: 12_to_200V inverter. Ver3 Start schematic.
Parts:
- added C21, C29: 10nF, __MyCommonLib1:RSMD_0805
- added C22: 10uFx16V, __MyCommonLib1:CE_5.2MM
- added C23, C25, C26, C27, C28, C30: 0.1uF, __MyCommonLib1:RSMD_0805
- added C24: 470uFx25V, __MyCommonLib1:CE_6.3MM
- added D10, D11, D12: LL4148, __MyCommonLib1:SOD-80
- added D7, D8: 1N4001, __MyCommonLib1:DO-41_10MM
- added IC1: LM317, __MyCommonLib1:D2PAK
- added IC2: 74HC595, __MyCommonLib1:SOIC16
- added IC3: ATTINY45, __MyCommonLib1:SOIC8(0.15'')
- added LED1, LED8: RED, __MyCommonLib1:LED3MM
- added LED2, LED7: GREEN, __MyCommonLib1:LED3MM
- added LED3, LED4, LED5, LED6: YELLOW, __MyCommonLib1:LED3MM
- added R120: 10K, __MyCommonLib1:R_ADJ_STAND
- added R56: 1M0, __MyCommonLib1:RSMD_0805
- added R57: 22K, __MyCommonLib1:RSMD_0805
- added R58: 110K, __MyCommonLib1:RSMD_0805
- added R59: 5K6, __MyCommonLib1:RSMD_0805
- added R60: 27K, __MyCommonLib1:RSMD_0805
- added R61: 0.1Ohm, __MyCommonLib1:R_1.0W
- added R62, R65, R66, R67, R68, R69, R70, R71, R74: 1K0, __MyCommonLib1:RSMD_0805
- added R63: 3K0, __MyCommonLib1:RSMD_0805
- added R64: 1K0, __MyCommonLib1:RSMD_1206
- added R72: 4K7, __MyCommonLib1:RSMD_0805
- added R73: 10K, __MyCommonLib1:RSMD_0805
- added R75: 10K, __MyCommonLib1:RSMD_1206_BIG_GAP
- added R76: 3K3, __MyCommonLib1:RSMD_0805
- added X3: VCC_IN, __MyCommonLib1:PIN1X1_3.5MM_SIDE_BOARD
- added X4: GND_FROM_CHARGE, __MyCommonLib1:PIN1X1_3.5MM_SIDE_BOARD
- added X5: GND_TO_ACC, __MyCommonLib1:PIN1X1_3.5MM_SIDE_BOARD
- added X6: CHARGE_IN, __MyCommonLib1:PIN1X1_3.5MM_SIDE_BOARD
- moved D107 174.0 mm to (-64.2, -87.2), turned to 180 degrees
- moved ZD101 44.6 mm to (-31.8, -63.2), turned to 270 degrees
- moved D105 34.6 mm to (-31.7, -76.0), turned to 90 degrees
- moved TR102 1.08 mm to (-52.8, -71.0), turned to 180 degrees
Connections:
- new net +5V: C22.PLUS, C23.PAD_0, C26.PAD_0, C27.PAD_0, D11.CATHODE, D12.CATHODE, IC1.2, IC2.10, IC2.16, IC3.8, R62.PAD_1, R72.PAD_0
- new net GND: C19.1, C22.MINUS, C23.PAD_1, C24.MINUS, C25.PAD_1, C26.PAD_1, C27.PAD_1, C28.PAD_1, C29.PAD_1, C30.PAD_1, CE3.MINUS, CE4.MINUS, D10.ANODE, IC103.3, IC2.13, IC2.8, IC3.2, IC3.4, LED1.CATHODE, LED2.CATHODE, LED3.CATHODE, LED4.CATHODE, LED5.CATHODE, LED6.CATHODE, LED7.CATHODE, LED8.CATHODE, R48.PAD_1, R49.PAD_1, R57.PAD_0, R59.PAD_0, R61.PAD1, R63.PAD_0, R76.PAD_0, TR102.11, X4.1
- new net I_SHUNT_ADC: C28.PAD_0, D10.CATHODE, D11.ANODE, IC3.3, R73.PAD_1
- new net LED_DATA: IC2.14, IC3.5
- new net LED_LATCH: C29.PAD_0, IC2.12, R74.PAD_1
- new net LED_SCK: IC2.11, IC3.6, R74.PAD_0
- new net N$68: C20.PAD_0, C21.PAD_0, IC103.2, R120.2, R59.PAD_1, R60.PAD_0
- new net N$69: C21.PAD_1, R56.PAD_1
- new net N$70: R61.PAD_0, R73.PAD_0, X5.1
- new net N$71: D7.ANODE, R75.PAD_0, X3.1
- new net N$72: D8.ANODE, X6.1
- new net N$73: C24.PLUS, C25.PAD_0, D7.CATHODE, D8.CATHODE, IC1.3
- new net N$74: IC1.1, R62.PAD_0, R63.PAD_1
- new net N$75: IC2.15, R64.PAD_0
- new net N$76: IC2.1, R65.PAD_0
- new net N$77: IC2.2, R66.PAD_0
- new net N$78: IC2.3, R67.PAD_0
- new net N$79: IC2.4, R68.PAD_0
- new net N$80: IC2.5, R69.PAD_0
- new net N$81: IC2.6, R70.PAD_0
- new net N$82: IC2.7, R71.PAD_0
- new net N$83: LED1.ANODE, R64.PAD_1
- new net N$84: LED3.ANODE, R66.PAD_1
- new net N$85: LED6.ANODE, R69.PAD_1
- new net N$86: LED8.ANODE, R71.PAD_1
- new net N$87: LED2.ANODE, R65.PAD_1
- new net N$88: LED5.ANODE, R68.PAD_1
- new net N$89: LED7.ANODE, R70.PAD_1
- new net N$90: LED4.ANODE, R67.PAD_1
- new net N$91: IC3.1, R72.PAD_1
- new net VOLTAGE_ADC: C30.PAD_0, D12.ANODE, IC3.7, R75.PAD_1, R76.PAD_1
- net N$57: now also R120.3, R57.PAD_1; no longer C19.1, CE3.MINUS, CE4.MINUS, R48.PAD_1, R49.PAD_1, TR102.11
- net N$59: now also R50.PAD_0, R51.PAD_0, R58.PAD_1, R60.PAD_1
- net N$62: now also C20.PAD_1, R56.PAD_0
- net N$63: now also R120.1, R58.PAD_0; no longer IC103.3

Commit message: 12 to 200V converter. Ver3. Schematic almost done.
Parts:
- removed C28: 0.1uF, __MyCommonLib1:RSMD_0805
- removed D10, D11: LL4148, __MyCommonLib1:SOD-80
- removed D7, D8: 1N4001, __MyCommonLib1:DO-41_10MM
- removed X4: GND_FROM_CHARGE, __MyCommonLib1:PIN1X1_3.5MM_SIDE_BOARD
- removed X5: GND_TO_ACC, __MyCommonLib1:PIN1X1_3.5MM_SIDE_BOARD
- removed X6: CHARGE_IN, __MyCommonLib1:PIN1X1_3.5MM_SIDE_BOARD
- added C31, C33: 0.1uF, __MyCommonLib1:RSMD_0805
- added C32, C34: 0.1uF*, __MyCommonLib1:RSMD_0805
- added CE5: 22uF x 50V, __MyCommonLib1:CE_5.2MM
- added D13: FR101, __MyCommonLib1:DO-41_10MM
- added D14, D15: LL4148, __MyCommonLib1:SOD-80
- added IC11: LM358SOIC8, __MyCommonLib1:SOIC8
- added R77, R78, R85, R86, R87, R91: 10K, __MyCommonLib1:RSMD_0805
- added R79, R80, R88: 1K0, __MyCommonLib1:RSMD_0805
- added R81: 5K1, __MyCommonLib1:RSMD_0805
- added R82: 330R, __MyCommonLib1:RSMD_0805
- added R83: 0.1R, __MyCommonLib1:R_1.0W
- added R84: 240R, __MyCommonLib1:RSMD_0805
- added R89: 470K, __MyCommonLib1:RSMD_0805
- added R90: 200K, __MyCommonLib1:RSMD_0805
- added R92, R93: 20R, __MyCommonLib1:RSMD_0805
- added T10, T106, T9: BSS84, __MyCommonLib1:SOT23_SMALL_PADS
- added T7, T8: BC847, __MyCommonLib1:SOT23_SMALL_PADS
- CE3: device __MyCommonLib1:CE_5.2MM -> __MyCommonLib1:CE_13MM
- R61: value 0.1Ohm -> 10K; device __MyCommonLib1:R_1.0W -> __MyCommonLib1:RSMD_0805
- R73: value 10K -> 1K0
- X3: value VCC_IN -> LAMP1_SWITCH; device __MyCommonLib1:PIN1X1_3.5MM_SIDE_BOARD -> __MyCommonLib1:PIN2X1_2.54MM
- moved X3 167.9 mm to (-144.6, -554.5)
- moved R61 125.0 mm to (-148.6, -534.4)
- moved R73 111.7 mm to (-148.6, -537.5)
- moved IC2 23.4 mm to (-102.2, -398.1), turned to 90 degrees
Connections:
- removed net CONV_GND: C1.PAD_1, C2.MINUS, C5.PAD_0, C6.MINUS, C7.PAD_0, C8.MINUS, C9.PAD_1, R1.PAD_0, R12.PAD_0, R13.PAD_0, R15.PAD1, R17.PAD_1, R20.PAD_1, R4.PAD_1, R53.PAD_1, R55.PAD_1, R9.PAD_0, T1.3, T16.2, T2.3, T3.3, T4.3, U1.4, U1.7, ZD2.ANODE
- removed net I_SHUNT_ADC: C28.PAD_0, D10.CATHODE, D11.ANODE, IC3.3, R73.PAD_1
- removed net N$72: D8.ANODE, X6.1
- removed net N$73: C24.PLUS, C25.PAD_0, D7.CATHODE, D8.CATHODE, IC1.3
- new net -VBAT: C1.PAD_1, C2.MINUS, C5.PAD_0, C6.MINUS, C7.PAD_0, C8.MINUS, C9.PAD_1, R1.PAD_0, R12.PAD_0, R13.PAD_0, R15.PAD1, R17.PAD_1, R20.PAD_1, R4.PAD_1, R53.PAD_1, R55.PAD_1, R83.PAD_0, R88.PAD_0, R9.PAD_0, T1.3, T16.2, T2.3, T3.3, T4.3, U1.4, U1.7, ZD2.ANODE
- new net CHARGER_ENABLED: CE5.PLUS, D13.CATHODE, R78.PAD_0
- new net I_CS_ADC: C34.PAD_0, IC3.3, R91.PAD_1
- new net N$100: C31.PAD_0, IC11.7, R81.PAD_0, R89.PAD_1
- new net N$101: R84.PAD_1, R86.PAD_0, R87.PAD_0, R89.PAD_0
- new net N$102: D14.CATHODE, D15.ANODE, IC11.2, IC11.5, R88.PAD_1
- new net N$103: C32.PAD_0, IC11.1, R90.PAD_1, R91.PAD_0
- new net N$104: R93.PAD_1, T9.2
- new net N$92: R81.PAD_1, T8.1
- new net N$94: R78.PAD_1, R79.PAD_1, T7.1
- new net N$95: R77.PAD_1, R80.PAD_1, T106.1
- new net N$96: R92.PAD_1, T10.2
- new net N$97: C32.PAD_1, IC11.3, R85.PAD_1, R90.PAD_0
- new net N$98: CE3.PLUS, D107.CATHODE, L1.1, R77.PAD_0, T106.2
- new net N$99: C31.PAD_1, IC11.6, R86.PAD_1
- new net VOLTAGE_SENSE: R50.PAD_0, R51.PAD_0, R58.PAD_1, R60.PAD_1, R75.PAD_0, T106.3
- net +12V_BAT: now also CE4.PLUS, L1.2, R61.PAD_0, R92.PAD_0, R93.PAD_0
- net +5V: now also C33.PAD_0, D15.CATHODE, IC11.8, R87.PAD_1; no longer D11.CATHODE
- net GND: now also C33.PAD_1, C34.PAD_1, CE5.MINUS, D14.ANODE, IC11.4, R79.PAD_0, R82.PAD_1, R83.PAD1, R84.PAD_0, R85.PAD_0, T7.2; no longer C28.PAD_1, D10.ANODE, IC3.2, R61.PAD1, X4.1
- net N$58: now also D13.ANODE
- net N$59: now also R61.PAD_1, R73.PAD_1, T10.1, T9.1; no longer CE3.PLUS, D107.CATHODE, L1.1, R50.PAD_0, R51.PAD_0, R58.PAD_1, R60.PAD_1
- net N$60: now also R82.PAD_0, T8.2; no longer CE4.PLUS, L1.2
- net N$62: now also T8.3
- net N$70: now also C24.PLUS, C25.PAD_0, IC1.3, T10.3, T9.3; no longer R61.PAD_0, R73.PAD_0, X5.1
- net N$71: now also R80.PAD_0, T7.3; no longer D7.ANODE, R75.PAD_0, X3.1
- net VOLTAGE_ADC: now also IC3.2; no longer IC3.7
Routing:
- net CONV_GND: track 31.6 -> 0.00 mm, vias 2 -> 0
- net -VBAT: track 0.00 -> 31.6 mm, vias 0 -> 2
