File: 12_to_200V_inverter/schematic/12to220inverterVer3.brd (EAGLE design)
At the start: 150 x 100 mm, 245 parts, among them IC1 UC3842, IC10 TL494, IC2 PC817, IC3 LM358SOIC8, IC4 TL431, IC5 LM317, IC6 74HC595, IC7 74HC595, IC8 ATTINY45, IC9 TL431, J1 0, J2 0, J3 0, J4 0, T1 AO4407AL, T10 16N60, T11 BC847, T12 BC847, T13 BSS84, T15 BC847, T16 BSS84, T17 BC847, T18 BC847, T19 BSS84, T2 IRF830, T20 BSS84, T21 BC847, T22 BC847, T23 BSS84, T24 BC847, T3 IRF830, T4 BC847, T5 BC857, T6 BC857, T7 IRFZ24N, T8 IRFZ24N, T9 BC857, X1 BAT+, X2 LAMP1, X3 LAMP1, X4 BAT-, X5 220VAC, X6 LAMP1_SWITCH, X7 LAMP1_SWITCH, X8 MCU_PROGRAMMING

Commit message: 12to200V inverter. restore
Parts:
- added TR4: Self made transformer. From TR8 sat reciever., __MyCommonLib1:TRANS_29.5X23_1234567_910
- moved C7 142.3 mm to (36.4, 25.6)
- moved R3 138.9 mm to (8.90, 48.8), turned to 90 degrees
- moved R2 136.5 mm to (4.20, 50.4)
- moved R9 135.8 mm to (29.3, 25.6)
- moved C41 64.0 mm to (64.0, 95.0), turned to 90 degrees
- moved R80 25.7 mm to (80.0, 45.0), turned to 0 degrees
- moved D27 18.8 mm to (29.0, 76.0)
- moved D28 18.8 mm to (26.0, 76.0)
- moved D25 13.4 mm to (44.0, 83.0), turned to 0 degrees
- moved R76 10.3 mm to (83.0, 51.0), turned to 90 degrees
- moved L1 9.06 mm to (61.0, 57.0)
- moved R90 8.06 mm to (38.0, 90.0), turned to 0 degrees
- moved C15 7.62 mm to (86.0, 34.0)
- moved R5 7.62 mm to (21.0, 78.0), turned to 180 degrees
- moved C6 5.83 mm to (50.0, 32.0), turned to 0 degrees
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Connections:
- new net ANY_LAMP_ON: D24.ANODE, D25.ANODE, D27.CATHODE, D28.CATHODE
- net GND: now also TR4.7
- net LAMP1_ON: no longer D24.ANODE
- net LAMP2_ON: no longer D25.ANODE
- net N$130: now also D25.CATHODE; no longer D27.CATHODE, D28.CATHODE
- net N$32: now also TR4.10
- net N$34: now also TR4.1, TR4.9
- net N$35: now also TR4.2
- net N$48: now also TR4.5
- net N$50: now also TR4.4
- net N$58: now also TR4.6
- net N$93: no longer D25.CATHODE
Routing:
- net GND: track 263.3 -> 315.5 mm
- net +5V: track 78.2 -> 109.9 mm, vias 8 -> 10
- net LAMP2_ON: track 28.7 -> 7.58 mm
- net ANY_LAMP_ON: track 0.00 -> 20.3 mm
- net N$24: track 18.7 -> 0.00 mm
- net VOLTAGE_ADC: track 0.00 -> 18.4 mm
- net +12V_BAT: track 150.9 -> 139.6 mm
- net CHARGE_CURR_ADC: track 0.00 -> 10.9 mm
- net +12V_CONVERTER: track 49.0 -> 39.6 mm
- net N$58: track 0.00 -> 9.27 mm
- net N$64: track 44.0 -> 35.1 mm
- net LAMP1_ON: track 25.1 -> 16.3 mm
- net -VBAT: track 202.1 -> 197.5 mm
- net N$73: track 10.1 -> 5.78 mm
- net LED_DATA(MOSI): track 0.00 -> 4.17 mm
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
Commit message: 10 to 200V inverter. Ver3. Routing.
Parts:
- removed J1: 0, __MyCommonLib1:RSMD_1206_BIG_GAP
- D10, D8: device __MyCommonLib1:DO-41_10MM -> __MyCommonLib1:DO-41_15MM
- D13: device __MyCommonLib1:DO-41_10MM -> __MyCommonLib1:DO-41_12.5MM
- R30: device __MyCommonLib1:R_1.0W_VERTICAL -> __MyCommonLib1:R_1.0W
- R68, R76: device __MyCommonLib1:RSMD_0805 -> __MyCommonLib1:RSMD_1206_BIG_GAP
- moved C36 182.8 mm to (51.9, 78.9)
- moved R80 26.5 mm to (54.0, 40.0), turned to 270 degrees
- moved CE5 20.1 mm to (119.0, 39.2)
- moved D20 12.1 mm to (88.0, 52.0), turned to 0 degrees
- moved R30 10.9 mm to (124.8, 25.8), turned to 270 degrees
- moved L1 9.49 mm to (70.0, 54.0)
- moved R90 9.43 mm to (33.0, 82.0)
- moved R35 8.41 mm to (106.6, 6.40)
- moved C21 7.00 mm to (83.0, 56.0)
- moved J2 6.91 mm to (118.4, 44.4)
- moved C26 6.40 mm to (100.0, 59.0)
- moved D24 6.40 mm to (34.0, 77.0), turned to 270 degrees
- moved R76 6.32 mm to (77.0, 49.0), turned to 180 degrees
- moved R40 6.00 mm to (98.0, 40.0), turned to 0 degrees
- moved D22 5.60 mm to (72.5, 64.5)
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Connections:
- removed net N$40: IC2.4, J1.PAD_0
- net N$35: no longer HS1.PACKAGE
- net N$55: now also IC2.4; no longer J1.PAD_1
Routing:
- net N$50: track 94.1 -> 53.3 mm
- net CHARGE_CURR_ADC: track 10.9 -> 47.9 mm, vias 0 -> 2
- net N$40: track 36.2 -> 0.00 mm
- net N$102: track 0.00 -> 29.8 mm
- net N$8: track 28.7 -> 0.00 mm
- net N$55: track 5.32 -> 32.9 mm
- net N$62: track 0.00 -> 22.0 mm
- net N$68: track 0.00 -> 21.6 mm
- net -VBAT: track 197.5 -> 218.7 mm
- net N$98: track 0.00 -> 18.2 mm
- net N$33: track 19.6 -> 36.0 mm, vias 0 -> 2
- net N$48: track 0.00 -> 14.7 mm
- net N$100: track 0.00 -> 14.4 mm
- net GND: track 315.5 -> 302.5 mm
- net N$125: track 0.00 -> 11.7 mm
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- added copper zone on layer 16, net CHARGER_POWER
- added copper zone on layer 16, net GND
- added copper zone on layer 16, net N$110
- added copper zone on layer 16, net N$13
- added copper zone on layer 16, net N$22
- added copper zone on layer 16, net N$27
- added copper zone on layer 16, net N$28
- added copper zone on layer 16, net N$29
- added copper zone on layer 16, net N$32
- added copper zone on layer 16, net N$34
- added copper zone on layer 16, net N$35
- added copper zone on layer 16, net N$36
- added copper zone on layer 16, net N$50
- added copper zone on layer 16, net N$58
- added copper zone on layer 16, net N$98

Commit message: 10 to 200V inverter. Ver3. Routing.
Parts:
- added C39: 0.1uF x 50V, __MyCommonLib1:RSMD_0805
- R72, R78: device __MyCommonLib1:RSMD_0805 -> __MyCommonLib1:RSMD_1206_BIG_GAP
- moved C35 9.77 mm to (105.1, 86.0)
- moved R73 8.25 mm to (95.0, 78.0)
- moved R92 6.68 mm to (87.6, 81.0)
- moved R94 6.08 mm to (75.0, 78.0)
- moved T22 6.08 mm to (75.0, 74.0)
- moved T15 5.83 mm to (86.0, 72.0)
- moved R54 5.39 mm to (89.0, 76.0)
- moved R59 5.39 mm to (117.0, 65.0), turned to 180 degrees
- moved R77 5.39 mm to (95.0, 70.0), turned to 90 degrees
- moved IC6 5.00 mm to (93.1, 87.9)
- moved R8 4.88 mm to (79.8, 81.0), turned to 180 degrees
- moved R61 4.24 mm to (113.0, 62.0), turned to 90 degrees
- moved R13 4.12 mm to (70.0, 78.0), turned to 0 degrees
- moved R58 4.12 mm to (80.0, 70.0), turned to 180 degrees
- moved C32 4.00 mm to (108.0, 86.0)
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Connections:
- removed net N$61: IC2.2, R59.PAD_1
- new net N$40: IC2.1, R59.PAD_1
- net GND: now also C39.PAD_0
- net N$62: now also R59.PAD_0; no longer IC2.1
- net N$98: now also C39.PAD_1, IC2.2; no longer R59.PAD_0
Routing:
- net GND: track 302.5 -> 407.2 mm, vias 2 -> 6
- net +5V: track 115.5 -> 169.8 mm, vias 10 -> 6
- net N$98: track 18.2 -> 59.3 mm, vias 0 -> 2
- net LED_DATA(MOSI): track 6.10 -> 46.1 mm, vias 0 -> 2
- net +12V_BAT: track 142.5 -> 179.7 mm
- net N$108: track 0.00 -> 17.9 mm
- net CHARGE_CURR_ADC: track 47.9 -> 58.1 mm
- net N$94: track 0.00 -> 9.10 mm
- net N$16: track 6.37 -> 14.5 mm
- net N$95: track 2.76 -> 9.78 mm
- net N$78: track 7.17 -> 13.5 mm
- net N$105: track 47.5 -> 42.5 mm
- net SENSE_BAT_VOLTAGE: track 40.5 -> 45.3 mm
- net N$106: track 0.00 -> 4.68 mm
- net N$71: track 0.00 -> 4.27 mm
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
Commit message: 10 to 200V inverter. Ver3. Routing.
Parts:
- removed J4: 0, __MyCommonLib1:RSMD_1206_BIG_GAP
- moved R107 26.7 mm to (81.6, 91.4)
- moved RT1 17.1 mm to (142.0, 56.0), turned to 180 degrees
- moved C36 14.0 mm to (62.6, 88.0), turned to 90 degrees
- moved D26 9.85 mm to (50.4, 87.4), turned to 90 degrees
- moved X5 6.20 mm to (128.8, 58.2)
- moved C34 5.80 mm to (59.2, 81.0)
- moved C35 4.92 mm to (104.0, 90.8), turned to 180 degrees
- moved C32 4.90 mm to (109.0, 90.8)
- moved R97 3.80 mm to (53.2, 81.0)
- moved R98 3.60 mm to (56.4, 81.0)
- moved IC8 2.40 mm to (57.6, 87.0)
- moved C33 2.26 mm to (132.6, 88.6)
- moved IC7 2.26 mm to (125.6, 88.6)
- moved R95 2.24 mm to (113.0, 93.0)
- moved R13 1.65 mm to (69.6, 76.4)
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Connections:
- removed net N$110: RT1.PAD_0, X5.2
- removed net N$13: F2.PAD1, X5.1
- removed net N$63: J4.PAD_1, X8.4
- new net N$61: F2.PAD1, RT1.PAD_0
- new net N$70: RT1.PAD1, X5.1
- net CONV_TEMP_ADC(SCK): now also X8.4; no longer J4.PAD_0
- net N$22: now also X5.2; no longer RT1.PAD1
Routing:
- net GND: track 407.2 -> 286.8 mm, vias 6 -> 8
- net +5V: track 169.8 -> 55.2 mm
- net N$98: track 59.3 -> 44.2 mm
- net N$80: track 13.2 -> 21.1 mm
- net CONV_TEMP_ADC(SCK): track 27.8 -> 35.1 mm, vias 0 -> 2
- net LED_DATA(MOSI): track 46.1 -> 39.3 mm, vias 2 -> 0
- net CHARGE_CURR_ADC: track 58.1 -> 64.0 mm
- net ~RST: track 24.5 -> 30.2 mm
- net N$17: track 9.72 -> 4.04 mm
- net VOLTAGE_ADC: track 19.0 -> 13.6 mm
- net N$63: track 3.91 -> 0.00 mm
- net LED_SCK(MISO): track 73.3 -> 76.4 mm
- net N$105: track 42.5 -> 45.3 mm
- net N$107: track 47.2 -> 44.8 mm
- net N$82: track 25.1 -> 27.4 mm
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- added copper zone on layer 16, net +5V
- added copper zone on layer 16, net N$61
- added copper zone on layer 16, net N$70
- removed copper zone on layer 16, net N$110
- removed copper zone on layer 16, net N$13

Commit message: 10 to 200V inverter. Ver3. Routing.
Parts:
- moved R10 12.7 mm to (17.6, 66.8), turned to 180 degrees
- moved R8 9.77 mm to (69.6, 79.2)
- moved R12 8.23 mm to (20.6, 71.6), turned to 270 degrees
- moved D25 7.00 mm to (40.0, 77.0), turned to 270 degrees
- moved R114 6.08 mm to (47.4, 82.8), turned to 90 degrees
- moved R116 5.57 mm to (39.0, 82.8)
- moved D17 5.39 mm to (44.6, 78.8)
- moved R5 4.81 mm to (16.4, 79.4)
- moved R93 4.80 mm to (42.2, 88.0)
- moved T23 3.96 mm to (43.2, 82.8), turned to 90 degrees
- moved R3 3.76 mm to (10.0, 52.4), turned to 0 degrees
- moved R2 3.69 mm to (7.00, 48.0)
- moved D27 3.22 mm to (30.6, 73.2)
- moved R18 2.67 mm to (23.4, 55.6)
- moved R28 2.61 mm to (33.6, 54.8)
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Connections:
- net +200VDC_I_SENSE: now also R10.PAD_1, R12.PAD_1
- net -VBAT: no longer R10.PAD_1, R12.PAD_1
Routing:
- net -VBAT: track 218.7 -> 64.6 mm
- net +12V_BAT: track 178.5 -> 94.7 mm
- net +200VDC_I_SENSE: track 32.2 -> 3.10 mm
- net +12V_CONVERTER: track 39.6 -> 23.4 mm
- net GND: track 286.8 -> 276.2 mm
- net CONVERTER_ON: track 13.6 -> 23.9 mm
- net N$73: track 0.28 -> 9.68 mm
- net N$16: track 14.9 -> 5.56 mm
- net N$64: track 35.1 -> 26.2 mm
- net N$15: track 0.00 -> 8.77 mm
- net ANY_LAMP_ON: track 23.3 -> 15.5 mm
- net LAMP2_ON: track 7.58 -> 0.00 mm
- net N$17: track 4.04 -> 11.2 mm
- net CONV_PWM2: track 38.1 -> 44.9 mm
- net N$19: track 0.00 -> 6.33 mm
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- added copper zone on layer 16, net +12V_BAT
- added copper zone on layer 16, net +12V_CONVERTER
- added copper zone on layer 16, net +200VDC_I_SENSE
- added copper zone on layer 16, net +200VDC_OUT
- added copper zone on layer 16, net -VBAT
- added copper zone on layer 16, net LAMP1_ON
- added copper zone on layer 16, net LAMP2_ON
- added copper zone on layer 16, net N$10
- added copper zone on layer 16, net N$25
- added copper zone on layer 16, net N$30
- added copper zone on layer 16, net N$64
- added copper zone on layer 16, net N$65
- added copper zone on layer 16, net N$66
- added copper zone on layer 16, net N$67
- added copper zone on layer 16, net N$8
- added copper zone on layer 16, net N$91

Commit message: 12 to 200V inverter. Almost routed.
Parts:
- R7: device __MyCommonLib1:RSMD_1206_BIG_GAP -> __MyCommonLib1:RSMD_0805
- moved D23 30.0 mm to (59.4, 57.0), turned to 180 degrees
- moved R7 11.8 mm to (68.0, 68.0)
- moved C38 3.54 mm to (53.4, 29.0), turned to 270 degrees
- moved D2 3.30 mm to (42.0, 72.6)
- moved R1 3.22 mm to (45.4, 73.8)
- moved R90 2.53 mm to (33.0, 81.0), turned to 270 degrees
- moved C7 2.00 mm to (36.0, 25.0), turned to 270 degrees
- moved D24 2.00 mm to (36.0, 77.0)
- moved R4 1.34 mm to (52.0, 75.4)
- moved D17 1.28 mm to (43.6, 79.6)
- moved D16 1.08 mm to (64.0, 57.6)
- moved D25 1.00 mm to (39.0, 77.0)
- moved T1 1.00 mm to (54.0, 68.0)
- moved R114 0.85 mm to (46.8, 83.4)
- moved T23 0.85 mm to (42.6, 83.4)
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Routing:
- net N$93: track 6.15 -> 45.4 mm
- net N$14: track 5.84 -> 22.4 mm, vias 0 -> 2
- net +12V_BAT: track 94.7 -> 105.1 mm, vias 4 -> 10
- net N$17: track 11.2 -> 3.33 mm
- net N$26: track 0.00 -> 6.64 mm
- net N$109: track 6.10 -> 11.3 mm
- net ANY_LAMP_ON: track 15.5 -> 11.2 mm
- net GND: track 276.2 -> 273.6 mm
- net N$9: track 7.51 -> 9.06 mm
- net N$73: track 9.68 -> 10.8 mm
- net -VBAT: track 64.6 -> 65.5 mm
- net N$126: track 6.56 -> 5.71 mm
- net SENSE_BAT_VOLTAGE: track 46.8 -> 47.6 mm
- added copper zone on layer 16, net N$24

Commit message: 12 to 200V inverter. Routed.
Parts:
- moved R50 2.00 mm to (108.0, 23.0), turned to 180 degrees
- moved R30 1.40 mm to (123.4, 25.8)
- moved R53 0.60 mm to (112.4, 23.0), turned to 180 degrees
- moved LED1 0.40 mm to (146.6, 82.0)
- moved LED3 0.40 mm to (146.6, 77.0)
- moved LED5 0.40 mm to (146.6, 72.0)
- moved LED7 0.40 mm to (146.6, 67.0)
- moved F2 0.20 mm to (135.6, 50.0)
Routing:
- net N$38: track 60.3 -> 44.4 mm
- net N$50: track 53.3 -> 50.2 mm
- net LED_SCK(MISO): track 76.0 -> 78.8 mm
- net N$20: track 12.8 -> 10.1 mm
- net N$100: track 17.4 -> 19.4 mm
- net N$78: track 14.6 -> 16.4 mm
- net N$4: track 9.99 -> 11.6 mm
- net CONVERTER_ON: track 23.9 -> 25.5 mm
- net SENSE_BAT_VOLTAGE: track 47.6 -> 48.8 mm
- net N$43: track 10.5 -> 9.45 mm
- net N$55: track 32.9 -> 31.9 mm
- net N$37: track 11.0 -> 10.1 mm
- net +5V: track 55.2 -> 56.1 mm
- net N$23: track 19.4 -> 18.5 mm
- net GND: track 273.6 -> 272.8 mm
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- added copper zone on layer 16, net N$38
- added copper zone on layer 16, net N$45
