File: 12_to_200V_inverter/schematic/12to220inverterVer3.brd (EAGLE design)
At the start: 160 x 100 mm, 254 parts, among them IC1 UC3842, IC10 TL494, IC2 PC817, IC3 LM358, IC4 TL431, IC5 LM317, IC6 74HC595, IC7 74HC595, IC8 ATTINY45, IC9 TL431, J100 0, J2 0, J3 0, T10 16N60, T11 BC847, T12 BC847, T13 AO3401, T14 AO3401, T15 BC847, T16 BSS84, T17 BC847, T18 BC847, T19 BSS84, T2 IRF830, T21 BC847, T22 BC847, T23 BSS84, T24 BC847, T3 IRF830, T4 BC847, T5 BC857, T6 BC857, T7 IRFZ24N, T8 IRFZ24N, T9 BC857, U100 DF06S, X1 BAT+, X2 LAMP1, X3 LAMP1, X4 BAT-, X5 220VAC, X6 LAMP1_SWITCH, X7 LAMP1_SWITCH, X8 MCU_PROGRAMMING

Commit message: 12 to 200V inverter. New board with ETD transformers. Route.
Parts:
- removed D11: SR3A0, __MyCommonLib1:DO-27_15MM
- added D101: MBR20100CT, __MyCommonLib1:TO-220(VER2)_BIG_PADS
- CE2: device __MyCommonLib1:CE_13MM -> __MyCommonLib1:CE_10MM
- D2: device __MyCommonLib1:DO-41_5MM -> __MyCommonLib1:DO-41_10MM
- D23: device __MyCommonLib1:SOD-80 -> __MyCommonLib1:DO-35_10MM
- IC8: device __MyCommonLib1:SOIC8(0.15'') -> __MyCommonLib1:PSOP8(0.208'')
- moved D5 66.1 mm to (39.0, 47.2)
- moved R14 63.5 mm to (35.0, 50.9)
- moved T5 53.8 mm to (35.0, 46.9)
- moved D6 50.6 mm to (25.0, 44.0)
- moved R15 41.9 mm to (28.1, 45.5), turned to 90 degrees
- moved T6 39.9 mm to (21.2, 44.5)
- moved D19 26.0 mm to (115.5, 59.0), turned to 0 degrees
- moved D2 23.8 mm to (68.9, 73.0), turned to 0 degrees
- moved R4 22.0 mm to (70.0, 70.0), turned to 180 degrees
- moved R1 19.7 mm to (74.0, 69.0)
- moved ZD4 17.7 mm to (68.9, 73.0), turned to 180 degrees
- moved T14 15.8 mm to (70.0, 66.4)
- moved R80 11.3 mm to (55.0, 42.9), turned to 180 degrees
- moved D23 10.4 mm to (60.5, 53.1), turned to 90 degrees
- moved C9 10.3 mm to (-5.40, 32.7)
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Connections:
- net CHARGER_POWER: now also D101.2, D23.A; no longer D11.CATHODE, D23.ANODE
- net N$58: now also D101.1, D101.3; no longer D11.ANODE
- net N$93: now also D23.C; no longer D23.CATHODE
Routing:
- net N$32: track 0.00 -> 85.7 mm
- net GND: track 256.4 -> 323.5 mm
- net +12V_BAT: track 80.6 -> 140.9 mm
- net -VBAT: track 61.3 -> 113.6 mm, vias 0 -> 2
- net N$22: track 0.00 -> 47.7 mm
- net N$58: track 0.00 -> 32.7 mm
- net N$29: track 0.00 -> 28.2 mm
- net N$61: track 0.00 -> 27.6 mm
- net CHARGER_POWER: track 0.00 -> 26.5 mm
- net N$98: track 34.8 -> 58.6 mm
- net N$28: track 0.00 -> 23.8 mm
- net N$14: track 41.9 -> 19.2 mm, vias 2 -> 0
- net N$102: track 42.4 -> 20.8 mm
- net N$27: track 0.00 -> 18.6 mm
- net N$8: track 0.00 -> 16.7 mm
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
Commit message: 12 to 200V inverter. New board with ETD transformers. Finally routed.
Parts:
- added J101: 0, __MyCommonLib1:RSMD_0805
- D23: device __MyCommonLib1:DO-35_10MM -> __MyCommonLib1:DO-35_15MM
- D3, ZD2: device __MyCommonLib1:DO-41_5MM -> __MyCommonLib1:DO-41_10MM
- D4: device __MyCommonLib1:DO-41_12.5MM -> __MyCommonLib1:DO-41_10MM
- R76: device __MyCommonLib1:RSMD_1206_BIG_GAP -> __MyCommonLib1:RSMD_0805
- R80: device __MyCommonLib1:R_1.0W_VERTICAL -> __MyCommonLib1:R_1.0W
- moved D4 54.7 mm to (16.1, 42.0)
- moved C16 36.4 mm to (78.0, 2.20)
- moved C9 14.5 mm to (9.00, 34.0), turned to 180 degrees
- moved R3 12.6 mm to (11.0, 57.0)
- moved R48 10.8 mm to (86.4, 32.0), turned to 180 degrees
- moved C15 9.98 mm to (86.4, 34.7)
- moved R80 9.07 mm to (64.0, 44.0), turned to 0 degrees
- moved R2 8.55 mm to (5.00, 57.0)
- moved R47 8.07 mm to (86.4, 29.3), turned to 180 degrees
- moved R14 8.01 mm to (41.0, 45.6), turned to 270 degrees
- moved D101 7.86 mm to (64.0, 50.0)
- moved C6 7.75 mm to (44.5, 36.9)
- moved D2 5.97 mm to (74.0, 69.9), turned to 90 degrees
- moved D5 5.57 mm to (37.0, 42.0), turned to 180 degrees
- moved IC7 5.46 mm to (137.0, 82.9), turned to 90 degrees
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Connections:
- new net N$104: IC7.12, J101.PAD_1
- net LED_LATCH: now also J101.PAD_0; no longer IC7.12
- net N$48: now also C15.PAD_1; no longer R47.PAD_0, R48.PAD_0
- net N$49: now also C15.PAD_0, R47.PAD_0, R48.PAD_0; no longer C15.PAD_1, R47.PAD_1, R48.PAD_1
- net N$50: now also R47.PAD_1, R48.PAD_1; no longer C15.PAD_0
Routing:
- net +12V_BAT: track 140.9 -> 51.7 mm, vias 6 -> 4
- net N$32: track 85.7 -> 6.32 mm
- net GND: track 323.5 -> 249.6 mm, vias 8 -> 9
- net N$22: track 47.7 -> 2.86 mm
- net N$58: track 32.7 -> 0.00 mm
- net N$29: track 28.2 -> 0.00 mm
- net N$61: track 27.6 -> 0.00 mm
- net CHARGER_POWER: track 26.5 -> 0.00 mm
- net +5V: track 60.2 -> 86.1 mm
- net N$28: track 23.8 -> 0.00 mm
- net CONV_PWM2: track 21.7 -> 44.1 mm, vias 0 -> 2
- net N$82: track 0.00 -> 17.7 mm
- net N$27: track 18.6 -> 2.86 mm
- net N$81: track 0.00 -> 15.1 mm
- net N$104: track 0.00 -> 14.2 mm, vias 1 -> 0
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- added copper zone on layer 16, net CHARGER_POWER
- added copper zone on layer 16, net N$15
- added copper zone on layer 16, net N$22
- added copper zone on layer 16, net N$24
- added copper zone on layer 16, net N$25
- added copper zone on layer 16, net N$27
- added copper zone on layer 16, net N$28
- added copper zone on layer 16, net N$29
- added copper zone on layer 16, net N$30
- added copper zone on layer 16, net N$36
- added copper zone on layer 16, net N$37
- added copper zone on layer 16, net N$40
- added copper zone on layer 16, net N$58
- added copper zone on layer 16, net N$61
- added copper zone on layer 16, net N$70
Other:
- board text added: "BAT+"

Commit message: 12 to 200V inverter. New board with ETD transformers. Finally routed.
Parts:
- IC4: device __MyCommonLib1:TO-92A(PINS_SWAPED) -> __MyCommonLib1:TO-92A
- moved RT1 2.28 mm to (154.0, 52.4)
- moved X5 2.28 mm to (145.2, 53.0)
- moved C11 2.11 mm to (149.9, 44.6)
- moved R29 2.11 mm to (146.9, 37.9)
- moved R32 2.11 mm to (151.9, 37.9)
- moved TR2 2.11 mm to (149.4, 32.8)
- moved RV1 2.11 mm to (153.5, 21.5)
- moved U100 1.50 mm to (141.4, 21.8)
- moved IC4 1.20 mm to (125.0, 73.0), flipped to the top
- moved F2 0.70 mm to (136.0, 50.5)
- moved C12 0.50 mm to (150.0, 15.8)
Routing:
- net GND: track 249.6 -> 241.4 mm
- net N$32: track 6.32 -> 0.00 mm
- net N$68: track 21.6 -> 15.9 mm
- net N$62: track 18.8 -> 14.9 mm
- added copper zone on layer 16, net N$62
- added copper zone on layer 16, net N$68

Commit message: 12 to 200V inverter. New board with ETD transformers. Finally routed.
Parts:
- added R110: *, __MyCommonLib1:RSMD_1206
- F2: device __MyCommonLib1:FUSE_20X5.6MM -> __MyCommonLib1:FUSE_20X5MM_VERT_WIRE
- moved C7 7.00 mm to (28.0, 26.0), turned to 0 degrees
- moved R9 7.00 mm to (35.0, 26.0), turned to 0 degrees
- moved R35 0.61 mm to (111.5, 5.50)
Connections:
- net N$24: now also R110.PAD_0, R9.PAD_0; no longer C7.PAD_1
- net N$25: now also C7.PAD_1; no longer R9.PAD_0
- net N$26: now also R110.PAD_1
Routing:
- net N$34: track 5.00 -> 0.00 mm
- net N$24: track 0.00 -> 4.04 mm
- net N$26: track 3.90 -> 7.94 mm
- added copper zone on layer 16, net N$34
- added copper zone on layer 16, net N$43

Commit message: 12 to 200V inverter. New board with ETD transformers. Finally routed.
Parts:
- moved RT1 0.85 mm to (154.6, 53.0)
Changed lines of the file:
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@@
 <element name="TR2" library="__MyCommonLib1" package="EMI_CM_21X17" value="EMI" x="149.4" y="32.8" rot="R270"/>
 <element name="C12" library="__MyCommonLib1" package="MKP_18X6" value="0.1uF x 275VAC X2" x="150" y="15.8" rot="R90"/>
-<element name="RT1" library="__MyCommonLib1" package="NTC_9.0X4.2" value="5 Ohm" x="154" y="52.4" rot="R90"/>
+<element name="RT1" library="__MyCommonLib1" package="NTC_9.0X4.2" value="5 Ohm" x="154.6" y="53" rot="R90"/>
 <element name="CE1" library="__MyCommonLib1" package="CE_13MM" value="22uF x 400V" x="102.5" y="7.1" rot="R270"/>
 <element name="R29" library="__MyCommonLib1" package="RSMD_0805" value="240K" x="146.9" y="37.9" smashed="yes" rot="MR0">
@@
 <vertex x="150.2" y="48"/>
 <vertex x="152.8" y="48"/>
-<vertex x="153.6" y="48.8"/>
-<vertex x="153.6" y="50.6"/>
+<vertex x="154.2" y="49.4"/>
+<vertex x="154.2" y="50.1"/>
 </polygon>
 </signal>
@@
 <vertex x="134.1" y="59.8"/>
 <vertex x="135.9" y="58"/>
-<vertex x="151.7" y="58"/>
-<vertex x="155.2" y="54.5"/>
-<vertex x="156.1" y="54.5"/>
-<vertex x="156.5" y="54.9"/>
+<vertex x="152.2" y="58"/>
+<vertex x="155.3" y="54.9"/>
+<vertex x="156.1" y="54.9"/>
+<vertex x="156.5" y="55.3"/>
 <vertex x="156.5" y="56.6"/>
 <vertex x="155.9" y="57.2"/>
 <vertex x="154.8" y="57.2"/>
 <vertex x="153.2" y="58.8"/>
-<vertex x="140.7" y="58.8"/>
-<vertex x="137.6" y="61.9"/>
+<vertex x="140" y="58.8"/>
+<vertex x="136.9" y="61.9"/>
 </polygon>
 </signal>

Commit message: 12 to 200V inverter. Timny changes to schematic and board.
Parts:
- F2: value 0.3A -> 2A
- R100, R101, R102, R103, R104, R105, R106, R99: value 1K0 -> 2K2
- R115: value 1K -> 1K0
- RT2, RT3: value 22K_20deg -> 100K_20deg
- flipped D23 to the top, turned to 180 degrees

Commit message: 12 to 200V inverter. Last steps.
Parts:
- R81: value 240R -> 470R
- turned ZD4 to 0 degrees
Connections:
- net N$14: now also ZD4.ANODE; no longer ZD4.CATHODE
- net N$9: now also ZD4.CATHODE; no longer ZD4.ANODE
Changed lines of the file:
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@@
 <grid distance="0.1" unitdist="mm" unit="mm" style="lines" multiple="10" display="yes" altdistance="0.025" altunitdist="inch" altunit="inch"/>
 <layers>
-<layer number="1" name="Top" color="4" fill="1" visible="no" active="yes"/>
+<layer number="1" name="Top" color="4" fill="1" visible="yes" active="yes"/>
 <layer number="2" name="Route2" color="1" fill="3" visible="no" active="no"/>
 <layer number="3" name="Route3" color="4" fill="3" visible="no" active="no"/>
@@
 <layer number="14" name="Route14" color="1" fill="6" visible="no" active="no"/>
 <layer number="15" name="Route15" color="4" fill="6" visible="no" active="no"/>
-<layer number="16" name="Bottom" color="1" fill="1" visible="no" active="yes"/>
+<layer number="16" name="Bottom" color="1" fill="1" visible="yes" active="yes"/>
 <layer number="17" name="Pads" color="2" fill="1" visible="yes" active="yes"/>
 <layer number="18" name="Vias" color="2" fill="1" visible="yes" active="yes"/>
 <layer number="19" name="Unrouted" color="6" fill="1" visible="yes" active="yes"/>
 <layer number="20" name="Dimension" color="15" fill="1" visible="yes" active="yes"/>
-<layer number="21" name="tPlace" color="7" fill="1" visible="no" active="yes"/>
+<layer number="21" name="tPlace" color="7" fill="1" visible="yes" active="yes"/>
 <layer number="22" name="bPlace" color="7" fill="1" visible="yes" active="yes"/>
-<layer number="23" name="tOrigins" color="15" fill="1" visible="no" active="yes"/>
+<layer number="23" name="tOrigins" color="15" fill="1" visible="yes" active="yes"/>
 <layer number="24" name="bOrigins" color="15" fill="1" visible="yes" active="yes"/>
 <layer number="25" name="tNames" color="7" fill="1" visible="no" active="yes"/>
 <layer number="26" name="bNames" color="7" fill="1" visible="no" active="yes"/>
 <layer number="27" name="tValues" color="7" fill="1" visible="no" active="yes"/>
-<layer number="28" name="bValues" color="7" fill="1" visible="yes" active="yes"/>
+<layer number="28" name="bValues" color="7" fill="1" visible="no" active="yes"/>
 <layer number="29" name="tStop" color="7" fill="3" visible="no" active="yes"/>
 <layer number="30" name="bStop" color="7" fill="6" visible="no" active="yes"/>
@@
 <layer number="38" name="bTest" color="7" fill="1" visible="no" active="yes"/>
 <layer number="39" name="tKeepout" color="4" fill="11" visible="no" active="yes"/>
-<layer number="40" name="bKeepout" color="1" fill="11" visible="yes" active="yes"/>
+<layer number="40" name="bKeepout" color="1" fill="11" visible="no" active="yes"/>
 <layer number="41" name="tRestrict" color="4" fill="10" visible="no" active="yes"/>
 <layer number="42" name="bRestrict" color="1" fill="10" visible="no" active="yes"/>
@@
 <text x="12.1" y="46" size="1.778" layer="16" font="vector" ratio="25" rot="MR90">BAT-</text>
 <text x="46" y="10" size="1.778" layer="16" font="vector" ratio="25" rot="MR90">BAT+</text>
+<wire x1="18" y1="49" x2="18" y2="43" width="0.1" layer="21"/>
+<wire x1="18" y1="43" x2="29" y2="43" width="0.1" layer="21"/>
+<wire x1="29" y1="43" x2="29" y2="36" width="0.1" layer="21"/>
+<wire x1="29" y1="36" x2="32" y2="36" width="0.1" layer="21"/>
+<wire x1="32" y1="36" x2="32" y2="43" width="0.1" layer="21"/>
+<wire x1="32" y1="43" x2="44" y2="43" width="0.1" layer="21"/>
+<wire x1="44" y1="43" x2="44" y2="36" width="0.1" layer="21"/>
+<wire x1="44" y1="36" x2="48" y2="36" width="0.1" layer="21"/>
+<wire x1="48" y1="36" x2="53" y2="41" width="0.1" layer="21"/>
+<wire x1="53" y1="41" x2="53" y2="53" width="0.1" layer="21"/>
+<wire x1="53" y1="53" x2="45" y2="53" width="0.1" layer="21"/>
+<wire x1="45" y1="53" x2="44" y2="54" width="0.1" layer="21"/>
+<wire x1="44" y1="54" x2="44" y2="58" width="0.1" layer="21"/>
+<wire x1="44" y1="58" x2="27" y2="58" width="0.1" layer="21"/>
+<wire x1="27" y1="58" x2="27" y2="51" width="0.1" layer="21"/>
+<wire x1="27" y1="51" x2="25" y2="49" width="0.1" layer="21"/>
+<wire x1="25" y1="49" x2="18" y2="49" width="0.1" layer="21"/>
 </plain>
 <attributes>
@@
 <attribute name="VALUE" x="62" y="43" size="1.016" layer="27" font="vector" ratio="20"/>
 </element>
-<element name="R81" library="__MyCommonLib1" package="RSMD_0805" value="240R" x="109" y="67" smashed="yes" rot="MR270">
+<element name="R81" library="__MyCommonLib1" package="RSMD_0805" value="470R" x="109" y="67" smashed="yes" rot="MR270">
 <attribute name="NAME" x="109" y="67" size="1.016" layer="26" font="vector" ratio="20" rot="MR270"/>
 <attribute name="VALUE" x="109.6" y="69" size="1.016" layer="28" font="vector" ratio="20" rot="MR270"/>
@@
 <attribute name="VALUE" x="72.5" y="64.7" size="1.016" layer="28" font="vector" ratio="20" rot="MR0"/>
 </element>
-<element name="ZD4" library="__MyCommonLib1" package="SOD-80" value="5V6" x="68.9" y="75" smashed="yes" rot="MR180">
-<attribute name="NAME" x="68.9" y="75" size="1.016" layer="26" font="vector" ratio="20" rot="MR180"/>
-<attribute name="VALUE" x="67.4" y="77.7" size="1.016" layer="28" font="vector" ratio="20" rot="MR180"/>
+<element name="ZD4" library="__MyCommonLib1" package="SOD-80" value="5V6" x="68.9" y="75" smashed="yes" rot="MR0">
+<attribute name="NAME" x="68.9" y="75" size="1.016" layer="26" font="vector" ratio="20" rot="MR0"/>
+<attribute name="VALUE" x="70.4" y="72.3" size="1.016" layer="28" font="vector" ratio="20" rot="MR0"/>
 </element>
 <element name="ZD5" library="__MyCommonLib1" package="SOD-80" value="5V6" x="28" y="85.5" smashed="yes" rot="MR90">
@@
 <contactref element="R7" pad="PAD_1"/>
 <contactref element="T14" pad="1"/>
-<contactref element="ZD4" pad="CATHODE"/>
 <wire x1="72.4" y1="67.4" x2="76.2" y2="67.4" width="0.6" layer="16"/>
 <wire x1="77.9" y1="67.95" x2="77.95" y2="68" width="0.6" layer="16"/>
 <wire x1="68.95" y1="72" x2="68.65" y2="72.3" width="0.8" layer="16"/>
 <wire x1="68.65" y1="72.3" x2="67.9" y2="72.3" width="0.8" layer="16"/>
-<wire x1="67.025" y1="75" x2="67.2" y2="74.825" width="0.8" layer="16"/>
-<wire x1="67.2" y1="74.825" x2="67.2" y2="73" width="0.8" layer="16"/>
+<wire x1="67.2" y1="75" x2="67.2" y2="73" width="0.8" layer="16"/>
 <wire x1="67.2" y1="73" x2="67.9" y2="72.3" width="0.8" layer="16"/>
 <wire x1="68.95" y1="72" x2="68.95" y2="70.85" width="0.8" layer="16"/>
@@
 <wire x1="77.9" y1="67.95" x2="76.75" y2="67.95" width="1" layer="16"/>
 <wire x1="76.75" y1="67.95" x2="76.2" y2="67.4" width="1" layer="16"/>
+<contactref element="ZD4" pad="ANODE"/>
+<wire x1="67.025" y1="75" x2="67.2" y2="75" width="0.8" layer="16"/>
 </signal>
 <signal name="N$16">
@@
 <contactref element="D2" pad="CATHODE"/>
 <contactref element="R1" pad="PAD_1"/>
-<contactref element="ZD4" pad="ANODE"/>
-<wire x1="70.775" y1="75" x2="71" y2="74.775" width="0.6" layer="16"/>
 <wire x1="71" y1="74.775" x2="71" y2="72.05" width="0.6" layer="16"/>
 <wire x1="74" y1="72.55" x2="73.95" y2="72.5" width="0.6" layer="16"/>
@@
 <wire x1="74" y1="72.55" x2="74" y2="74.98" width="0.6" layer="16"/>
 <wire x1="71" y1="72.05" x2="71.05" y2="72" width="0.6" layer="16"/>
+<contactref element="ZD4" pad="CATHODE"/>
+<wire x1="70.775" y1="75" x2="71" y2="75" width="0.8" layer="16"/>
+<wire x1="71" y1="75" x2="71" y2="74.775" width="0.8" layer="16"/>
 </signal>
 <signal name="+200VDC_I_SENSE">
@@
 <vertex x="55.7" y="40.9"/>
 <vertex x="55.7" y="44.9"/>
-<vertex x="54.9" y="45.7"/>
-<vertex x="47.5" y="45.7"/>
+<vertex x="54.7" y="45.9"/>
+<vertex x="47.3" y="45.9"/>
 <vertex x="44.7" y="48.5"/>
 <vertex x="44.7" y="49.4"/>
@@
 <via x="155" y="92" extent="1-16" drill="3.5" diameter="6"/>
 </signal>
+<signal name="N$119">
+<via x="32" y="48" extent="1-16" drill="3" diameter="3.2"/>
+</signal>
+<signal name="N$120">
+<via x="49" y="42" extent="1-16" drill="3" diameter="3.2"/>
+</signal>
 </signals>
