File: 12_to_200V_inverter/schematic/12to220inverterVer3.sch (EAGLE design)
At the start: 245 parts, among them IC1 UC3842, IC10 TL494, IC2 PC817, IC3 LM358SOIC8, IC4 TL431, IC5 LM317, IC6 74HC595, IC7 74HC595, IC8 ATTINY45, T1 AO4407AL, T10 16N60, T11 BC847, T12 BC847, T13 BSS84, T14 BC857, T15 BC847, T16 BSS84, T17 BC847, T18 BC847, T19 BSS84, T2 IRF830, T20 BSS84, T21 BC847, T22 BC847, T23 BSS84, T24 BC847, T3 IRF830, T4 BC847, T5 BC857, T6 BC857, T7 IRFZ24N, T8 IRFZ24N, T9 BC857, X1 BAT+, X2 LAMP1, X3 LAMP1, X4 BAT-, X5 220VAC, X6 LAMP1_SWITCH, X7 LAMP1_SWITCH, X8 MCU_PROGRAMMING

Commit message: 12 to 200V converter. Ver3.
Parts:
- added HS1: 21X16MM, __MyCommonLib1:HEATSINK_21X16MM
- D10, D12, D13, D8, D9: device __MyCommonLib1:1N4001DO-41_10MM -> __MyCommonLib1:1N4001DO-41_5MM
- ZD2: device __MyCommonLib1:ZENNERDO-41_10MM -> __MyCommonLib1:ZENNERDO-41_5MM
Connections:
- net N$35: now also HS1.PIN0
Other:
- moved on the sheet: C15, C16, CE4, D14, R47, R48, R50, T10

Commit message: 12 to 200V converter. Ver3. Start simplification.
Parts:
- removed R31, R37, R38: 120K, __MyCommonLib1:RSMD_1206
- removed R33, R34, R36: 33K, __MyCommonLib1:RSMD_1206
- D10, D12, D13, D8, D9: device __MyCommonLib1:1N4001DO-41_5MM -> __MyCommonLib1:1N4001DO-41_10MM
- R30: device __MyCommonLib1:RSMD_1206 -> __MyCommonLib1:R1.0W
- R35: device __MyCommonLib1:RSMD_1206 -> __MyCommonLib1:R1.0W_VERT
- ZD2: device __MyCommonLib1:ZENNERDO-41_5MM -> __MyCommonLib1:ZENNERDO-41_10MM
Connections:
- removed net N$40: R31.PIN0, R38.PIN1
- removed net N$41: R30.PIN0, R37.PIN1
- removed net N$52: R33.PIN1, R34.PIN0
- removed net N$53: R35.PIN1, R36.PIN0
- net N$32: now also R35.PIN1; no longer R31.PIN1, R34.PIN1, R36.PIN1
- net N$36: no longer R33.PIN0
- net N$38: now also R30.PIN0; no longer R37.PIN0, R38.PIN0
Other:
- moved on the sheet: R30, R35

Commit message: 12 to 200V converter. Ver3. Start simplification.
Parts:
- removed R51: 5K6, __MyCommonLib1:RSMD_0805
- removed R56: 560R, __MyCommonLib1:RSMD_0805
- removed T14: BC857, __MyCommonLib1:BC857SOT23_SMALL_PADS
- added J1: 0, __MyCommonLib1:RSMD_1206_BIG_GAP
- R30: device __MyCommonLib1:R1.0W -> __MyCommonLib1:R1.0W_VERT
Connections:
- removed net N$54: R51.PIN0, R56.PIN1, T14.B
- new net N$40: IC2.COLLECTOR, J1.PIN0
- net N$23: no longer R51.PIN1
- net N$43: no longer T14.E
- net N$50: no longer R56.PIN0, T14.C
- net N$55: now also J1.PIN1; no longer IC2.COLLECTOR
Other:
- moved on the sheet: IC2, R50, R53, R57

Commit message: 12 to 200V converter. Ver3. Start simplification.
Parts:
- added C37: 0.1uF, __MyCommonLib1:CSMD_0805
- added C38: 1000uFx25V, __MyCommonLib1:CE10MM
- added IC9: TL431, __MyCommonLib1:TL431SOT23
- added J2: 0, __MyCommonLib1:RSMD_1206_BIG_GAP
- added R31: 1K0, __MyCommonLib1:RSMD_0805
- R72: value 10K -> 4K7
Connections:
- removed net N$57: R66.END_B, R75.PIN1
- removed net N$63: R63.PIN0, R66.END_A
- new net N$41: IC2.EMITER, J2.PIN0
- new net N$52: R63.PIN0, R66.END_B
- new net N$53: R66.END_A, R75.PIN1
- new net N$54: C37.PIN0, IC9.CATHODE, IC9.REFERENCE, R31.PIN1, R72.PIN1
- net +12V_BAT: now also C38.PLUS
- net -VBAT: now also C38.MINUS
- net GND: now also C37.PIN1, IC9.ANODE
- net N$100: now also IC3G$1.OUT; no longer IC3G$2.OUT
- net N$102: now also IC3G$1.IN+; no longer IC3G$2.IN+
- net N$103: now also IC3G$2.OUT; no longer IC3G$1.OUT
- net N$131: now also IC3G$2.IN+; no longer IC3G$1.IN+
- net N$32: now also C16.PIN1
- net N$50: now also J2.PIN1; no longer C16.PIN1, IC2.EMITER
- net N$97: now also IC3G$2.IN-; no longer IC3G$1.IN-
- net N$98: now also R31.PIN0; no longer R72.PIN1
- net N$99: now also IC3G$1.IN-; no longer IC3G$2.IN-
Other:
- moved on the sheet: C16, C21, C22, C24, C41, D29, D30, D4, IC2, IC3G$1, IC3G$2, IC3G$3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

Commit message: 12 to 200V converter. Ver3. Routing.
Parts:
- removed C9: 0.1uF x 10V, __MyCommonLib1:CSMD_0805
- D1, D3: device __MyCommonLib1:1N4001DO-41_10MM -> __MyCommonLib1:1N4001DO-41_5MM
- R11: device __MyCommonLib1:R1.0W_VERT -> __MyCommonLib1:R1.0W
Connections:
- removed net N$15: C2.MINUS, D3.ANODE, R3.PIN0, TR1.PRI_START
- net -VBAT: now also C2.MINUS, D3.ANODE, R3.PIN0, TR1.PRI_START; no longer C9.PIN1
- net N$7: no longer C9.PIN0
Other:
- moved on the sheet: R19
Changed lines of the file:
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@@
 <part name="R9" library="__MyCommonLib1" deviceset="R" device="SMD_1206" value="20R"/>
 <part name="C1" library="__MyCommonLib1" deviceset="CE" device="13MM" value="20uF x 450V"/>
-<part name="D3" library="__MyCommonLib1" deviceset="1N4001" device="DO-41_10MM" value="UF4007"/>
-<part name="R11" library="__MyCommonLib1" deviceset="R" device="1.0W_VERT" value="1R0"/>
+<part name="D3" library="__MyCommonLib1" deviceset="1N4001" device="DO-41_5MM" value="UF4007"/>
+<part name="R11" library="__MyCommonLib1" deviceset="R" device="1.0W" value="1R0"/>
 <part name="C4" library="__MyCommonLib1" deviceset="C" device="SMD_0805" value="0.47uFx25V"/>
 <part name="C3" library="__MyCommonLib1" deviceset="CE" device="6.3MM" value="100uFx25V"/>
@@
 <part name="R26" library="__MyCommonLib1" deviceset="R" device="SMD_0805" value="51K"/>
 <part name="ZD1" library="__MyCommonLib1" deviceset="ZENNER" device="(SOD_80)" value="4.7V"/>
-<part name="D1" library="__MyCommonLib1" deviceset="1N4001" device="DO-41_10MM" value="UF4007"/>
+<part name="D1" library="__MyCommonLib1" deviceset="1N4001" device="DO-41_5MM" value="UF4007"/>
 <part name="C2" library="__MyCommonLib1" deviceset="CE" device="13MM" value="20uF x 450V"/>
 <part name="R27" library="__MyCommonLib1" deviceset="R" device="SMD_0805" value="10K"/>
@@
 <part name="D7" library="__MyCommonLib1" deviceset="LL4147" device="SOD-80" value="MBR0540"/>
 <part name="R18" library="__MyCommonLib1" deviceset="R" device="SMD_0805" value="150R"/>
-<part name="C9" library="__MyCommonLib1" deviceset="C" device="SMD_0805" value="0.1uF x 10V"/>
 <part name="FRAME1" library="frames" deviceset="A4L-LOC" device="" value="12_TO_200VDC_CONVERTER"/>
 <part name="X5" library="__MyCommonLib1" deviceset="PIN1X2" device="BRD_CONN_12X10.2" value="220VAC"/>
@@
 <attribute name="VALUE" x="31.75" y="46.99" size="1.27" layer="96" font="vector" ratio="20"/>
 </instance>
-<instance part="R19" gate="R$1" x="58.42" y="60.96" smashed="yes" rot="R180">
-<attribute name="NAME" x="60.96" y="63.5" size="1.27" layer="95" font="vector" ratio="20"/>
-<attribute name="VALUE" x="60.96" y="60.96" size="1.27" layer="96" font="vector" ratio="20"/>
+<instance part="R19" gate="R$1" x="53.34" y="60.96" smashed="yes" rot="R180">
+<attribute name="NAME" x="55.88" y="63.5" size="1.27" layer="95" font="vector" ratio="20"/>
+<attribute name="VALUE" x="55.88" y="60.96" size="1.27" layer="96" font="vector" ratio="20"/>
 </instance>
 <instance part="D7" gate="D1" x="25.4" y="68.58" smashed="yes" rot="R270">
@@
 <attribute name="NAME" x="30.48" y="66.04" size="1.27" layer="95" font="vector" ratio="20"/>
 <attribute name="VALUE" x="35.56" y="66.04" size="1.27" layer="96" font="vector" ratio="20"/>
-</instance>
-<instance part="C9" gate="C$1" x="53.34" y="58.42" smashed="yes" rot="MR180">
-<attribute name="NAME" x="48.26" y="71.12" size="1.27" layer="95" font="vector" ratio="20" rot="MR180"/>
-<attribute name="VALUE" x="48.26" y="69.85" size="1.27" layer="96" font="vector" ratio="20" rot="MR180"/>
 </instance>
 <instance part="T2" gate="G$1" x="205.74" y="147.32" smashed="yes">
@@
 <pinref part="D4" gate="D$1" pin="CATHODE"/>
 <wire x1="22.86" y1="137.16" x2="22.86" y2="139.7" width="0.1524" layer="91"/>
+<pinref part="C6" gate="C$1" pin="PIN1"/>
 <wire x1="22.86" y1="139.7" x2="27.94" y2="139.7" width="0.1524" layer="91"/>
-<pinref part="C6" gate="C$1" pin="PIN1"/>
 <wire x1="27.94" y1="139.7" x2="33.02" y2="139.7" width="0.1524" layer="91"/>
 <wire x1="33.02" y1="139.7" x2="38.1" y2="139.7" width="0.1524" layer="91"/>
 <wire x1="38.1" y1="139.7" x2="38.1" y2="137.16" width="0.1524" layer="91"/>
+<junction x="33.02" y="139.7"/>
 <pinref part="C38" gate="C$1" pin="PLUS"/>
-<wire x1="27.94" y1="139.7" x2="27.94" y2="137.16" width="0.1524" layer="91"/>
-<junction x="33.02" y="139.7"/>
+<wire x1="27.94" y1="137.16" x2="27.94" y2="139.7" width="0.1524" layer="91"/>
 <junction x="27.94" y="139.7"/>
 </segment>
@@
 <net name="N$7" class="0">
 <segment>
-<wire x1="58.42" y1="68.58" x2="53.34" y2="68.58" width="0.1524" layer="91"/>
 <wire x1="53.34" y1="68.58" x2="48.26" y2="68.58" width="0.1524" layer="91"/>
 <wire x1="48.26" y1="68.58" x2="48.26" y2="60.96" width="0.1524" layer="91"/>
@@
 <pinref part="C8" gate="C$1" pin="PLUS"/>
 <pinref part="R19" gate="R$1" pin="PIN0"/>
-<wire x1="58.42" y1="66.04" x2="58.42" y2="68.58" width="0.1524" layer="91"/>
+<wire x1="53.34" y1="66.04" x2="53.34" y2="68.58" width="0.1524" layer="91"/>
 <pinref part="R18" gate="R$1" pin="PIN0"/>
 <wire x1="40.64" y1="68.58" x2="43.18" y2="68.58" width="0.1524" layer="91"/>
-<pinref part="C9" gate="C$1" pin="PIN0"/>
-<wire x1="53.34" y1="60.96" x2="53.34" y2="68.58" width="0.1524" layer="91"/>
-<junction x="53.34" y="68.58"/>
 </segment>
 </net>
@@
 <segment>
 <pinref part="IC10" gate="G$1" pin="1IN+"/>
-<wire x1="88.9" y1="45.72" x2="58.42" y2="45.72" width="0.1524" layer="91"/>
+<wire x1="88.9" y1="45.72" x2="53.34" y2="45.72" width="0.1524" layer="91"/>
 <pinref part="R21" gate="R$1" pin="PIN0"/>
 <pinref part="R19" gate="R$1" pin="PIN1"/>
-<wire x1="58.42" y1="45.72" x2="36.83" y2="45.72" width="0.1524" layer="91"/>
-<wire x1="58.42" y1="55.88" x2="58.42" y2="45.72" width="0.1524" layer="91"/>
-<junction x="58.42" y="45.72"/>
+<wire x1="53.34" y1="45.72" x2="36.83" y2="45.72" width="0.1524" layer="91"/>
+<wire x1="53.34" y1="55.88" x2="53.34" y2="45.72" width="0.1524" layer="91"/>
+<junction x="53.34" y="45.72"/>
 </segment>
 </net>
@@
 <pinref part="ZD1" gate="G$1" pin="ANODE"/>
 <wire x1="43.18" y1="50.8" x2="43.18" y2="55.88" width="0.1524" layer="91"/>
-<pinref part="C9" gate="C$1" pin="PIN1"/>
-<wire x1="53.34" y1="50.8" x2="53.34" y2="55.88" width="0.1524" layer="91"/>
 <wire x1="43.18" y1="50.8" x2="48.26" y2="50.8" width="0.1524" layer="91"/>
-<wire x1="48.26" y1="50.8" x2="53.34" y2="50.8" width="0.1524" layer="91"/>
 <wire x1="48.26" y1="50.8" x2="48.26" y2="55.88" width="0.1524" layer="91"/>
 <pinref part="C8" gate="C$1" pin="MINUS"/>
@@
 <wire x1="68.58" y1="55.88" x2="68.58" y2="50.8" width="0.1524" layer="91"/>
 <wire x1="68.58" y1="50.8" x2="76.2" y2="50.8" width="0.1524" layer="91"/>
-<wire x1="53.34" y1="50.8" x2="68.58" y2="50.8" width="0.1524" layer="91"/>
-<junction x="53.34" y="50.8"/>
+<wire x1="48.26" y1="50.8" x2="68.58" y2="50.8" width="0.1524" layer="91"/>
 <junction x="68.58" y="50.8"/>
 <pinref part="R20" gate="R$1" pin="PIN0"/>
@@
 <junction x="83.82" y="111.76"/>
 <pinref part="R11" gate="R$1" pin="PIN1"/>
-<wire x1="167.64" y1="111.76" x2="198.12" y2="111.76" width="0.1524" layer="91"/>
+<wire x1="167.64" y1="111.76" x2="182.88" y2="111.76" width="0.1524" layer="91"/>
+<wire x1="182.88" y1="111.76" x2="198.12" y2="111.76" width="0.1524" layer="91"/>
 <wire x1="198.12" y1="111.76" x2="218.44" y2="111.76" width="0.1524" layer="91"/>
 <wire x1="218.44" y1="111.76" x2="218.44" y2="119.38" width="0.1524" layer="91"/>
@@
 <wire x1="27.94" y1="129.54" x2="22.86" y2="129.54" width="0.1524" layer="91"/>
 <wire x1="22.86" y1="129.54" x2="22.86" y2="132.08" width="0.1524" layer="91"/>
-<pinref part="C38" gate="C$1" pin="MINUS"/>
-<wire x1="27.94" y1="132.08" x2="27.94" y2="129.54" width="0.1524" layer="91"/>
 <pinref part="C6" gate="C$1" pin="PIN0"/>
 <wire x1="38.1" y1="132.08" x2="38.1" y2="129.54" width="0.1524" layer="91"/>
 <wire x1="38.1" y1="129.54" x2="33.02" y2="129.54" width="0.1524" layer="91"/>
+<junction x="33.02" y="129.54"/>
+<pinref part="C38" gate="C$1" pin="MINUS"/>
+<wire x1="27.94" y1="132.08" x2="27.94" y2="129.54" width="0.1524" layer="91"/>
 <junction x="27.94" y="129.54"/>
-<junction x="33.02" y="129.54"/>
-</segment>
-</net>
-<net name="N$15" class="0">
-<segment>
 <pinref part="D3" gate="D$1" pin="ANODE"/>
 <wire x1="134.62" y1="157.48" x2="134.62" y2="152.4" width="0.1524" layer="91"/>
@@
 <junction x="144.78" y="152.4"/>
 <pinref part="TR1" gate="G$1" pin="PRI_START"/>
+<wire x1="149.86" y1="152.4" x2="182.88" y2="152.4" width="0.1524" layer="91"/>
+<wire x1="182.88" y1="152.4" x2="182.88" y2="111.76" width="0.1524" layer="91"/>
+<junction x="182.88" y="111.76"/>
+<junction x="149.86" y="152.4"/>
 </segment>
 </net>
@@
 <segment>
 <pinref part="R5" gate="R$1" pin="PIN1"/>
-<wire x1="185.42" y1="144.78" x2="172.72" y2="144.78" width="0.1524" layer="91"/>
-<label x="182.88" y="147.32" size="1.27" layer="95" font="vector" ratio="20" rot="R180"/>
-</segment>
-</net>
+<wire x1="185.42" y1="144.78" x2="170.18" y2="144.78" width="0.1524" layer="91"/>
+<label x="180.34" y="147.32" size="1.27" layer="95" font="vector" ratio="20" rot="R180"/>
+</segment>
+</net>

Commit message: 12 to 200V converter. Ver3. Routing.
Parts:
- D4: device __MyCommonLib1:1N4001DO-41_10MM -> __MyCommonLib1:1N4001DO-41_12.5MM
- IC5: device __MyCommonLib1:LM317(D2PAK) -> __MyCommonLib1:LM317TO-220(VER2)_BIG_PADS
- R73: device __MyCommonLib1:RSMD_0805 -> __MyCommonLib1:R0207
- R80: device __MyCommonLib1:R1.0W -> __MyCommonLib1:R1.0W_VERT
- R97, R98: device __MyCommonLib1:RSMD_1206_BIG_GAP -> __MyCommonLib1:RSMD_0805
- T10: device __MyCommonLib1:IRF830TO-220_VER2 -> __MyCommonLib1:IRF830TO-220_VER2_BIG_PADS
- T2, T3, T7, T8: device __MyCommonLib1:IRF830TO-220 -> __MyCommonLib1:IRF830TO-220_VER2_BIG_PADS
- X6, X7: device __MyCommonLib1:PIN1X22.54MM -> __MyCommonLib1:PIN1X22.54MM_WITH_CLAMP
Connections:
- removed net N$70: D21.ANODE, T19.DRAIN, T20.DRAIN
- new net N$15: D21.CATHODE, R84.PIN0, R85.PIN0, R86.PIN0
- net +12V_BAT: now also D21.ANODE; no longer R84.PIN0, R85.PIN0, R86.PIN0
- net CONVERTER_ON: now also IC6.QH; no longer IC6.QB
- net N$91: now also T19.DRAIN, T20.DRAIN; no longer D21.CATHODE
Other:
- moved on the sheet: D21, D23, D24, D25, R84, R85, R86, R89, R90, R91, T19, T20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

Commit message: 12 to 200V converter. Ver3. Routing.
Parts:
- added J3, J4: 0, __MyCommonLib1:RSMD_1206_BIG_GAP
- D2: device __MyCommonLib1:1N4001DO-41_10MM -> __MyCommonLib1:1N4001DO-41_5MM
- D21: device __MyCommonLib1:1N4001DO-41_10MM -> __MyCommonLib1:1N4001DO-41_12.5MM
- R7: device __MyCommonLib1:RSMD_0805 -> __MyCommonLib1:RSMD_1206_BIG_GAP
- R93: device __MyCommonLib1:RSMD_1206_BIG_GAP -> __MyCommonLib1:RSMD_0805
Connections:
- new net N$57: J3.PIN1, X8.3
- new net N$63: J4.PIN1, X8.4
- net -VBAT: no longer R13.PIN0, T4.E
- net BUZZER_ON: now also IC6.QF; no longer IC6.QA
- net CONVERTER_ON: now also IC6.QG; no longer IC6.QH
- net CONV_TEMP_ADC(SCK): now also J4.PIN0; no longer X8.4
- net GND: now also R13.PIN0, T4.E
- net LED_DATA(MOSI): now also J3.PIN0; no longer X8.3
- net SENSE_BAT_VOLTAGE: now also IC6.QH; no longer IC6.QD
- net ~ADD_CHARGE_VOLTAGE: now also IC6.QD; no longer IC6.QC
Other:
- moved on the sheet: R13, R7, R8, T4, X8

Commit message: 12 to 200V converter. Ver3. Routing.
Parts:
- added C9: 0.47uFx25V, __MyCommonLib1:CSMD_1206
- R1: device __MyCommonLib1:RSMD_0805 -> __MyCommonLib1:RSMD_1206
Connections:
- net +12V_BAT: now also C9.PIN1
- net -VBAT: now also C9.PIN0
Changed lines of the file:
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@@
 <part name="D21" library="__MyCommonLib1" deviceset="1N4001" device="DO-41_12.5MM" value="1N4001"/>
 <part name="T1" library="__MyCommonLib1" deviceset="AO4407" device="(SO8)" value="AO4407AL"/>
-<part name="R1" library="__MyCommonLib1" deviceset="R" device="SMD_0805" value="1R0"/>
+<part name="R1" library="__MyCommonLib1" deviceset="R" device="SMD_1206" value="1R0"/>
 <part name="X8" library="__MyCommonLib1" deviceset="PIN2X3" device="2.54MM_LOOSE_PADS" value="MCU_PROGRAMMING"/>
 <part name="GND98" library="supply1" deviceset="GND" device=""/>
@@
 <part name="J3" library="__MyCommonLib1" deviceset="R" device="SMD_1206_BIG_GAP" value="0"/>
 <part name="J4" library="__MyCommonLib1" deviceset="R" device="SMD_1206_BIG_GAP" value="0"/>
+<part name="C9" library="__MyCommonLib1" deviceset="C" device="SMD_1206" value="0.47uFx25V"/>
 </parts>
 <sheets>
@@
 <instance part="GND39" gate="1" x="68.58" y="86.36" smashed="yes" rot="MR0">
 <attribute name="VALUE" x="67.31" y="83.185" size="1.27" layer="96" font="vector" ratio="20" rot="MR0"/>
+</instance>
+<instance part="C9" gate="C$1" x="43.18" y="134.62" smashed="yes" rot="MR0">
+<attribute name="NAME" x="40.64" y="129.54" size="1.27" layer="95" font="vector" ratio="20" rot="MR180"/>
+<attribute name="VALUE" x="40.64" y="128.27" size="1.27" layer="96" font="vector" ratio="20" rot="MR180"/>
 </instance>
 </instances>
@@
 <wire x1="27.94" y1="137.16" x2="27.94" y2="139.7" width="0.1524" layer="91"/>
 <junction x="27.94" y="139.7"/>
+<pinref part="C9" gate="C$1" pin="PIN1"/>
+<wire x1="38.1" y1="139.7" x2="43.18" y2="139.7" width="0.1524" layer="91"/>
+<wire x1="43.18" y1="139.7" x2="43.18" y2="137.16" width="0.1524" layer="91"/>
+<junction x="38.1" y="139.7"/>
 </segment>
 <segment>
@@
 <junction x="182.88" y="111.76"/>
 <junction x="149.86" y="152.4"/>
-</segment>
-</net>
+<pinref part="C9" gate="C$1" pin="PIN0"/>
+<wire x1="38.1" y1="129.54" x2="43.18" y2="129.54" width="0.1524" layer="91"/>
+<wire x1="43.18" y1="129.54" x2="43.18" y2="132.08" width="0.1524" layer="91"/>
+<junction x="38.1" y="129.54"/>
+</segment>
+</net>
