File: 12_to_200V_inverter/schematic/12to220inverterVer3.sch (EAGLE design)
At the start: 245 parts, among them IC1 UC3842, IC10 TL494, IC2 PC817, IC3 LM358SOIC8, IC4 TL431, IC5 LM317, IC6 74HC595, IC7 74HC595, IC8 ATTINY45, IC9 TL431, J1 0, J2 0, J3 0, J4 0, T1 AO4407AL, T10 16N60, T11 BC847, T12 BC847, T13 BSS84, T15 BC847, T16 BSS84, T17 BC847, T18 BC847, T19 BSS84, T2 IRF830, T20 BSS84, T21 BC847, T22 BC847, T23 BSS84, T24 BC847, T3 IRF830, T4 BC847, T5 BC857, T6 BC857, T7 IRFZ24N, T8 IRFZ24N, T9 BC857, X1 BAT+, X2 LAMP1, X3 LAMP1, X4 BAT-, X5 220VAC, X6 LAMP1_SWITCH, X7 LAMP1_SWITCH, X8 MCU_PROGRAMMING

Commit message: 12to200V inverter. restore
Parts:
- added TR4: Self made transformer. From TR8 sat reciever., __MyCommonLib1:TRANS_FLYBACK_AUX_SINGLE_OUT(TRANS29.5X23)
Connections:
- new net ANY_LAMP_ON: D24.ANODE, D25.ANODE, D27.CATHODE, D28.CATHODE
- net GND: now also TR4.SEC_START
- net LAMP1_ON: no longer D24.ANODE
- net LAMP2_ON: no longer D25.ANODE
- net N$130: now also D25.CATHODE; no longer D27.CATHODE, D28.CATHODE
- net N$32: now also TR4.PRI2_START
- net N$34: now also TR4.PRI1_START, TR4.PRI2_END
- net N$35: now also TR4.PRI1_END
- net N$48: now also TR4.AUX_END
- net N$50: now also TR4.AUX_START
- net N$58: now also TR4.SEC_END
- net N$93: no longer D25.CATHODE
Other:
- moved on the sheet: D25, D27, D28, X6, X7

Commit message: 10 to 200V inverter. Ver3. Routing.
Parts:
- removed J1: 0, __MyCommonLib1:RSMD_1206_BIG_GAP
- D10, D8: device __MyCommonLib1:1N4001DO-41_10MM -> __MyCommonLib1:1N4001DO-41_15MM
- D13: device __MyCommonLib1:1N4001DO-41_10MM -> __MyCommonLib1:1N4001DO-41_12.5MM
- R30: device __MyCommonLib1:R1.0W_VERT -> __MyCommonLib1:R1.0W
- R68, R76: device __MyCommonLib1:RSMD_0805 -> __MyCommonLib1:RSMD_1206_BIG_GAP
Connections:
- removed net N$40: IC2.COLLECTOR, J1.PIN0
- net N$35: no longer HS1.PIN0
- net N$55: now also IC2.COLLECTOR; no longer J1.PIN1
Other:
- moved on the sheet: C14, C16, CE2, CE3, CE4, D11, D16, L1, R41, R42, R49, R54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

Commit message: 10 to 200V inverter. Ver3. Routing.
Parts:
- added C39: 0.1uF x 50V, __MyCommonLib1:CSMD_0805
- R72, R78: device __MyCommonLib1:RSMD_0805 -> __MyCommonLib1:RSMD_1206_BIG_GAP
Connections:
- removed net N$61: IC2.LED_CATHODE, R59.PIN1
- new net N$40: IC2.LED_ANODE, R59.PIN1
- net GND: now also C39.PIN0
- net N$62: now also R59.PIN0; no longer IC2.LED_ANODE
- net N$98: now also C39.PIN1, IC2.LED_CATHODE; no longer R59.PIN0
Other:
- moved on the sheet: IC2, J2, R59

Commit message: 10 to 200V inverter. Ver3. Routing.
Parts:
- removed J4: 0, __MyCommonLib1:RSMD_1206_BIG_GAP
Connections:
- removed net N$110: RT1.PIN0, X5.2
- removed net N$13: F2.PIN1, X5.1
- removed net N$63: J4.PIN1, X8.4
- new net N$61: F2.PIN1, RT1.PIN0
- new net N$70: RT1.PIN1, X5.1
- net CONV_TEMP_ADC(SCK): now also X8.4; no longer J4.PIN0
- net N$22: now also X5.2; no longer RT1.PIN1
Other:
- moved on the sheet: F2, RT1, X5
Changed lines of the file:
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@@
 <part name="GND39" library="supply1" deviceset="GND" device=""/>
 <part name="J3" library="__MyCommonLib1" deviceset="R" device="SMD_1206_BIG_GAP" value="0"/>
-<part name="J4" library="__MyCommonLib1" deviceset="R" device="SMD_1206_BIG_GAP" value="0"/>
 <part name="C9" library="__MyCommonLib1" deviceset="C" device="SMD_1206" value="0.47uFx25V"/>
 <part name="TR4" library="__MyCommonLib1" deviceset="TRANS_FLYBACK_AUX_SINGLE_OUT" device="(TRANS29.5X23)" value="Self made transformer. From TR8 sat reciever."/>
@@
 <attribute name="SHEET" x="230.505" y="5.08" size="2.54" layer="94" font="vector"/>
 </instance>
-<instance part="X5" gate="G$1" x="8.89" y="149.86" smashed="yes" rot="R180">
-<attribute name="NAME" x="10.16" y="146.05" size="1.27" layer="95" font="vector" ratio="20" rot="R180"/>
-<attribute name="VALUE" x="10.16" y="147.32" size="1.27" layer="96" font="vector" ratio="20" rot="R180"/>
-</instance>
-<instance part="F2" gate="G$1" x="22.86" y="149.86" smashed="yes" rot="MR270">
-<attribute name="NAME" x="20.32" y="147.32" size="1.27" layer="95" font="vector" ratio="20" rot="MR180"/>
-<attribute name="VALUE" x="25.4" y="147.32" size="1.27" layer="96" font="vector" ratio="20" rot="MR180"/>
+<instance part="X5" gate="G$1" x="8.89" y="162.56" smashed="yes" rot="R180">
+<attribute name="NAME" x="12.7" y="171.45" size="1.27" layer="95" font="vector" ratio="20" rot="R180"/>
+<attribute name="VALUE" x="12.7" y="170.18" size="1.27" layer="96" font="vector" ratio="20" rot="R180"/>
+</instance>
+<instance part="F2" gate="G$1" x="17.78" y="149.86" smashed="yes" rot="MR270">
+<attribute name="NAME" x="15.24" y="147.32" size="1.27" layer="95" font="vector" ratio="20" rot="MR180"/>
+<attribute name="VALUE" x="20.32" y="147.32" size="1.27" layer="96" font="vector" ratio="20" rot="MR180"/>
 </instance>
 <instance part="C11" gate="C$1" x="30.48" y="157.48" smashed="yes" rot="MR180">
-<attribute name="NAME" x="27.94" y="156.21" size="1.27" layer="95" font="vector" ratio="20" rot="MR0"/>
-<attribute name="VALUE" x="29.21" y="158.75" size="1.27" layer="96" font="vector" ratio="20" rot="MR0"/>
+<attribute name="NAME" x="30.48" y="168.91" size="1.27" layer="95" font="vector" ratio="20" rot="MR0"/>
+<attribute name="VALUE" x="26.67" y="168.91" size="1.27" layer="96" font="vector" ratio="20" rot="MR180"/>
 </instance>
 <instance part="TR2" gate="G$1" x="55.88" y="157.48" smashed="yes" rot="R270">
@@
 <attribute name="VALUE" x="55.88" y="147.32" size="1.27" layer="96" font="vector" ratio="20" rot="MR180"/>
 </instance>
-<instance part="RT1" gate="G$1" x="22.86" y="165.1" smashed="yes" rot="MR180">
-<attribute name="NAME" x="20.32" y="170.18" size="1.27" layer="95" font="vector" ratio="20" rot="MR180"/>
-<attribute name="VALUE" x="20.32" y="171.45" size="1.27" layer="96" font="vector" ratio="20" rot="MR180"/>
+<instance part="RT1" gate="G$1" x="17.78" y="154.94" smashed="yes" rot="MR180">
+<attribute name="NAME" x="15.24" y="160.02" size="1.27" layer="95" font="vector" ratio="20" rot="MR180"/>
+<attribute name="VALUE" x="15.24" y="161.29" size="1.27" layer="96" font="vector" ratio="20" rot="MR180"/>
 </instance>
 <instance part="D8" gate="D$1" x="86.36" y="165.1" smashed="yes" rot="R270">
@@
 </busses>
 <nets>
-<net name="N$13" class="0">
-<segment>
-<pinref part="X5" gate="G$1" pin="1"/>
-<pinref part="F2" gate="G$1" pin="PIN1"/>
-<wire x1="12.7" y1="149.86" x2="17.78" y2="149.86" width="0.1524" layer="91"/>
-</segment>
-</net>
 <net name="N$22" class="0">
 <segment>
@@
 <wire x1="33.02" y1="160.02" x2="33.02" y2="165.1" width="0.1524" layer="91"/>
 <junction x="33.02" y="165.1"/>
-<pinref part="RT1" gate="G$1" pin="PIN1"/>
-<wire x1="27.94" y1="165.1" x2="30.48" y2="165.1" width="0.1524" layer="91"/>
-<junction x="30.48" y="165.1"/>
 <pinref part="TR2" gate="G$1" pin="W1_START"/>
 <wire x1="50.8" y1="165.1" x2="50.8" y2="162.56" width="0.1524" layer="91"/>
+<pinref part="X5" gate="G$1" pin="2"/>
+<wire x1="12.7" y1="165.1" x2="30.48" y2="165.1" width="0.1524" layer="91"/>
+<junction x="30.48" y="165.1"/>
 </segment>
 </net>
@@
 <pinref part="F2" gate="G$1" pin="PIN0"/>
 <pinref part="C11" gate="C$1" pin="PIN1"/>
-<wire x1="27.94" y1="149.86" x2="30.48" y2="149.86" width="0.1524" layer="91"/>
+<wire x1="22.86" y1="149.86" x2="30.48" y2="149.86" width="0.1524" layer="91"/>
 <wire x1="30.48" y1="149.86" x2="30.48" y2="154.94" width="0.1524" layer="91"/>
 <wire x1="30.48" y1="149.86" x2="33.02" y2="149.86" width="0.1524" layer="91"/>
@@
 </segment>
 </net>
-<net name="N$110" class="0">
-<segment>
-<pinref part="X5" gate="G$1" pin="2"/>
-<wire x1="12.7" y1="152.4" x2="15.24" y2="152.4" width="0.1524" layer="91"/>
-<wire x1="15.24" y1="152.4" x2="15.24" y2="165.1" width="0.1524" layer="91"/>
-<wire x1="15.24" y1="165.1" x2="17.78" y2="165.1" width="0.1524" layer="91"/>
-<pinref part="RT1" gate="G$1" pin="PIN0"/>
-</segment>
-</net>
 <net name="N$111" class="0">
 <segment>
@@
 </segment>
 </net>
+<net name="N$61" class="0">
+<segment>
+<pinref part="RT1" gate="G$1" pin="PIN0"/>
+<wire x1="12.7" y1="154.94" x2="10.16" y2="154.94" width="0.1524" layer="91"/>
+<wire x1="10.16" y1="154.94" x2="10.16" y2="149.86" width="0.1524" layer="91"/>
+<pinref part="F2" gate="G$1" pin="PIN1"/>
+<wire x1="10.16" y1="149.86" x2="12.7" y2="149.86" width="0.1524" layer="91"/>
+</segment>
+</net>
+<net name="N$70" class="0">
+<segment>
+<pinref part="RT1" gate="G$1" pin="PIN1"/>
+<wire x1="22.86" y1="154.94" x2="25.4" y2="154.94" width="0.1524" layer="91"/>
+<wire x1="25.4" y1="154.94" x2="25.4" y2="162.56" width="0.1524" layer="91"/>
+<pinref part="X5" gate="G$1" pin="1"/>
+<wire x1="25.4" y1="162.56" x2="12.7" y2="162.56" width="0.1524" layer="91"/>
+</segment>
+</net>
 </nets>
 </sheet>
@@
 <attribute name="VALUE" x="80.01" y="66.04" size="1.27" layer="96" font="vector" ratio="20"/>
 </instance>
-<instance part="J4" gate="R$1" x="106.68" y="63.5" smashed="yes" rot="R90">
-<attribute name="NAME" x="109.22" y="66.04" size="1.27" layer="95" font="vector" ratio="20" rot="R180"/>
-<attribute name="VALUE" x="105.41" y="66.04" size="1.27" layer="96" font="vector" ratio="20" rot="R180"/>
-</instance>
 </instances>
 <busses>
@@
 <net name="LED_SCK(MISO)" class="0">
 <segment>
+<label x="152.4" y="97.79" size="1.27" layer="95" font="vector" ratio="20" rot="R180"/>
+<wire x1="132.08" y1="96.52" x2="154.94" y2="96.52" width="0.1524" layer="91"/>
 <pinref part="IC6" gate="G$1" pin="SER_CLK"/>
-<wire x1="132.08" y1="96.52" x2="149.86" y2="96.52" width="0.1524" layer="91"/>
-<label x="142.24" y="97.79" size="1.27" layer="95" font="vector" ratio="20" rot="R180"/>
 <pinref part="R95" gate="R$1" pin="PIN0"/>
-<wire x1="149.86" y1="96.52" x2="167.64" y2="96.52" width="0.1524" layer="91"/>
+<wire x1="154.94" y1="96.52" x2="167.64" y2="96.52" width="0.1524" layer="91"/>
 <wire x1="134.62" y1="88.9" x2="132.08" y2="88.9" width="0.1524" layer="91"/>
 <wire x1="132.08" y1="88.9" x2="132.08" y2="93.98" width="0.1524" layer="91"/>
-<wire x1="132.08" y1="93.98" x2="149.86" y2="93.98" width="0.1524" layer="91"/>
-<wire x1="149.86" y1="93.98" x2="149.86" y2="96.52" width="0.1524" layer="91"/>
-<junction x="149.86" y="96.52"/>
+<wire x1="132.08" y1="93.98" x2="154.94" y2="93.98" width="0.1524" layer="91"/>
+<wire x1="154.94" y1="93.98" x2="154.94" y2="96.52" width="0.1524" layer="91"/>
+<junction x="154.94" y="96.52"/>
 </segment>
 <segment>
@@
 </segment>
 <segment>
-<pinref part="IC7" gate="G$1" pin="SER_CLK"/>
-<wire x1="167.64" y1="58.42" x2="154.94" y2="58.42" width="0.1524" layer="91"/>
-<label x="162.56" y="60.96" size="1.27" layer="95" font="vector" ratio="20" rot="R180"/>
-</segment>
-<segment>
 <pinref part="X8" gate="G$1" pin="6"/>
 <wire x1="121.92" y1="60.96" x2="99.06" y2="60.96" width="0.1524" layer="91"/>
 <label x="121.92" y="62.865" size="1.27" layer="95" font="vector" ratio="20" rot="R180"/>
 </segment>
+<segment>
+<pinref part="IC7" gate="G$1" pin="SER_CLK"/>
+<wire x1="167.64" y1="58.42" x2="147.32" y2="58.42" width="0.1524" layer="91"/>
+<label x="162.56" y="60.96" size="1.27" layer="95" font="vector" ratio="20" rot="R180"/>
+</segment>
 </net>
 <net name="LED_DATA(MOSI)" class="0">
 <segment>
-<pinref part="IC6" gate="G$1" pin="SER_IN"/>
 <wire x1="167.64" y1="99.06" x2="132.08" y2="99.06" width="0.1524" layer="91"/>
-<label x="142.24" y="100.33" size="1.27" layer="95" font="vector" ratio="20" rot="R180"/>
+<label x="152.4" y="100.33" size="1.27" layer="95" font="vector" ratio="20" rot="R180"/>
+<pinref part="IC6" gate="G$1" pin="SER_IN"/>
 </segment>
 <segment>
@@
 </segment>
 <segment>
-<wire x1="134.62" y1="63.5" x2="111.76" y2="63.5" width="0.1524" layer="91"/>
-<label x="134.62" y="65.405" size="1.27" layer="95" font="vector" ratio="20" rot="R180"/>
-<pinref part="J4" gate="R$1" pin="PIN0"/>
+<wire x1="121.92" y1="63.5" x2="99.06" y2="63.5" width="0.1524" layer="91"/>
+<label x="121.92" y="65.405" size="1.27" layer="95" font="vector" ratio="20" rot="R180"/>
+<pinref part="X8" gate="G$1" pin="4"/>
 </segment>
 </net>
@@
 </segment>
 </net>
-<net name="N$63" class="0">
-<segment>
-<pinref part="X8" gate="G$1" pin="4"/>
-<pinref part="J4" gate="R$1" pin="PIN1"/>
-<wire x1="101.6" y1="63.5" x2="99.06" y2="63.5" width="0.1524" layer="91"/>
-</segment>
-</net>

Commit message: 10 to 200V inverter. Ver3. Routing.
Connections:
- net +200VDC_I_SENSE: now also R10.PIN1, R12.PIN1
- net -VBAT: no longer R10.PIN1, R12.PIN1
Other:
- moved on the sheet: R10, R11, R12
Changed lines of the file:
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@@
 <attribute name="VALUE" x="132.08" y="157.48" size="1.27" layer="96" font="vector" ratio="20" rot="MR0"/>
 </instance>
-<instance part="R11" gate="R$1" x="218.44" y="124.46" smashed="yes" rot="R180">
-<attribute name="NAME" x="220.98" y="119.38" size="1.27" layer="95" font="vector" ratio="20"/>
-<attribute name="VALUE" x="220.98" y="121.92" size="1.27" layer="96" font="vector" ratio="20"/>
+<instance part="R11" gate="R$1" x="218.44" y="119.38" smashed="yes" rot="R180">
+<attribute name="NAME" x="220.98" y="114.3" size="1.27" layer="95" font="vector" ratio="20"/>
+<attribute name="VALUE" x="220.98" y="116.84" size="1.27" layer="96" font="vector" ratio="20"/>
 </instance>
 <instance part="C4" gate="C$1" x="88.9" y="157.48" smashed="yes" rot="MR0">
@@
 <attribute name="VALUE" x="191.77" y="148.59" size="1.27" layer="96" font="vector" ratio="20" rot="MR180"/>
 </instance>
-<instance part="R10" gate="R$1" x="198.12" y="124.46" smashed="yes" rot="MR180">
-<attribute name="NAME" x="200.66" y="127" size="1.27" layer="95" font="vector" ratio="20" rot="MR180"/>
-<attribute name="VALUE" x="200.66" y="125.73" size="1.27" layer="96" font="vector" ratio="20" rot="MR180"/>
+<instance part="R10" gate="R$1" x="200.66" y="137.16" smashed="yes" rot="MR90">
+<attribute name="NAME" x="195.58" y="134.62" size="1.27" layer="95" font="vector" ratio="20" rot="MR180"/>
+<attribute name="VALUE" x="195.58" y="133.35" size="1.27" layer="96" font="vector" ratio="20" rot="MR180"/>
 </instance>
 <instance part="R6" gate="R$1" x="236.22" y="144.78" smashed="yes" rot="MR270">
@@
 <attribute name="VALUE" x="238.76" y="148.59" size="1.27" layer="96" font="vector" ratio="20" rot="MR180"/>
 </instance>
-<instance part="R12" gate="R$1" x="228.6" y="124.46" smashed="yes" rot="MR180">
-<attribute name="NAME" x="231.14" y="125.73" size="1.27" layer="95" font="vector" ratio="20" rot="MR180"/>
-<attribute name="VALUE" x="231.14" y="124.46" size="1.27" layer="96" font="vector" ratio="20" rot="MR180"/>
+<instance part="R12" gate="R$1" x="226.06" y="137.16" smashed="yes" rot="MR270">
+<attribute name="NAME" x="228.6" y="133.35" size="1.27" layer="95" font="vector" ratio="20" rot="MR0"/>
+<attribute name="VALUE" x="228.6" y="132.08" size="1.27" layer="96" font="vector" ratio="20" rot="MR0"/>
 </instance>
 <instance part="T1" gate="G$1" x="71.12" y="162.56" smashed="yes" rot="MR90">
@@
 <wire x1="208.28" y1="137.16" x2="218.44" y2="137.16" width="0.1524" layer="91"/>
 <wire x1="218.44" y1="137.16" x2="218.44" y2="139.7" width="0.1524" layer="91"/>
-<wire x1="218.44" y1="129.54" x2="218.44" y2="132.08" width="0.1524" layer="91"/>
+<wire x1="218.44" y1="124.46" x2="218.44" y2="127" width="0.1524" layer="91"/>
 <junction x="218.44" y="137.16"/>
-<wire x1="218.44" y1="132.08" x2="218.44" y2="137.16" width="0.1524" layer="91"/>
-<wire x1="218.44" y1="132.08" x2="200.66" y2="132.08" width="0.1524" layer="91"/>
-<junction x="218.44" y="132.08"/>
-<label x="217.17" y="134.62" size="1.27" layer="95" font="vector" ratio="20" rot="R180"/>
+<wire x1="218.44" y1="127" x2="218.44" y2="137.16" width="0.1524" layer="91"/>
+<wire x1="218.44" y1="127" x2="200.66" y2="127" width="0.1524" layer="91"/>
+<junction x="218.44" y="127"/>
+<label x="217.17" y="129.54" size="1.27" layer="95" font="vector" ratio="20" rot="R180"/>
+<pinref part="R10" gate="R$1" pin="PIN1"/>
+<wire x1="205.74" y1="137.16" x2="208.28" y2="137.16" width="0.1524" layer="91"/>
+<pinref part="R12" gate="R$1" pin="PIN1"/>
+<wire x1="218.44" y1="137.16" x2="220.98" y2="137.16" width="0.1524" layer="91"/>
+<junction x="208.28" y="137.16"/>
 </segment>
 <segment>
@@
 <pinref part="R11" gate="R$1" pin="PIN1"/>
 <wire x1="167.64" y1="111.76" x2="182.88" y2="111.76" width="0.1524" layer="91"/>
-<wire x1="182.88" y1="111.76" x2="198.12" y2="111.76" width="0.1524" layer="91"/>
-<wire x1="198.12" y1="111.76" x2="218.44" y2="111.76" width="0.1524" layer="91"/>
-<wire x1="218.44" y1="111.76" x2="218.44" y2="119.38" width="0.1524" layer="91"/>
+<wire x1="182.88" y1="111.76" x2="218.44" y2="111.76" width="0.1524" layer="91"/>
+<wire x1="218.44" y1="111.76" x2="218.44" y2="114.3" width="0.1524" layer="91"/>
 <junction x="167.64" y="111.76"/>
-<pinref part="R10" gate="R$1" pin="PIN1"/>
-<wire x1="198.12" y1="119.38" x2="198.12" y2="111.76" width="0.1524" layer="91"/>
-<junction x="198.12" y="111.76"/>
-<pinref part="R12" gate="R$1" pin="PIN1"/>
-<wire x1="228.6" y1="119.38" x2="228.6" y2="111.76" width="0.1524" layer="91"/>
 <wire x1="228.6" y1="111.76" x2="218.44" y2="111.76" width="0.1524" layer="91"/>
 <junction x="218.44" y="111.76"/>
@@
 <wire x1="195.58" y1="144.78" x2="198.12" y2="144.78" width="0.1524" layer="91"/>
 <wire x1="198.12" y1="144.78" x2="200.66" y2="144.78" width="0.1524" layer="91"/>
-<wire x1="198.12" y1="144.78" x2="198.12" y2="129.54" width="0.1524" layer="91"/>
+<wire x1="198.12" y1="144.78" x2="198.12" y2="139.7" width="0.1524" layer="91"/>
+<wire x1="198.12" y1="139.7" x2="193.04" y2="139.7" width="0.1524" layer="91"/>
+<wire x1="193.04" y1="139.7" x2="193.04" y2="137.16" width="0.1524" layer="91"/>
+<wire x1="193.04" y1="137.16" x2="195.58" y2="137.16" width="0.1524" layer="91"/>
 <junction x="198.12" y="144.78"/>
 <pinref part="R10" gate="R$1" pin="PIN0"/>
@@
 <pinref part="R12" gate="R$1" pin="PIN0"/>
 <wire x1="228.6" y1="144.78" x2="226.06" y2="144.78" width="0.1524" layer="91"/>
-<wire x1="228.6" y1="129.54" x2="228.6" y2="144.78" width="0.1524" layer="91"/>
+<wire x1="231.14" y1="137.16" x2="233.68" y2="137.16" width="0.1524" layer="91"/>
+<wire x1="233.68" y1="137.16" x2="233.68" y2="139.7" width="0.1524" layer="91"/>
+<wire x1="233.68" y1="139.7" x2="228.6" y2="139.7" width="0.1524" layer="91"/>
+<wire x1="228.6" y1="139.7" x2="228.6" y2="144.78" width="0.1524" layer="91"/>
 <junction x="228.6" y="144.78"/>
 </segment>
