File: 12_to_200V_inverter/schematic/12to220inverterVer3.sch (EAGLE design)
At the start: 254 parts, among them IC1 UC3842, IC10 TL494, IC2 PC817, IC3 LM358, IC4 TL431, IC5 LM317, IC6 74HC595, IC7 74HC595, IC8 ATTINY45, IC9 TL431, J100 0, J2 0, J3 0, T10 16N60, T11 BC847, T12 BC847, T13 AO3401, T14 AO3401, T15 BC847, T16 BSS84, T17 BC847, T18 BC847, T19 BSS84, T2 IRF830, T21 BC847, T22 BC847, T23 BSS84, T24 BC847, T3 IRF830, T4 BC847, T5 BC857, T6 BC857, T7 IRFZ24N, T8 IRFZ24N, T9 BC857, U100 DF06S, X1 BAT+, X2 LAMP1, X3 LAMP1, X4 BAT-, X5 220VAC, X6 LAMP1_SWITCH, X7 LAMP1_SWITCH, X8 MCU_PROGRAMMING

Commit message: 12 to 200V inverter. New board with ETD transformers. Route.
Parts:
- removed D11: SR3A0, __MyCommonLib1:SR360_15MM
- added D101: MBR20100CT, __MyCommonLib1:MBR20100CT
- CE2: device __MyCommonLib1:CE13MM -> __MyCommonLib1:CE10MM
- D2: device __MyCommonLib1:1N4001DO-41_5MM -> __MyCommonLib1:1N4001DO-41_10MM
- D23: device __MyCommonLib1:LL4147SOD-80 -> __MyCommonLib1:LL4147(DO-35_10MM)
- IC8: device __MyCommonLib1:ATTINY45(SOIC8-0.15'') -> __MyCommonLib1:ATTINY45(PSOP8_0.208'')
Connections:
- net CHARGER_POWER: now also D101.CATHODE; no longer D11.CATHODE
- net N$58: now also D101.ANODE1, D101.ANODE2; no longer D11.ANODE
Other:
- moved on the sheet: C14, R41, R42

Commit message: 12 to 200V inverter. New board with ETD transformers. Finally routed.
Parts:
- added J101: 0, __MyCommonLib1:RSMD_0805
- D23: device __MyCommonLib1:LL4147(DO-35_10MM) -> __MyCommonLib1:LL4147(DO-35_15MM)
- D3: device __MyCommonLib1:1N4001DO-41_5MM -> __MyCommonLib1:1N4001DO-41_10MM
- D4: device __MyCommonLib1:1N4001DO-41_12.5MM -> __MyCommonLib1:1N4001DO-41_10MM
- R76: device __MyCommonLib1:RSMD_1206_BIG_GAP -> __MyCommonLib1:RSMD_0805
- R80: device __MyCommonLib1:R1.0W_VERT -> __MyCommonLib1:R1.0W
- ZD2: device __MyCommonLib1:ZENNERDO-41_5MM -> __MyCommonLib1:ZENNERDO-41_10MM
Connections:
- new net N$104: IC7.LATCH, J101.PIN1
- net LED_LATCH: now also J101.PIN0; no longer IC7.LATCH
- net N$48: now also C15.PIN1; no longer R47.PIN0, R48.PIN0
- net N$49: now also C15.PIN0, R47.PIN0, R48.PIN0; no longer C15.PIN1, R47.PIN1, R48.PIN1
- net N$50: now also R47.PIN1, R48.PIN1; no longer C15.PIN0
Other:
- moved on the sheet: C15, R47, R48

Commit message: 12 to 200V inverter. New board with ETD transformers. Finally routed.
Parts:
- IC4: device __MyCommonLib1:TL431TO-92A_PINS_SWAPPED -> __MyCommonLib1:TL431TO-92A
Changed lines of the file:
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@@
 <setting verticaltext="up"/>
 </settings>
-<grid distance="0.05" unitdist="inch" unit="inch" style="lines" multiple="2" display="yes" altdistance="0.01" altunitdist="inch" altunit="inch"/>
+<grid distance="0.1" unitdist="inch" unit="inch" style="lines" multiple="1" display="no" altdistance="0.01" altunitdist="inch" altunit="inch"/>
 <layers>
 <layer number="1" name="Top" color="4" fill="1" visible="yes" active="no"/>
@@
 <part name="L1" library="__MyCommonLib1" deviceset="L" device="(7MM)" value="20uH"/>
 <part name="CE3" library="__MyCommonLib1" deviceset="CE" device="6.3MM" value="47uF x 25V"/>
-<part name="IC4" library="__MyCommonLib1" deviceset="TL431" device="TO-92A_PINS_SWAPPED" value="TL431"/>
+<part name="IC4" library="__MyCommonLib1" deviceset="TL431" device="TO-92A" value="TL431"/>
 <part name="R59" library="__MyCommonLib1" deviceset="R" device="SMD_0805" value="5K6"/>
 <part name="R61" library="__MyCommonLib1" deviceset="R" device="SMD_0805" value="10K"/>

Commit message: 12 to 200V inverter. New board with ETD transformers. Finally routed.
Parts:
- added R110: *, __MyCommonLib1:RSMD_1206
- F2: device __MyCommonLib1:FUSE20X5.6MM -> __MyCommonLib1:FUSE(20X5MM_VERT_WIRE)
Connections:
- net N$24: now also R110.PIN0, R9.PIN0; no longer C7.PIN1
- net N$25: now also C7.PIN1; no longer R9.PIN0
- net N$26: now also R110.PIN1
Other:
- moved on the sheet: C7, D5, R14, R9, T5, T7, TR100

Commit message: 12 to 200V inverter. Timny changes to schematic and board.
Parts:
- F2: value 0.3A -> 2A
- R100, R101, R102, R103, R104, R105, R106, R99: value 1K0 -> 2K2
- R115: value 1K -> 1K0
- RT2, RT3: value 22K_20deg -> 100K_20deg

Commit message: 12 to 200V inverter. Last steps.
Parts:
- R81: value 240R -> 470R
Connections:
- net N$14: now also ZD4.ANODE; no longer ZD4.CATHODE
- net N$9: now also ZD4.CATHODE; no longer ZD4.ANODE
Other:
- moved on the sheet: ZD4
Changed lines of the file:
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@@
 <setting verticaltext="up"/>
 </settings>
-<grid distance="0.1" unitdist="inch" unit="inch" style="lines" multiple="1" display="no" altdistance="0.01" altunitdist="inch" altunit="inch"/>
+<grid distance="0.1" unitdist="inch" unit="inch" style="lines" multiple="1" display="yes" altdistance="0.01" altunitdist="inch" altunit="inch"/>
 <layers>
 <layer number="1" name="Top" color="4" fill="1" visible="no" active="no"/>
@@
 <part name="GND19" library="supply1" deviceset="GND" device=""/>
 <part name="R80" library="__MyCommonLib1" deviceset="R" device="1.0W" value="0.1R"/>
-<part name="R81" library="__MyCommonLib1" deviceset="R" device="SMD_0805" value="240R"/>
+<part name="R81" library="__MyCommonLib1" deviceset="R" device="SMD_0805" value="470R"/>
 <part name="C26" library="__MyCommonLib1" deviceset="C" device="SMD_0805" value="0.1uF"/>
 <part name="R79" library="__MyCommonLib1" deviceset="R" device="SMD_0805" value="10K"/>
@@
 <attribute name="VALUE" x="67.31" y="167.64" size="1.27" layer="96" font="vector" ratio="20" rot="MR180"/>
 </instance>
-<instance part="ZD4" gate="G$1" x="58.42" y="147.32" smashed="yes" rot="R270">
+<instance part="ZD4" gate="G$1" x="58.42" y="147.32" smashed="yes" rot="R90">
 <attribute name="NAME" x="55.88" y="144.78" size="1.27" layer="95" font="vector" ratio="20" rot="R180"/>
 <attribute name="VALUE" x="58.42" y="143.51" size="1.27" layer="96" font="vector" ratio="20"/>
@@
 <junction x="68.58" y="152.4"/>
 <pinref part="T14" gate="G$1" pin="GATE"/>
-<pinref part="ZD4" gate="G$1" pin="CATHODE"/>
+<pinref part="ZD4" gate="G$1" pin="ANODE"/>
 <wire x1="68.58" y1="147.32" x2="68.58" y2="152.4" width="0.1524" layer="91"/>
 <wire x1="60.96" y1="147.32" x2="68.58" y2="147.32" width="0.1524" layer="91"/>
@@
 <wire x1="50.8" y1="162.56" x2="48.26" y2="162.56" width="0.1524" layer="91"/>
 <junction x="48.26" y="162.56"/>
-<pinref part="ZD4" gate="G$1" pin="ANODE"/>
-<wire x1="55.88" y1="147.32" x2="48.26" y2="147.32" width="0.1524" layer="91"/>
 <wire x1="48.26" y1="147.32" x2="48.26" y2="152.4" width="0.1524" layer="91"/>
 <junction x="48.26" y="152.4"/>
-</segment>
-</net>
+<pinref part="ZD4" gate="G$1" pin="CATHODE"/>
+<wire x1="55.88" y1="147.32" x2="48.26" y2="147.32" width="0.1524" layer="91"/>
+</segment>
+</net>
