File: HumidityMetter/schematic/HumidityMetter.brd (EAGLE design)
At the start: 160 x 100 mm, 2 parts

Commit message: Humidity metter. Start schematic routing.
Parts:
- removed U$1: STM32F103C8T6(LQFP48)(LQFP48), __MyCommonLib1:LQFP48
- removed U$2: LCD_0802B(0802B), __MyCommonLib1:LCD_0802B
- added C1, C10, C11, C12, C13, C14, C2, C5, C6, C8, C9: 0.1uF, __MyCommonLib1:RSMD_0805
- added C3: 100uFx16V, __MyCommonLib1:CE_6.3MM
- added C4, C7: 10uF x 10V, __MyCommonLib1:CE_5.2MM
- added D1: LL4148, __MyCommonLib1:SOD-80
- added IC1, IC2: LM317, __MyCommonLib1:D2PAK
- added IC3: STM32F103C8T6, __MyCommonLib1:LQFP48
- added IC4: AM2320, __MyCommonLib1:AM2320_HOR
- added J1, J2, J3, J4: 0, __MyCommonLib1:RSMD_0805
- added K1: POWER_ON, __MyCommonLib1:KEY_7X4.5
- added LCD1: LCD_0802B, __MyCommonLib1:LCD_0802B
- added R1: 1 Ohm, __MyCommonLib1:RSMD_1206
- added R10: 3K9, __MyCommonLib1:RSMD_0805
- added R11, R3, R5: 1K0, __MyCommonLib1:RSMD_0805
- added R12, R13, R14, R15, R21, R22, R23: 390R, __MyCommonLib1:RSMD_0805
- added R16, R17, R18, R19: 2K0, __MyCommonLib1:RSMD_0805
- added R2, R30, R4: 10K, __MyCommonLib1:RSMD_0805
- added R20: 10K, __MyCommonLib1:R_ADJ_STAND
- added R24: 18K, __MyCommonLib1:RSMD_0805
- added R25: 6K8, __MyCommonLib1:RSMD_0805
- added R26, R27: 4K7, __MyCommonLib1:RSMD_0805
- added R28, R29: 200R, __MyCommonLib1:RSMD_0805
- added R6, R8: *, __MyCommonLib1:RSMD_0805
- added R7: 3K0, __MyCommonLib1:RSMD_0805
- added R9: 2K2, __MyCommonLib1:RSMD_0805
- added T1: BSS84, __MyCommonLib1:SOT23
- added T2: BC847, __MyCommonLib1:SOT23_SMALL_PADS
- added X1: +9V, __MyCommonLib1:PIN1X1_D3.5MM
- added X2: GND, __MyCommonLib1:PIN1X1_D3.5MM
- added X3: ISP, __MyCommonLib1:PIN4X1_2.54MM
Connections:
- new net +3.3V: C6.PAD_1, C7.PLUS, D1.CATHODE, IC2.2, J1.PAD_0, J3.PAD_0, R30.PAD_0, R9.PAD_1, X3.1
- new net +5V: C1.PAD_1, C4.PLUS, C5.PAD_1, C8.PAD_1, IC1.2, IC4.1, LCD1.2, LCD1.A, R20.1, R26.PAD_0, R27.PAD_0, R5.PAD_1
- new net ADC_9V: C9.PAD_1, D1.ANODE, R24.PAD_1, R25.PAD_0
- new net BOOT0: IC3.44, J1.PAD_1, J2.PAD_0
- new net BOOT1: IC3.20, J3.PAD_1, J4.PAD_0
- new net GND: C1.PAD_0, C10.PAD_0, C11.PAD_0, C12.PAD_0, C13.PAD_0, C14.PAD_0, C2.PAD_0, C3.MINUS, C4.MINUS, C5.PAD_0, C6.PAD_0, C7.MINUS, C8.PAD_0, C9.PAD_0, IC3.23, IC3.35, IC3.47, IC3.8, IC4.3, J2.PAD_1, J4.PAD_1, K1.1, K1.2, LCD1.1, LCD1.K, R10.PAD_1, R16.PAD_1, R17.PAD_1, R18.PAD_1, R19.PAD_1, R20.3, R25.PAD_1, R4.PAD_1, R6.PAD_1, R7.PAD_1, R8.PAD_1, T2.2, X2.1, X3.4
- new net I2C_SCL: IC3.21, R29.PAD_0
- new net I2C_SDA: IC3.22, R28.PAD_0
- new net LCD_D4: IC3.28, R15.PAD_1
- new net LCD_D5: IC3.27, R14.PAD_1
- new net LCD_D6: IC3.26, R13.PAD_1
- new net LCD_D7: IC3.25, R12.PAD_1
- new net LCD_E: IC3.43, R21.PAD_1
- new net LCD_R/~W: IC3.45, R22.PAD_1
- new net LCD_RS: IC3.46, R23.PAD_1
- new net N$1: R1.PAD_1, X1.1
- new net N$10: LCD1.14, R12.PAD_0
- new net N$11: LCD1.13, R13.PAD_0
- new net N$12: LCD1.12, R14.PAD_0
- new net N$13: LCD1.11, R15.PAD_0
- new net N$14: IC4.2, R26.PAD_1, R28.PAD_1
- new net N$15: LCD1.10, R16.PAD_0
- new net N$16: LCD1.9, R17.PAD_0
- new net N$17: LCD1.8, R18.PAD_0
- new net N$18: LCD1.7, R19.PAD_0
- new net N$19: C10.PAD_1, C11.PAD_1, C12.PAD_1, C13.PAD_1, IC3.24, IC3.36, IC3.48, IC3.9
- new net N$2: R1.PAD_0, R2.PAD_0, T1.2
- new net N$20: IC4.4, R27.PAD_1, R29.PAD_1
- new net N$21: LCD1.4, R23.PAD_0
- new net N$22: LCD1.5, R22.PAD_0
- new net N$23: LCD1.6, R21.PAD_0
- new net N$3: K1.3, K1.4, R2.PAD_1, R3.PAD_0, T1.1
- new net N$4: R3.PAD_1, T2.3
- new net N$5: R11.PAD_1, R4.PAD_0, T2.1
- new net N$6: C2.PAD_1, C3.PLUS, IC1.3, IC2.3, R24.PAD_0, T1.3
- new net N$7: IC1.1, R5.PAD_0, R6.PAD_0, R7.PAD_0
- new net N$8: IC2.1, R10.PAD_0, R8.PAD_0, R9.PAD_0
- new net N$9: LCD1.3, R20.2
- new net NRST: C14.PAD_1, IC3.7, R30.PAD_1
- new net PWR_HOLD: R11.PAD_0
- new net SWDCLK: IC3.37, X3.3
- new net SWDIO: IC3.34, X3.2
Routing:
- net +5V: track 0.00 -> 21.9 mm
- net N$20: track 0.00 -> 9.69 mm
- net N$14: track 0.00 -> 9.69 mm
- net GND: track 0.00 -> 7.15 mm
Other:
- board size 160 x 100 mm -> 107.9 x 59.4 mm

Commit message: Humidity metter.
Parts:
- added D10: 1N4007, __MyCommonLib1:DO-41_10MM
- R1: device __MyCommonLib1:RSMD_1206 -> __MyCommonLib1:R0207
- moved X3 290.1 mm to (25.0, 50.0), turned to 180 degrees
- moved C14 285.1 mm to (48.0, 41.0), turned to 270 degrees
- moved R30 277.9 mm to (48.0, 37.0), turned to 90 degrees
- moved J2 275.5 mm to (40.0, 49.0), turned to 180 degrees
- moved J1 274.7 mm to (40.0, 52.0)
- moved J4 270.2 mm to (49.0, 32.0), turned to 90 degrees
- moved J3 265.5 mm to (46.0, 32.0), turned to 270 degrees
- moved C13 259.2 mm to (45.0, 37.0), turned to 270 degrees
- moved C10 255.8 mm to (42.0, 46.0), turned to 180 degrees
- moved C11 253.6 mm to (29.0, 45.0), turned to 90 degrees
- moved R23 246.7 mm to (40.0, 56.0)
- moved R22 245.0 mm to (60.1, 48.0)
- moved C12 244.7 mm to (31.8, 30.6)
- moved R21 241.4 mm to (37.3, 59.0)
- moved D1 219.1 mm to (18.0, 20.0)
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Connections:
- removed net N$19: C10.PAD_1, C11.PAD_1, C12.PAD_1, C13.PAD_1, IC3.24, IC3.36, IC3.48, IC3.9
- net +3.3V: now also C10.PAD_1, C11.PAD_1, C12.PAD_1, C13.PAD_1, IC3.24, IC3.36, IC3.48, IC3.9
- net +5V: now also R20.3; no longer R20.1
- net GND: now also D10.ANODE, R20.1; no longer R20.3
- net LCD_D4: now also IC3.25; no longer IC3.28
- net LCD_D5: now also IC3.28; no longer IC3.27
- net LCD_D7: now also IC3.27; no longer IC3.25
- net N$1: now also R1.PAD1; no longer R1.PAD_1
- net N$2: now also D10.CATHODE
Routing:
- net GND: track 7.15 -> 114.9 mm
- net +3.3V: track 0.00 -> 92.0 mm, vias 0 -> 6
- net +5V: track 21.9 -> 109.9 mm
- net LCD_D5: track 0.00 -> 81.0 mm
- net LCD_D7: track 0.00 -> 75.3 mm
- net LCD_D6: track 0.00 -> 68.7 mm
- net LCD_D4: track 0.00 -> 61.8 mm
- net I2C_SCL: track 0.00 -> 59.7 mm, vias 0 -> 2
- net I2C_SDA: track 0.00 -> 56.5 mm, vias 0 -> 2
- net N$23: track 0.00 -> 30.4 mm
- net LCD_R/~W: track 0.00 -> 29.7 mm, vias 0 -> 2
- net N$21: track 0.00 -> 26.3 mm
- net N$12: track 0.00 -> 24.8 mm
- net N$9: track 0.00 -> 24.8 mm
- net N$10: track 0.00 -> 20.1 mm
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Other:
- board size 107.9 x 59.4 mm -> 100 x 68 mm

Commit message: Humidity metter. Routing.
Parts:
- added R31, R32: *, __MyCommonLib1:RSMD_0805
- R10: value 3K9 -> *
- R6: value * -> 3K0
- R7: value 3K0 -> *
- R8: value * -> 3K9
- moved J2 22.1 mm to (18.0, 51.0), turned to 270 degrees
- moved J1 14.0 mm to (26.0, 51.0), turned to 90 degrees
- moved R24 11.7 mm to (21.0, 22.0), turned to 180 degrees
- moved R22 11.2 mm to (49.0, 46.0)
- moved C3 8.08 mm to (11.0, 14.0), turned to 0 degrees
- moved C8 7.62 mm to (51.0, 52.0)
- moved D1 7.20 mm to (24.9, 22.0), turned to 90 degrees
- moved R5 7.00 mm to (53.0, 15.0)
- moved R6 7.00 mm to (54.0, 8.00)
- moved R7 7.00 mm to (54.0, 11.0)
- moved R21 6.43 mm to (35.0, 53.0), turned to 270 degrees
- moved C6 6.38 mm to (31.0, 13.0), turned to 0 degrees
- moved C1 5.80 mm to (80.4, 28.1)
- moved R26 5.80 mm to (80.4, 33.2)
- moved R27 5.80 mm to (80.4, 25.5)
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Connections:
- net +3.3V: now also R31.PAD_1
- net +5V: now also R32.PAD_1
- net ADC_9V: now also IC3.13
- net LCD_R/~W: now also IC3.46; no longer IC3.45
- net LCD_RS: now also IC3.45; no longer IC3.46
- net N$7: now also R32.PAD_0
- net N$8: now also R31.PAD_0
- net PWR_HOLD: now also IC3.31
Routing:
- net ADC_9V: track 0.00 -> 43.6 mm, vias 0 -> 2
- net N$6: track 0.00 -> 30.3 mm, vias 0 -> 2
- net GND: track 114.9 -> 86.2 mm, vias 0 -> 2
- net N$3: track 0.00 -> 19.5 mm
- net N$7: track 0.00 -> 19.3 mm
- net N$8: track 0.00 -> 16.5 mm
- net LCD_R/~W: track 29.7 -> 13.4 mm, vias 2 -> 0
- net PWR_HOLD: track 0.00 -> 15.1 mm
- net BOOT0: track 14.9 -> 29.6 mm
- net N$22: track 9.04 -> 22.5 mm
- net +5V: track 109.9 -> 98.9 mm, vias 0 -> 4
- net N$23: track 30.4 -> 39.5 mm
- net LCD_E: track 18.0 -> 9.22 mm
- net N$4: track 0.00 -> 6.86 mm
- net I2C_SDA: track 56.5 -> 50.5 mm
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- added copper zone on layer 16, net +3.3V
- added copper zone on layer 16, net +5V
- added copper zone on layer 16, net GND
- added copper zone on layer 16, net N$2

Commit message: Humidity metter. Routing.
Parts:
- added LED1: ERROR(RED), __MyCommonLib1:LED_0805
- added R33: 1K0, __MyCommonLib1:RSMD_0805
- R11: device __MyCommonLib1:RSMD_0805 -> __MyCommonLib1:RSMD_1206_BIG_GAP
- moved R24 4.02 mm to (17.0, 22.0)
- moved D1 3.90 mm to (21.0, 22.0)
- moved C9 3.62 mm to (18.0, 27.0), turned to 270 degrees
- moved R11 2.00 mm to (19.0, 41.0), turned to 0 degrees
- moved C11 1.41 mm to (30.0, 48.0)
- moved R25 1.00 mm to (21.0, 27.0), turned to 90 degrees
- moved C2 1.00 mm to (11.0, 19.0), turned to 180 degrees
- moved X2 1.00 mm to (2.01, 12.0)
- moved X1 0.86 mm to (2.00, 46.0)
Connections:
- new net ERROR_LED: IC3.40, R33.PAD_0
- new net N$19: LED1.ANODE, R33.PAD_1
- net GND: now also LED1.CATHODE
Routing:
- net N$19: track 0.00 -> 19.1 mm
- net GND: track 86.2 -> 73.9 mm
- net N$12: track 26.4 -> 36.3 mm
- net ERROR_LED: track 0.00 -> 9.84 mm
- net ADC_9V: track 43.6 -> 37.6 mm
- net N$30: track 0.00 -> 4.00 mm
- net N$29: track 0.00 -> 4.00 mm
- net N$28: track 0.00 -> 4.00 mm
- net N$3: track 19.5 -> 23.2 mm
- net N$6: track 30.3 -> 26.6 mm
- net PWR_HOLD: track 15.1 -> 11.8 mm
- net N$5: track 5.76 -> 6.57 mm
- net +3.3V: track 97.9 -> 98.7 mm
- net SWDCLK: track 22.5 -> 21.9 mm
- added copper zone on layer 16, net N$1
- added copper zone on layer 16, net N$6
Other:
- board text added: "ERROR"

Commit message: Himidity metter. Board routed.
Parts:
- R24: device __MyCommonLib1:RSMD_0805 -> __MyCommonLib1:RSMD_1206_BIG_GAP
- R26, R27, R28, R29: device __MyCommonLib1:RSMD_0805 -> __MyCommonLib1:R0207
- moved R29 15.3 mm to (68.1, 32.0)
- moved C1 12.4 mm to (90.0, 36.0)
- moved R28 12.3 mm to (68.2, 29.0)
- moved C2 10.0 mm to (11.0, 9.00)
- moved R27 5.63 mm to (77.0, 30.0), turned to 270 degrees
- moved R26 3.29 mm to (80.0, 29.9), turned to 270 degrees
- moved C9 1.41 mm to (17.0, 28.0)
- moved D1 1.00 mm to (21.0, 23.0)
- moved R24 1.00 mm to (17.0, 23.0), turned to 90 degrees
- moved R25 1.00 mm to (21.0, 28.0)
Connections:
- net N$14: now also R26.PAD1, R28.PAD1; no longer R26.PAD_1, R28.PAD_1
- net N$20: now also R27.PAD1, R29.PAD1; no longer R27.PAD_1, R29.PAD_1
Routing:
- net I2C_SCL: track 58.1 -> 32.9 mm, vias 2 -> 0
- net N$20: track 12.7 -> 32.6 mm
- net +5V: track 98.9 -> 79.8 mm, vias 4 -> 8
- net I2C_SDA: track 50.5 -> 33.6 mm, vias 2 -> 0
- net N$14: track 12.7 -> 24.8 mm
- net N$12: track 36.3 -> 25.3 mm
- net ADC_9V: track 37.6 -> 46.5 mm
- net GND: track 73.9 -> 82.1 mm, vias 2 -> 6
- net +3.3V: track 98.7 -> 102.9 mm
- net N$29: track 4.00 -> 0.00 mm
- net N$28: track 4.00 -> 8.00 mm
- net N$23: track 39.5 -> 37.5 mm
- net N$21: track 31.0 -> 29.9 mm
- net N$10: track 20.9 -> 20.2 mm
- net LCD_D5: track 80.8 -> 81.4 mm
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Other:
- board text added: "07.08.2024"
- board text added: "HUMIDITY"
- board text added: "LED"
- board text added: "METTER"
- board text added: "VER1.0"
