File: HumidityMetter/schematic/HumidityMetter.brd (EAGLE design)
At the start: 100 x 68 mm, 65 parts, among them IC1 LM317, IC2 LM317, IC3 STM32F103C8T6, IC4 AM2320, J1 0, J2 0, J3 0, J4 0, K1 POWER_ON, T1 BSS84, T2 BC847, X1 +9V, X2 GND, X3 ISP

Commit message: Himidity metter. Board routed.
Parts:
- added D2: 1N4007, __MyCommonLib1:DO-41_10MM
- moved X3 2.00 mm to (22.0, 48.0)
- moved J1 1.00 mm to (26.0, 52.0)
- moved J2 1.00 mm to (18.0, 52.0)
- moved LED1 1.00 mm to (15.0, 52.0)
- moved R11 1.00 mm to (19.0, 40.0)
- moved R4 1.00 mm to (14.0, 40.0)
- moved T2 1.00 mm to (10.0, 40.0)
Connections:
- net +3.3V: now also D2.CATHODE
- net GND: now also D2.ANODE
Routing:
- net SWDIO: track 11.6 -> 14.0 mm
- net N$4: track 6.86 -> 5.86 mm

Commit message: Himidity metter. Board routed. Fix tiny problems.
Parts:
- LCD1: device __MyCommonLib1:LCD_0802B -> __MyCommonLib1:LCD_0802B(CHINA_CLONE)
- moved R3 3.00 mm to (8.00, 36.0), turned to 180 degrees
- moved R1 0.05 mm to (5.00, 36.0)
Routing:
- net +5V: track 79.8 -> 81.5 mm
- net N$4: track 5.86 -> 4.14 mm
- net N$3: track 23.2 -> 24.9 mm
- net N$28: track 8.00 -> 6.40 mm
- net N$30: track 4.00 -> 3.20 mm
- net GND: track 82.1 -> 82.4 mm, vias 6 -> 8

Commit message: Himidity metter. Board routed. Fix tiny problems.
Parts:
- moved C4 0.40 mm to (36.6, 16.0)
- moved C5 0.40 mm to (36.6, 13.0)
Routing:
- net GND: track 82.4 -> 80.4 mm
- added copper zone on layer 16, net ADC_9V
- added copper zone on layer 16, net BOOT0
- added copper zone on layer 16, net BOOT1
- added copper zone on layer 16, net ERROR_LED
- added copper zone on layer 16, net I2C_SCL
- added copper zone on layer 16, net I2C_SDA
- added copper zone on layer 16, net LCD_D4
- added copper zone on layer 16, net LCD_D5
- added copper zone on layer 16, net LCD_D7
- added copper zone on layer 16, net LCD_E
- added copper zone on layer 16, net LCD_RS
- added copper zone on layer 16, net PWR_HOLD
- added copper zone on layer 16, net SWDCLK
- added copper zone on layer 16, net SWDIO

Commit message: Himidity metter. Board routed. Fix tiny problems.
Parts:
- flipped R1 to the top
- flipped R26 to the top
- flipped R27 to the top
- flipped R28 to the top, turned to 0 degrees
- flipped R29 to the top, turned to 0 degrees

Commit message: Humidity metter. Add key reading and switching between temp, humidity, preassure and battery voltage(dummy).
Parts:
- added D3, D4: LL4148, __MyCommonLib1:SOD-80
- added R34: 10K, __MyCommonLib1:RSMD_0805
Connections:
- new net KEY: D3.CATHODE, D4.CATHODE, K1.3, K1.4
- new net N$24: D3.ANODE, IC3.29, IC3.30, R34.PAD_0
- net +3.3V: now also R34.PAD_1
- net N$3: now also D4.ANODE; no longer K1.3, K1.4
Routing:
- net N$3: track 24.9 -> 15.3 mm
Changed lines of the file:
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@@
 <layer number="14" name="Route14" color="1" fill="6" visible="no" active="no"/>
 <layer number="15" name="Route15" color="4" fill="6" visible="no" active="no"/>
-<layer number="16" name="Bottom" color="1" fill="1" visible="no" active="yes"/>
+<layer number="16" name="Bottom" color="1" fill="1" visible="yes" active="yes"/>
 <layer number="17" name="Pads" color="2" fill="1" visible="yes" active="yes"/>
 <layer number="18" name="Vias" color="2" fill="1" visible="yes" active="yes"/>
-<layer number="19" name="Unrouted" color="6" fill="1" visible="no" active="yes"/>
+<layer number="19" name="Unrouted" color="6" fill="1" visible="yes" active="yes"/>
 <layer number="20" name="Dimension" color="15" fill="1" visible="yes" active="yes"/>
 <layer number="21" name="tPlace" color="7" fill="1" visible="yes" active="yes"/>
@@
 <attribute name="VALUE" x="18.96" y="41.97" size="1.27" layer="27" font="vector" ratio="20"/>
 </element>
+<element name="D3" library="__MyCommonLib1" package="SOD-80" value="LL4148" x="-1.5" y="-7"/>
+<element name="R34" library="__MyCommonLib1" package="RSMD_0805" value="10K" x="-2.2" y="-10.1"/>
+<element name="D4" library="__MyCommonLib1" package="SOD-80" value="LL4148" x="-1.5" y="-13.2"/>
 </elements>
 <signals>
@@
 <contactref element="R3" pad="PAD_0"/>
 <contactref element="T1" pad="1"/>
-<contactref element="K1" pad="3"/>
-<contactref element="K1" pad="4"/>
-<wire x1="8.75" y1="25.5" x2="8.75" y2="32.5" width="2" layer="16"/>
 <wire x1="-0.05" y1="31" x2="-0.05" y2="32.45" width="0.8" layer="16"/>
 <wire x1="-0.05" y1="32.45" x2="1.6" y2="34.1" width="0.8" layer="16"/>
@@
 <wire x1="-0.05" y1="27.35" x2="-0.1" y2="27.3" width="0.8" layer="16"/>
 <wire x1="6.95" y1="36" x2="6.95" y2="34.3" width="0.8" layer="16"/>
-<wire x1="6.95" y1="34.3" x2="8.75" y2="32.5" width="0.8" layer="16"/>
 <wire x1="1.6" y1="34.1" x2="4" y2="34.1" width="0.8" layer="16"/>
 <wire x1="4" y1="34.1" x2="5.7" y2="35.8" width="0.8" layer="16"/>
 <wire x1="6.95" y1="36" x2="6.75" y2="35.8" width="0.8" layer="16"/>
 <wire x1="6.75" y1="35.8" x2="5.7" y2="35.8" width="0.8" layer="16"/>
+<contactref element="D4" pad="ANODE"/>
+<wire x1="0.375" y1="-13.2" x2="-0.1" y2="27.3" width="0" layer="19" extent="1-16"/>
 </signal>
 <signal name="N$4">
@@
 <vertex x="43.1" y="36.5"/>
 </polygon>
+<contactref element="R34" pad="PAD_1"/>
+<wire x1="21.98" y1="13.06" x2="-1.15" y2="-10.1" width="0" layer="19" extent="1-16"/>
 </signal>
 <signal name="PWR_HOLD">
@@
 <wire x1="0.4" y1="6" x2="3.6" y2="6" width="0.8" layer="16"/>
 </signal>
+<signal name="N$24">
+<contactref element="R34" pad="PAD_0"/>
+<contactref element="D3" pad="ANODE"/>
+<contactref element="IC3" pad="29"/>
+<contactref element="IC3" pad="30"/>
+<wire x1="31.75" y1="38.75" x2="31.75" y2="38.25" width="0" layer="19" extent="16-16"/>
+<wire x1="0.375" y1="-7" x2="31.75" y2="38.25" width="0" layer="19" extent="1-16"/>
+<wire x1="-3.25" y1="-10.1" x2="0.375" y2="-7" width="0" layer="19" extent="1-1"/>
+</signal>
+<signal name="KEY">
+<contactref element="D3" pad="CATHODE"/>
+<contactref element="K1" pad="3"/>
+<contactref element="K1" pad="4"/>
+<contactref element="D4" pad="CATHODE"/>
+<wire x1="8.75" y1="25.5" x2="8.75" y2="32.5" width="0" layer="19" extent="1-1"/>
+<wire x1="-3.375" y1="-7" x2="8.75" y2="25.5" width="0" layer="19" extent="1-1"/>
+<wire x1="-3.375" y1="-13.2" x2="-3.375" y2="-7" width="0" layer="19" extent="1-1"/>
+</signal>
 </signals>
