File: HumidityMetter/schematic/HumidityMetter.sch (EAGLE design)
At the start: 2 parts

Commit message: Humidity metter. Start schematic routing.
Parts:
- removed U$1: STM32F103C8T6(LQFP48)(LQFP48), __MyCommonLib1:STM32F103C8T6(LQFP48)(LQFP48)
- removed U$2: LCD_0802B(0802B), __MyCommonLib1:LCD_0802B(0802B)
- added C1, C10, C11, C12, C13, C14, C2, C5, C6, C8, C9: 0.1uF, __MyCommonLib1:CSMD_0805
- added C3: 100uFx16V, __MyCommonLib1:CE6.3MM
- added C4, C7: 10uF x 10V, __MyCommonLib1:CE5.2MM
- added D1: LL4148, __MyCommonLib1:LL4147SOD-80
- added IC1, IC2: LM317, __MyCommonLib1:LM317(D2PAK)
- added IC3: STM32F103C8T6, __MyCommonLib1:STM32F103C8T6(LQFP48)(LQFP48)
- added IC4: AM2320, __MyCommonLib1:AM2320(HOR)
- added J1, J2, J3, J4: 0, __MyCommonLib1:RSMD_0805
- added K1: POWER_ON, __MyCommonLib1:KEY(7X4.5)
- added LCD1: LCD_0802B, __MyCommonLib1:LCD_0802B(0802B)
- added R1: 1 Ohm, __MyCommonLib1:RSMD_1206
- added R10: 3K9, __MyCommonLib1:RSMD_0805
- added R11, R3, R5: 1K0, __MyCommonLib1:RSMD_0805
- added R12, R13, R14, R15, R21, R22, R23: 390R, __MyCommonLib1:RSMD_0805
- added R16, R17, R18, R19: 2K0, __MyCommonLib1:RSMD_0805
- added R2, R30, R4: 10K, __MyCommonLib1:RSMD_0805
- added R20: 10K, __MyCommonLib1:R_ADJSTAND_6.5_X_3.5MM
- added R24: 18K, __MyCommonLib1:RSMD_0805
- added R25: 6K8, __MyCommonLib1:RSMD_0805
- added R26, R27: 4K7, __MyCommonLib1:RSMD_0805
- added R28, R29: 200R, __MyCommonLib1:RSMD_0805
- added R6, R8: *, __MyCommonLib1:RSMD_0805
- added R7: 3K0, __MyCommonLib1:RSMD_0805
- added R9: 2K2, __MyCommonLib1:RSMD_0805
- added T1: BSS84, __MyCommonLib1:BSS84(SOT23)
- added T2: BC847, __MyCommonLib1:BC847SOT23_SMALL_PADS
- added X1: +9V, __MyCommonLib1:PIN1X13.5MM_DRILL
- added X2: GND, __MyCommonLib1:PIN1X13.5MM_DRILL
- added X3: ISP, __MyCommonLib1:PIN4X1(2.54MM)
Connections:
- new net +3.3V: C6.PIN1, C7.PLUS, D1.CATHODE, IC2.OUT, J1.PIN0, J3.PIN0, R30.PIN0, R9.PIN1, X3.1
- new net +5V: C1.PIN1, C4.PLUS, C5.PIN1, C8.PIN1, IC1.OUT, IC4.VDD, LCD1.A, LCD1.VDD, R20.END_A, R26.PIN0, R27.PIN0, R5.PIN1
- new net ADC_9V: C9.PIN1, D1.ANODE, R24.PIN1, R25.PIN0
- new net BOOT0: IC3.BOOT0, J1.PIN1, J2.PIN0
- new net BOOT1: IC3.PB2/BOOT1, J3.PIN1, J4.PIN0
- new net GND: C1.PIN0, C10.PIN0, C11.PIN0, C12.PIN0, C13.PIN0, C14.PIN0, C2.PIN0, C3.MINUS, C4.MINUS, C5.PIN0, C6.PIN0, C7.MINUS, C8.PIN0, C9.PIN0, IC3.VSS1, IC3.VSS2, IC3.VSS3, IC3.VSSA, IC4.GND, J2.PIN1, J4.PIN1, K1.1, LCD1.K, LCD1.VSS, R10.PIN1, R16.PIN1, R17.PIN1, R18.PIN1, R19.PIN1, R20.END_B, R25.PIN1, R4.PIN1, R6.PIN1, R7.PIN1, R8.PIN1, T2.E, X2.1, X3.4
- new net I2C_SCL: IC3.PB10/I2C2_SCL/USART3_TX, R29.PIN0
- new net I2C_SDA: IC3.PB11/I2C2_SDA/USART3_RX, R28.PIN0
- new net LCD_D4: IC3.PB15/SPI2_MOSI/TIM1_CH3N, R15.PIN1
- new net LCD_D5: IC3.PB14/SPI2_MISO/USART3_RTS/TIM1_CH2N, R14.PIN1
- new net LCD_D6: IC3.PB13/SPI2_SCK/USART3_CTS/TIM1_CH1, R13.PIN1
- new net LCD_D7: IC3.PB12/SPI2_NSS/I2C2_SMBAI/USART3_CK/TIM1_BKIN, R12.PIN1
- new net LCD_E: IC3.PB7/I2C1_SDA/TIM4_CH2, R21.PIN1
- new net LCD_R/~W: IC3.PB8/TIM4_CH3, R22.PIN1
- new net LCD_RS: IC3.PB9/TIM4_CH4, R23.PIN1
- new net N$1: R1.PIN1, X1.1
- new net N$10: LCD1.DB7, R12.PIN0
- new net N$11: LCD1.DB6, R13.PIN0
- new net N$12: LCD1.DB5, R14.PIN0
- new net N$13: LCD1.DB4, R15.PIN0
- new net N$14: IC4.SDA, R26.PIN1, R28.PIN1
- new net N$15: LCD1.DB3, R16.PIN0
- new net N$16: LCD1.DB2, R17.PIN0
- new net N$17: LCD1.DB1, R18.PIN0
- new net N$18: LCD1.DB0, R19.PIN0
- new net N$19: C10.PIN1, C11.PIN1, C12.PIN1, C13.PIN1, IC3.VDD1, IC3.VDD2, IC3.VDD3, IC3.VDDA
- new net N$2: R1.PIN0, R2.PIN0, T1.SOURCE
- new net N$20: IC4.SCL, R27.PIN1, R29.PIN1
- new net N$21: LCD1.RS, R23.PIN0
- new net N$22: LCD1.R/~W, R22.PIN0
- new net N$23: LCD1.E, R21.PIN0
- new net N$3: K1.2, R2.PIN1, R3.PIN0, T1.GATE
- new net N$4: R3.PIN1, T2.C
- new net N$5: R11.PIN1, R4.PIN0, T2.B
- new net N$6: C2.PIN1, C3.PLUS, IC1.IN, IC2.IN, R24.PIN0, T1.DRAIN
- new net N$7: IC1.ADJ, R5.PIN0, R6.PIN0, R7.PIN0
- new net N$8: IC2.ADJ, R10.PIN0, R8.PIN0, R9.PIN0
- new net N$9: LCD1.VO, R20.ADJ
- new net NRST: C14.PIN1, IC3.NRST, R30.PIN1
- new net PWR_HOLD: R11.PIN0
- new net SWDCLK: IC3.PA14/JTCK/SWCLK, X3.3
- new net SWDIO: IC3.PA13/JTMS/SWDIO, X3.2

Commit message: Humidity metter.
Parts:
- added D10: 1N4007, __MyCommonLib1:1N4001DO-41_10MM
- R1: device __MyCommonLib1:RSMD_1206 -> __MyCommonLib1:R0207
Connections:
- removed net N$19: C10.PIN1, C11.PIN1, C12.PIN1, C13.PIN1, IC3.VDD1, IC3.VDD2, IC3.VDD3, IC3.VDDA
- net +3.3V: now also C10.PIN1, C11.PIN1, C12.PIN1, C13.PIN1, IC3.VDD1, IC3.VDD2, IC3.VDD3, IC3.VDDA
- net +5V: now also R20.END_B; no longer R20.END_A
- net GND: now also D10.ANODE, R20.END_A; no longer R20.END_B
- net LCD_D4: now also IC3.PB12/SPI2_NSS/I2C2_SMBAI/USART3_CK/TIM1_BKIN; no longer IC3.PB15/SPI2_MOSI/TIM1_CH3N
- net LCD_D5: now also IC3.PB15/SPI2_MOSI/TIM1_CH3N; no longer IC3.PB14/SPI2_MISO/USART3_RTS/TIM1_CH2N
- net LCD_D7: now also IC3.PB14/SPI2_MISO/USART3_RTS/TIM1_CH2N; no longer IC3.PB12/SPI2_NSS/I2C2_SMBAI/USART3_CK/TIM1_BKIN
- net N$2: now also D10.CATHODE
Other:
- moved on the sheet: C2, C3, C4, C5, C6, C7, C9, D1, IC1, IC2, K1, R10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

Commit message: Humidity metter. Routing.
Parts:
- added R31, R32: *, __MyCommonLib1:RSMD_0805
- R10: value 3K9 -> *
- R6: value * -> 3K0
- R7: value 3K0 -> *
- R8: value * -> 3K9
Connections:
- net +3.3V: now also R31.PIN1
- net +5V: now also R32.PIN1
- net ADC_9V: now also IC3.PA3/USART2_RX/ADC12_IN3/TIM2_CH4
- net LCD_R/~W: now also IC3.PB9/TIM4_CH4; no longer IC3.PB8/TIM4_CH3
- net LCD_RS: now also IC3.PB8/TIM4_CH3; no longer IC3.PB9/TIM4_CH4
- net N$7: now also R32.PIN0
- net N$8: now also R31.PIN0
- net PWR_HOLD: now also IC3.PA10/USART1_RX/TIM1_CH3
Other:
- moved on the sheet: C6, C7, IC2, R10, R6, R7, R8, R9

Commit message: Humidity metter. Routing.
Parts:
- added LED1: ERROR(RED), __MyCommonLib1:LED3MM(SMD0805)
- added R33: 1K0, __MyCommonLib1:RSMD_0805
- R11: device __MyCommonLib1:RSMD_0805 -> __MyCommonLib1:RSMD_1206_BIG_GAP
Connections:
- new net ERROR_LED: IC3.PB4/JNTRST, R33.PIN0
- new net N$19: LED1.ANODE, R33.PIN1
- net GND: now also LED1.CATHODE
Other:
- moved on the sheet: C1, IC4, R26, R27, R28, R29, X3

Commit message: Himidity metter. Board routed.
Parts:
- R24: device __MyCommonLib1:RSMD_0805 -> __MyCommonLib1:RSMD_1206_BIG_GAP
- R26, R27, R28, R29: device __MyCommonLib1:RSMD_0805 -> __MyCommonLib1:R0207
Changed lines of the file:
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@@
 <setting verticaltext="up"/>
 </settings>
-<grid distance="0.025" unitdist="inch" unit="inch" style="lines" multiple="4" display="yes" altdistance="0.01" altunitdist="inch" altunit="inch"/>
+<grid distance="0.1" unitdist="inch" unit="inch" style="lines" multiple="1" display="no" altdistance="0.01" altunitdist="inch" altunit="inch"/>
 <layers>
 <layer number="1" name="Top" color="4" fill="1" visible="yes" active="no"/>
@@
 <part name="R22" library="__MyCommonLib1" deviceset="R" device="SMD_0805" value="390R"/>
 <part name="R23" library="__MyCommonLib1" deviceset="R" device="SMD_0805" value="390R"/>
-<part name="R24" library="__MyCommonLib1" deviceset="R" device="SMD_0805" value="18K"/>
+<part name="R24" library="__MyCommonLib1" deviceset="R" device="SMD_1206_BIG_GAP" value="18K"/>
 <part name="R25" library="__MyCommonLib1" deviceset="R" device="SMD_0805" value="6K8"/>
 <part name="C9" library="__MyCommonLib1" deviceset="C" device="SMD_0805" value="0.1uF"/>
@@
 <part name="C1" library="__MyCommonLib1" deviceset="C" device="SMD_0805" value="0.1uF"/>
 <part name="GND28" library="supply1" deviceset="GND" device=""/>
-<part name="R26" library="__MyCommonLib1" deviceset="R" device="SMD_0805" value="4K7"/>
-<part name="R27" library="__MyCommonLib1" deviceset="R" device="SMD_0805" value="4K7"/>
-<part name="R28" library="__MyCommonLib1" deviceset="R" device="SMD_0805" value="200R"/>
-<part name="R29" library="__MyCommonLib1" deviceset="R" device="SMD_0805" value="200R"/>
+<part name="R26" library="__MyCommonLib1" deviceset="R" device="0207" value="4K7"/>
+<part name="R27" library="__MyCommonLib1" deviceset="R" device="0207" value="4K7"/>
+<part name="R28" library="__MyCommonLib1" deviceset="R" device="0207" value="200R"/>
+<part name="R29" library="__MyCommonLib1" deviceset="R" device="0207" value="200R"/>
 <part name="D10" library="__MyCommonLib1" deviceset="1N4001" device="DO-41_10MM" value="1N4007"/>
 <part name="GND29" library="supply1" deviceset="GND" device=""/>

Commit message: Himidity metter. Board routed.
Parts:
- added D2: 1N4007, __MyCommonLib1:1N4001DO-41_10MM
Connections:
- net +3.3V: now also D2.CATHODE
- net GND: now also D2.ANODE
Other:
- moved on the sheet: LED1, R33, X3
Changed lines of the file:
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@@
 <setting verticaltext="up"/>
 </settings>
-<grid distance="0.1" unitdist="inch" unit="inch" style="lines" multiple="1" display="no" altdistance="0.01" altunitdist="inch" altunit="inch"/>
+<grid distance="0.1" unitdist="inch" unit="inch" style="lines" multiple="1" display="yes" altdistance="0.01" altunitdist="inch" altunit="inch"/>
 <layers>
 <layer number="1" name="Top" color="4" fill="1" visible="yes" active="no"/>
@@
 <part name="LED1" library="__MyCommonLib1" deviceset="LED3MM" device="(SMD0805)" value="ERROR(RED)"/>
 <part name="GND30" library="supply1" deviceset="GND" device=""/>
+<part name="D2" library="__MyCommonLib1" deviceset="1N4001" device="DO-41_10MM" value="1N4007"/>
+<part name="GND31" library="supply1" deviceset="GND" device=""/>
 </parts>
 <sheets>
@@
 <attribute name="VALUE" x="26.035" y="135.255" size="1.27" layer="96" font="vector" ratio="20"/>
 </instance>
-<instance part="X3" gate="G$1" x="68.58" y="157.48" smashed="yes" rot="MR0">
-<attribute name="NAME" x="71.12" y="162.56" size="1.27" layer="95" font="vector" ratio="20" rot="MR0"/>
-<attribute name="VALUE" x="68.58" y="149.86" size="1.27" layer="96" font="vector" ratio="20" rot="MR180"/>
-</instance>
-<instance part="GND26" gate="1" x="76.2" y="147.32" smashed="yes">
-<attribute name="VALUE" x="74.93" y="145.415" size="1.27" layer="96" font="vector" ratio="20"/>
+<instance part="X3" gate="G$1" x="66.04" y="152.4" smashed="yes" rot="MR0">
+<attribute name="NAME" x="66.04" y="144.78" size="1.27" layer="95" font="vector" ratio="20" rot="MR180"/>
+<attribute name="VALUE" x="66.04" y="142.24" size="1.27" layer="96" font="vector" ratio="20" rot="MR180"/>
+</instance>
+<instance part="GND26" gate="1" x="73.66" y="142.24" smashed="yes">
+<attribute name="VALUE" x="72.39" y="140.335" size="1.27" layer="96" font="vector" ratio="20"/>
 </instance>
 <instance part="IC4" gate="G$1" x="129.54" y="144.78" smashed="yes">
@@
 <attribute name="VALUE" x="170.18" y="162.56" size="1.27" layer="96" font="vector" ratio="20" rot="MR180"/>
 </instance>
-<instance part="R33" gate="R$1" x="48.26" y="165.1" smashed="yes" rot="R180">
-<attribute name="NAME" x="51.435" y="165.1" size="1.27" layer="95" font="vector" ratio="20"/>
-<attribute name="VALUE" x="51.435" y="162.56" size="1.27" layer="96" font="vector" ratio="20"/>
-</instance>
-<instance part="LED1" gate="LED$1" x="48.26" y="152.4" smashed="yes" rot="R180">
-<attribute name="NAME" x="50.8" y="152.4" size="1.27" layer="95" font="vector" ratio="20"/>
-<attribute name="VALUE" x="50.8" y="149.86" size="1.27" layer="96" font="vector" ratio="20"/>
-</instance>
-<instance part="GND30" gate="1" x="48.26" y="137.16" smashed="yes">
-<attribute name="VALUE" x="45.72" y="133.985" size="1.27" layer="96" font="vector" ratio="20"/>
+<instance part="R33" gate="R$1" x="43.18" y="165.1" smashed="yes" rot="R180">
+<attribute name="NAME" x="46.355" y="165.1" size="1.27" layer="95" font="vector" ratio="20"/>
+<attribute name="VALUE" x="46.355" y="162.56" size="1.27" layer="96" font="vector" ratio="20"/>
+</instance>
+<instance part="LED1" gate="LED$1" x="43.18" y="152.4" smashed="yes" rot="R180">
+<attribute name="NAME" x="45.72" y="152.4" size="1.27" layer="95" font="vector" ratio="20"/>
+<attribute name="VALUE" x="45.72" y="149.86" size="1.27" layer="96" font="vector" ratio="20"/>
+</instance>
+<instance part="GND30" gate="1" x="43.18" y="137.16" smashed="yes">
+<attribute name="VALUE" x="40.64" y="133.985" size="1.27" layer="96" font="vector" ratio="20"/>
+</instance>
+<instance part="D2" gate="D$1" x="66.04" y="160.02" smashed="yes" rot="R270">
+<attribute name="NAME" x="63.5" y="163.83" size="1.27" layer="95" font="vector" ratio="20"/>
+<attribute name="VALUE" x="63.5" y="162.56" size="1.27" layer="96" font="vector" ratio="20"/>
+</instance>
+<instance part="GND31" gate="1" x="60.96" y="154.94" smashed="yes">
+<attribute name="VALUE" x="59.69" y="153.035" size="1.27" layer="96" font="vector" ratio="20"/>
 </instance>
 </instances>
@@
 <pinref part="X3" gate="G$1" pin="4"/>
 <pinref part="GND26" gate="1" pin="GND"/>
-<wire x1="73.66" y1="152.4" x2="76.2" y2="152.4" width="0.1524" layer="91"/>
-<wire x1="76.2" y1="152.4" x2="76.2" y2="149.86" width="0.1524" layer="91"/>
+<wire x1="71.12" y1="147.32" x2="73.66" y2="147.32" width="0.1524" layer="91"/>
+<wire x1="73.66" y1="147.32" x2="73.66" y2="144.78" width="0.1524" layer="91"/>
 </segment>
 <segment>
@@
 <pinref part="LED1" gate="LED$1" pin="CATHODE"/>
 <pinref part="GND30" gate="1" pin="GND"/>
-<wire x1="48.26" y1="139.7" x2="48.26" y2="149.86" width="0.1524" layer="91"/>
+<wire x1="43.18" y1="139.7" x2="43.18" y2="149.86" width="0.1524" layer="91"/>
+</segment>
+<segment>
+<pinref part="D2" gate="D$1" pin="ANODE"/>
+<pinref part="GND31" gate="1" pin="GND"/>
+<wire x1="63.5" y1="160.02" x2="60.96" y2="160.02" width="0.1524" layer="91"/>
+<wire x1="60.96" y1="160.02" x2="60.96" y2="157.48" width="0.1524" layer="91"/>
 </segment>
 </net>
@@
 <segment>
 <pinref part="X3" gate="G$1" pin="1"/>
-<wire x1="83.82" y1="160.02" x2="73.66" y2="160.02" width="0.1524" layer="91"/>
-<label x="83.82" y="161.29" size="1.27" layer="95" font="vector" ratio="20" rot="R180"/>
+<wire x1="81.28" y1="154.94" x2="73.66" y2="154.94" width="0.1524" layer="91"/>
+<label x="81.28" y="156.21" size="1.27" layer="95" font="vector" ratio="20" rot="R180"/>
+<pinref part="D2" gate="D$1" pin="CATHODE"/>
+<wire x1="73.66" y1="154.94" x2="71.12" y2="154.94" width="0.1524" layer="91"/>
+<wire x1="68.58" y1="160.02" x2="73.66" y2="160.02" width="0.1524" layer="91"/>
+<wire x1="73.66" y1="160.02" x2="73.66" y2="154.94" width="0.1524" layer="91"/>
+<junction x="73.66" y="154.94"/>
 </segment>
 <segment>
@@
 <segment>
 <pinref part="X3" gate="G$1" pin="2"/>
-<wire x1="83.82" y1="157.48" x2="73.66" y2="157.48" width="0.1524" layer="91"/>
-<label x="83.82" y="158.75" size="1.27" layer="95" font="vector" ratio="20" rot="R180"/>
+<wire x1="81.28" y1="152.4" x2="71.12" y2="152.4" width="0.1524" layer="91"/>
+<label x="81.28" y="153.67" size="1.27" layer="95" font="vector" ratio="20" rot="R180"/>
 </segment>
 <segment>
@@
 <segment>
 <pinref part="X3" gate="G$1" pin="3"/>
-<wire x1="83.82" y1="154.94" x2="73.66" y2="154.94" width="0.1524" layer="91"/>
-<label x="83.82" y="156.21" size="1.27" layer="95" font="vector" ratio="20" rot="R180"/>
+<wire x1="81.28" y1="149.86" x2="71.12" y2="149.86" width="0.1524" layer="91"/>
+<label x="81.28" y="151.13" size="1.27" layer="95" font="vector" ratio="20" rot="R180"/>
 </segment>
 <segment>
@@
 <segment>
 <pinref part="R33" gate="R$1" pin="PIN0"/>
-<wire x1="48.26" y1="170.18" x2="48.26" y2="172.72" width="0.1524" layer="91"/>
-<wire x1="48.26" y1="172.72" x2="60.96" y2="172.72" width="0.1524" layer="91"/>
-<label x="50.8" y="173.355" size="1.27" layer="95" font="vector" ratio="20"/>
+<wire x1="43.18" y1="170.18" x2="43.18" y2="172.72" width="0.1524" layer="91"/>
+<wire x1="43.18" y1="172.72" x2="55.88" y2="172.72" width="0.1524" layer="91"/>
+<label x="45.72" y="173.355" size="1.27" layer="95" font="vector" ratio="20"/>
 </segment>
 </net>
@@
 <pinref part="R33" gate="R$1" pin="PIN1"/>
 <pinref part="LED1" gate="LED$1" pin="ANODE"/>
-<wire x1="48.26" y1="160.02" x2="48.26" y2="154.94" width="0.1524" layer="91"/>
-</segment>
-</net>
+<wire x1="43.18" y1="160.02" x2="43.18" y2="154.94" width="0.1524" layer="91"/>
+</segment>
+</net>

Commit message: Himidity metter. Board routed. Fix tiny problems.
Parts:
- LCD1: device __MyCommonLib1:LCD_0802B(0802B) -> __MyCommonLib1:LCD_0802B(0802B_CHINA_CLONE)
Changed lines of the file:
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@@
 <setting verticaltext="up"/>
 </settings>
-<grid distance="0.1" unitdist="inch" unit="inch" style="lines" multiple="1" display="yes" altdistance="0.01" altunitdist="inch" altunit="inch"/>
+<grid distance="0.1" unitdist="inch" unit="inch" style="lines" multiple="1" display="no" altdistance="0.01" altunitdist="inch" altunit="inch"/>
 <layers>
 <layer number="1" name="Top" color="4" fill="1" visible="yes" active="no"/>
@@
 <part name="FRAME1" library="frames" deviceset="A4L-LOC" device="" value="HUMIDITY METTER"/>
 <part name="IC3" library="__MyCommonLib1" deviceset="STM32F103C8T6(LQFP48)" device="(LQFP48)" value="STM32F103C8T6"/>
-<part name="LCD1" library="__MyCommonLib1" deviceset="LCD_0802B" device="(0802B)" value="LCD_0802B"/>
+<part name="LCD1" library="__MyCommonLib1" deviceset="LCD_0802B" device="(0802B_CHINA_CLONE)" value="LCD_0802B"/>
 <part name="IC1" library="__MyCommonLib1" deviceset="LM317" device="(D2PAK)" value="LM317"/>
 <part name="X1" library="__MyCommonLib1" deviceset="PIN1X1" device="3.5MM_DRILL" value="+9V"/>
