File: HumidityMetter/schematic/HumidityMetter_v2.brd (EAGLE design)
At the start: 100 x 68 mm, 64 parts, among them IC1 LM317, IC10 AMS1117-3.3, IC3 STM32F103C8T6, IC4 AM2320, J1 0, J2 0, J3 0, J4 0, K1 POWER_ON, T1 BSS84, T2 BC847, X1 +9V, X2 GND, X3 ISP

Commit message: Humidity metter v2. Change schematic/board.
Parts:
- removed IC1: LM317, __MyCommonLib1:D2PAK
- removed IC4: AM2320, __MyCommonLib1:AM2320_HOR
- removed R32: *, __MyCommonLib1:RSMD_0805
- added C15: 0.1uF x 16V, __MyCommonLib1:RSMD_0603
- added C16: 3.3nF x 16V, __MyCommonLib1:RSMD_0603
- added C17, C7: 10uF x 10V, __MyCommonLib1:RSMD_1206
- added IC11: MP1482, __MyCommonLib1:SOIC8
- added L1: 39uH, __MyCommonLib1:COIL_7MM
- added L2: 20uH, __MyCommonLib1:RSMD_1206
- added R8: 100K, __MyCommonLib1:RSMD_0603
- added X4: SENSOR, __MyCommonLib1:JST_XH2.5MM_4PIN
- C1, J1, J2, R21, R22, R23, R33: device __MyCommonLib1:RSMD_0805 -> __MyCommonLib1:RSMD_0603
- C2: value 0.1uF -> 10uF x 16V; device __MyCommonLib1:RSMD_0805 -> __MyCommonLib1:RSMD_1206
- C3: value 100uFx16V -> 10uF x 16V; device __MyCommonLib1:CE_6.3MM -> __MyCommonLib1:RSMD_1206
- C4: value 10uF x 10V -> 10nF x 16V; device __MyCommonLib1:CE_5.2MM -> __MyCommonLib1:RSMD_0603
- C5: value 0.1uF -> 10uF x 10V; device __MyCommonLib1:RSMD_0805 -> __MyCommonLib1:RSMD_1206
- R26, R27, R28, R29: device __MyCommonLib1:R0207 -> __MyCommonLib1:RSMD_0603
- R5: value 1K0 -> 5K6; device __MyCommonLib1:RSMD_0805 -> __MyCommonLib1:RSMD_0603
- R6: value 3K0 -> 36K; device __MyCommonLib1:RSMD_0805 -> __MyCommonLib1:RSMD_0603
- R7: value * -> 8K2; device __MyCommonLib1:RSMD_0805 -> __MyCommonLib1:RSMD_0603
- moved R7 100.1 mm to (-12.1, -64.2), flipped to the top, turned to 0 degrees
- moved R5 98.1 mm to (-12.1, -58.4), flipped to the top, turned to 0 degrees
- moved R6 95.8 mm to (-12.1, -61.3), flipped to the top, turned to 0 degrees
- moved C4 75.4 mm to (-10.7, -42.7)
- moved C5 75.3 mm to (-10.7, -45.6), flipped to the top, turned to 0 degrees
- moved C3 51.0 mm to (-10.7, -32.2)
- moved R29 18.0 mm to (86.1, 32.1), flipped to the bottom
- moved R28 17.7 mm to (85.9, 29.6), flipped to the bottom, turned to 180 degrees
- moved R27 14.8 mm to (91.7, 32.1), flipped to the bottom, turned to 0 degrees
- moved R26 11.6 mm to (91.6, 29.6), flipped to the bottom, turned to 0 degrees
- moved C1 2.20 mm to (91.7, 34.6), turned to 180 degrees
Connections:
- removed net N$24: D3.ANODE, IC3.29, IC3.30, R34.PAD_0
- removed net N$6: C2.PAD_1, C3.PLUS, IC1.3, R24.PAD_0, T1.3
- removed net N$7 (its old number): IC1.1, R32.PAD_0, R5.PAD_0, R6.PAD_0, R7.PAD_0
- new net N$25: IC11.7, R8.PAD_0
- new net N$26: D4.ANODE, R3.PAD_1, T2.3
- new net N$27: C4.PAD_0, IC11.3, L1.1
- new net N$29: C4.PAD_1, IC11.1
- new net N$31: C5.PAD_1, C7.PAD_1, L1.2, L2.PAD_0, R6.PAD_0
- new net N$32: C15.PAD_1, IC11.8
- new net N$34: C16.PAD_1, IC11.6
- new net N$35: C16.PAD_0, R5.PAD_0
- new net N$36: IC11.5, R6.PAD_1, R7.PAD_0
- new net N$8: C2.PAD_1, C3.PAD_1, IC11.2, R24.PAD_0, R8.PAD_1, T1.3
- net +3.3V: now also C1.PAD_1, R26.PAD_0, R27.PAD_0, R34.PAD_0, X4.1; no longer R34.PAD_1
- net +5V: now also C17.PAD_1, L2.PAD_1; no longer C1.PAD_1, C4.PLUS, C5.PAD_1, IC1.2, IC4.1, R26.PAD_0, R27.PAD_0, R32.PAD_1, R5.PAD_1
- net GND: now also C15.PAD_0, C17.PAD_0, C3.PAD_0, C7.PAD_0, IC11.4, R5.PAD_1, X4.4; no longer C3.MINUS, C4.MINUS, IC4.3, R6.PAD_1
- net KEY: now also D3.ANODE, IC3.29, R34.PAD_1; no longer D3.CATHODE, D4.CATHODE, K1.3, K1.4
- net N$14: now also R26.PAD_1, R28.PAD_1, X4.2; no longer IC4.2, R26.PAD1, R28.PAD1
- net N$20: now also R27.PAD_1, R29.PAD_1, X4.3; no longer IC4.4, R27.PAD1, R29.PAD1
- net N$3: no longer D4.ANODE
- net N$4: now also D3.CATHODE, D4.CATHODE, K1.3, K1.4; no longer R3.PAD_1, T2.3
Routing:
- net N$20: track 32.6 -> 0.00 mm
- net I2C_SCL: track 32.9 -> 3.04 mm
- net I2C_SDA: track 33.6 -> 4.79 mm
- net N$6: track 26.6 -> 0.00 mm, vias 2 -> 0
- net N$14: track 24.8 -> 0.00 mm
- net N$7 (its old number): track 19.3 -> 0.00 mm
- net +5V: track 81.5 -> 64.4 mm, vias 8 -> 6
- net N$4: track 4.14 -> 0.00 mm
- net N$26: track 0.00 -> 4.14 mm
- net GND: track 80.7 -> 78.5 mm
- added copper zone on layer 16, net N$2
- removed copper zone on layer 16, net N$7

Commit message: Humidity metter v2. Change schematic/board 2.
Parts:
- removed D10: 1N4007, __MyCommonLib1:DO-41_10MM
- added D11: B120, __MyCommonLib1:DO-214AC
- D2: value 1N4007 -> B120; device __MyCommonLib1:DO-41_10MM -> __MyCommonLib1:DO-214AC
- moved R5 104.1 mm to (64.0, 12.6), flipped to the bottom, turned to 180 degrees
- moved C16 99.9 mm to (61.0, 12.6), flipped to the bottom
- moved C15 95.2 mm to (61.0, 10.0), flipped to the bottom
- moved C4 81.4 mm to (53.0, 8.00), flipped to the bottom
- moved R8 80.5 mm to (60.2, 16.9), flipped to the bottom
- moved L1 76.7 mm to (47.0, 14.0), turned to 180 degrees
- moved X3 73.8 mm to (90.8, 21.2), turned to 270 degrees
- moved IC11 67.9 mm to (55.2, 12.0), flipped to the bottom, turned to 180 degrees
- moved LED1 67.3 mm to (75.8, 23.2), turned to 180 degrees
- moved IC10 54.6 mm to (80.8, 10.4)
- moved J2 51.4 mm to (64.0, 29.0), turned to 90 degrees
- moved R33 50.8 mm to (75.0, 26.0), turned to 0 degrees
- moved C11 48.4 mm to (76.9, 36.0), turned to 270 degrees
- moved J1 42.7 mm to (62.0, 29.0), turned to 270 degrees
- moved D2 33.9 mm to (-7.80, 27.2), flipped to the bottom, turned to 90 degrees
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Connections:
- net +3.3V: now also D11.CATHODE; no longer D2.CATHODE
- net GND: now also D11.ANODE; no longer D10.ANODE
- net N$7: now also D2.CATHODE; no longer D10.CATHODE
Routing:
- net LCD_D5: track 81.7 -> 14.8 mm
- net LCD_D7: track 74.9 -> 13.0 mm
- net +5V: track 64.4 -> 4.79 mm, vias 6 -> 0
- net LCD_D6: track 68.9 -> 11.1 mm
- net +3.3V: track 102.7 -> 47.0 mm, vias 8 -> 1
- net LCD_D4: track 63.2 -> 9.64 mm
- net GND: track 78.5 -> 39.4 mm, vias 8 -> 4
- net LCD_E: track 9.52 -> 38.5 mm, vias 0 -> 2
- net I2C_SDA: track 4.79 -> 31.8 mm, vias 0 -> 2
- net LCD_R/~W: track 14.0 -> 40.8 mm, vias 0 -> 2
- net I2C_SCL: track 3.04 -> 28.6 mm, vias 0 -> 2
- net LCD_RS: track 9.72 -> 32.9 mm, vias 0 -> 2
- net N$22: track 22.8 -> 0.00 mm
- net N$19: track 18.8 -> 0.00 mm
- net N$13: track 18.7 -> 0.00 mm
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- removed copper zone on layer 16, net ADC_9V
- removed copper zone on layer 16, net BOOT0
- removed copper zone on layer 16, net BOOT1
- removed copper zone on layer 16, net ERROR_LED
- removed copper zone on layer 16, net I2C_SCL
- removed copper zone on layer 16, net I2C_SDA
- removed copper zone on layer 16, net LCD_D4
- removed copper zone on layer 16, net LCD_D5
- removed copper zone on layer 16, net LCD_D7
- removed copper zone on layer 16, net LCD_E
- removed copper zone on layer 16, net LCD_RS
- removed copper zone on layer 16, net PWR_HOLD
- removed copper zone on layer 16, net SWDCLK
- removed copper zone on layer 16, net SWDIO

Commit message: Humidity metter v2. Change schematic/board 2.
Parts:
- removed D3, D4: LL4148, __MyCommonLib1:SOD-80
- added D55: BAT54C, __MyCommonLib1:SOT23_SMALL_PADS
- C9, R2, R25, R3, R34, R4: device __MyCommonLib1:RSMD_0805 -> __MyCommonLib1:RSMD_0603
- LCD1: device __MyCommonLib1:LCD_0802B(CHINA_CLONE) -> __MyCommonLib1:LCD_0802B_2SCREW(CHINA_CLONE)
- R1: device __MyCommonLib1:R0207 -> __MyCommonLib1:RSMD_1206
- R11, R24: device __MyCommonLib1:RSMD_1206_BIG_GAP -> __MyCommonLib1:RSMD_0603
- R20: device __MyCommonLib1:R_ADJ_STAND -> __MyCommonLib1:R_ADJ_HOR
- moved R7 88.9 mm to (29.5, 14.4), turned to 90 degrees
- moved R6 85.4 mm to (27.5, 14.4), turned to 270 degrees
- moved L2 84.6 mm to (36.0, 12.6), turned to 180 degrees
- moved C17 77.9 mm to (35.9, 8.50), turned to 180 degrees
- moved C7 74.6 mm to (15.9, 20.6)
- moved C5 68.1 mm to (15.9, 17.1)
- moved C3 50.7 mm to (13.5, 12.4), turned to 270 degrees
- moved R34 48.5 mm to (26.6, 28.9), turned to 90 degrees
- moved X3 42.6 mm to (51.8, 38.4), turned to 90 degrees
- moved J4 41.8 mm to (26.7, 41.4), turned to 90 degrees
- moved J3 41.5 mm to (24.8, 41.4), turned to 270 degrees
- moved R27 40.5 mm to (55.2, 22.4)
- moved C10 40.0 mm to (33.5, 39.8), turned to 0 degrees
- moved R28 39.2 mm to (49.9, 22.4)
- moved D11 38.9 mm to (53.1, 30.9)
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Connections:
- removed net N$4: D3.CATHODE, D4.CATHODE, K1.3, K1.4
- new net N$2: D55.3, K1.3, K1.4
- net ADC_9V: now also IC3.15; no longer IC3.13
- net I2C_SCL: now also IC3.42; no longer IC3.21
- net I2C_SDA: now also IC3.43; no longer IC3.22
- net KEY: now also D55.2, IC3.13; no longer D3.ANODE, IC3.29
- net LCD_D5: now also IC3.27; no longer IC3.28
- net LCD_D7: now also IC3.28; no longer IC3.27
- net LCD_E: now also IC3.22; no longer IC3.43
- net LCD_R/~W: now also IC3.21; no longer IC3.46
- net LCD_RS: now also IC3.46; no longer IC3.45
- net N$1: now also R1.PAD_1; no longer R1.PAD1
- net N$14: now also R29.PAD_1; no longer R28.PAD_1
- net N$20: now also R28.PAD_1; no longer R29.PAD_1
- net N$26: now also D55.1; no longer D4.ANODE
- net PWR_HOLD: now also IC3.17; no longer IC3.31
Routing:
- net N$8: track 0.00 -> 49.4 mm, vias 0 -> 2
- net N$23: track 52.9 -> 8.82 mm
- net GND: track 39.4 -> 77.5 mm
- net N$21: track 45.2 -> 9.29 mm
- net LCD_RS: track 32.9 -> 0.00 mm, vias 2 -> 0
- net LCD_E: track 38.5 -> 12.7 mm, vias 2 -> 0
- net KEY: track 0.00 -> 25.3 mm
- net LCD_R/~W: track 40.8 -> 21.4 mm, vias 2 -> 0
- net N$31: track 0.00 -> 15.8 mm
- net N$7: track 0.00 -> 15.6 mm
- net SWDCLK: track 25.6 -> 10.0 mm
- net I2C_SDA: track 31.8 -> 17.0 mm, vias 2 -> 0
- net N$27: track 0.00 -> 14.6 mm
- net ADC_9V: track 30.6 -> 16.4 mm, vias 1 -> 0
- net I2C_SCL: track 28.6 -> 15.4 mm, vias 2 -> 0
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- removed copper zone on layer 16, net +3.3V
- removed copper zone on layer 16, net +5V
- removed copper zone on layer 16, net GND
- removed copper zone on layer 16, net N$1
- removed copper zone on layer 16, net N$2
- removed copper zone on layer 16, net N$6
Other:
- board size 100 x 68 mm -> 60.2 x 58 mm
- board text removed: "ERROR"
- board text removed: "LED"

Commit message: Humidity metter v2. Change schematic/board 3.
Parts:
- added J5, J7: 0, __MyCommonLib1:RSMD_1206_BIG_GAP
- added J6: 0, __MyCommonLib1:RSMD_0805
- R12: device __MyCommonLib1:RSMD_0603 -> __MyCommonLib1:RSMD_0805
- X1, X2: device __MyCommonLib1:PIN1X1_D3.5MM -> __MyCommonLib1:PIN1X1_3.5MM_PWR
- moved R33 49.3 mm to (23.3, 40.9), turned to 0 degrees
- moved LED1 45.7 mm to (20.2, 42.0), turned to 90 degrees
- moved L2 18.4 mm to (21.8, 24.3)
- moved C17 16.9 mm to (26.7, 22.7), turned to 90 degrees
- moved D2 15.4 mm to (4.30, 20.6), turned to 270 degrees
- moved C6 9.34 mm to (43.9, 17.7), turned to 0 degrees
- moved R1 8.29 mm to (5.20, 38.5)
- moved J2 7.79 mm to (45.5, 33.3)
- moved X1 7.21 mm to (11.9, 41.2)
- moved R34 7.09 mm to (33.6, 30.0)
- moved J4 3.76 mm to (23.3, 43.0), turned to 0 degrees
- moved IC10 3.55 mm to (40.2, 11.3)
- moved R12 3.52 mm to (46.1, 44.6)
- moved R30 3.42 mm to (38.3, 23.5), turned to 180 degrees
- moved J1 3.04 mm to (46.1, 30.8), turned to 90 degrees
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Connections:
- new net N$24: J7.PAD_1, R6.PAD_0
- new net N$4: J5.PAD_1, LCD1.3
- new net N$6: IC3.34, J6.PAD_0
- net +5V: now also R20.1; no longer R20.3
- net ADC_9V: now also IC3.13; no longer IC3.15
- net ERROR_LED: now also IC3.17; no longer IC3.40
- net GND: now also R20.3; no longer R20.1
- net KEY: now also IC3.12; no longer IC3.13
- net LCD_D4: now also IC3.26; no longer IC3.25
- net LCD_D5: now also IC3.28; no longer IC3.27
- net LCD_D6: now also IC3.27; no longer IC3.26
- net LCD_D7: now also IC3.39; no longer IC3.28
- net LCD_E: now also IC3.25; no longer IC3.22
- net LCD_R/~W: now also IC3.22; no longer IC3.21
- net LCD_RS: now also IC3.21; no longer IC3.46
- net N$31: now also J7.PAD_0; no longer R6.PAD_0
- net N$9: now also J5.PAD_0; no longer LCD1.3
- net PWR_HOLD: now also IC3.15; no longer IC3.17
- net SWDIO: now also J6.PAD_1; no longer IC3.34
Routing:
- net +5V: track 0.00 -> 71.5 mm, vias 0 -> 2
- net +3.3V: track 42.1 -> 74.1 mm, vias 1 -> 10
- net GND: track 77.5 -> 105.6 mm, vias 4 -> 8
- net N$9: track 24.9 -> 5.55 mm
- net N$6: track 0.00 -> 15.9 mm
- net LCD_RS: track 0.00 -> 15.7 mm
- net SWDIO: track 20.4 -> 4.87 mm, vias 2 -> 0
- net BOOT1: track 0.00 -> 14.3 mm
- net ERROR_LED: track 0.00 -> 13.0 mm
- net N$2: track 0.00 -> 10.3 mm
- net N$1: track 8.16 -> 0.00 mm
- net LCD_R/~W: track 21.4 -> 14.0 mm
- net N$4: track 0.00 -> 6.64 mm
- net N$31: track 15.8 -> 21.4 mm
- net N$27: track 14.6 -> 19.9 mm
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- added copper zone on layer 16, net +3.3V
- added copper zone on layer 16, net +5V
- added copper zone on layer 16, net GND
- added copper zone on layer 16, net N$1
- added copper zone on layer 16, net N$7

Commit message: Humidity metter v2. Change schematic/board 4.
Parts:
- moved R34 7.40 mm to (26.2, 29.8)
- moved D1 5.20 mm to (23.6, 30.7)
- moved C9 1.00 mm to (19.0, 32.8)
- moved C6 0.98 mm to (44.3, 18.6)
- moved R25 0.90 mm to (20.9, 32.8)
- moved R24 0.76 mm to (17.1, 32.8), turned to 270 degrees
- moved R26 0.30 mm to (55.6, 24.9)
- moved R27 0.30 mm to (55.6, 22.4)
- moved R28 0.30 mm to (49.6, 22.4)
- moved R29 0.30 mm to (49.6, 24.9)
Connections:
- net ADC_9V: now also IC3.12; no longer IC3.13
- net KEY: now also IC3.11; no longer IC3.12
Routing:
- net +3.3V: track 74.1 -> 83.2 mm
- net N$28: track 0.00 -> 5.20 mm
- net N$27: track 19.9 -> 15.0 mm
- net N$31: track 21.4 -> 17.7 mm
- net ADC_9V: track 16.4 -> 19.8 mm
- net SWDIO: track 4.87 -> 2.26 mm
- net N$30: track 0.00 -> 2.60 mm
- net LCD_D7: track 10.6 -> 13.0 mm
- net N$23: track 8.82 -> 6.91 mm
- net N$21: track 9.29 -> 7.46 mm
- net N$15: track 8.20 -> 6.41 mm
- net KEY: track 26.5 -> 28.2 mm
- net N$12: track 10.9 -> 9.12 mm
- net N$17: track 8.26 -> 6.53 mm
- net SWDCLK: track 9.76 -> 11.3 mm
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- added copper zone on layer 16, net N$11
- added copper zone on layer 16, net N$12
- added copper zone on layer 16, net N$13
- added copper zone on layer 16, net N$15
- added copper zone on layer 16, net N$16
- added copper zone on layer 16, net N$17
- added copper zone on layer 16, net N$18
- added copper zone on layer 16, net N$21
- added copper zone on layer 16, net N$22
- added copper zone on layer 16, net N$23
- added copper zone on layer 16, net N$27
- added copper zone on layer 16, net N$31
- added copper zone on layer 16, net N$4
- added copper zone on layer 16, net SWDCLK
- added copper zone on layer 16, net SWDIO
Other:
- board text added: "03.01.2024"
- board text added: "CLK"
- board text added: "DIO"
- board text added: "GND"
- board text added: "VCC"
- board text added: "VER2.0"
- board text removed: "07.08.2024"
- board text removed: "VER1.0"
