File: HumidityMetter/schematic/HumidityMetter_v2.brd (EAGLE design)
At the start: 60.2 x 58 mm, 72 parts, among them IC10 AMS1117-3.3, IC11 MP1482, IC3 STM32F103C8T6, J1 0, J2 0, J3 0, J4 0, J5 0, J6 0, J7 0, K1 POWER_ON, T1 BSS84, T2 BC847, X1 +9V, X2 GND, X3 ISP, X4 SENSOR

Commit message: Humidity metter v2. Change schematic/board 5.
Parts:
- C16: value 3.3nF x 16V -> 4.7nF x 16V
- R16, R17, R18, R19: value 2K0 -> 2K2
- R5: value 5K6 -> 1K5
- T1: value BSS84 -> AO3401
- T2: value BC847 -> 2N7002
Routing:
- net PLUS_SIGN: track 0.00 -> 5.20 mm
- net N$28: track 5.20 -> 0.00 mm
- net N$30: track 2.60 -> 0.00 mm
- net MINUS_SIGN: track 0.00 -> 2.60 mm
