File: HumidityMetter/schematic/HumidityMetter_v2.sch (EAGLE design)
At the start: 64 parts, among them IC1 LM317, IC10 AMS1117-3.3, IC3 STM32F103C8T6, IC4 AM2320, J1 0, J2 0, J3 0, J4 0, K1 POWER_ON, T1 BSS84, T2 BC847, X1 +9V, X2 GND, X3 ISP

Commit message: Humidity metter v2. Change schematic/board.
Parts:
- removed IC1: LM317, __MyCommonLib1:LM317(D2PAK)
- removed IC4: AM2320, __MyCommonLib1:AM2320(HOR)
- removed R32: *, __MyCommonLib1:RSMD_0805
- added C15: 0.1uF x 16V, __MyCommonLib1:CSMD_0603
- added C16: 3.3nF x 16V, __MyCommonLib1:CSMD_0603
- added C17, C7: 10uF x 10V, __MyCommonLib1:CSMD_1206
- added IC11: MP1482, __MyCommonLib1:MP1482(SO-8)
- added L1: 39uH, __MyCommonLib1:L(7MM)
- added L2: 20uH, __MyCommonLib1:L(1206)
- added R8: 100K, __MyCommonLib1:RSMD_0603
- added X4: SENSOR, __MyCommonLib1:PIN4X1(JST_XH2.5)
- C1: device __MyCommonLib1:CSMD_0805 -> __MyCommonLib1:CSMD_0603
- C2: value 0.1uF -> 10uF x 16V; device __MyCommonLib1:CSMD_0805 -> __MyCommonLib1:CSMD_1206
- C3: value 100uFx16V -> 10uF x 16V; device __MyCommonLib1:CE6.3MM -> __MyCommonLib1:CSMD_1206
- C4: value 10uF x 10V -> 10nF x 16V; device __MyCommonLib1:CE5.2MM -> __MyCommonLib1:CSMD_0603
- C5: value 0.1uF -> 10uF x 10V; device __MyCommonLib1:CSMD_0805 -> __MyCommonLib1:CSMD_1206
- J1, J2, R21, R22, R23, R33: device __MyCommonLib1:RSMD_0805 -> __MyCommonLib1:RSMD_0603
- R26, R27, R28, R29: device __MyCommonLib1:R0207 -> __MyCommonLib1:RSMD_0603
- R5: value 1K0 -> 5K6; device __MyCommonLib1:RSMD_0805 -> __MyCommonLib1:RSMD_0603
- R6: value 3K0 -> 36K; device __MyCommonLib1:RSMD_0805 -> __MyCommonLib1:RSMD_0603
- R7: value * -> 8K2; device __MyCommonLib1:RSMD_0805 -> __MyCommonLib1:RSMD_0603
Connections:
- removed net N$24: D3.ANODE, IC3.PA8/USART1_CK/TIM1_CH1/MCO, IC3.PA9/USART1_TX/TIM1_CH2, R34.PIN0
- removed net N$6: C2.PIN1, C3.PLUS, IC1.IN, R24.PIN0, T1.DRAIN
- removed net N$7 (its old number): IC1.ADJ, R32.PIN0, R5.PIN0, R6.PIN0, R7.PIN0
- new net N$25: IC11.EN, R8.PIN0
- new net N$26: D4.ANODE, R3.PIN1, T2.C
- new net N$27: C4.PIN0, IC11.SW, L1.START
- new net N$29: C4.PIN1, IC11.BS
- new net N$31: C5.PIN1, C7.PIN1, L1.END, L2.END, R6.PIN0
- new net N$32: C15.PIN1, IC11.SS
- new net N$34: C16.PIN1, IC11.COMP
- new net N$35: C16.PIN0, R5.PIN0
- new net N$36: IC11.FB, R6.PIN1, R7.PIN0
- new net N$8: C2.PIN1, C3.PIN1, IC11.IN, R24.PIN0, R8.PIN1, T1.DRAIN
- net +3.3V: now also C1.PIN1, R26.PIN0, R27.PIN0, R34.PIN0, X4.1; no longer R34.PIN1
- net +5V: now also C17.PIN1, L2.START; no longer C1.PIN1, C4.PLUS, C5.PIN1, IC1.OUT, IC4.VDD, R26.PIN0, R27.PIN0, R32.PIN1, R5.PIN1
- net GND: now also C15.PIN0, C17.PIN0, C3.PIN0, C7.PIN0, IC11.GND, R5.PIN1, X4.4; no longer C3.MINUS, C4.MINUS, IC4.GND, R6.PIN1
- net KEY: now also D3.ANODE, IC3.PA8/USART1_CK/TIM1_CH1/MCO, R34.PIN1; no longer D3.CATHODE, D4.CATHODE, K1.2
- net N$14: now also X4.2; no longer IC4.SDA
- net N$20: now also X4.3; no longer IC4.SCL
- net N$3: no longer D4.ANODE
- net N$4: now also D3.CATHODE, D4.CATHODE, K1.2; no longer R3.PIN1, T2.C
Other:
- moved on the sheet: C1, C2, C5, C6, C8, C9, D1, D10, D3, D4, IC10, K1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

Commit message: Humidity metter v2. Change schematic/board 2.
Parts:
- removed D10: 1N4007, __MyCommonLib1:1N4001DO-41_10MM
- added D11: B120, __MyCommonLib1:B120(DO-214AC)
- D2: value 1N4007 -> B120; device __MyCommonLib1:1N4001DO-41_10MM -> __MyCommonLib1:B120(DO-214AC)
Connections:
- net +3.3V: now also D11.CATHODE; no longer D2.CATHODE
- net GND: now also D11.ANODE; no longer D10.ANODE
- net N$7: now also D2.CATHODE; no longer D10.CATHODE
Changed lines of the file:
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@@
 <part name="R28" library="__MyCommonLib1" deviceset="R" device="SMD_0603" value="200R"/>
 <part name="R29" library="__MyCommonLib1" deviceset="R" device="SMD_0603" value="200R"/>
-<part name="D10" library="__MyCommonLib1" deviceset="1N4001" device="DO-41_10MM" value="1N4007"/>
 <part name="GND29" library="supply1" deviceset="GND" device=""/>
 <part name="R33" library="__MyCommonLib1" deviceset="R" device="SMD_0603" value="1K0"/>
 <part name="LED1" library="__MyCommonLib1" deviceset="LED3MM" device="(SMD0805)" value="ERROR(RED)"/>
 <part name="GND30" library="supply1" deviceset="GND" device=""/>
-<part name="D2" library="__MyCommonLib1" deviceset="1N4001" device="DO-41_10MM" value="1N4007"/>
 <part name="GND31" library="supply1" deviceset="GND" device=""/>
 <part name="D3" library="__MyCommonLib1" deviceset="LL4147" device="SOD-80" value="LL4148"/>
@@
 <part name="GND32" library="supply1" deviceset="GND" device=""/>
 <part name="X4" library="__MyCommonLib1" deviceset="PIN4X1" device="(JST_XH2.5)" value="SENSOR"/>
+<part name="D11" library="__MyCommonLib1" deviceset="B120" device="(DO-214AC)" value="B120"/>
+<part name="D2" library="__MyCommonLib1" deviceset="B120" device="(DO-214AC)" value="B120"/>
 </parts>
 <sheets>
@@
 <attribute name="VALUE" x="109.22" y="143.51" size="1.27" layer="96" font="vector" ratio="20" rot="R180"/>
 </instance>
-<instance part="D10" gate="D$1" x="467.36" y="180.34" smashed="yes">
-<attribute name="NAME" x="469.9" y="181.61" size="1.27" layer="95" font="vector" ratio="20"/>
-<attribute name="VALUE" x="469.9" y="180.34" size="1.27" layer="96" font="vector" ratio="20"/>
-</instance>
 <instance part="GND29" gate="1" x="467.36" y="172.72" smashed="yes" rot="MR0">
 <attribute name="VALUE" x="469.265" y="170.815" size="1.27" layer="96" font="vector" ratio="20" rot="MR0"/>
@@
 <attribute name="VALUE" x="40.64" y="133.985" size="1.27" layer="96" font="vector" ratio="20"/>
 </instance>
-<instance part="D2" gate="D$1" x="66.04" y="160.02" smashed="yes" rot="R270">
-<attribute name="NAME" x="63.5" y="163.83" size="1.27" layer="95" font="vector" ratio="20"/>
-<attribute name="VALUE" x="63.5" y="162.56" size="1.27" layer="96" font="vector" ratio="20"/>
-</instance>
 <instance part="GND31" gate="1" x="60.96" y="154.94" smashed="yes">
 <attribute name="VALUE" x="59.69" y="153.035" size="1.27" layer="96" font="vector" ratio="20"/>
@@
 <attribute name="NAME" x="121.92" y="152.4" size="1.27" layer="95" font="vector" ratio="20"/>
 <attribute name="VALUE" x="120.65" y="138.43" size="1.27" layer="96" font="vector" ratio="20"/>
+</instance>
+<instance part="D11" gate="G$1" x="66.04" y="160.02" smashed="yes" rot="R270">
+<attribute name="NAME" x="62.23" y="162.56" size="1.27" layer="95" font="vector" ratio="20"/>
+<attribute name="VALUE" x="67.31" y="162.56" size="1.27" layer="96" font="vector" ratio="20"/>
+</instance>
+<instance part="D2" gate="G$1" x="467.36" y="180.34" smashed="yes">
+<attribute name="NAME" x="469.9" y="180.34" size="1.27" layer="95" font="vector" ratio="20"/>
+<attribute name="VALUE" x="469.9" y="179.07" size="1.27" layer="96" font="vector" ratio="20"/>
 </instance>
 </instances>
@@
 </segment>
 <segment>
-<pinref part="D10" gate="D$1" pin="ANODE"/>
 <pinref part="GND29" gate="1" pin="GND"/>
 <wire x1="467.36" y1="175.26" x2="467.36" y2="177.8" width="0.1524" layer="91"/>
+<pinref part="D2" gate="G$1" pin="ANODE"/>
 </segment>
 <segment>
@@
 </segment>
 <segment>
-<pinref part="D2" gate="D$1" pin="ANODE"/>
 <pinref part="GND31" gate="1" pin="GND"/>
-<wire x1="63.5" y1="160.02" x2="60.96" y2="160.02" width="0.1524" layer="91"/>
 <wire x1="60.96" y1="160.02" x2="60.96" y2="157.48" width="0.1524" layer="91"/>
+<pinref part="D11" gate="G$1" pin="ANODE"/>
+<wire x1="60.96" y1="160.02" x2="63.5" y2="160.02" width="0.1524" layer="91"/>
 </segment>
 <segment>
@@
 <wire x1="81.28" y1="154.94" x2="73.66" y2="154.94" width="0.1524" layer="91"/>
 <label x="81.28" y="156.21" size="1.27" layer="95" font="vector" ratio="20" rot="R180"/>
-<pinref part="D2" gate="D$1" pin="CATHODE"/>
 <wire x1="73.66" y1="154.94" x2="71.12" y2="154.94" width="0.1524" layer="91"/>
-<wire x1="68.58" y1="160.02" x2="73.66" y2="160.02" width="0.1524" layer="91"/>
 <wire x1="73.66" y1="160.02" x2="73.66" y2="154.94" width="0.1524" layer="91"/>
 <junction x="73.66" y="154.94"/>
+<pinref part="D11" gate="G$1" pin="CATHODE"/>
+<wire x1="68.58" y1="160.02" x2="73.66" y2="160.02" width="0.1524" layer="91"/>
 </segment>
 <segment>
@@
 <pinref part="R1" gate="R$1" pin="PIN0"/>
 <wire x1="472.44" y1="185.42" x2="467.36" y2="185.42" width="0.1524" layer="91"/>
-<pinref part="D10" gate="D$1" pin="CATHODE"/>
 <wire x1="467.36" y1="182.88" x2="467.36" y2="185.42" width="0.1524" layer="91"/>
 <pinref part="T1" gate="G$1" pin="SOURCE"/>
@@
 <junction x="462.28" y="185.42"/>
 <junction x="467.36" y="185.42"/>
-</segment>
-</net>
+<pinref part="D2" gate="G$1" pin="CATHODE"/>
+</segment>
+</net>

Commit message: Humidity metter v2. Change schematic/board 2.
Parts:
- removed D3, D4: LL4148, __MyCommonLib1:LL4147SOD-80
- added D55: BAT54C, __MyCommonLib1:BAT54C(SOT23)
- C9: device __MyCommonLib1:CSMD_0805 -> __MyCommonLib1:CSMD_0603
- LCD1: device __MyCommonLib1:LCD_0802B(0802B_CHINA_CLONE) -> __MyCommonLib1:LCD_0802BLCD_0802B_2SCREW(CHINA_CLONE)
- R1: device __MyCommonLib1:R0207 -> __MyCommonLib1:RSMD_1206
- R11, R24: device __MyCommonLib1:RSMD_1206_BIG_GAP -> __MyCommonLib1:RSMD_0603
- R2, R25, R3, R34, R4: device __MyCommonLib1:RSMD_0805 -> __MyCommonLib1:RSMD_0603
- R20: device __MyCommonLib1:R_ADJSTAND_6.5_X_3.5MM -> __MyCommonLib1:R_ADJHOR_7X7MM
Connections:
- removed net N$4: D3.CATHODE, D4.CATHODE, K1.2
- new net N$2: D55.CATHODE, K1.2
- net ADC_9V: now also IC3.PA5/SPI1_SCK/ADC12_IN5; no longer IC3.PA3/USART2_RX/ADC12_IN3/TIM2_CH4
- net I2C_SCL: now also IC3.PB6/I2C1_SCL/TIM4_CH1; no longer IC3.PB10/I2C2_SCL/USART3_TX
- net I2C_SDA: now also IC3.PB7/I2C1_SDA/TIM4_CH2; no longer IC3.PB11/I2C2_SDA/USART3_RX
- net KEY: now also D55.ANODE2, IC3.PA3/USART2_RX/ADC12_IN3/TIM2_CH4; no longer D3.ANODE, IC3.PA8/USART1_CK/TIM1_CH1/MCO
- net LCD_D5: now also IC3.PB14/SPI2_MISO/USART3_RTS/TIM1_CH2N; no longer IC3.PB15/SPI2_MOSI/TIM1_CH3N
- net LCD_D7: now also IC3.PB15/SPI2_MOSI/TIM1_CH3N; no longer IC3.PB14/SPI2_MISO/USART3_RTS/TIM1_CH2N
- net LCD_E: now also IC3.PB11/I2C2_SDA/USART3_RX; no longer IC3.PB7/I2C1_SDA/TIM4_CH2
- net LCD_R/~W: now also IC3.PB10/I2C2_SCL/USART3_TX; no longer IC3.PB9/TIM4_CH4
- net LCD_RS: now also IC3.PB9/TIM4_CH4; no longer IC3.PB8/TIM4_CH3
- net N$14: now also R29.PIN1; no longer R28.PIN1
- net N$20: now also R28.PIN1; no longer R29.PIN1
- net N$26: now also D55.ANODE1; no longer D4.ANODE
- net PWR_HOLD: now also IC3.PA7/SPI1_MOSI/ADC12_IN7/TIM3_CH2; no longer IC3.PA10/USART1_RX/TIM1_CH3
Other:
- moved on the sheet: C2, C3, R28, R29, R34

Commit message: Humidity metter v2. Change schematic/board 3.
Parts:
- added J5, J7: 0, __MyCommonLib1:RSMD_1206_BIG_GAP
- added J6: 0, __MyCommonLib1:RSMD_0805
- R12: device __MyCommonLib1:RSMD_0603 -> __MyCommonLib1:RSMD_0805
- X1, X2: device __MyCommonLib1:PIN1X13.5MM_DRILL -> __MyCommonLib1:PIN1X13.5MM_PWR
Connections:
- new net N$24: J7.PIN1, R6.PIN0
- new net N$4: J5.PIN1, LCD1.VO
- new net N$6: IC3.PA13/JTMS/SWDIO, J6.PIN0
- net +5V: now also R20.END_A; no longer R20.END_B
- net ADC_9V: now also IC3.PA3/USART2_RX/ADC12_IN3/TIM2_CH4; no longer IC3.PA5/SPI1_SCK/ADC12_IN5
- net ERROR_LED: now also IC3.PA7/SPI1_MOSI/ADC12_IN7/TIM3_CH2; no longer IC3.PB4/JNTRST
- net GND: now also R20.END_B; no longer R20.END_A
- net KEY: now also IC3.PA2/USART2_TX/ADC12_IN2/TIM2_CH3; no longer IC3.PA3/USART2_RX/ADC12_IN3/TIM2_CH4
- net LCD_D4: now also IC3.PB13/SPI2_SCK/USART3_CTS/TIM1_CH1; no longer IC3.PB12/SPI2_NSS/I2C2_SMBAI/USART3_CK/TIM1_BKIN
- net LCD_D5: now also IC3.PB15/SPI2_MOSI/TIM1_CH3N; no longer IC3.PB14/SPI2_MISO/USART3_RTS/TIM1_CH2N
- net LCD_D6: now also IC3.PB14/SPI2_MISO/USART3_RTS/TIM1_CH2N; no longer IC3.PB13/SPI2_SCK/USART3_CTS/TIM1_CH1
- net LCD_D7: now also IC3.PB3/JTDO; no longer IC3.PB15/SPI2_MOSI/TIM1_CH3N
- net LCD_E: now also IC3.PB12/SPI2_NSS/I2C2_SMBAI/USART3_CK/TIM1_BKIN; no longer IC3.PB11/I2C2_SDA/USART3_RX
- net LCD_R/~W: now also IC3.PB11/I2C2_SDA/USART3_RX; no longer IC3.PB10/I2C2_SCL/USART3_TX
- net LCD_RS: now also IC3.PB10/I2C2_SCL/USART3_TX; no longer IC3.PB9/TIM4_CH4
- net N$31: now also J7.PIN0; no longer R6.PIN0
- net N$9: now also J5.PIN0; no longer LCD1.VO
- net PWR_HOLD: now also IC3.PA5/SPI1_SCK/ADC12_IN5; no longer IC3.PA7/SPI1_MOSI/ADC12_IN7/TIM3_CH2
- net SWDIO: now also J6.PIN1; no longer IC3.PA13/JTMS/SWDIO
Other:
- moved on the sheet: C8, R20

Commit message: Humidity metter v2. Change schematic/board 4.
Connections:
- net ADC_9V: now also IC3.PA2/USART2_TX/ADC12_IN2/TIM2_CH3; no longer IC3.PA3/USART2_RX/ADC12_IN3/TIM2_CH4
- net KEY: now also IC3.PA1/USART2_RTS/ADC12_IN1/TIM2_CH2; no longer IC3.PA2/USART2_TX/ADC12_IN2/TIM2_CH3
Changed lines of the file:
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@@
 </segment>
 <segment>
-<wire x1="33.02" y1="91.44" x2="22.86" y2="91.44" width="0.1524" layer="91"/>
-<label x="30.48" y="92.71" size="1.27" layer="95" font="vector" ratio="20" rot="R180"/>
-<pinref part="IC3" gate="G$1" pin="PA3/USART2_RX/ADC12_IN3/TIM2_CH4"/>
+<wire x1="33.02" y1="93.98" x2="22.86" y2="93.98" width="0.1524" layer="91"/>
+<label x="30.48" y="95.25" size="1.27" layer="95" font="vector" ratio="20" rot="R180"/>
+<pinref part="IC3" gate="G$1" pin="PA2/USART2_TX/ADC12_IN2/TIM2_CH3"/>
 </segment>
 </net>
@@
 </segment>
 <segment>
-<wire x1="33.02" y1="93.98" x2="22.86" y2="93.98" width="0.1524" layer="91"/>
-<label x="30.48" y="95.25" size="1.27" layer="95" font="vector" ratio="20" rot="R180"/>
-<pinref part="IC3" gate="G$1" pin="PA2/USART2_TX/ADC12_IN2/TIM2_CH3"/>
-</segment>
-</net>
+<wire x1="33.02" y1="96.52" x2="22.86" y2="96.52" width="0.1524" layer="91"/>
+<label x="30.48" y="97.79" size="1.27" layer="95" font="vector" ratio="20" rot="R180"/>
+<pinref part="IC3" gate="G$1" pin="PA1/USART2_RTS/ADC12_IN1/TIM2_CH2"/>
+</segment>
+</net>
