File: HumidityMetter/schematic/HumidityMetter_v2.sch (EAGLE design)
At the start: 72 parts, among them IC10 AMS1117-3.3, IC11 MP1482, IC3 STM32F103C8T6, J1 0, J2 0, J3 0, J4 0, J5 0, J6 0, J7 0, K1 POWER_ON, T1 BSS84, T2 BC847, X1 +9V, X2 GND, X3 ISP, X4 SENSOR

Commit message: Humidity metter v2. Change schematic/board 5.
Parts:
- C16: value 3.3nF x 16V -> 4.7nF x 16V
- R16, R17, R18, R19: value 2K0 -> 2K2
- R5: value 5K6 -> 1K5
- T1: value BSS84 -> AO3401
- T2: value BC847 -> 2N7002; device __MyCommonLib1:BC847SOT23_SMALL_PADS -> __MyCommonLib1:2N7002SOT23_SMALL_PADS
Connections:
- net GND: now also T2.SOURCE; no longer T2.E
- net N$26: now also T2.DRAIN; no longer T2.C
- net N$5: now also T2.GATE; no longer T2.B
Other:
- moved on the sheet: R11, R4
