File: PowerSupply_1600W/CurrentRestrictionBoard/CurrentRestrictionBoard_V1_0.sch (EAGLE design)
At the start: 0 parts

Commit message: PS 1600W Current restriction board.
Parts:
- added C1, C4: *, __MyCommonLib1:CSMD_0805
- added C2: 0.47uF x 16V, __MyCommonLib1:CSMD_0805
- added C3: 1n0 16V, __MyCommonLib1:CSMD_0805
- added C5: 0.1uF x 16V, __MyCommonLib1:CSMD_0805
- added D1: LL4148, __MyCommonLib1:LL4147SOD-80
- added R1: 22K, __MyCommonLib1:RSMD_0805
- added R2: 10R, __MyCommonLib1:RSMD_1206
- added R3, R7: 5K1, __MyCommonLib1:RSMD_0805
- added R4: RSMD_0805, __MyCommonLib1:RSMD_0805
- added R5: *, __MyCommonLib1:RSMD_0805
- added R6: 680K, __MyCommonLib1:RSMD_0805
- added R8: 10K, __MyCommonLib1:RSMD_0805
- added U1: LM358, __MyCommonLib1:LM358SOIC8
- added U2: TL431, __MyCommonLib1:TL431SOT23
- added X1: GND, __MyCommonLib1:PIN1X1PAD_2.5X2.5
- added X2: +12V, __MyCommonLib1:PIN1X1PAD_2.5X2.5
- added X3: CS_IN, __MyCommonLib1:PIN1X1PAD_2.5X2.5
- added X4: VReg_OUT, __MyCommonLib1:PIN1X1PAD_2.5X2.5
Connections:
- new net +12V: C2.PIN1, R2.PIN0, R7.PIN1, U1G$3.VCC
- new net GND: C1.PIN0, C2.PIN0, C5.PIN0, R8.PIN0, U1G$3.GND, U2.ANODE, X1.1
- new net N$1: R2.PIN1, X2.1
- new net N$10: C5.PIN1, R1.PIN1, R7.PIN0, U2.CATHODE, U2.REFERENCE
- new net N$2: R4.PIN1, X3.1
- new net N$3: C1.PIN1, R4.PIN0, U1G$1.IN+
- new net N$4: C3.PIN0, C4.PIN0, R1.PIN0, R6.PIN1, R8.PIN1, U1G$1.IN-
- new net N$5: C3.PIN1, R5.PIN0, R6.PIN0, U1G$1.OUT, U1G$2.IN+
- new net N$6: C4.PIN1, R5.PIN1
- new net N$7: D1.CATHODE, R3.PIN1, U1G$2.IN-
- new net N$8: D1.ANODE, U1G$2.OUT
- new net N$9: R3.PIN0, X4.1

Commit message: PS 1600W Current restriction board. Route done.
Parts:
- added J1: 0, __MyCommonLib1:RSMD_0805
- C1, C3, C4, C5: device __MyCommonLib1:CSMD_0805 -> __MyCommonLib1:CSMD_0603
- D1: value LL4148 -> BAT54A; device __MyCommonLib1:LL4147SOD-80 -> __MyCommonLib1:BAT54ASOT23_SMALL_PADS
- R1, R3, R5, R6, R8: device __MyCommonLib1:RSMD_0805 -> __MyCommonLib1:RSMD_0603
- R2: device __MyCommonLib1:RSMD_1206 -> __MyCommonLib1:RSMD_0805
- R4: value RSMD_0805 -> *; device __MyCommonLib1:RSMD_0805 -> __MyCommonLib1:RSMD_0603
Connections:
- new net N$11: J1.PIN0, U1G$2.IN+
- net N$5: now also J1.PIN1; no longer U1G$2.IN+
- net N$7: now also D1.CATHODE1, D1.CATHODE2; no longer D1.CATHODE
Other:
- moved on the sheet: R3, U1G$2, X4
Changed lines of the file:
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@@
 <part name="U1" library="__MyCommonLib1" deviceset="LM358" device="SOIC8" value="LM358"/>
 <part name="FRAME4" library="frames" deviceset="A4L-LOC" device="" value="12_TO_200VDC_CONVERTER"/>
-<part name="C1" library="__MyCommonLib1" deviceset="C" device="SMD_0805" value="*"/>
-<part name="D1" library="__MyCommonLib1" deviceset="LL4147" device="SOD-80" value="LL4148"/>
-<part name="R1" library="__MyCommonLib1" deviceset="R" device="SMD_0805" value="22K"/>
+<part name="C1" library="__MyCommonLib1" deviceset="C" device="SMD_0603" value="*"/>
+<part name="R1" library="__MyCommonLib1" deviceset="R" device="SMD_0603" value="22K"/>
 <part name="U2" library="__MyCommonLib1" deviceset="TL431" device="SOT23" value="TL431"/>
 <part name="X1" library="__MyCommonLib1" deviceset="PIN1X1" device="PAD_2.5X2.5" value="GND"/>
@@
 <part name="X3" library="__MyCommonLib1" deviceset="PIN1X1" device="PAD_2.5X2.5" value="CS_IN"/>
 <part name="X4" library="__MyCommonLib1" deviceset="PIN1X1" device="PAD_2.5X2.5" value="VReg_OUT"/>
-<part name="R2" library="__MyCommonLib1" deviceset="R" device="SMD_1206" value="10R"/>
-<part name="R3" library="__MyCommonLib1" deviceset="R" device="SMD_0805" value="5K1"/>
+<part name="R2" library="__MyCommonLib1" deviceset="R" device="SMD_0805" value="10R"/>
+<part name="R3" library="__MyCommonLib1" deviceset="R" device="SMD_0603" value="5K1"/>
 <part name="C2" library="__MyCommonLib1" deviceset="C" device="SMD_0805" value="0.47uF x 16V"/>
 <part name="GND1" library="supply1" deviceset="GND" device=""/>
 <part name="GND2" library="supply1" deviceset="GND" device=""/>
 <part name="GND3" library="supply1" deviceset="GND" device=""/>
-<part name="R4" library="__MyCommonLib1" deviceset="R" device="SMD_0805"/>
+<part name="R4" library="__MyCommonLib1" deviceset="R" device="SMD_0603" value="*"/>
 <part name="GND4" library="supply1" deviceset="GND" device=""/>
-<part name="C3" library="__MyCommonLib1" deviceset="C" device="SMD_0805" value="1n0 16V"/>
-<part name="C4" library="__MyCommonLib1" deviceset="C" device="SMD_0805" value="*"/>
-<part name="R5" library="__MyCommonLib1" deviceset="R" device="SMD_0805" value="*"/>
-<part name="R6" library="__MyCommonLib1" deviceset="R" device="SMD_0805" value="680K"/>
-<part name="C5" library="__MyCommonLib1" deviceset="C" device="SMD_0805" value="0.1uF x 16V"/>
+<part name="C3" library="__MyCommonLib1" deviceset="C" device="SMD_0603" value="1n0 16V"/>
+<part name="C4" library="__MyCommonLib1" deviceset="C" device="SMD_0603" value="*"/>
+<part name="R5" library="__MyCommonLib1" deviceset="R" device="SMD_0603" value="*"/>
+<part name="R6" library="__MyCommonLib1" deviceset="R" device="SMD_0603" value="680K"/>
+<part name="C5" library="__MyCommonLib1" deviceset="C" device="SMD_0603" value="0.1uF x 16V"/>
 <part name="GND5" library="supply1" deviceset="GND" device=""/>
 <part name="GND6" library="supply1" deviceset="GND" device=""/>
 <part name="R7" library="__MyCommonLib1" deviceset="R" device="SMD_0805" value="5K1"/>
-<part name="R8" library="__MyCommonLib1" deviceset="R" device="SMD_0805" value="10K"/>
+<part name="R8" library="__MyCommonLib1" deviceset="R" device="SMD_0603" value="10K"/>
 <part name="GND7" library="supply1" deviceset="GND" device=""/>
+<part name="J1" library="__MyCommonLib1" deviceset="R" device="SMD_0805" value="0"/>
+<part name="D1" library="__MyCommonLib1" deviceset="BAT54A" device="SOT23_SMALL_PADS" value="BAT54A"/>
 </parts>
 <sheets>
@@
 <attribute name="VALUE" x="77.47" y="105.41" size="1.27" layer="96" font="vector" ratio="20"/>
 </instance>
-<instance part="U1" gate="G$2" x="116.84" y="104.14" smashed="yes">
-<attribute name="NAME" x="113.03" y="104.14" size="1.27" layer="95" font="vector" ratio="20"/>
-<attribute name="VALUE" x="113.03" y="102.87" size="1.27" layer="96" font="vector" ratio="20"/>
+<instance part="U1" gate="G$2" x="119.38" y="104.14" smashed="yes">
+<attribute name="NAME" x="115.57" y="104.14" size="1.27" layer="95" font="vector" ratio="20"/>
+<attribute name="VALUE" x="115.57" y="102.87" size="1.27" layer="96" font="vector" ratio="20"/>
 </instance>
 <instance part="U1" gate="G$3" x="58.42" y="152.4" smashed="yes">
@@
 <attribute name="VALUE" x="54.61" y="101.6" size="1.27" layer="96" font="vector" ratio="20"/>
 </instance>
-<instance part="D1" gate="D1" x="129.54" y="104.14" smashed="yes" rot="R270">
-<attribute name="NAME" x="127" y="100.33" size="1.27" layer="95" font="vector" ratio="20"/>
-<attribute name="VALUE" x="127" y="99.06" size="1.27" layer="96" font="vector" ratio="20"/>
-</instance>
 <instance part="R1" gate="R$1" x="40.64" y="73.66" smashed="yes" rot="R90">
 <attribute name="NAME" x="38.1" y="77.47" size="1.27" layer="95" font="vector" ratio="20"/>
@@
 <attribute name="VALUE" x="36.83" y="113.03" size="1.27" layer="96" font="vector" ratio="20" rot="MR0"/>
 </instance>
-<instance part="X4" gate="X$1" x="158.75" y="104.14" smashed="yes" rot="MR180">
-<attribute name="NAME" x="156.21" y="99.06" size="1.27" layer="95" font="vector" ratio="20" rot="MR180"/>
-<attribute name="VALUE" x="156.21" y="100.33" size="1.27" layer="96" font="vector" ratio="20" rot="MR180"/>
+<instance part="X4" gate="X$1" x="168.91" y="104.14" smashed="yes" rot="MR180">
+<attribute name="NAME" x="166.37" y="99.06" size="1.27" layer="95" font="vector" ratio="20" rot="MR180"/>
+<attribute name="VALUE" x="166.37" y="100.33" size="1.27" layer="96" font="vector" ratio="20" rot="MR180"/>
 </instance>
 <instance part="R2" gate="R$1" x="43.18" y="160.02" smashed="yes" rot="R90">
@@
 <attribute name="VALUE" x="40.64" y="162.56" size="1.27" layer="96" font="vector" ratio="20"/>
 </instance>
-<instance part="R3" gate="R$1" x="142.24" y="104.14" smashed="yes" rot="R90">
-<attribute name="NAME" x="137.16" y="107.95" size="1.27" layer="95" font="vector" ratio="20"/>
-<attribute name="VALUE" x="137.16" y="106.68" size="1.27" layer="96" font="vector" ratio="20"/>
+<instance part="R3" gate="R$1" x="152.4" y="104.14" smashed="yes" rot="R90">
+<attribute name="NAME" x="147.32" y="107.95" size="1.27" layer="95" font="vector" ratio="20"/>
+<attribute name="VALUE" x="147.32" y="106.68" size="1.27" layer="96" font="vector" ratio="20"/>
 </instance>
 <instance part="C2" gate="C$1" x="50.8" y="154.94" smashed="yes">
@@
 <instance part="GND7" gate="1" x="48.26" y="55.88" smashed="yes">
 <attribute name="VALUE" x="45.72" y="53.34" size="1.27" layer="96"/>
+</instance>
+<instance part="J1" gate="R$1" x="104.14" y="106.68" smashed="yes" rot="R90">
+<attribute name="NAME" x="101.6" y="107.95" size="1.27" layer="95" font="vector" ratio="20"/>
+<attribute name="VALUE" x="106.68" y="109.22" size="1.27" layer="96" font="vector" ratio="20" rot="R180"/>
+</instance>
+<instance part="D1" gate="G$1" x="134.62" y="104.14" smashed="yes" rot="R90">
+<attribute name="NAME" x="132.08" y="110.49" size="1.27" layer="95" font="vector" ratio="20"/>
+<attribute name="VALUE" x="132.08" y="109.22" size="1.27" layer="96" font="vector" ratio="20"/>
 </instance>
 </instances>
@@
 <junction x="96.52" y="93.98"/>
 <junction x="96.52" y="99.06"/>
-<pinref part="U1" gate="G$2" pin="IN+"/>
-<wire x1="109.22" y1="106.68" x2="96.52" y2="106.68" width="0.1524" layer="91"/>
+<pinref part="J1" gate="R$1" pin="PIN1"/>
+<wire x1="99.06" y1="106.68" x2="96.52" y2="106.68" width="0.1524" layer="91"/>
 <junction x="96.52" y="106.68"/>
 </segment>
@@
 <segment>
 <pinref part="U1" gate="G$2" pin="IN-"/>
-<wire x1="109.22" y1="101.6" x2="106.68" y2="101.6" width="0.1524" layer="91"/>
-<wire x1="106.68" y1="101.6" x2="106.68" y2="96.52" width="0.1524" layer="91"/>
-<wire x1="106.68" y1="96.52" x2="134.62" y2="96.52" width="0.1524" layer="91"/>
-<wire x1="134.62" y1="96.52" x2="134.62" y2="104.14" width="0.1524" layer="91"/>
-<pinref part="D1" gate="D1" pin="CATHODE"/>
-<wire x1="134.62" y1="104.14" x2="132.08" y2="104.14" width="0.1524" layer="91"/>
+<wire x1="111.76" y1="101.6" x2="109.22" y2="101.6" width="0.1524" layer="91"/>
+<wire x1="109.22" y1="101.6" x2="109.22" y2="96.52" width="0.1524" layer="91"/>
+<wire x1="109.22" y1="96.52" x2="144.78" y2="96.52" width="0.1524" layer="91"/>
+<wire x1="144.78" y1="96.52" x2="144.78" y2="104.14" width="0.1524" layer="91"/>
 <pinref part="R3" gate="R$1" pin="PIN1"/>
-<wire x1="137.16" y1="104.14" x2="134.62" y2="104.14" width="0.1524" layer="91"/>
-<junction x="134.62" y="104.14"/>
+<wire x1="147.32" y1="104.14" x2="144.78" y2="104.14" width="0.1524" layer="91"/>
+<junction x="144.78" y="104.14"/>
+<pinref part="D1" gate="G$1" pin="CATHODE2"/>
+<wire x1="137.16" y1="106.68" x2="139.7" y2="106.68" width="0.1524" layer="91"/>
+<pinref part="D1" gate="G$1" pin="CATHODE1"/>
+<wire x1="137.16" y1="101.6" x2="139.7" y2="101.6" width="0.1524" layer="91"/>
+<wire x1="139.7" y1="101.6" x2="139.7" y2="104.14" width="0.1524" layer="91"/>
+<wire x1="139.7" y1="104.14" x2="139.7" y2="106.68" width="0.1524" layer="91"/>
+<wire x1="144.78" y1="104.14" x2="139.7" y2="104.14" width="0.1524" layer="91"/>
+<junction x="139.7" y="104.14"/>
 </segment>
 </net>
@@
 <segment>
 <pinref part="U1" gate="G$2" pin="OUT"/>
-<pinref part="D1" gate="D1" pin="ANODE"/>
-<wire x1="124.46" y1="104.14" x2="127" y2="104.14" width="0.1524" layer="91"/>
+<pinref part="D1" gate="G$1" pin="ANODE"/>
+<wire x1="129.54" y1="104.14" x2="127" y2="104.14" width="0.1524" layer="91"/>
 </segment>
 </net>
@@
 <pinref part="R3" gate="R$1" pin="PIN0"/>
 <pinref part="X4" gate="X$1" pin="1"/>
-<wire x1="154.94" y1="104.14" x2="147.32" y2="104.14" width="0.1524" layer="91"/>
+<wire x1="165.1" y1="104.14" x2="157.48" y2="104.14" width="0.1524" layer="91"/>
 </segment>
 </net>
@@
 </segment>
 </net>
+<net name="N$11" class="0">
+<segment>
+<pinref part="J1" gate="R$1" pin="PIN0"/>
+<pinref part="U1" gate="G$2" pin="IN+"/>
+<wire x1="109.22" y1="106.68" x2="111.76" y2="106.68" width="0.1524" layer="91"/>
+</segment>
+</net>
