File: PowerSupply_1600W/CurrentRestrictionBoard/CurrentRestrictionBoard_V1_0_TO_PRINT.brd (EAGLE design)
At the start: 21.5 x 15.1 mm, 21 parts, among them J1 0, U1 LM358, U2 TL431, X1 GND, X2 +12V, X3 CS_IN, X4 VReg_OUT

Commit message: PS1600W. Current restriction board.
Parts:
- added C10: 0.1uF x 16V, __MyCommonLib1:RSMD_0603
- added C6, C9, R12, R13: *, __MyCommonLib1:RSMD_0603
- added C7: 0.47uF x 16V, __MyCommonLib1:RSMD_0805
- added C8: 1n0 16V, __MyCommonLib1:RSMD_0603
- added D2: BAT54A, __MyCommonLib1:SOT23_SMALL_PADS
- added J2: 0, __MyCommonLib1:RSMD_0805
- added R10: 10R, __MyCommonLib1:RSMD_0805
- added R11: 5K1, __MyCommonLib1:RSMD_0603
- added R14: 680K, __MyCommonLib1:RSMD_0603
- added R15: 5K1, __MyCommonLib1:RSMD_0805
- added R16: 10K, __MyCommonLib1:RSMD_0603
- added R9: 22K, __MyCommonLib1:RSMD_0603
- added U3: LM358, __MyCommonLib1:SOIC8
- added U4: TL431, __MyCommonLib1:SOT23
- added X5: GND, __MyCommonLib1:PIN1X1_2.5X2.5MM
- added X6: +12V, __MyCommonLib1:PIN1X1_2.5X2.5MM
- added X7: CS_IN, __MyCommonLib1:PIN1X1_2.5X2.5MM
- added X8: VReg_OUT, __MyCommonLib1:PIN1X1_2.5X2.5MM
Connections:
- new net +12V1: C7.PAD_1, R10.PAD_0, R15.PAD_1, U3.8
- new net GND1: C10.PAD_0, C6.PAD_0, C7.PAD_0, R16.PAD_0, U3.4, U4.3, X5.1
- new net N$12: R10.PAD_1, X6.1
- new net N$13: R12.PAD_1, X7.1
- new net N$14: C6.PAD_1, R12.PAD_0, U3.3
- new net N$15: C8.PAD_1, J2.PAD_1, R13.PAD_0, R14.PAD_0, U3.1
- new net N$16: C9.PAD_1, R13.PAD_1
- new net N$17: D2.1, D2.2, R11.PAD_1, U3.6
- new net N$18: D2.3, U3.7
- new net N$19: R11.PAD_0, X8.1
- new net N$20: C10.PAD_1, R15.PAD_0, R9.PAD_1, U4.1, U4.2
- new net N$21: C8.PAD_0, C9.PAD_0, R14.PAD_1, R16.PAD_1, R9.PAD_0, U3.2
- new net N$22: J2.PAD_0, U3.5
Routing:
- net N$22: track 0.00 -> 16.7 mm
- net GND1: track 0.00 -> 14.4 mm
- net N$21: track 0.00 -> 13.9 mm
- net N$14: track 0.00 -> 12.0 mm
- net N$15: track 0.00 -> 11.2 mm
- net N$20: track 0.00 -> 9.99 mm
- net N$17: track 0.00 -> 7.82 mm
- net +12V1: track 0.00 -> 6.59 mm
- net N$18: track 0.00 -> 3.82 mm
- net N$19: track 0.00 -> 2.94 mm
- net N$12: track 0.00 -> 2.92 mm
- net N$13: track 0.00 -> 2.57 mm
- net S$4: track 0.00 -> 2.00 mm
- net S$3: track 0.00 -> 2.00 mm
- net S$2: track 0.00 -> 2.00 mm
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- added copper zone on layer 1, net +12V1
- added copper zone on layer 1, net GND1
Other:
- board size 21.5 x 15.1 mm -> 21.5 x 31.2 mm
