File: SoftStartBoard/schematic/SoftStart_V1_0.brd (EAGLE design)
At the start: 70 x 50 mm, 74 parts, among them T1 PK616BA, T2 PK616BA, T3 PK616BA, T4 PK616BA, T6 BC857, T7 BC847SOT23, T8 2N7002, U1 TP2274, U2 AMS1117, U3 MC34063, X1 +12V, X10 ON/OFF, X2 GND, X3 LAMP, X4 LAMP, X5 SET_DUTY_CYCLE(10K)

Commit message: SoftStart. Almost routed PCB.
Parts:
- added C18: 0.1uF x 16V, __MyCommonLib1:RSMD_0805
- added R18: 20R*, __MyCommonLib1:RSMD_1206
- C4: device __MyCommonLib1:RSMD_0805 -> __MyCommonLib1:RSMD_1206
- R23: device __MyCommonLib1:RSMD_0805 -> __MyCommonLib1:RSMD_1206_BIG_GAP
- moved R17 335.9 mm to (20.8, 6.00), turned to 180 degrees
- moved R34 334.3 mm to (29.5, 8.30), turned to 270 degrees
- moved C17 330.5 mm to (16.3, 6.00), turned to 180 degrees
- moved R28 330.4 mm to (43.7, 43.9), turned to 90 degrees
- moved R29 330.2 mm to (43.7, 39.7), turned to 90 degrees
- moved R31 321.0 mm to (19.8, 20.1), turned to 90 degrees
- moved ZD3 320.4 mm to (17.1, 3.10)
- moved R33 318.8 mm to (25.5, 7.10)
- moved R32 317.6 mm to (16.2, 14.0), turned to 180 degrees
- moved T8 305.3 mm to (16.3, 10.0), turned to 180 degrees
- moved D5 305.0 mm to (24.3, 9.80)
- moved R30 303.6 mm to (20.9, 13.5)
- moved R10 296.5 mm to (20.0, 10.0), turned to 90 degrees
- moved C10 276.2 mm to (46.2, 34.7), turned to 180 degrees
- moved T7 238.7 mm to (34.1, 31.3), turned to 270 degrees
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Connections:
- new net N$30: C18.PAD_1, R18.PAD_1, T7.3
- net +10V: now also R18.PAD_0; no longer T7.3
- net GND: now also C18.PAD_0
- net N$11: now also D5.CATHODE, R34.PAD_0; no longer D5.ANODE, R34.PAD_1
- net N$12: now also U1.5; no longer U1.3
- net N$13: now also U1.7; no longer U1.1
- net N$14: now also U1.6; no longer U1.2
- net N$15: now also U1.2; no longer U1.6
- net N$16: now also U1.10; no longer U1.12
- net N$17: now also U1.9; no longer U1.13
- net N$18: now also U1.13, U1.8; no longer U1.14, U1.9
- net N$19: now also D5.ANODE, U1.1; no longer R34.PAD_0, U1.7
- net N$20: now also R34.PAD_1; no longer D5.CATHODE
- net N$24: now also U1.12; no longer U1.10
- net N$25: now also U1.14; no longer U1.8
- net N$40: now also U1.3; no longer U1.5
Routing:
- net GND: track 0.00 -> 92.2 mm, vias 0 -> 4
- net +10V: track 0.00 -> 84.6 mm
- net N$36: track 0.00 -> 38.9 mm, vias 0 -> 2
- net N$18: track 0.00 -> 21.7 mm
- net N$10: track 0.00 -> 21.3 mm, vias 0 -> 2
- net N$13: track 0.00 -> 20.2 mm
- net N$33: track 0.00 -> 18.4 mm
- net N$12: track 0.00 -> 17.8 mm
- net N$24: track 0.00 -> 17.1 mm
- net +13V_RAW: track 0.00 -> 15.7 mm
- net N$26: track 0.00 -> 14.6 mm
- net N$31: track 0.00 -> 12.8 mm
- net N$9: track 0.00 -> 12.7 mm, vias 0 -> 2
- net N$5: track 0.00 -> 12.3 mm
- net N$20: track 0.00 -> 12.2 mm
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- added copper zone on layer 16, net +10V
- added copper zone on layer 16, net +12V
- added copper zone on layer 16, net GND
- added copper zone on layer 16, net N$2
- added copper zone on layer 16, net N$4
- added copper zone on layer 16, net N$8
Other:
- board size 70 x 50 mm -> 60 x 60 mm

Commit message: SoftStart. Routed PCB.
Parts:
- T7: value BC847SOT23 -> BC847
- moved R4 0.54 mm to (42.9, 8.80)
- moved L2 0.30 mm to (51.0, 32.5)
- moved R15 0.10 mm to (31.3, 20.1)
Routing:
- net N$8: track 0.00 -> 5.40 mm
- net N$4: track 0.00 -> 5.30 mm
- net +12V: track 0.00 -> 4.00 mm
- net N$42: track 0.00 -> 3.20 mm
- net N$38: track 0.00 -> 1.80 mm
- net +10V: track 84.6 -> 83.1 mm
- net GND: track 92.2 -> 93.0 mm
- net N$17: track 8.20 -> 8.95 mm
- net N$20: track 12.2 -> 11.5 mm

Commit message: Soft start. Adjust time/voltage define resistors.
Parts:
- C1, C8: value 47uFx16V -> 22uFx16V
- R10: value 4K7 -> 5K1
- R11: value 36K -> 10K
- R12: value 100K -> 82K
- R16: value 10K -> 8K2
- R9: value 51K -> 13K
Changed lines of the file:
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@@
 <layer number="21" name="tPlace" color="7" fill="1" visible="yes" active="yes"/>
 <layer number="22" name="bPlace" color="7" fill="1" visible="yes" active="yes"/>
-<layer number="23" name="tOrigins" color="15" fill="1" visible="no" active="yes"/>
-<layer number="24" name="bOrigins" color="15" fill="1" visible="no" active="yes"/>
+<layer number="23" name="tOrigins" color="15" fill="1" visible="yes" active="yes"/>
+<layer number="24" name="bOrigins" color="15" fill="1" visible="yes" active="yes"/>
 <layer number="25" name="tNames" color="7" fill="1" visible="no" active="yes"/>
 <layer number="26" name="bNames" color="7" fill="1" visible="no" active="yes"/>
@@
 <element name="U1" library="__MyCommonLib1" package="SOIC14" value="TP2274" x="26" y="20" rot="MR180"/>
 <element name="U2" library="__MyCommonLib1" package="SOT223(WAVE_SOLDERING)" value="AMS1117" x="50.9" y="16.4" rot="MR90"/>
-<element name="C1" library="__MyCommonLib1" package="CE_6.3MM" value="47uFx16V" x="38" y="13" rot="R90"/>
+<element name="C1" library="__MyCommonLib1" package="CE_6.3MM" value="22uFx16V" x="38" y="13" rot="R90"/>
 <element name="C2" library="__MyCommonLib1" package="CE_10MM" value="470uFx25V" x="45.6" y="51.4"/>
 <element name="X1" library="__MyCommonLib1" package="RPI_6.3" value="+12V" x="3" y="42" rot="R90"/>
@@
 <element name="R7" library="__MyCommonLib1" package="RSMD_0805" value="20R" x="29" y="33.4" rot="MR180"/>
 <element name="R8" library="__MyCommonLib1" package="RSMD_0805" value="10K" x="29.9" y="36.9" rot="MR90"/>
-<element name="R9" library="__MyCommonLib1" package="RSMD_0805" value="51K" x="17.9" y="23.5" rot="MR180"/>
-<element name="R11" library="__MyCommonLib1" package="RSMD_0805" value="36K" x="16.9" y="20.1" rot="MR90"/>
-<element name="R12" library="__MyCommonLib1" package="RSMD_0805" value="100K" x="22.6" y="26.6" rot="MR0"/>
+<element name="R9" library="__MyCommonLib1" package="RSMD_0805" value="13K" x="17.9" y="23.5" rot="MR180"/>
+<element name="R11" library="__MyCommonLib1" package="RSMD_0805" value="10K" x="16.9" y="20.1" rot="MR90"/>
+<element name="R12" library="__MyCommonLib1" package="RSMD_0805" value="82K" x="22.6" y="26.6" rot="MR0"/>
 <element name="R13" library="__MyCommonLib1" package="RSMD_0805" value="51K" x="31.3" y="25.2" rot="MR270"/>
 <element name="R14" library="__MyCommonLib1" package="RSMD_0805" value="51K" x="27.1" y="26.6" rot="MR0"/>
 <element name="R15" library="__MyCommonLib1" package="RSMD_0805" value="51K" x="31.3" y="20.1" rot="MR270"/>
-<element name="R16" library="__MyCommonLib1" package="RSMD_0805" value="10K" x="34" y="25.2" rot="MR270"/>
+<element name="R16" library="__MyCommonLib1" package="RSMD_0805" value="8K2" x="34" y="25.2" rot="MR270"/>
 <element name="C6" library="__MyCommonLib1" package="RSMD_0805" value="1nF x 16V" x="34" y="20.2" rot="MR90"/>
 <element name="C7" library="__MyCommonLib1" package="RSMD_0805" value="0.1uF x 16V" x="25.2" y="13.5" rot="MR0"/>
-<element name="C8" library="__MyCommonLib1" package="CE_6.3MM" value="47uFx16V" x="16.9" y="16.6"/>
+<element name="C8" library="__MyCommonLib1" package="CE_6.3MM" value="22uFx16V" x="16.9" y="16.6"/>
 <element name="X5" library="__MyCommonLib1" package="PIN3X1_2.54MM_WITH_CLAMP" value="SET_DUTY_CYCLE(10K)" x="37" y="5" rot="R270"/>
 <element name="R22" library="__MyCommonLib1" package="RSMD_0805" value="5K1" x="33.1" y="5.8" rot="MR0"/>
@@
 <element name="R28" library="__MyCommonLib1" package="RSMD_0805" value="15K" x="43.7" y="43.9" rot="MR90"/>
 <element name="R29" library="__MyCommonLib1" package="RSMD_0805" value="1K6" x="43.7" y="39.7" rot="MR90"/>
-<element name="R10" library="__MyCommonLib1" package="RSMD_0805" value="4K7" x="20" y="10" rot="MR90"/>
+<element name="R10" library="__MyCommonLib1" package="RSMD_0805" value="5K1" x="20" y="10" rot="MR90"/>
 <element name="R30" library="__MyCommonLib1" package="RSMD_0805" value="20K" x="20.9" y="13.5" rot="MR0"/>
 <element name="D5" library="__MyCommonLib1" package="SOD-80" value="LL4148" x="24.3" y="9.8" rot="MR0"/>
