File: SoftStartBoard/schematic/SoftStart_V1_0.brd (EAGLE design)
At the start: 60 x 60 mm, 76 parts, among them T1 PK616BA, T2 PK616BA, T3 PK616BA, T4 PK616BA, T6 BC857, T7 BC847, T8 2N7002, U1 TP2274, U2 AMS1117, U3 MC34063, X1 +12V, X10 ON/OFF, X2 GND, X3 LAMP, X4 LAMP, X5 SET_DUTY_CYCLE(10K)

Commit message: Update soft start board. SWR metter.
Parts:
- removed C1, C8: 22uFx16V, __MyCommonLib1:CE_6.3MM
- removed C10: 220pFx25V, __MyCommonLib1:RSMD_0805
- removed C11, C13, C16: 1.0uFx25V, __MyCommonLib1:RSMD_1206
- removed C12, C14, C15: 47uFx25V, __MyCommonLib1:CE_6.3MM
- removed C17, C18, C7, C9: 0.1uF x 16V, __MyCommonLib1:RSMD_0805
- removed C2: 470uFx25V, __MyCommonLib1:CE_10MM
- removed C3: 1000uFx25V, __MyCommonLib1:CE_10MM
- removed C4: 0.1uFx25V, __MyCommonLib1:RSMD_1206
- removed C5: 0.1uFx25V, __MyCommonLib1:RSMD_0805
- removed C6: 1nF x 16V, __MyCommonLib1:RSMD_0805
- removed D1, D2, D3: B120, __MyCommonLib1:DO-214AC
- removed D5: LL4148, __MyCommonLib1:SOD-80
- removed F1: 20A, __MyCommonLib1:FUSE_AUTO_MINI_ON_TERMINALS
- removed L1: 680uHx0.17A, __MyCommonLib1:LCHB0608
- removed L2: 680uH x 0.07A, __MyCommonLib1:LCHB0608
- removed L3: 1.0mH x 0.05A, __MyCommonLib1:LCHB0608
- removed R1: 4K7, __MyCommonLib1:RSMD_0805
- removed R10, R22, R25, R34: 5K1, __MyCommonLib1:RSMD_0805
- removed R11, R17, R33, R8: 10K, __MyCommonLib1:RSMD_0805
- removed R12: 82K, __MyCommonLib1:RSMD_0805
- removed R13, R14, R15: 51K, __MyCommonLib1:RSMD_0805
- removed R16: 8K2, __MyCommonLib1:RSMD_0805
- removed R18: 20R*, __MyCommonLib1:RSMD_1206
- removed R2: 47K, __MyCommonLib1:RSMD_0805
- removed R23: 10K, __MyCommonLib1:RSMD_1206_BIG_GAP
- removed R24: 1M0, __MyCommonLib1:RSMD_0805
- removed R26: 2K0, __MyCommonLib1:RSMD_0805
- removed R27: 2R0, __MyCommonLib1:RSMD_1206_BIG_GAP
- removed R28: 15K, __MyCommonLib1:RSMD_0805
- removed R29: 1K6, __MyCommonLib1:RSMD_0805
- removed R3: 10R*, __MyCommonLib1:RSMD_1206_BIG_GAP
- removed R30: 20K, __MyCommonLib1:RSMD_0805
- removed R31: 510K*, __MyCommonLib1:RSMD_0805
- removed R32, R6, R7: 20R, __MyCommonLib1:RSMD_0805
- removed R4: 9K1, __MyCommonLib1:RSMD_0805
- removed R5: 1K3, __MyCommonLib1:RSMD_0805
- removed R9: 13K, __MyCommonLib1:RSMD_0805
- removed T1, T2, T3, T4: PK616BA, __MyCommonLib1:PDFN_5X6P
- removed T6: BC857, __MyCommonLib1:SOT23
- removed T7: BC847, __MyCommonLib1:SOT23
- removed T8: 2N7002, __MyCommonLib1:SOT23
- removed U1: TP2274, __MyCommonLib1:SOIC14
- removed U2: AMS1117, __MyCommonLib1:SOT223(WAVE_SOLDERING)
- removed U3: MC34063, __MyCommonLib1:SOIC8
- removed X1: +12V, __MyCommonLib1:RPI_6.3
- removed X10: ON/OFF, __MyCommonLib1:PIN2X1_2.54_WITH_CLAMP
- removed X2: GND, __MyCommonLib1:RPI_6.3
- removed X3, X4: LAMP, __MyCommonLib1:RPI_6.3
- removed X5: SET_DUTY_CYCLE(10K), __MyCommonLib1:PIN3X1_2.54MM_WITH_CLAMP
- removed ZD1, ZD2, ZD3: 5V6, __MyCommonLib1:SOD-80
Connections:
- removed net +10V: C1.PLUS, C5.PAD_1, C7.PAD_1, R14.PAD_1, R18.PAD_0, R31.PAD_1, R33.PAD_1, R5.PAD_0, R9.PAD_1, U1.4, U2.2, U2.4, X5.1
- removed net +12V: C3.PLUS, D1.ANODE, D3.CATHODE, F1.PAD0, X3.PAD1, X3.PAD2
- removed net +13V_RAW: C15.PLUS, C16.PAD_0, L3.2, U2.3
- removed net GND: C1.MINUS, C10.PAD_0, C13.PAD_1, C14.MINUS, C15.MINUS, C16.PAD_1, C17.PAD_0, C18.PAD_0, C2.MINUS, C3.MINUS, C4.PAD_0, C5.PAD_0, C7.PAD_0, C8.MINUS, C9.PAD_0, L2.2, R10.PAD_0, R11.PAD_0, R15.PAD_1, R2.PAD_0, R29.PAD_0, R4.PAD_0, R8.PAD_1, T1.S1, T1.S2, T1.S3, T2.S1, T2.S2, T2.S3, T3.S1, T3.S2, T3.S3, T4.S1, T4.S2, T4.S3, T6.3, T8.2, U1.11, U3.2, U3.4, X10.1, X5.3, ZD2.ANODE, ZD3.ANODE
- removed net N$1: R1.PAD_0, R2.PAD_1, T1.G, T2.G, ZD1.CATHODE
- removed net N$10: R6.PAD_0, T4.G
- removed net N$11: D5.CATHODE, R34.PAD_0
- removed net N$12: R12.PAD_0, R13.PAD_0, U1.5
- removed net N$13: R12.PAD_1, R16.PAD_0, U1.7
- removed net N$14: R11.PAD_1, R9.PAD_0, U1.6
- removed net N$15: R10.PAD_1, R30.PAD_1, U1.2
- removed net N$16: R14.PAD_0, R15.PAD_0, U1.10
- removed net N$17: C6.PAD_1, R16.PAD_1, U1.9
- removed net N$18: C6.PAD_0, R13.PAD_1, U1.13, U1.8
- removed net N$19: D5.ANODE, R30.PAD_0, U1.1
- removed net N$2: T1.D, T1.D1, T1.D2, T1.D3, T1.D4, T2.D, T2.D1, T2.D2, T2.D3, T2.D4, X2.PAD1, X2.PAD2
- removed net N$20: C9.PAD_1, R22.PAD_1, R23.PAD_0, R34.PAD_1
- removed net N$22: C17.PAD_1, R17.PAD_0, T8.1, ZD3.CATHODE
- removed net N$23: R22.PAD_0, X5.2
- removed net N$24: R23.PAD_1, R24.PAD_0, U1.12
- removed net N$25: R24.PAD_1, R25.PAD_0, U1.14
- removed net N$26: R25.PAD_1, T6.1, T7.1
- removed net N$27: R6.PAD_1, R7.PAD_1, R8.PAD_0, T6.2, T7.2
- removed net N$3: ZD1.ANODE, ZD2.CATHODE
- removed net N$30: C18.PAD_1, R18.PAD_1, T7.3
- removed net N$31: C11.PAD_1, C12.PLUS, L1.2, U3.1
- removed net N$32: C11.PAD_0, C12.MINUS, D2.ANODE, L2.1
- removed net N$33: C2.PLUS, C4.PAD_1, R27.PAD_1, R3.PAD_0, U3.6
- removed net N$34: R26.PAD_0, U3.8
- removed net N$35: C10.PAD_1, U3.3
- removed net N$36: C13.PAD_0, C14.PLUS, D2.CATHODE, L3.1, R28.PAD_1
- removed net N$37: R28.PAD_0, R29.PAD_1, U3.5
- removed net N$39: R32.PAD_0, T8.3
- removed net N$4: F1.PAD1, R1.PAD_1, X1.PAD1, X1.PAD2
- removed net N$40: C8.PLUS, R31.PAD_0, R32.PAD_1, U1.3
- removed net N$41: R17.PAD_1, R33.PAD_0, X10.2
- removed net N$5: L1.1, R26.PAD_1, R27.PAD_0, U3.7
- removed net N$6: D1.CATHODE, R3.PAD_1
- removed net N$7: R4.PAD_1, R5.PAD_1, U2.1
- removed net N$8: D3.ANODE, T3.D, T3.D1, T3.D2, T3.D3, T3.D4, T4.D, T4.D1, T4.D2, T4.D3, T4.D4, X4.PAD1, X4.PAD2
- removed net N$9: R7.PAD_0, T3.G
Routing:
- net +10V: track 83.1 -> 0.00 mm
- net GND: track 93.0 -> 18.5 mm, vias 4 -> 2
- net N$36: track 39.0 -> 0.00 mm, vias 2 -> 0
- net N$1: track 28.4 -> 0.00 mm, vias 4 -> 0
- net N$10: track 21.3 -> 0.00 mm, vias 2 -> 0
- net N$18: track 21.2 -> 0.00 mm
- net N$13: track 20.2 -> 0.00 mm
- net N$33: track 18.4 -> 0.00 mm
- net N$12: track 17.5 -> 0.00 mm
- net N$24: track 17.0 -> 0.00 mm
- net +13V_RAW: track 15.7 -> 0.00 mm
- net N$26: track 14.8 -> 0.00 mm
- net N$31: track 12.8 -> 0.00 mm
- net N$9: track 12.6 -> 0.00 mm, vias 2 -> 0
- net N$5: track 12.3 -> 0.00 mm
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