File: SoftStartBoard/schematic/SoftStart_V1_0.sch (EAGLE design)
At the start: 74 parts, among them T1 PK616BA, T2 PK616BA, T3 PK616BA, T4 PK616BA, T6 BC857, T7 BC847SOT23, T8 2N7002, U1 TP2274, U2 AMS1117, U3 MC34063, X1 +12V, X10 ON/OFF, X2 GND, X3 LAMP, X4 LAMP, X5 SET_DUTY_CYCLE(10K)

Commit message: SoftStart. Almost routed PCB.
Parts:
- added C18: 0.1uF x 16V, __MyCommonLib1:CSMD_0805
- added R18: 20R*, __MyCommonLib1:RSMD_1206
- C4: device __MyCommonLib1:CSMD_0805 -> __MyCommonLib1:CSMD_1206
- R23: device __MyCommonLib1:RSMD_0805 -> __MyCommonLib1:RSMD_1206_BIG_GAP
Connections:
- new net N$30: C18.PIN1, R18.PIN1, T7.C
- net +10V: now also R18.PIN0; no longer T7.C
- net GND: now also C18.PIN0
- net N$11: now also D5.CATHODE, R34.PIN0; no longer D5.ANODE, R34.PIN1
- net N$12: now also U1OP2.IN+; no longer U1OP1.IN+
- net N$13: now also U1OP2.OUT; no longer U1OP1.OUT
- net N$14: now also U1OP2.IN-; no longer U1OP1.IN-
- net N$15: now also U1OP1.IN-; no longer U1OP2.IN-
- net N$16: now also U1OP3.IN+; no longer U1OP4.IN+
- net N$17: now also U1OP3.IN-; no longer U1OP4.IN-
- net N$18: now also U1OP3.OUT, U1OP4.IN-; no longer U1OP3.IN-, U1OP4.OUT
- net N$19: now also D5.ANODE, U1OP1.OUT; no longer R34.PIN0, U1OP2.OUT
- net N$20: now also R34.PIN1; no longer D5.CATHODE
- net N$24: now also U1OP4.IN+; no longer U1OP3.IN+
- net N$25: now also U1OP4.OUT; no longer U1OP3.OUT
- net N$40: now also U1OP1.IN+; no longer U1OP2.IN+
Other:
- moved on the sheet: D5, R34, U1OP1, U1OP2, U1OP3, U1OP4

Commit message: SoftStart. Routed PCB.
Parts:
- T7: value BC847SOT23 -> BC847
Changed lines of the file:
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@@
 <part name="R25" library="__MyCommonLib1" deviceset="R" device="SMD_0805" value="5K1"/>
 <part name="T6" library="__MyCommonLib1" deviceset="BC857" device="SOT23" value="BC857"/>
-<part name="T7" library="__MyCommonLib1" deviceset="BC847" device="SOT23"/>
+<part name="T7" library="__MyCommonLib1" deviceset="BC847" device="SOT23" value="BC847"/>
 <part name="GND23" library="supply1" deviceset="GND" device=""/>
 <part name="C9" library="__MyCommonLib1" deviceset="C" device="SMD_0805" value="0.1uF x 16V"/>

Commit message: Soft start. Adjust time/voltage define resistors.
Parts:
- C1, C8: value 47uFx16V -> 22uFx16V
- R10: value 4K7 -> 5K1
- R11: value 36K -> 10K
- R12: value 100K -> 82K
- R16: value 10K -> 8K2
- R9: value 51K -> 13K
Other:
- note added: "+4.347V"
- note added: "+5V"
- note added: "0.0V to 2.0V rise"
- note added: "Trise = 5.5sec"
- note added: "Umax=7.05V"
- note added: "Umin=0.832V"
- note removed: "+3.310V"
- note removed: "+4.0V"
- note removed: "Umax=4.9981V"
- note removed: "Umin=0.9181V"
- moved on the sheet: R10
