File: SoftStartBoard/schematic/SoftStart_V1_0.sch (EAGLE design)
At the start: 76 parts, among them T1 PK616BA, T2 PK616BA, T3 PK616BA, T4 PK616BA, T6 BC857, T7 BC847, T8 2N7002, U1 TP2274, U2 AMS1117, U3 MC34063, X1 +12V, X10 ON/OFF, X2 GND, X3 LAMP, X4 LAMP, X5 SET_DUTY_CYCLE(10K)

Commit message: Update soft start board. SWR metter.
Parts:
- removed C1, C8: 22uFx16V, __MyCommonLib1:CE6.3MM
- removed C10: 220pFx25V, __MyCommonLib1:CSMD_0805
- removed C11, C13, C16: 1.0uFx25V, __MyCommonLib1:CSMD_1206
- removed C12, C14, C15: 47uFx25V, __MyCommonLib1:CE6.3MM
- removed C17, C18, C7, C9: 0.1uF x 16V, __MyCommonLib1:CSMD_0805
- removed C2: 470uFx25V, __MyCommonLib1:CE10MM
- removed C3: 1000uFx25V, __MyCommonLib1:CE10MM
- removed C4: 0.1uFx25V, __MyCommonLib1:CSMD_1206
- removed C5: 0.1uFx25V, __MyCommonLib1:CSMD_0805
- removed C6: 1nF x 16V, __MyCommonLib1:CSMD_0805
- removed D1, D2, D3: B120, __MyCommonLib1:B120(DO-214AC)
- removed D5: LL4148, __MyCommonLib1:LL4147SOD-80
- removed F1: 20A, __MyCommonLib1:FUSEAUTO_MINI_TERMINALS
- removed L1: 680uHx0.17A, __MyCommonLib1:L(LCHB0608)
- removed L2: 680uH x 0.07A, __MyCommonLib1:L(LCHB0608)
- removed L3: 1.0mH x 0.05A, __MyCommonLib1:L(LCHB0608)
- removed R1: 4K7, __MyCommonLib1:RSMD_0805
- removed R10, R22, R25, R34: 5K1, __MyCommonLib1:RSMD_0805
- removed R11, R17, R33, R8: 10K, __MyCommonLib1:RSMD_0805
- removed R12: 82K, __MyCommonLib1:RSMD_0805
- removed R13, R14, R15: 51K, __MyCommonLib1:RSMD_0805
- removed R16: 8K2, __MyCommonLib1:RSMD_0805
- removed R18: 20R*, __MyCommonLib1:RSMD_1206
- removed R2: 47K, __MyCommonLib1:RSMD_0805
- removed R23: 10K, __MyCommonLib1:RSMD_1206_BIG_GAP
- removed R24: 1M0, __MyCommonLib1:RSMD_0805
- removed R26: 2K0, __MyCommonLib1:RSMD_0805
- removed R27: 2R0, __MyCommonLib1:RSMD_1206_BIG_GAP
- removed R28: 15K, __MyCommonLib1:RSMD_0805
- removed R29: 1K6, __MyCommonLib1:RSMD_0805
- removed R3: 10R*, __MyCommonLib1:RSMD_1206_BIG_GAP
- removed R30: 20K, __MyCommonLib1:RSMD_0805
- removed R31: 510K*, __MyCommonLib1:RSMD_0805
- removed R32, R6, R7: 20R, __MyCommonLib1:RSMD_0805
- removed R4: 9K1, __MyCommonLib1:RSMD_0805
- removed R5: 1K3, __MyCommonLib1:RSMD_0805
- removed R9: 13K, __MyCommonLib1:RSMD_0805
- removed T1, T2, T3, T4: PK616BA, __MyCommonLib1:PK616BA(PDFN_5X6P)
- removed T6: BC857, __MyCommonLib1:BC857SOT23
- removed T7: BC847, __MyCommonLib1:BC847SOT23
- removed T8: 2N7002, __MyCommonLib1:2N7002SOT23
- removed U1: TP2274, __MyCommonLib1:LM324
- removed U2: AMS1117, __MyCommonLib1:AMS1117SOT223_WS
- removed U3: MC34063, __MyCommonLib1:MC34063(SO-8)
- removed X1: +12V, __MyCommonLib1:RPI_MALE6.3_TWO_HOLES
- removed X10: ON/OFF, __MyCommonLib1:PIN1X22.54MM_WITH_CLAMP
- removed X2: GND, __MyCommonLib1:RPI_MALE6.3_TWO_HOLES
- removed X3, X4: LAMP, __MyCommonLib1:RPI_MALE6.3_TWO_HOLES
- removed X5: SET_DUTY_CYCLE(10K), __MyCommonLib1:PIN1X3(2.54MM_WITH_CLAMP)
- removed ZD1, ZD2, ZD3: 5V6, __MyCommonLib1:ZENNER(SOD_80)
Connections:
- removed net +10V: C1.PLUS, C5.PIN1, C7.PIN1, R14.PIN1, R18.PIN0, R31.PIN1, R33.PIN1, R5.PIN0, R9.PIN1, U1PWR.VCC, U2.OUT, X5.1
- removed net +12V: C3.PLUS, D1.ANODE, D3.CATHODE, F1.PIN0, X3.1
- removed net +13V_RAW: C15.PLUS, C16.PIN0, L3.END, U2.IN
- removed net GND: C1.MINUS, C10.PIN0, C13.PIN1, C14.MINUS, C15.MINUS, C16.PIN1, C17.PIN0, C18.PIN0, C2.MINUS, C3.MINUS, C4.PIN0, C5.PIN0, C7.PIN0, C8.MINUS, C9.PIN0, L2.END, R10.PIN0, R11.PIN0, R15.PIN1, R2.PIN0, R29.PIN0, R4.PIN0, R8.PIN1, T1.SOURCE, T2.SOURCE, T3.SOURCE, T4.SOURCE, T6.C, T8.SOURCE, U1PWR.GND, U3.GND, U3.SW_E, X10.1, X5.3, ZD2.ANODE, ZD3.ANODE
- removed net N$1: R1.PIN0, R2.PIN1, T1.GATE, T2.GATE, ZD1.CATHODE
- removed net N$10: R6.PIN0, T4.GATE
- removed net N$11: D5.CATHODE, R34.PIN0
- removed net N$12: R12.PIN0, R13.PIN0, U1OP2.IN+
- removed net N$13: R12.PIN1, R16.PIN0, U1OP2.OUT
- removed net N$14: R11.PIN1, R9.PIN0, U1OP2.IN-
- removed net N$15: R10.PIN1, R30.PIN1, U1OP1.IN-
- removed net N$16: R14.PIN0, R15.PIN0, U1OP3.IN+
- removed net N$17: C6.PIN1, R16.PIN1, U1OP3.IN-
- removed net N$18: C6.PIN0, R13.PIN1, U1OP3.OUT, U1OP4.IN-
- removed net N$19: D5.ANODE, R30.PIN0, U1OP1.OUT
- removed net N$2: T1.DRAIN, T2.DRAIN, X2.1
- removed net N$20: C9.PIN1, R22.PIN1, R23.PIN0, R34.PIN1
- removed net N$22: C17.PIN1, R17.PIN0, T8.GATE, ZD3.CATHODE
- removed net N$23: R22.PIN0, X5.2
- removed net N$24: R23.PIN1, R24.PIN0, U1OP4.IN+
- removed net N$25: R24.PIN1, R25.PIN0, U1OP4.OUT
- removed net N$26: R25.PIN1, T6.B, T7.B
- removed net N$27: R6.PIN1, R7.PIN1, R8.PIN0, T6.E, T7.E
- removed net N$3: ZD1.ANODE, ZD2.CATHODE
- removed net N$30: C18.PIN1, R18.PIN1, T7.C
- removed net N$31: C11.PIN1, C12.PLUS, L1.END, U3.SW_C
- removed net N$32: C11.PIN0, C12.MINUS, D2.ANODE, L2.START
- removed net N$33: C2.PLUS, C4.PIN1, R27.PIN1, R3.PIN0, U3.VCC
- removed net N$34: R26.PIN0, U3.DR_C
- removed net N$35: C10.PIN1, U3.CT
- removed net N$36: C13.PIN0, C14.PLUS, D2.CATHODE, L3.START, R28.PIN1
- removed net N$37: R28.PIN0, R29.PIN1, U3.INV_IN
- removed net N$39: R32.PIN0, T8.DRAIN
- removed net N$4: F1.PIN1, R1.PIN1, X1.1
- removed net N$40: C8.PLUS, R31.PIN0, R32.PIN1, U1OP1.IN+
- removed net N$41: R17.PIN1, R33.PIN0, X10.2
- removed net N$5: L1.START, R26.PIN1, R27.PIN0, U3.I_PEAK
- removed net N$6: D1.CATHODE, R3.PIN1
- removed net N$7: R4.PIN1, R5.PIN1, U2.ADJ
- removed net N$8: D3.ANODE, T3.DRAIN, T4.DRAIN, X4.1
- removed net N$9: R7.PIN0, T3.GATE
Other:
- note removed: "+4.347V"
- note removed: "+5V"
- note removed: "0.0V to 2.0V rise"
- note removed: "50KHz_Saw_1.0_to_5.0V"
- note removed: "Trise = 5.5sec"
- note removed: "Umax=7.05V"
- note removed: "Umin=0.832V"
